File: ATMEGA-SCHEMATICS/SNAKE_GAME/SNAKE_GAME.kicad_pcb (KiCad board)
At the start: 2 copper layers, 31 parts, among them U1 ATmega168A-P, U4 LM2576T-ADJ, Y1 Crystal

Commit message: .
Parts:
- removed C6, C7: C_Small, Capacitor_THT:CP_Radial_D5.0mm_P2.50mm
- removed D2: 1N5822, Diode_THT:D_DO-201AD_P15.24mm_Horizontal
- removed R23, R25: 4.7k, Resistor_THT:R_Axial_DIN0207_L6.3mm_D2.5mm_P10.16mm_Horizontal
- removed R26: 1k, Resistor_THT:R_Axial_DIN0207_L6.3mm_D2.5mm_P10.16mm_Horizontal
- removed U4: LM2576T-ADJ, Package_TO_SOT_THT:TO-220-5_Vertical
- added 220UF1: C_Polarized, Capacitor_THT:C_Disc_D3.0mm_W1.6mm_P2.50mm, F.Cu at (124.0, -81.8)
- added H1: MountingHole, MountingHole:MountingHole_3.2mm_M3, F.Cu at (145.5, -99.2)
- added H2: MountingHole, MountingHole:MountingHole_3.2mm_M3, F.Cu at (145.5, -4.75)
- added H3: MountingHole, MountingHole:MountingHole_3.2mm_M3, F.Cu at (13.0, -4.75)
- added H4: MountingHole, MountingHole:MountingHole_3.2mm_M3, F.Cu at (13.0, -99.2)
- added J1: GRID, TerminalBlock:TerminalBlock_MaiXu_MX126-5.0-03P_1x03_P5.00mm, F.Cu at (108.0, -92.8)
- added J10: VCC, TerminalBlock:TerminalBlock_MaiXu_MX126-5.0-04P_1x04_P5.00mm, F.Cu at (132.0, -13.5)
- added J11: PJ-102A, Connector_BarrelJack:BarrelJack_Horizontal, F.Cu at (138.8, -82.8)
- added J3: Conn_01x03_Pin, Connector_PinSocket_2.54mm:PinSocket_1x03_P2.54mm_Vertical, F.Cu at (121.8, -96.2)
- added J4: USB_ASP, Connector_IDC:IDC-Header_2x05_P2.54mm_Vertical, F.Cu at (117.0, -8.21)
- added J5: BUTTONS, TerminalBlock:TerminalBlock_MaiXu_MX126-5.0-03P_1x03_P5.00mm, F.Cu at (33.0, -67.2)
- added J6: JOYSTICK, TerminalBlock:TerminalBlock_MaiXu_MX126-5.0-04P_1x04_P5.00mm, F.Cu at (33.0, -48.2)
- added J7: UART_TERM, Connector_PinSocket_2.54mm:PinSocket_1x04_P2.54mm_Vertical, F.Cu at (127.0, -69.5)
- added J8: PCF_SCREEN, TerminalBlock:TerminalBlock_MaiXu_MX126-5.0-04P_1x04_P5.00mm, F.Cu at (67.9, -88.1)
- added J9: GROUND, TerminalBlock:TerminalBlock_MaiXu_MX126-5.0-04P_1x04_P5.00mm, F.Cu at (132.0, -37.5)
- added SW1: SW_Push, Button_Switch_THT:SW_PUSH_6mm, F.Cu at (129.8, -97.8)
- moved R16 185.4 mm to (24.1, -67.2), turned to 180 degrees
- moved R24 181.8 mm to (98.0, -86.6), turned to -90 degrees
- moved R15 177.2 mm to (24.1, -62.2), turned to 180 degrees
- moved R14 169.0 mm to (24.1, -57.2), turned to 180 degrees
- moved R22 158.0 mm to (83.9, -69.0), turned to 90 degrees
- moved R6 157.1 mm to (51.6, -67.5), turned to 180 degrees
- moved R7 156.4 mm to (51.6, -62.8), turned to 180 degrees
- moved R21 155.3 mm to (77.9, -69.1), turned to 90 degrees
- moved R13 155.0 mm to (51.6, -57.2), turned to 180 degrees
- moved R20 153.6 mm to (24.6, -48.2), turned to 180 degrees
- moved R19 146.2 mm to (24.6, -43.2), turned to 180 degrees
- moved C4 143.4 mm to (72.8, -41.5)
- moved Y1 143.1 mm to (73.8, -30.1), turned to 90 degrees
- moved R18 139.0 mm to (24.6, -38.2), turned to 180 degrees
- moved C2 133.2 mm to (63.5, -37.6), turned to 180 degrees
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Connections:
- C1 pad 2: Net-(U1-AVCC) -> VCC
- C4 pad 2: Net-(U1-AVCC) -> VCC
- U1 pad 16: /CS -> unconnected-(U1-PB2-Pad16)
- U1 pad 20: Net-(U1-AVCC) -> VCC
- U1 pad 26: /SCREEN_INT -> unconnected-(U1-PC3-Pad26)
- U1 pad 7: Net-(U1-AVCC) -> VCC
Routing:
- net VCC: track 0.00 -> 382.4 mm
- net /RESET: track 0.00 -> 151.6 mm, vias 0 -> 5
- net Net-(U1-PB0): track 0.00 -> 71.4 mm, vias 0 -> 2
- net Net-(U1-PD6): track 0.00 -> 70.8 mm, vias 0 -> 2
- net /SDA: track 0.00 -> 70.5 mm
- net Net-(U1-PD7): track 0.00 -> 69.2 mm, vias 0 -> 2
- net /DIN_GRID: track 0.00 -> 61.9 mm
- net /TXD: track 0.00 -> 60.8 mm, vias 0 -> 2
- net /RXD: track 0.00 -> 49.0 mm, vias 0 -> 2
- net Net-(U1-PD5): track 0.00 -> 41.8 mm
- net /SCL: track 0.00 -> 40.6 mm
- net Net-(U1-PD4): track 0.00 -> 39.9 mm
- net Net-(U1-PD3): track 0.00 -> 39.1 mm
- net Net-(U1-PD2): track 0.00 -> 38.1 mm
- net /MOSI: track 0.00 -> 36.4 mm, vias 0 -> 2
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- added copper zone on F.Cu, net GND
- added copper zone on B.Cu, net VCC
Other:
- board outline added: 139.5 x 101.5 mm

Commit message: .
Parts:
- moved H3 6.60 mm to (15.8, -10.8)
- moved J4 6.33 mm to (116.2, -14.5)
- moved H2 6.00 mm to (145.5, -10.8)
- moved H4 2.75 mm to (15.8, -99.2)
- moved J5 2.00 mm to (35.0, -67.2)
- moved J6 2.00 mm to (35.0, -48.2)
- moved R13 2.00 mm to (53.6, -57.2)
- moved R14 2.00 mm to (26.1, -57.2)
- moved R15 2.00 mm to (26.1, -62.2)
- moved R16 2.00 mm to (26.1, -67.2)
- moved R17 2.00 mm to (26.6, -33.8)
- moved R18 2.00 mm to (26.6, -38.2)
- moved R19 2.00 mm to (26.6, -43.2)
- moved R2 2.00 mm to (53.1, -48.2)
- moved R20 2.00 mm to (26.6, -48.2)
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Routing:
- net /RESET: track 151.6 -> 145.7 mm
- net /MOSI: track 36.4 -> 31.6 mm
- net VCC: track 382.4 -> 378.5 mm
- net Net-(U1-PD4): track 39.9 -> 37.2 mm
- net /SCK: track 31.1 -> 29.1 mm
- net Net-(U1-PD7): track 69.2 -> 67.2 mm
- net Net-(U1-PD6): track 70.8 -> 68.8 mm
- net Net-(U1-PD3): track 39.1 -> 37.1 mm
- net Net-(U1-PD2): track 38.1 -> 36.1 mm
- net Net-(U1-PB0): track 71.4 -> 69.4 mm
- net /MISO: track 26.7 -> 25.0 mm
- net Net-(U1-PD5): track 41.8 -> 41.0 mm
Other:
- board size 139.5 x 101.5 mm -> 136.8 x 95.5 mm

Commit message: .
Parts:
- moved J9 13.3 mm to (121.0, -30.0)
- moved 220UF1 13.3 mm to (113.0, -74.2)
- moved C1 13.3 mm to (95.3, -30.6)
- moved C2 13.3 mm to (52.5, -30.1)
- moved C3 13.3 mm to (52.8, -19.6)
- moved C4 13.3 mm to (61.8, -34.0)
- moved C5 13.3 mm to (94.2, -36.0)
- moved H1 13.3 mm to (134.5, -91.8)
- moved H2 13.3 mm to (134.5, -3.25)
- moved H3 13.3 mm to (4.75, -3.25)
- moved H4 13.3 mm to (4.75, -91.8)
- moved J1 13.3 mm to (97.0, -85.2)
- moved J10 13.3 mm to (121.0, -5.99)
- moved J11 13.3 mm to (127.8, -75.3)
- moved J3 13.3 mm to (110.8, -88.8)
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
Commit message: .
Parts:
- added 1k: 100, Resistor_THT:R_Axial_DIN0207_L6.3mm_D2.5mm_P10.16mm_Horizontal, F.Cu at (98.3, -60.0)
- added G***: LOGO, Connector_Pin:snake, F.Cu at (23.5, -78.5)
- added H5: MountingHole, MountingHole:MountingHole_3.2mm_M3, F.Cu at (149.9, -72.5)
- added H6: MountingHole, MountingHole:MountingHole_3.2mm_M3, F.Cu at (149.9, -64.6)
- added H7: MountingHole, MountingHole:MountingHole_3.2mm_M3, F.Cu at (149.9, -56.6)
- added PWR_ON_LED: LED, LED_THT:LED_D1.8mm_W3.3mm_H2.4mm, F.Cu at (118.2, -80.0)
- renumbered R5 to 100, R13 to 100, R6 to 100, R4 to 100, R3 to 100, R7 to 100, R2 to 100, C4 to 100nF, C1 to 100nF, C5 to 100nF, Y1 to 20MHz, C2 to 20pF, C3 to 20pF, R18 to 4k7, R17 to 4k7, R14 to 4k7, R20 to 4k7, R19 to 4k7, R16 to 4k7, J10 to 5V, J9 to GND, J11 to PJ_102A, R15 to R4k7, SW1 to RESET_SW, J7 to UART_TERM, J4 to USBASP--
Connections:
- USBASP-- pad 3: unconnected-(J4-Pin_3-Pad3) -> GND
- USBASP-- pad 4: unconnected-(J4-Pin_4-Pad4) -> GND
- USBASP-- pad 6: unconnected-(J4-Pin_6-Pad6) -> GND
Routing:
- net GND: track 0.00 -> 173.4 mm, vias 0 -> 10
- net Net-(D1-K): track 0.00 -> 32.1 mm, vias 0 -> 1
- net VCC: track 378.5 -> 387.5 mm
Other:
- board text added: "═════════════════════════════ Project: Snake Game MCU: ATmega168A Board: Custom PCB Course: UMB-CS341-F25 Semester: Fall 2025 Author: Lucas Nascimento ══════════════════════════════"

Commit message: .
Parts:
- removed J3: Conn_01x03_Pin, Connector_PinSocket_2.54mm:PinSocket_1x03_P2.54mm_Vertical
- added 4k7: 4.7k, Resistor_THT:R_Axial_DIN0207_L6.3mm_D2.5mm_P10.16mm_Horizontal, F.Cu at (138.5, 33.2)
- moved H5 150.0 mm to (142.0, 77.2)
- moved H7 138.9 mm to (98.0, 72.2)
- moved H6 138.0 mm to (78.0, 53.2)
- moved G*** 127.0 mm to (59.5, 43.2)
- moved 100nF 126.3 mm to (95.3, 87.8)
- moved 100nF 126.3 mm to (128.8, 91.1)
- moved 100nF 126.3 mm to (127.8, 85.8)
- moved 20MHz 126.3 mm to (96.3, 99.1)
- moved 20pF 126.3 mm to (86.0, 91.6)
- moved 20pF 126.3 mm to (86.3, 102.1)
- moved 220UF1 126.3 mm to (146.5, 47.5)
- moved 4K7 126.3 mm to (48.6, 67.0)
- moved 4K7 126.3 mm to (49.1, 95.5)
- moved 4K7 126.3 mm to (48.6, 72.0)
- moved 4K7 126.3 mm to (49.1, 81.0)
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- renumbered R4k7 to 4K7, 4k7 to 4K7, U1 to ATMEGA168, J1 to GRID, J6 to JOYSTICK, J8 to PCF_SCREEN, PWR_ON_LED to PWR_LED, 1k to R1, 100 to R13, 100 to R2, 100 to R3, 100 to R4, 4k7 to R4K7, 100 to R5, 100 to R6, 100 to R7, RESET_SW to RESET_SWT, USBASP-- to USBASP
Connections:
- RESET_SWT pad 2: Net-(J3-Pin_2) -> GND
Routing:
- net Net-(J3-Pin_2): track 19.6 -> 0.00 mm
- net GND: track 173.4 -> 187.3 mm, vias 10 -> 9
- net VCC: track 387.5 -> 377.4 mm
- net /RESET: track 145.7 -> 150.3 mm
Other:
- board text added: "BUTTONS"
- board text added: "DIN"
- board text added: "DOWN"
- board text added: "EXIT"
- board text added: "GND"
- board text added: "LEFT"
- board text added: "MISO"
- board text added: "MOSI"
- board text added: "RESET"
- board text added: "RIGHT"
- board text added: "RXD"
- board text added: "SCK"
- board text added: "SCL"
- board text added: "SDA"
- board text added: "SEL."
- board text added: "START"
- board text added: "TXD"
- board text added: "UP"
- board text added: "VCC"
