File: ATMEGA-SCHEMATICS/SNAKE_GAME/SNAKE_GAME.kicad_pcb (KiCad board)
At the start: 2 copper layers, 136.8 x 95.5 mm, 46 parts, among them J5 BUTTONS

Commit message: .
Parts:
- removed 100nF (x3), 20pF (x2): C_Small, Capacitor_THT:CP_Radial_D5.0mm_P2.50mm
- removed 20MHz: Crystal, Crystal:Resonator-2Pin_W6.0mm_H3.0mm
- removed 220UF1: C_Polarized, Capacitor_THT:C_Disc_D3.0mm_W1.6mm_P2.50mm
- removed 4K7 (x5), 4k7, R21, R22, R24, R4K7 (x2): 4.7k, Resistor_THT:R_Axial_DIN0207_L6.3mm_D2.5mm_P10.16mm_Horizontal
- removed 5V: VCC, TerminalBlock:TerminalBlock_MaiXu_MX126-5.0-04P_1x04_P5.00mm
- removed ATMEGA168: ATmega168A-P, Package_DIP:DIP-28_W7.62mm
- removed GND: GROUND, TerminalBlock:TerminalBlock_MaiXu_MX126-5.0-04P_1x04_P5.00mm
- removed GRID: GRID, TerminalBlock:TerminalBlock_MaiXu_MX126-5.0-03P_1x03_P5.00mm
- removed J5: BUTTONS, TerminalBlock:TerminalBlock_MaiXu_MX126-5.0-03P_1x03_P5.00mm
- removed JOYSTICK: JOYSTICK, TerminalBlock:TerminalBlock_MaiXu_MX126-5.0-04P_1x04_P5.00mm
- removed PCF_SCREEN: PCF_SCREEN, TerminalBlock:TerminalBlock_MaiXu_MX126-5.0-04P_1x04_P5.00mm
- removed PJ_102A: PJ-102A, Connector_BarrelJack:BarrelJack_Horizontal
- removed PWR_LED: LED, LED_THT:LED_D1.8mm_W3.3mm_H2.4mm
- removed R5, R6: 100, Resistor_THT:R_Axial_DIN0207_L6.3mm_D2.5mm_P10.16mm_Horizontal
- removed RESET_SWT: SW_Push, Button_Switch_THT:SW_PUSH_6mm
- removed UART_TERM: UART_TERM, Connector_PinSocket_2.54mm:PinSocket_1x04_P2.54mm_Vertical
- removed USBASP: USB_ASP, Connector_IDC:IDC-Header_2x05_P2.54mm_Vertical
- added 220UF2: C_Polarized, Capacitor_THT:C_Disc_D3.0mm_W1.6mm_P2.50mm, F.Cu at (300.5, 14.1)
- added AUDIO-SCREEN1: ATmega168A-P, Package_DIP:DIP-28_W7.62mm, F.Cu at (111.4, 60.5)
- added C10: C_Small, Capacitor_THT:CP_Radial_D5.0mm_P2.50mm, F.Cu at (40.5, 56.0)
- added C11: C_Small, Capacitor_THT:CP_Radial_D5.0mm_P2.50mm, F.Cu at (131.5, 76.0)
- added C12: C_Small, Capacitor_THT:CP_Radial_D5.0mm_P2.50mm, F.Cu at (133.7, 85.0)
- added C13: C_Small, Capacitor_THT:CP_Radial_D5.0mm_P2.50mm, F.Cu at (78.0, 51.5)
- added C14: C_Small, Capacitor_THT:CP_Radial_D5.0mm_P2.50mm, F.Cu at (95.5, 77.0)
- added C15: C_Small, Capacitor_THT:CP_Radial_D5.0mm_P2.50mm, F.Cu at (95.5, 87.0)
- added C6: C_Small, Capacitor_THT:CP_Radial_D5.0mm_P2.50mm, F.Cu at (77.5, 44.3)
- added C7: C_Small, Capacitor_THT:CP_Radial_D5.0mm_P2.50mm, F.Cu at (47.0, 43.0)
- added C8: C_Small, Capacitor_THT:CP_Radial_D5.0mm_P2.50mm, F.Cu at (102.0, 71.0)
- added C9: C_Small, Capacitor_THT:CP_Radial_D5.0mm_P2.50mm, F.Cu at (41.0, 47.5)
- added D2: LED, LED_THT:LED_D1.8mm_W3.3mm_H2.4mm, F.Cu at (300.6, 10.5)
- added GRID_CONTROLLER1: ATmega168A-P, Package_DIP:DIP-28_W7.62mm, F.Cu at (58.4, 30.9)
- added J12: USB_ASP, Connector_IDC:IDC-Header_2x05_P2.54mm_Vertical, F.Cu at (146.5, 96.5)
- added J13: UART_TERM, Connector_PinSocket_2.54mm:PinSocket_1x04_P2.54mm_Vertical, F.Cu at (299.0, 75.9)
- added J14: BUTTONS, TerminalBlock:TerminalBlock_MaiXu_MX126-5.0-03P_1x03_P5.00mm, F.Cu at (95.0, 114.5)
- added J15: PJ-102A, Connector_BarrelJack:BarrelJack_Horizontal, F.Cu at (182.5, 28.1)
- added J17: JOYSTICK, TerminalBlock:TerminalBlock_MaiXu_MX126-5.0-04P_1x04_P5.00mm, F.Cu at (82.0, 114.5)
- added J19: PCF_SCREEN, TerminalBlock:TerminalBlock_MaiXu_MX126-5.0-04P_1x04_P5.00mm, F.Cu at (79.0, 19.5)
- added J20: GROUND, TerminalBlock:TerminalBlock_MaiXu_MX126-5.0-04P_1x04_P5.00mm, F.Cu at (136.5, 52.0)
- added J21: VCC, TerminalBlock:TerminalBlock_MaiXu_MX126-5.0-04P_1x04_P5.00mm, F.Cu at (125.5, 37.5)
- added J3: GRID, TerminalBlock:TerminalBlock_MaiXu_MX126-5.0-03P_1x03_P5.00mm, F.Cu at (23.5, 24.8)
- added R10: 100, Resistor_THT:R_Axial_DIN0207_L6.3mm_D2.5mm_P10.16mm_Horizontal, F.Cu at (240.1, 63.5)
- added R11: 100, Resistor_THT:R_Axial_DIN0207_L6.3mm_D2.5mm_P10.16mm_Horizontal, F.Cu at (240.1, 67.5)
- added R12: 100, Resistor_THT:R_Axial_DIN0207_L6.3mm_D2.5mm_P10.16mm_Horizontal, F.Cu at (281.1, 140.0)
- added R14: 100, Resistor_THT:R_Axial_DIN0207_L6.3mm_D2.5mm_P10.16mm_Horizontal, F.Cu at (229.3, 30.8)
- added R23: 4.7k, Resistor_THT:R_Axial_DIN0207_L6.3mm_D2.5mm_P10.16mm_Horizontal, F.Cu at (273.0, 55.4)
- added R25: 100, Resistor_THT:R_Axial_DIN0207_L6.3mm_D2.5mm_P10.16mm_Horizontal, F.Cu at (281.1, 145.5)
- added R26: 100, Resistor_THT:R_Axial_DIN0207_L6.3mm_D2.5mm_P10.16mm_Horizontal, F.Cu at (240.1, 79.7)
- added R27: 4.7k, Resistor_THT:R_Axial_DIN0207_L6.3mm_D2.5mm_P10.16mm_Horizontal, F.Cu at (240.1, 83.7)
- added R29: 4.7k, Resistor_THT:R_Axial_DIN0207_L6.3mm_D2.5mm_P10.16mm_Horizontal, F.Cu at (273.0, 59.4)
- added R30: 4.7k, Resistor_THT:R_Axial_DIN0207_L6.3mm_D2.5mm_P10.16mm_Horizontal, F.Cu at (273.0, 63.5)
- added R33: 4.7k, Resistor_THT:R_Axial_DIN0207_L6.3mm_D2.5mm_P10.16mm_Horizontal, F.Cu at (273.0, 67.5)
- added R34: 4.7k, Resistor_THT:R_Axial_DIN0207_L6.3mm_D2.5mm_P10.16mm_Horizontal, F.Cu at (273.0, 71.6)
- added R35: 4.7k, Resistor_THT:R_Axial_DIN0207_L6.3mm_D2.5mm_P10.16mm_Horizontal, F.Cu at (273.0, 75.6)
- added R36: 4.7k, Resistor_THT:R_Axial_DIN0207_L6.3mm_D2.5mm_P10.16mm_Horizontal, F.Cu at (273.0, 79.7)
- added R37: 100, Resistor_THT:R_Axial_DIN0207_L6.3mm_D2.5mm_P10.16mm_Horizontal, F.Cu at (229.3, 34.8)
- added R38: 4.7k, Resistor_THT:R_Axial_DIN0207_L6.3mm_D2.5mm_P10.16mm_Horizontal, F.Cu at (240.1, 87.8)
- added R39: 4.7k, Resistor_THT:R_Axial_DIN0207_L6.3mm_D2.5mm_P10.16mm_Horizontal, F.Cu at (229.3, 38.9)
- added R40: 4.7k, Resistor_THT:R_Axial_DIN0207_L6.3mm_D2.5mm_P10.16mm_Horizontal, F.Cu at (229.3, 42.9)
- added R43: 4.7k, Resistor_THT:R_Axial_DIN0207_L6.3mm_D2.5mm_P10.16mm_Horizontal, F.Cu at (229.3, 47.0)
- added R8: 100, Resistor_THT:R_Axial_DIN0207_L6.3mm_D2.5mm_P10.16mm_Horizontal, F.Cu at (240.1, 55.4)
- added R9: 100, Resistor_THT:R_Axial_DIN0207_L6.3mm_D2.5mm_P10.16mm_Horizontal, F.Cu at (280.0, 123.5)
- added SWG_RESET: SWG_Push, Button_Switch_THT:SW_PUSH_6mm, F.Cu at (165.0, 17.0)
- added SWS_RESET: SWS_Push, Button_Switch_THT:SW_PUSH_6mm, F.Cu at (152.0, 17.2)
- added U5: LM2576T-ADJ, Package_TO_SOT_THT:TO-220-5_Vertical, F.Cu at (183.1, 61.5)
- added Y2: Crystal, Crystal:Resonator-2Pin_W6.0mm_H3.0mm, F.Cu at (47.0, 55.0)
- added Y3: Crystal, Crystal:Resonator-2Pin_W6.0mm_H3.0mm, F.Cu at (102.0, 84.5)
- moved H3 247.7 mm to (241.6, -23.0)
- moved R2 225.1 mm to (295.0, 30.7), turned to 0 degrees
- moved H4 208.2 mm to (241.6, -15.1)
- moved H6 191.1 mm to (249.5, -30.9)
- moved H7 179.0 mm to (249.5, -23.0)
- moved R3 169.5 mm to (229.3, 14.6), turned to 0 degrees
- moved R4 169.5 mm to (229.3, 18.6), turned to 0 degrees
- moved H2 166.6 mm to (241.6, -30.9)
- moved R13 159.8 mm to (229.3, 26.7), turned to 0 degrees
- moved R7 159.4 mm to (229.3, 22.6), turned to 0 degrees
- moved H5 158.3 mm to (249.5, -38.9)
- moved G*** 117.0 mm to (107.5, -63.5)
- moved R1 110.1 mm to (229.3, 10.5)
- moved H1 100.8 mm to (241.6, -38.9)
Connections:
- R1 pad 1: GND -> Net-(AUDIO-SCREEN1-PD2)
- R1 pad 2: Net-(D1-K) -> /AUDIO-SCREEN_CONTROLLER/JS_UP
- R13 pad 2: /B_SELECT -> /AUDIO-SCREEN_CONTROLLER/JS_RIGHT
- R2 pad 1: Net-(U1-PD2) -> GND
- R2 pad 2: /JS_UP -> Net-(D2-K)
- R3 pad 2: /JS_DOWN -> /AUDIO-SCREEN_CONTROLLER/JS_DOWN
- R4 pad 2: /JS_LEFT -> /AUDIO-SCREEN_CONTROLLER/JS_LEFT
- R7 pad 2: /B_START -> /AUDIO-SCREEN_CONTROLLER/B_START
Routing:
- net VCC: track 377.4 -> 47.6 mm
- net /RESET: track 150.3 -> 0.00 mm, vias 5 -> 0
- net /SDA: track 70.5 -> 0.00 mm
- net Net-(AUDIO-SCREEN1-PC0): track 69.4 -> 0.00 mm, vias 2 -> 0
- net Net-(U1-PD6): track 68.8 -> 0.00 mm, vias 2 -> 0
- net Net-(AUDIO-SCREEN1-PD7): track 67.2 -> 0.00 mm, vias 2 -> 0
- net GND: track 187.3 -> 121.3 mm, vias 9 -> 0
- net /DIN_GRID: track 61.9 -> 0.00 mm
- net /TXD: track 60.8 -> 0.00 mm, vias 2 -> 0
- net /RXD: track 49.0 -> 0.00 mm, vias 2 -> 0
- net Net-(U1-PD5): track 41.0 -> 0.00 mm
- net /SCL: track 40.6 -> 0.00 mm
- net Net-(AUDIO-SCREEN1-PD4): track 37.2 -> 0.00 mm
- net Net-(AUDIO-SCREEN1-PD3): track 37.1 -> 0.00 mm
- net Net-(U1-PD2): track 36.1 -> 0.00 mm
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- removed copper zone on F.Cu, net GND
- removed copper zone on B.Cu, net VCC
Other:
- board outline removed
- board text removed: "BUTTONS"
- board text removed: "DIN"
- board text removed: "DOWN"
- board text removed: "EXIT"
- board text removed: "GND"
- board text removed: "LEFT"
- board text removed: "MISO"
- board text removed: "MOSI"
- board text removed: "RESET"
- board text removed: "RIGHT"
- board text removed: "RXD"
- board text removed: "SCK"
- board text removed: "SCL"
- board text removed: "SDA"
- board text removed: "SEL."
- board text removed: "START"
- board text removed: "TXD"
- board text removed: "UP"
- board text removed: "VCC"
