File: ATMEGA-SCHEMATICS/SNAKE_GAME/SNAKE_GAME.kicad_pcb (KiCad board)
At the start: 2 copper layers, 81 parts, among them J1 UART_ESP, J12 USB_ASP, J13 UART_TERM, J14 BUTTONS, J15 PJ-102A, J17 JOYSTICK, J19 PCF_SCREEN, J20 GROUND, J21 VCC, J3 GRID, SW2 SWG_Push, SW3 SWS_Push, U1 ESP-12E, U2 FT232RL, U5 LM2576T-ADJ, Y2 Crystal, Y3 Crystal

Commit message: .
Parts:
- added C10: 100nF, Capacitor_THT:C_Disc_D7.5mm_W5.0mm_P5.00mm, F.Cu at (283.6, -95.0)
- added C16: 100nF, Capacitor_THT:C_Disc_D7.5mm_W5.0mm_P5.00mm, F.Cu at (283.6, -88.5)
- added C19: 100nF, Capacitor_THT:C_Disc_D7.5mm_W5.0mm_P5.00mm, F.Cu at (283.6, -81.9)
- added C20: 100nF, Capacitor_THT:C_Disc_D7.5mm_W5.0mm_P5.00mm, F.Cu at (283.6, -75.4)
- added C24: 100nF, Capacitor_THT:C_Disc_D7.5mm_W5.0mm_P5.00mm, F.Cu at (283.6, -68.8)
- added C25: 100nF, Capacitor_THT:C_Disc_D7.5mm_W5.0mm_P5.00mm, F.Cu at (283.6, -62.3)
- added C26: 100nF, Capacitor_THT:C_Disc_D7.5mm_W5.0mm_P5.00mm, F.Cu at (283.6, -55.7)
- added C27: 100nF, Capacitor_THT:C_Disc_D7.5mm_W5.0mm_P5.00mm, F.Cu at (325.9, -92.5)
- added C9: 100nF, Capacitor_THT:C_Disc_D7.5mm_W5.0mm_P5.00mm, F.Cu at (283.6, -101.6)
- added R15: 4.7k, Resistor_THT:R_Axial_DIN0207_L6.3mm_D2.5mm_P10.16mm_Horizontal, F.Cu at (292.2, -94.7)
- added R16: 4.7k, Resistor_THT:R_Axial_DIN0207_L6.3mm_D2.5mm_P10.16mm_Horizontal, F.Cu at (292.2, -90.7)
- added R17: 4.7k, Resistor_THT:R_Axial_DIN0207_L6.3mm_D2.5mm_P10.16mm_Horizontal, F.Cu at (292.2, -86.6)
- added R18: 4.7k, Resistor_THT:R_Axial_DIN0207_L6.3mm_D2.5mm_P10.16mm_Horizontal, F.Cu at (292.2, -82.6)
- added R19: 4.7k, Resistor_THT:R_Axial_DIN0207_L6.3mm_D2.5mm_P10.16mm_Horizontal, F.Cu at (292.2, -78.5)
- added R20: 4.7k, Resistor_THT:R_Axial_DIN0207_L6.3mm_D2.5mm_P10.16mm_Horizontal, F.Cu at (292.2, -74.5)
- added R21: 4.7k, Resistor_THT:R_Axial_DIN0207_L6.3mm_D2.5mm_P10.16mm_Horizontal, F.Cu at (292.2, -70.4)
- added R22: 4.7k, Resistor_THT:R_Axial_DIN0207_L6.3mm_D2.5mm_P10.16mm_Horizontal, F.Cu at (292.2, -66.4)
- added R5: 4.7k, Resistor_THT:R_Axial_DIN0207_L6.3mm_D2.5mm_P10.16mm_Horizontal, F.Cu at (292.2, -102.8)
- added R6: 4.7k, Resistor_THT:R_Axial_DIN0207_L6.3mm_D2.5mm_P10.16mm_Horizontal, F.Cu at (292.2, -98.8)
- added TS5A23159DGSR2: PAD_1&2, Lucas_lib:TS5A23159DGSR, F.Cu at (304.7, -74.6)
- added TS5A23159DGSR5: PAD_3&4, Lucas_lib:TS5A23159DGSR, F.Cu at (304.7, -65.5)
- added TS5A23159DGSR6: CONT_UART_RED_SWT, Lucas_lib:TS5A23159DGSR, F.Cu at (324.6, -96.5)
- added U3: PCF8574AP, Package_DIP:DIP-16_W7.62mm, F.Cu at (305.5, -102.8)
- moved J14 162.2 mm to (-54.5, 51.5)
- moved J17 162.2 mm to (-67.5, 51.5)
- moved AUDIO-SCREEN1 72.5 mm to (139.6, 127.3)
- moved C11 72.5 mm to (159.7, 142.8)
- moved C12 72.5 mm to (161.9, 151.8)
- moved C14 72.5 mm to (123.7, 143.8)
- moved C15 72.5 mm to (123.7, 153.8)
- moved C8 72.5 mm to (130.2, 137.8)
- moved Y3 72.5 mm to (130.2, 151.3)
- moved C13 65.0 mm to (75.5, 116.5)
- moved C1_Crystal1 65.0 mm to (38.5, 112.5)
- moved C2_Crystal1 65.0 mm to (38.0, 121.0)
- moved C6 65.0 mm to (75.0, 109.3)
- moved C7 65.0 mm to (44.5, 108.0)
- moved GRID_CONTROLLER1 65.0 mm to (55.9, 95.9)
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Connections:
- GRID_CONTROLLER1 pad 2: /CONTROLLERS/RXD -> /GRID_CONTROLLER/RXD
- GRID_CONTROLLER1 pad 3: /CONTROLLERS/TXD -> /GRID_CONTROLLER/TXD
- J13 pad 3: /CONTROLLERS/TXD -> /GRID_CONTROLLER/TXD
- J13 pad 4: /CONTROLLERS/RXD -> /GRID_CONTROLLER/RXD

Commit message: .
Parts:
- removed C1, C10 (x2), C16 (x2), C17, C18, C19 (x2), C20 (x2), C3, C4, C9 (x2): 100nF, Capacitor_THT:C_Disc_D7.5mm_W5.0mm_P5.00mm
- removed C2: 1uF, Capacitor_THT:C_Disc_D7.5mm_W5.0mm_P5.00mm
- removed C5: C_Small, Capacitor_THT:C_Disc_D7.5mm_W5.0mm_P5.00mm
- removed G***: LOGO, Connector_Pin:snake
- removed J1: UART_ESP, Connector_PinSocket_2.54mm:PinSocket_1x04_P2.54mm_Vertical
- removed R15, R16, R17, R18, R19, R20, R21, R22, R5, R6: 4.7k, Resistor_THT:R_Axial_DIN0207_L6.3mm_D2.5mm_P10.16mm_Horizontal
- removed SW2: SWG_Push, Button_Switch_THT:SW_PUSH_6mm
- removed SW3: SWS_Push, Button_Switch_THT:SW_PUSH_6mm
- removed TS5A23159DGSR1: CONT_UART_RED_SWT, Lucas_lib:TS5A23159DGSR
- removed TS5A23159DGSR2, TS5A23159DGSR4: PAD_1&2, Lucas_lib:TS5A23159DGSR
- removed TS5A23159DGSR2: PAD_3&4, Lucas_lib:TS5A23159DGSR
- removed U1: ESP-12E, RF_Module:ESP-12E
- removed U2: FT232RL, Package_SO:SSOP-28_5.3x10.2mm_P0.65mm
- removed U3: PCF8574AP, Package_DIP:DIP-16_W7.62mm
- removed U5: LM2576T-ADJ, Package_TO_SOT_THT:TO-220-5_Vertical
- added 23A1024/23LC1: ~, Package_DIP:CERDIP-8_W7.62mm_SideBrazed_Socket, F.Cu at (120.1, 89.7)
- added 47uF1: C_Polarized, Capacitor_THT:C_Disc_D3.0mm_W1.6mm_P2.50mm, F.Cu at (137.7, 28.9)
- added BZ1: Buzzer, Buzzer_Beeper:Buzzer_12x9.5RM7.6, F.Cu at (41.5, 62.6)
- added C22: 100nF, Capacitor_THT:C_Disc_D7.5mm_W5.0mm_P5.00mm, F.Cu at (111.1, 42.4)
- added C23: 100nF, Capacitor_THT:C_Disc_D7.5mm_W5.0mm_P5.00mm, F.Cu at (118.1, 107.3)
- added C28: 100nF, Capacitor_THT:C_Disc_D7.5mm_W5.0mm_P5.00mm, F.Cu at (104.3, 102.6)
- added C29: 100nF, Capacitor_THT:C_Disc_D7.5mm_W5.0mm_P5.00mm, F.Cu at (88.0, 114.0)
- added C77: 1uF, Capacitor_THT:C_Disc_D7.5mm_W5.0mm_P5.00mm, F.Cu at (136.9, 40.0)
- added D7: V_METER- LED, LED_THT:LED_D1.8mm_W3.3mm_H2.4mm, F.Cu at (144.2, 29.4)
- added J2: Vibrator, TerminalBlock:TerminalBlock_MaiXu_MX126-5.0-02P_1x02_P5.00mm, F.Cu at (33.6, 73.9)
- added R41: 100, Resistor_THT:R_Axial_DIN0207_L6.3mm_D2.5mm_P10.16mm_Horizontal, F.Cu at (38.6, 37.8)
- added R42: 100, Resistor_THT:R_Axial_DIN0207_L6.3mm_D2.5mm_P10.16mm_Horizontal, F.Cu at (33.1, 45.8)
- added R44: 4.7k, Resistor_THT:R_Axial_DIN0207_L6.3mm_D2.5mm_P10.16mm_Horizontal, F.Cu at (133.2, 114.5)
- added R45: 4.7k, Resistor_THT:R_Axial_DIN0207_L6.3mm_D2.5mm_P10.16mm_Horizontal, F.Cu at (57.3, 109.2)
- added R46: 4.7k, Resistor_THT:R_Axial_DIN0207_L6.3mm_D2.5mm_P10.16mm_Horizontal, F.Cu at (152.6, 90.4)
- added R54: 1k, Resistor_THT:R_Axial_DIN0207_L6.3mm_D2.5mm_P10.16mm_Horizontal, F.Cu at (144.3, 33.9)
- added R55: 4.7k, Resistor_THT:R_Axial_DIN0207_L6.3mm_D2.5mm_P10.16mm_Horizontal, F.Cu at (64.1, 111.7)
- added R56: 4.7k, Resistor_THT:R_Axial_DIN0207_L6.3mm_D2.5mm_P10.16mm_Horizontal, F.Cu at (87.5, 105.3)
- added R57: 4.7k, Resistor_THT:R_Axial_DIN0207_L6.3mm_D2.5mm_P10.16mm_Horizontal, F.Cu at (41.8, 88.5)
- added R59: 4.7k, Resistor_THT:R_Axial_DIN0207_L6.3mm_D2.5mm_P10.16mm_Horizontal, F.Cu at (80.3, 121.1)
- added SN74HC1: ~, Package_DIP:CERDIP-14_W7.62mm_SideBrazed_Socket, F.Cu at (95.9, 120.8)
- added SW4: SWS_Push, Button_Switch_THT:SW_PUSH_6mm, F.Cu at (157.2, 116.9)
- added SW6: SPI_PROG., Button_Switch_THT:SW_Slide_SPDT_Straight_CK_OS102011MS2Q, F.Cu at (47.3, 117.4)
- added TPS75533KCG1: ~, Package_TO_SOT_THT:TO-220-5_Vertical, F.Cu at (129.8, 39.1)
- C14, C15: footprint Capacitor_THT:C_Disc_D7.5mm_W5.0mm_P5.00mm -> Capacitor_THT:CP_Radial_D5.0mm_P2.50mm
- C24: value 100nF -> 1uF
- C25: value 100nF -> 22uF
- R2: value 100 -> 1k
- TS5A23159DGSR5: value PAD_3&4 -> SPI_CONTROL_MOSI-MISO; footprint Lucas_lib:TS5A23159DGSR -> LucasLib:TS5A23159DGSR
- TS5A23159DGSR6: value CONT_UART_RED_SWT -> SPI_CONTROL_SCK-RESET; footprint Lucas_lib:TS5A23159DGSR -> LucasLib:TS5A23159DGSR
- moved TS5A23159DGSR5 295.5 mm to (54.5, 91.7), turned to 180 degrees
- moved TS5A23159DGSR6 280.9 mm to (125.3, 101.5), turned to 180 degrees
- moved C26 280.0 mm to (49.1, 97.3), turned to 180 degrees
- moved C27 276.4 mm to (112.9, 83.7), turned to 90 degrees
- moved H5 276.1 mm to (25.5, 122.5), turned to -90 degrees
- moved H7 249.5 mm to (25.5, 86.9), turned to -90 degrees
- moved R33 225.3 mm to (49.1, 42.2), turned to -90 degrees
- moved H1 224.4 mm to (25.5, 21.7), turned to -90 degrees
- moved R34 221.0 mm to (54.0, 42.0), turned to -90 degrees
- moved R35 216.4 mm to (59.2, 42.1), turned to -90 degrees
- moved R36 212.3 mm to (64.0, 42.2), turned to -90 degrees
- moved R23 199.4 mm to (73.9, 42.3), turned to -90 degrees
- moved C24 197.7 mm to (120.1, 42.3), turned to 90 degrees
- moved R29 194.7 mm to (79.0, 42.4), turned to -90 degrees
- moved R30 189.5 mm to (84.6, 42.2), turned to -90 degrees
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Connections:
- net /AUDIO-SCREEN_CONTROLLER/B_EXIT renamed /AUDIO-SCREEN_CONTROLLER/B_EXIT_USR
- net /AUDIO-SCREEN_CONTROLLER/B_SELECT renamed /AUDIO-SCREEN_CONTROLLER/B_SELECT_USR
- net /AUDIO-SCREEN_CONTROLLER/B_START renamed /AUDIO-SCREEN_CONTROLLER/B_START_USR
- net /AUDIO-SCREEN_CONTROLLER/JS_DOWN renamed /AUDIO-SCREEN_CONTROLLER/JS_DOWN_USR
- net /AUDIO-SCREEN_CONTROLLER/JS_LEFT renamed /AUDIO-SCREEN_CONTROLLER/JS_LEFT_USR
- net /AUDIO-SCREEN_CONTROLLER/JS_RIGHT renamed /AUDIO-SCREEN_CONTROLLER/JS_RIGHT_USR
- net /AUDIO-SCREEN_CONTROLLER/JS_UP renamed /AUDIO-SCREEN_CONTROLLER/JS_UP_USR
- AUDIO-SCREEN1 pad 11: /AUDIO-SCREEN_CONTROLLER/DAC1 -> /AUDIO-SCREEN_CONTROLLER/DAC1_VIBRATOR
- AUDIO-SCREEN1 pad 12: /AUDIO-SCREEN_CONTROLLER/DAC2 -> /AUDIO-SCREEN_CONTROLLER/DAC2_BUZZER
- AUDIO-SCREEN1 pad 15: /AUDIO-SCREEN_CONTROLLER/INT3 -> REG_EN_LOW
- AUDIO-SCREEN1 pad 16: /AUDIO-SCREEN_CONTROLLER/INT4 -> unconnected-(AUDIO-SCREEN1-PB2-Pad16)
- AUDIO-SCREEN1 pad 2: /AUDIO-SCREEN_CONTROLLER/RXD -> /AUDIO-SCREEN_CONTROLLER/RXD_TERM_USR
- AUDIO-SCREEN1 pad 21: Net-(AUDIO-SCREEN1-AREF) -> VCC
- AUDIO-SCREEN1 pad 24: Net-(AUDIO-SCREEN1-PC0) -> Net-(AUDIO-SCREEN1-PC1)
- AUDIO-SCREEN1 pad 25: /AUDIO-SCREEN_CONTROLLER/INT1 -> /AUDIO-SCREEN_CONTROLLER/INT1_USR
- AUDIO-SCREEN1 pad 26: /AUDIO-SCREEN_CONTROLLER/INT2 -> PG
- AUDIO-SCREEN1 pad 27: /AUDIO-SCREEN_CONTROLLER/SDA -> /AUDIO-SCREEN_CONTROLLER/USR_SDA
- AUDIO-SCREEN1 pad 28: /AUDIO-SCREEN_CONTROLLER/SCL -> /AUDIO-SCREEN_CONTROLLER/USR_SCL
- AUDIO-SCREEN1 pad 3: /AUDIO-SCREEN_CONTROLLER/TXD -> /AUDIO-SCREEN_CONTROLLER/TXD_TERM_USR
- C11 pad 2: Net-(AUDIO-SCREEN1-AREF) -> VCC
- C24 pad 1: VCC -> GND
- C24 pad 2: GND -> VCC
- C25 pad 1: Net-(TS5A23159DGSR2-NC2) -> GND
- C25 pad 2: unconnected-(C25-Pad2) -> VCC
- C26 pad 1: Net-(TS5A23159DGSR5-NC2) -> VCC
- C26 pad 2: unconnected-(C26-Pad2) -> GND
- C27 pad 1: VCC -> Net-(23A1024/23LC1-SIO2)
- C27 pad 2: unconnected-(C27-Pad2) -> GND
- C6 pad 2: Net-(GRID_CONTROLLER1-AREF) -> VCC
- GRID_CONTROLLER1 pad 1: /AUDIO-SCREEN_CONTROLLER/RESET -> /CONTROLLERS/RESET_GRID
- GRID_CONTROLLER1 pad 15: /AUDIO-SCREEN_CONTROLLER/INT3 -> unconnected-(GRID_CONTROLLER1-PB1-Pad15)
- GRID_CONTROLLER1 pad 16: /AUDIO-SCREEN_CONTROLLER/INT4 -> unconnected-(GRID_CONTROLLER1-PB2-Pad16)
- GRID_CONTROLLER1 pad 17: /AUDIO-SCREEN_CONTROLLER/MOSI -> /CONTROLLERS/MOSI_GRID
- GRID_CONTROLLER1 pad 18: /AUDIO-SCREEN_CONTROLLER/MISO -> /CONTROLLERS/MISO_GRID
- GRID_CONTROLLER1 pad 19: /AUDIO-SCREEN_CONTROLLER/SCK -> /CONTROLLERS/SCK_GRID
- GRID_CONTROLLER1 pad 2: /GRID_CONTROLLER/RXD -> /AUDIO-SCREEN_CONTROLLER/RXD_TERM_USR
- GRID_CONTROLLER1 pad 21: Net-(GRID_CONTROLLER1-AREF) -> VCC
- GRID_CONTROLLER1 pad 24: /AUDIO-SCREEN_CONTROLLER/INT1 -> unconnected-(GRID_CONTROLLER1-PC1-Pad24)
- GRID_CONTROLLER1 pad 25: /AUDIO-SCREEN_CONTROLLER/INT2 -> unconnected-(GRID_CONTROLLER1-PC2-Pad25)
- GRID_CONTROLLER1 pad 26: unconnected-(GRID_CONTROLLER1-PC3-Pad26) -> /AUDIO-SCREEN_CONTROLLER/INT1_USR
- GRID_CONTROLLER1 pad 27: unconnected-(GRID_CONTROLLER1-PC4-Pad27) -> /AUDIO-SCREEN_CONTROLLER/USR_SDA
- GRID_CONTROLLER1 pad 28: unconnected-(GRID_CONTROLLER1-PC5-Pad28) -> /AUDIO-SCREEN_CONTROLLER/USR_SCL
- GRID_CONTROLLER1 pad 3: /GRID_CONTROLLER/TXD -> /AUDIO-SCREEN_CONTROLLER/TXD_TERM_USR
- J12 pad 1: /AUDIO-SCREEN_CONTROLLER/MOSI -> /CONTROLLERS/MOSI
- J12 pad 5: /AUDIO-SCREEN_CONTROLLER/RESET -> /CONTROLLERS/RESET
- J12 pad 7: /AUDIO-SCREEN_CONTROLLER/SCK -> /CONTROLLERS/SCK
- J12 pad 9: /AUDIO-SCREEN_CONTROLLER/MISO -> /CONTROLLERS/MISO
- J13 pad 3: /GRID_CONTROLLER/TXD -> /AUDIO-SCREEN_CONTROLLER/RXD_TERM_USR
- J13 pad 4: /GRID_CONTROLLER/RXD -> /AUDIO-SCREEN_CONTROLLER/TXD_TERM_USR
- J19 pad 3: /AUDIO-SCREEN_CONTROLLER/SDA -> /AUDIO-SCREEN_CONTROLLER/USR_SDA
- J19 pad 4: /AUDIO-SCREEN_CONTROLLER/SCL -> /AUDIO-SCREEN_CONTROLLER/USR_SCL
- J3 pad 1: VCC -> VCC_LED_GRID
- R14 pad 1: Net-(AUDIO-SCREEN1-PC0) -> Net-(AUDIO-SCREEN1-PC1)
- R27 pad 1: /AUDIO-SCREEN_CONTROLLER/RESET -> /CONTROLLERS/RESET_GRID
- R39 pad 2: /AUDIO-SCREEN_CONTROLLER/SCL -> /AUDIO-SCREEN_CONTROLLER/USR_SCL
- R40 pad 2: /AUDIO-SCREEN_CONTROLLER/SDA -> /AUDIO-SCREEN_CONTROLLER/USR_SDA
- TS5A23159DGSR5 pad 1: /AUDIO-SCREEN_CONTROLLER/PAD_3_SWT -> /CONTROLLERS/GRID_RAM_SIGNAL
- TS5A23159DGSR6 pad 1: unconnected-(TS5A23159DGSR6-IN1-Pad1) -> /CONTROLLERS/GRID_RAM_SIGNAL
Routing:
- net VCC: track 47.6 -> 262.5 mm, vias 0 -> 1
- net /AUDIO-SCREEN_CONTROLLER/JS_RIGHT_USR: track 0.00 -> 210.5 mm, vias 0 -> 4
- net REG_EN_LOW: track 0.00 -> 209.6 mm, vias 0 -> 2
- net GND: track 121.3 -> 299.9 mm, vias 0 -> 12
- net /CONTROLLERS/GRID_RAM_SIGNAL: track 0.00 -> 159.7 mm, vias 0 -> 5
- net /AUDIO-SCREEN_CONTROLLER/TXD_TERM_USR: track 0.00 -> 147.6 mm, vias 0 -> 2
- net /AUDIO-SCREEN_CONTROLLER/RXD_TERM_USR: track 0.00 -> 142.7 mm, vias 0 -> 2
- net /AUDIO-SCREEN_CONTROLLER/B_EXIT_USR: track 0.00 -> 137.4 mm, vias 0 -> 2
- net /AUDIO-SCREEN_CONTROLLER/JS_LEFT_USR: track 0.00 -> 137.0 mm, vias 0 -> 2
- net /AUDIO-SCREEN_CONTROLLER/JS_DOWN_USR: track 0.00 -> 134.6 mm, vias 0 -> 2
- net /AUDIO-SCREEN_CONTROLLER/USR_SDA: track 0.00 -> 129.5 mm, vias 0 -> 2
- net /CONTROLLERS/RESET_GRID: track 0.00 -> 126.2 mm, vias 0 -> 2
- net /AUDIO-SCREEN_CONTROLLER/JS_UP_USR: track 0.00 -> 125.6 mm, vias 0 -> 2
- net /AUDIO-SCREEN_CONTROLLER/B_SELECT_USR: track 0.00 -> 116.8 mm, vias 0 -> 2
- net /AUDIO-SCREEN_CONTROLLER/USR_SCL: track 0.00 -> 105.6 mm, vias 0 -> 2
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- added copper zone on F.Cu, net GND
- added copper zone on B.Cu, net VCC
Other:
- board outline added: 165 x 108 mm
- board text removed: "═════════════════════════════ Project: Snake Game MCU: ATmega168A Board: Custom PCB Course: UMB-CS341-F25 Semester: Fall 2025 Author: Lucas Nascimento ══════════════════════════════"

Commit message: ..
Parts:
- removed C26: 100nF, Capacitor_THT:C_Disc_D7.5mm_W5.0mm_P5.00mm
- removed TS5A23159DGSR5: SPI_CONTROL_MOSI-MISO, LucasLib:TS5A23159DGSR
- removed TS5A23159DGSR6: SPI_CONTROL_SCK-RESET, LucasLib:TS5A23159DGSR
- added C30: 100nF, Capacitor_THT:C_Disc_D7.5mm_W5.0mm_P5.00mm, F.Cu at (142.8, 111.8)
- added C31: 100nF, Capacitor_THT:C_Disc_D7.5mm_W5.0mm_P5.00mm, F.Cu at (53.5, 98.1)
- added C33: 1uF, Capacitor_THT:C_Disc_D7.5mm_W5.0mm_P5.00mm, F.Cu at (61.4, 93.1)
- added C34: 1uF, Capacitor_THT:C_Disc_D7.5mm_W5.0mm_P5.00mm, F.Cu at (137.8, 115.9)
- added U1: CD4066BE, Package_DIP:DIP-14_W7.62mm, F.Cu at (40.5, 95.4)
- added U2: CD4066BE, Package_DIP:DIP-14_W7.62mm, F.Cu at (135.8, 102.9)
- moved R44 18.8 mm to (152.0, 113.6), turned to 90 degrees
- moved J12 5.65 mm to (29.6, 109.1)
- moved C23 3.86 mm to (114.2, 107.2)
Connections:
- SN74HC1 pad 5: Net-(SN74HC1-1A) -> /CONTROLLERS/GRID_RAM_SIGNAL
- SN74HC1 pad 6: unconnected-(SN74HC1-3Y-Pad6) -> Net-(SN74HC1-3Y)
Routing:
- net Net-(SN74HC1-3Y): track 0.00 -> 201.9 mm, vias 0 -> 7
- net /CONTROLLERS/GRID_RAM_SIGNAL: track 159.7 -> 219.8 mm, vias 5 -> 7
- net /CONTROLLERS/MISO: track 26.9 -> 79.5 mm, vias 1 -> 2
- net /CONTROLLERS/SCK: track 103.7 -> 151.0 mm, vias 1 -> 2
- net VCC: track 262.5 -> 298.7 mm, vias 1 -> 5
- net /CONTROLLERS/MOSI_GRID: track 95.1 -> 129.2 mm, vias 1 -> 2
- net GND: track 299.9 -> 332.2 mm, vias 12 -> 15
- net /CONTROLLERS/RESET: track 103.0 -> 129.1 mm, vias 3 -> 4
- net /CONTROLLERS/MISO_GRID: track 103.5 -> 120.7 mm, vias 3 -> 6
- net Net-(SN74HC1-1A): track 84.1 -> 99.5 mm, vias 0 -> 2
- net /CONTROLLERS/SCK_GRID: track 57.1 -> 43.2 mm, vias 1 -> 0
- net /AUDIO-SCREEN_CONTROLLER/MOSI: track 15.4 -> 29.2 mm, vias 1 -> 0
- net /AUDIO-SCREEN_CONTROLLER/MISO: track 23.2 -> 33.2 mm, vias 1 -> 2
- net /CONTROLLERS/RESET_GRID: track 126.2 -> 135.6 mm
- net /CONTROLLERS/MOSI: track 26.2 -> 28.6 mm, vias 1 -> 2
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
Commit message: ..
Parts:
- removed H3: MountingHole, MountingHole:MountingHole_3.2mm_M3
- moved SW6 4.70 mm to (45.0, 121.5), turned to 0 degrees
Routing:
- net GND: track 332.2 -> 291.4 mm
- net VCC: track 298.7 -> 323.2 mm
- net /CONTROLLERS/GRID_RAM_SIGNAL: track 219.8 -> 236.8 mm, vias 7 -> 8
- net /GRID_CONTROLLER/DIN_GRID: track 68.7 -> 61.1 mm
- net /AUDIO-SCREEN_CONTROLLER/RXD_TERM_USR: track 142.7 -> 149.1 mm
- net /CONTROLLERS/MISO_GRID: track 120.7 -> 125.1 mm
- net /AUDIO-SCREEN_CONTROLLER/JS_DOWN_USR: track 134.6 -> 130.5 mm
- net /AUDIO-SCREEN_CONTROLLER/JS_RIGHT_USR: track 208.7 -> 212.7 mm
- net /AUDIO-SCREEN_CONTROLLER/TXD_TERM_USR: track 147.6 -> 151.5 mm
- net /AUDIO-SCREEN_CONTROLLER/B_SELECT_USR: track 116.8 -> 120.6 mm
- net /CONTROLLERS/MOSI: track 28.6 -> 32.2 mm
- net /CONTROLLERS/MISO: track 79.5 -> 83.0 mm
- net PG: track 98.5 -> 101.6 mm
- net /AUDIO-SCREEN_CONTROLLER/B_START_USR: track 103.4 -> 106.5 mm
- net /AUDIO-SCREEN_CONTROLLER/JS_UP_USR: track 125.6 -> 128.5 mm
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
Commit message: .
Parts:
- added H3: MountingHole, MountingHole:MountingHole_3.2mm_M3, F.Cu at (62.4, 23.0)
Changed lines of the file:
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@@
 		)
 	)
+	(footprint "MountingHole:MountingHole_3.2mm_M3"
+		(layer "F.Cu")
+		(at 62.4 23)
+		(descr "Mounting Hole 3.2mm, no annular, M3")
+		(tags "mounting hole 3.2mm no annular m3")
+		(property "Reference" "H3"
+			(at 0 -4.2 0)
+			(layer "F.SilkS")
+			(effects
+				(font
+					(size 1 1)
+					(thickness 0.15)
+				)
+			)
+		)
+		(property "Value" "MountingHole"
+			(at 0 4.2 0)
+			(layer "F.Fab")
+			(effects
+				(font
+					(size 1 1)
+					(thickness 0.15)
+				)
+			)
+		)
+		(property "Datasheet" ""
+			(at 0 0 0)
+			(unlocked yes)
+			(layer "F.Fab")
+			(hide yes)
+			(effects
+				(font
+					(size 1.27 1.27)
+					(thickness 0.15)
+				)
+			)
+		)
+		(property "Description" "Mounting Hole without connection"
+			(at 0 0 0)
+			(unlocked yes)
+			(layer "F.Fab")
+			(hide yes)
+			(effects
+				(font
+					(size 1.27 1.27)
+					(thickness 0.15)
+				)
+			)
+		)
+		(property ki_fp_filters "MountingHole*")
+		(sheetname "/")
+		(sheetfile "SNAKE_GAME.kicad_sch")
+		(attr exclude_from_pos_files exclude_from_bom)
+		(fp_circle
+			(center 0 0)
+			(end 3.2 0)
+			(stroke
+				(width 0.15)
+				(type solid)
+			)
+			(fill no)
+			(layer "Cmts.User")
+		)
+		(fp_circle
+			(center 0 0)
+			(end 3.45 0)
+			(stroke
+				(width 0.05)
+				(type solid)
+			)
+			(fill no)
+			(layer "F.CrtYd")
+		)
+		(fp_text user "${REFERENCE}"
+			(at 0 0 0)
+			(layer "F.Fab")
+			(effects
+				(font
+					(size 1 1)
+					(thickness 0.15)
+				)
+			)
+		)
+		(pad "" np_thru_hole circle
+			(at 0 0)
+			(size 3.2 3.2)
+			(drill 3.2)
+			(layers "*.Cu" "*.Mask")
+		)
+		(embedded_fonts no)
+	)
 	(footprint "Resistor_THT:R_Axial_DIN0207_L6.3mm_D2.5mm_P10.16mm_Horizontal"
 		(layer "F.Cu")
@@
 		(min_thickness 0.25)
 		(filled_areas_thickness no)
-		(fill
+		(fill yes
 			(thermal_gap 0.5)
 			(thermal_bridge_width 0.5)
@@
 		(min_thickness 0.25)
 		(filled_areas_thickness no)
-		(fill
+		(fill yes
 			(thermal_gap 0.5)
 			(thermal_bridge_width 0.5)
