File: ATMEGA-SCHEMATICS/SNAKE_GAME/SNAKE_GAME.kicad_sch (KiCad schematic)
At the start: 43 parts, among them J1 GRID, J10 VCC, J11 PJ-102A, J3 Conn_01x03_Pin, J4 USB_ASP, J5 BUTTONS, J6 JOYSTICK, J7 UART_TERM, J8 PCF_SCREEN, J9 GROUND, U1 ATmega168A-P, U4 LM2576T-ADJ, Y1 Crystal

Commit message: .
Parts:
- removed C6, C7: C_Small, Capacitor_THT:CP_Radial_D5.0mm_P2.50mm, symbol Device:C_Small
- removed D1: LED, symbol Device:LED
- removed D2: 1N5822, Diode_THT:D_DO-201AD_P15.24mm_Horizontal, symbol Diode:1N5822
- removed L2: 100uH, Library:SRN8040-101M, symbol Device:L
- removed R23, R25: 4.7k, Resistor_THT:R_Axial_DIN0207_L6.3mm_D2.5mm_P10.16mm_Horizontal, symbol Device:R
- removed R26: 1k, Resistor_THT:R_Axial_DIN0207_L6.3mm_D2.5mm_P10.16mm_Horizontal, symbol Device:R
- removed U4: LM2576T-ADJ, Package_TO_SOT_THT:TO-220-5_Vertical, symbol Regulator_Switching:LM2576T-ADJ
- added 220UF1: C_Polarized, Capacitor_THT:C_Disc_D3.0mm_W1.6mm_P2.50mm, symbol Device:C_Polarized
- added H1, H2, H3, H4: MountingHole, MountingHole:MountingHole_3.2mm_M3, symbol Mechanical:MountingHole
- added SW1: SW_Push, Button_Switch_THT:SW_PUSH_6mm, symbol Switch:SW_Push
- J1, J5: footprint (none) -> TerminalBlock:TerminalBlock_MaiXu_MX126-5.0-03P_1x03_P5.00mm
- J10, J6, J8, J9: footprint (none) -> TerminalBlock:TerminalBlock_MaiXu_MX126-5.0-04P_1x04_P5.00mm
- J11: footprint digikey-footprints:Barrel_Jack_5.5mmODx2.1mmID_PJ-102A -> Connector_BarrelJack:BarrelJack_Horizontal
- J3: footprint (none) -> Connector_PinSocket_2.54mm:PinSocket_1x03_P2.54mm_Vertical
- J4: footprint (none) -> Connector_IDC:IDC-Header_2x05_P2.54mm_Vertical
- J7: footprint (none) -> Connector_PinSocket_2.54mm:PinSocket_1x04_P2.54mm_Vertical
Connections:
- net GND: now also 220UF1.2
- net RESET: now also SW1.1; no longer J3.2 (Pin_2)
- net VCC: now also C1.2, C4.2, U1.20 (AVCC), U1.7 (VCC), 220UF1.1
- net CS: no longer names the net of U1.16 (PB2)
- net SCREEN_INT: no longer names the net of U1.26 (PC3)
- new net: J3.2 (Pin_2), SW1.2
- no-connect marks 5 -> 10
Other:
- moved on the sheet: J11, J3

Commit message: .
Parts:
- added D1: LED, LED_THT:LED_D1.8mm_W3.3mm_H2.4mm, symbol Device:LED
- added H5, H6, H7: MountingHole, MountingHole:MountingHole_3.2mm_M3, symbol Mechanical:MountingHole
- added R1: 100, Resistor_THT:R_Axial_DIN0207_L6.3mm_D2.5mm_P10.16mm_Horizontal, symbol Device:R
Connections:
- net GND: now also J4.3 (Pin_3), J4.4 (Pin_4), J4.6 (Pin_6), R1.1
- net VCC: now also D1.2 (A)
- new net: D1.1 (K), R1.2
- no-connect marks 10 -> 7

Commit message: .
Parts:
- removed J3: Conn_01x03_Pin, Connector_PinSocket_2.54mm:PinSocket_1x03_P2.54mm_Vertical, symbol Connector:Conn_01x03_Pin
- added R23: 4.7k, Resistor_THT:R_Axial_DIN0207_L6.3mm_D2.5mm_P10.16mm_Horizontal, symbol Device:R
Connections:
- net GND: now also SW1.2
- net RESET: now also R23.1
- net VCC: now also R23.2
Other:
- moved on the sheet: SW1
Changed lines of the file:
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@@
 	)
 	(junction
+		(at 76.2 78.74)
+		(diameter 0)
+		(color 0 0 0 0)
+	)
+	(junction
 		(at 144.78 152.4)
 		(diameter 0)
@@
 	)
 	(junction
+		(at 71.12 76.2)
+		(diameter 0)
+		(color 0 0 0 0)
+	)
+	(junction
 		(at 102.87 147.32)
 		(diameter 0)
@@
 	(wire
 		(pts
-			(xy 73.66 78.74) (xy 82.55 78.74)
-		)
-		(stroke
-			(width 0)
-			(type default)
-		)
-	)
-	(wire
-		(pts
 			(xy 232.41 35.56) (xy 236.22 35.56)
 		)
@@
 	(wire
 		(pts
-			(xy 73.66 76.2) (xy 54.61 76.2)
+			(xy 76.2 78.74) (xy 72.39 78.74)
 		)
 		(stroke
@@
 	(wire
 		(pts
+			(xy 71.12 76.2) (xy 54.61 76.2)
+		)
+		(stroke
+			(width 0)
+			(type default)
+		)
+	)
+	(wire
+		(pts
 			(xy 66.04 55.88) (xy 66.04 59.69)
 		)
@@
 	(wire
 		(pts
-			(xy 92.71 78.74) (xy 97.79 78.74)
+			(xy 86.36 78.74) (xy 97.79 78.74)
 		)
 		(stroke
@@
 	(wire
 		(pts
+			(xy 76.2 69.85) (xy 76.2 78.74)
+		)
+		(stroke
+			(width 0)
+			(type default)
+		)
+	)
+	(wire
+		(pts
+			(xy 72.39 76.2) (xy 71.12 76.2)
+		)
+		(stroke
+			(width 0)
+			(type default)
+		)
+	)
+	(wire
+		(pts
 			(xy 82.55 52.07) (xy 82.55 59.69)
 		)
@@
 	(wire
 		(pts
+			(xy 72.39 78.74) (xy 72.39 76.2)
+		)
+		(stroke
+			(width 0)
+			(type default)
+		)
+	)
+	(wire
+		(pts
 			(xy 124.46 149.86) (xy 128.27 149.86)
 		)
@@
 	(wire
 		(pts
-			(xy 73.66 78.74) (xy 73.66 76.2)
-		)
-		(stroke
-			(width 0)
-			(type default)
-		)
-	)
-	(wire
-		(pts
 			(xy 54.61 71.12) (xy 58.42 71.12)
 		)
@@
 	)
 	(label "RESET"
-		(at 73.66 76.2 0)
+		(at 76.2 69.85 0)
 		(effects
 			(font
@@
 	)
 	(symbol
-		(lib_id "Connector:Conn_01x03_Pin")
-		(at 102.87 78.74 180)
-		(unit 1)
-		(exclude_from_sim no)
-		(in_bom yes)
-		(on_board yes)
-		(dnp no)
-		(fields_autoplaced yes)
-		(property "Reference" "J3"
-			(at 104.14 77.4699 0)
-			(effects
-				(font
-					(size 1.27 1.27)
-				)
-				(justify right)
-			)
-		)
-		(property "Value" "Conn_01x03_Pin"
-			(at 104.14 80.0099 0)
-			(effects
-				(font
-					(size 1.27 1.27)
-				)
-				(justify right)
-			)
-		)
-		(property "Footprint" "Connector_PinSocket_2.54mm:PinSocket_1x03_P2.54mm_Vertical"
-			(at 102.87 78.74 0)
-			(effects
-				(font
-					(size 1.27 1.27)
-				)
-				(hide yes)
-			)
-		)
-		(property "Datasheet" "~"
-			(at 102.87 78.74 0)
-			(effects
-				(font
-					(size 1.27 1.27)
-				)
-				(hide yes)
-			)
-		)
-		(property "Description" "Generic connector, single row, 01x03, script generated"
-			(at 102.87 78.74 0)
-			(effects
-				(font
-					(size 1.27 1.27)
-				)
-				(hide yes)
-			)
-		)
-		(pin "3"
-		)
-		(pin "1"
-		)
-		(pin "2"
-		)
-		(instances
-			(project "SNAKE_GAME"
-				(path "/6a8c7582-1032-4e02-bf22-b5197316f506"
-					(reference "J3")
-					(unit 1)
-				)
-			)
-		)
-	)
-	(symbol
 		(lib_id "Connector:Conn_01x05_Pin")
 		(at 120.65 175.26 0)
@@
 	)
 	(symbol
+		(lib_id "Device:R")
+		(at 71.12 72.39 180)
+		(unit 1)
+		(exclude_from_sim no)
+		(in_bom yes)
+		(on_board yes)
+		(dnp no)
+		(property "Reference" "R23"
+			(at 69.088 72.39 90)
+			(effects
+				(font
+					(size 1.27 1.27)
+				)
+			)
+		)
+		(property "Value" "4.7k"
+			(at 71.12 72.136 90)
+			(effects
+				(font
+					(size 1.27 1.27)
+				)
+			)
+		)
+		(property "Footprint" "Resistor_THT:R_Axial_DIN0207_L6.3mm_D2.5mm_P10.16mm_Horizontal"
+			(at 72.898 72.39 90)
+			(effects
+				(font
+					(size 1.27 1.27)
+				)
+				(hide yes)
+			)
+		)
+		(property "Datasheet" "~"
+			(at 71.12 72.39 0)
+			(effects
+				(font
+					(size 1.27 1.27)
+				)
+				(hide yes)
+			)
+		)
+		(property "Description" "Resistor"
+			(at 71.12 72.39 0)
+			(effects
+				(font
+					(size 1.27 1.27)
+				)
+				(hide yes)
+			)
+		)
+		(pin "1"
+		)
+		(pin "2"
+		)
+		(instances
+			(project "SNAKE_GAME"
+				(path "/6a8c7582-1032-4e02-bf22-b5197316f506"
+					(reference "R23")
+					(unit 1)
+				)
+			)
+		)
+	)
+	(symbol
 		(lib_id "power:GND")
 		(at 43.18 149.86 0)
@@
 	(symbol
 		(lib_id "power:VCC")
-		(at 97.79 76.2 0)
+		(at 71.12 68.58 90)
 		(unit 1)
 		(exclude_from_sim no)
@@
 		(fields_autoplaced yes)
 		(property "Reference" "#PWR07"
-			(at 97.79 80.01 0)
+			(at 74.93 68.58 0)
 			(effects
 				(font
@@
 		)
 		(property "Value" "VCC"
-			(at 97.79 71.12 0)
+			(at 69.85 66.04 90)
 			(effects
 				(font
@@
 		)
 		(property "Footprint" ""
-			(at 97.79 76.2 0)
+			(at 71.12 68.58 0)
 			(effects
 				(font
@@
 		)
 		(property "Datasheet" ""
-			(at 97.79 76.2 0)
+			(at 71.12 68.58 0)
 			(effects
 				(font
@@
 		)
 		(property "Description" "Power symbol creates a global label with name \"VCC\""
-			(at 97.79 76.2 0)
+			(at 71.12 68.58 0)
 			(effects
 				(font
@@
 	(symbol
 		(lib_id "power:GND")
-		(at 97.79 81.28 0)
+		(at 97.79 78.74 0)
 		(unit 1)
 		(exclude_from_sim no)
@@
 		(fields_autoplaced yes)
 		(property "Reference" "#PWR06"
-			(at 97.79 87.63 0)
+			(at 97.79 85.09 0)
 			(effects
 				(font
@@
 		)
 		(property "Value" "GND"
-			(at 97.79 86.36 0)
+			(at 97.79 83.82 0)
 			(effects
 				(font
@@
 		)
 		(property "Footprint" ""
-			(at 97.79 81.28 0)
+			(at 97.79 78.74 0)
 			(effects
 				(font
@@
 		)
 		(property "Datasheet" ""
-			(at 97.79 81.28 0)
+			(at 97.79 78.74 0)
 			(effects
 				(font
@@
 		)
 		(property "Description" "Power symbol creates a global label with name \"GND\" , ground"
-			(at 97.79 81.28 0)
+			(at 97.79 78.74 0)
 			(effects
 				(font
@@
 	(symbol
 		(lib_id "Switch:SW_Push")
-		(at 87.63 78.74 0)
+		(at 81.28 78.74 0)
 		(unit 1)
 		(exclude_from_sim no)
@@
 		(fields_autoplaced yes)
 		(property "Reference" "SW1"
-			(at 87.63 71.12 0)
+			(at 81.28 71.12 0)
 			(effects
 				(font
@@
 		)
 		(property "Value" "SW_Push"
-			(at 87.63 73.66 0)
+			(at 81.28 73.66 0)
 			(effects
 				(font
@@
 		)
 		(property "Footprint" "Button_Switch_THT:SW_PUSH_6mm"
-			(at 87.63 73.66 0)
+			(at 81.28 73.66 0)
 			(effects
 				(font
@@
 		)
 		(property "Datasheet" "~"
-			(at 87.63 73.66 0)
+			(at 81.28 73.66 0)
 			(effects
 				(font
@@
 		)
 		(property "Description" "Push button switch, generic, two pins"
-			(at 87.63 78.74 0)
+			(at 81.28 78.74 0)
 			(effects
 				(font

Commit message: .
Parts:
- removed C1, C2, C3, C4, C5: C_Small, Capacitor_THT:CP_Radial_D5.0mm_P2.50mm, symbol Device:C_Small
- removed R13, R2, R3, R4, R5, R6, R7: 100, Resistor_THT:R_Axial_DIN0207_L6.3mm_D2.5mm_P10.16mm_Horizontal, symbol Device:R
- removed R23: 4.7k, Resistor_THT:R_Axial_DIN0207_L6.3mm_D2.5mm_P10.16mm_Horizontal, symbol Device:R
- removed SW1: SW_Push, Button_Switch_THT:SW_PUSH_6mm, symbol Switch:SW_Push
- removed U1: ATmega168A-P, Package_DIP:DIP-28_W7.62mm, symbol MCU_Microchip_ATmega:ATmega168A-P
- removed Y1: Crystal, Crystal:Resonator-2Pin_W6.0mm_H3.0mm, symbol Device:Crystal
- added U2: LM2576T-ADJ, Package_TO_SOT_THT:TO-220-5_Vertical, symbol Regulator_Switching:LM2576T-ADJ
Connections:
- no-connect marks 7 -> 2
Other:
- added sheet AUDIO-SCREEN_CONTROLLER (AUDIO-SCREEN_COTROLLER.kicad_sch)
- added sheet CONTROLLERS (CONTROLLERS.kicad_sch)
- added sheet GRID_CONTROLLER (GRID_CONTROLLER_sch.kicad_sch)
- added sheet POWER_SUPPLY (untitled.kicad_sch)

Commit message: .
Parts:
- removed 220UF1: C_Polarized, Capacitor_THT:C_Disc_D3.0mm_W1.6mm_P2.50mm, symbol Device:C_Polarized
- removed D1: LED, LED_THT:LED_D1.8mm_W3.3mm_H2.4mm, symbol Device:LED
- removed J1: GRID, TerminalBlock:TerminalBlock_MaiXu_MX126-5.0-03P_1x03_P5.00mm, symbol Connector:Conn_01x03_Pin
- removed J10: VCC, TerminalBlock:TerminalBlock_MaiXu_MX126-5.0-04P_1x04_P5.00mm, symbol Connector:Conn_01x05_Pin
- removed J11: PJ-102A, Connector_BarrelJack:BarrelJack_Horizontal, symbol dk_Barrel-Power-Connectors:PJ-102A
- removed J4: USB_ASP, Connector_IDC:IDC-Header_2x05_P2.54mm_Vertical, symbol Connector_Generic:Conn_02x05_Odd_Even
- removed J5: BUTTONS, TerminalBlock:TerminalBlock_MaiXu_MX126-5.0-03P_1x03_P5.00mm, symbol Connector:Conn_01x03_Pin
- removed J6: JOYSTICK, TerminalBlock:TerminalBlock_MaiXu_MX126-5.0-04P_1x04_P5.00mm, symbol Connector:Conn_01x04_Pin
- removed J7: UART_TERM, Connector_PinSocket_2.54mm:PinSocket_1x04_P2.54mm_Vertical, symbol Connector:Conn_01x05_Pin
- removed J8: PCF_SCREEN, TerminalBlock:TerminalBlock_MaiXu_MX126-5.0-04P_1x04_P5.00mm, symbol Connector:Conn_01x04_Pin
- removed J9: GROUND, TerminalBlock:TerminalBlock_MaiXu_MX126-5.0-04P_1x04_P5.00mm, symbol Connector:Conn_01x05_Pin
- removed R1: 100, Resistor_THT:R_Axial_DIN0207_L6.3mm_D2.5mm_P10.16mm_Horizontal, symbol Device:R
- removed R14, R15, R16, R17, R18, R19, R20, R21, R22, R24: 4.7k, Resistor_THT:R_Axial_DIN0207_L6.3mm_D2.5mm_P10.16mm_Horizontal, symbol Device:R
- removed U2: LM2576T-ADJ, Package_TO_SOT_THT:TO-220-5_Vertical, symbol Regulator_Switching:LM2576T-ADJ
Connections:
- no-connect marks 2 -> 0
Other:
- moved on the sheet: H1, H2, H3, H4, H5, H6, H7

Commit message: .
Other:
- sheet AUDIO-SCREEN_CONTROLLER ports: added B_EXIT, B_SELECT, B_START, INT1, INT2, INT3, INT4, JS_DOWN, JS_LEFT, JS_RIGHT, JS_UP, MISO, MOSI, RESET, RXD, SCK, TXD; removed none
- sheet CONTROLLERS ports: added B_EXIT, B_SELECT, B_START, JS_DOWN, JS_LEFT, JS_RIGHT, JS_UP, MISO, MOSI, RESET, RXD, SCK, TXD; removed none
- sheet GRID_CONTROLLER ports: added B_EXIT, B_SELECT, B_START, INT1, INT2, INT3, INT4, JS_DOWN, JS_LEFT, JS_RIGHT, JS_UP, MISO, MOSI, RESET, RXD, SCK, TXD; removed none

Commit message: .
Other:
- added sheet ESP12E (ESP12E.kicad_sch)
Changed lines of the file:
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@@
+	)
+	(sheet
+		(at 149.86 96.52)
+		(size 45.72 31.75)
+		(exclude_from_sim no)
+		(in_bom yes)
+		(on_board yes)
+		(dnp no)
+		(fields_autoplaced yes)
+		(stroke
+			(width 0.1524)
+			(type solid)
+		)
+		(fill
+			(color 0 0 0 0.0000)
+		)
+		(property "Sheetname" "ESP12E"
+			(at 149.86 95.8084 0)
+			(effects
+				(font
+					(size 1.27 1.27)
+				)
+				(justify left bottom)
+			)
+		)
+		(property "Sheetfile" "ESP12E.kicad_sch"
+			(at 149.86 128.8546 0)
+			(effects
+				(font
+					(size 1.27 1.27)
+				)
+				(justify left top)
+			)
+		)
+		(instances
+			(project "SNAKE_GAME"
+				(path "/6a8c7582-1032-4e02-bf22-b5197316f506"
+					(page "6")
+				)
+			)
+		)
 	)
 	(sheet

Commit message: .
Other:
- sheet AUDIO-SCREEN_CONTROLLER ports: added RXD_ESP, RXD_TERM, TXD_ESP, TXD_TERM; removed none
- sheet CONTROLLERS ports: added PAD_1_DIN, PAD_2_DIN, PAD_3_DIN, PAD_4_DIN; removed none
- sheet ESP12E ports: added RXD_ESP, TXD_ESP; removed none
