File: ATMEGA-SCHEMATICS/SNAKE_GAME/SNAKE_GAME.kicad_sch (KiCad schematic)
At the start: 7 parts

Commit message: .
Parts:
- added R46: 4.7k, Resistor_THT:R_Axial_DIN0207_L6.3mm_D2.5mm_P10.16mm_Horizontal, symbol Device:R
Connections:
- new net AUDIO-SCREEN_CONTROLLER/INT1_USR: R46.1
- new net VCC: R46.2
Other:
- removed sheet ESP12E
- sheet AUDIO-SCREEN_CONTROLLER ports: added B_EXIT_USR, B_SELECT_USR, B_START_USR, INT1_USR, JS_DOWN_USR, JS_LEFT_USR, JS_RIGHT_USR, JS_UP_USR, RXD_TERM_USR, TXD_TERM_USR, USR_SCL, USR_SDA; removed B_EXIT, B_SELECT, B_START, INT1, INT2, INT3, INT4, JS_DOWN, JS_LEFT, JS_RIGHT, JS_UP, RXD, RXD_ESP, RXD_TERM, TXD, TXD_ESP, TXD_TERM
- sheet CONTROLLERS ports: added GRID_RAM_SIGNAL, MISO_GRID, MISO_USR, MOSI_GRID, MOSI_USR, RESET_GRID, RESET_USR, RXD_TERMINAL, SCK_GRID, SCK_USR, TXD_TERMINAL; removed MISO, MOSI, PAD_1_DIN, PAD_2_DIN, PAD_3_DIN, PAD_4_DIN, RESET, RXD, SCK, TXD
- sheet GRID_CONTROLLER ports: added B_EXIT_GRID, B_SELECT_GRID, B_START_GRID, GRID_MISO, GRID_MOSI, GRID_RESET, GRID_SCK, INT1_GRID, JS_DOWN_GRID, JS_LEFT_GRID, JS_RIGHT_GRID, JS_UP_GRID, RAM_SIGNAL, RXD_TERM_GRID, SCL_GRID, SDA_GRID, TXD_TERM_GRID; removed B_EXIT, B_SELECT, B_START, INT1, INT2, INT3, INT4, JS_DOWN, JS_LEFT, JS_RIGHT, JS_UP, MISO, MOSI, RESET, RXD, SCK, TXD
- note added: "BUTTONS"
- note added: "GRID_SPI_PROGRAMMER"
- note added: "JOYSTICK"
- note added: "UART_TERM."
- note added: "USR_SPI_PROGRAMMER"
