File: ATMEGA-SCHEMATICS/SNAKE_GAME/_autosave-SNAKE_GAME.kicad_pcb (KiCad board)
At the start: 2 copper layers, 81 parts, among them J1 UART_ESP, J12 USB_ASP, J13 UART_TERM, J14 BUTTONS, J15 PJ-102A, J17 JOYSTICK, J19 PCF_SCREEN, J20 GROUND, J21 VCC, J3 GRID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

Commit message: .
Parts:
- moved J14 162.2 mm to (-54.5, 51.5)
- moved J17 162.2 mm to (-67.5, 51.5)
- moved AUDIO-SCREEN1 72.5 mm to (139.6, 127.3)
- moved C11 72.5 mm to (159.7, 142.8)
- moved C12 72.5 mm to (161.9, 151.8)
- moved C14 72.5 mm to (123.7, 143.8)
- moved C15 72.5 mm to (123.7, 153.8)
- moved C8 72.5 mm to (130.2, 137.8)
- moved Y3 72.5 mm to (130.2, 151.3)
- moved C13 65.0 mm to (75.5, 116.5)
- moved C1_Crystal1 65.0 mm to (38.5, 112.5)
- moved C2_Crystal1 65.0 mm to (38.0, 121.0)
- moved C6 65.0 mm to (75.0, 109.3)
- moved C7 65.0 mm to (44.5, 108.0)
- moved GRID_CONTROLLER1 65.0 mm to (55.9, 95.9)
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