File: ATMEGA-SCHEMATICS/SNAKE_GAME/AUDIO-SCREEN_COTROLLER.kicad_sch (KiCad schematic)
At the start: 10 parts, among them SW3 SW_Push, U4 ATmega168A-P, Y3 Crystal

Commit message: .
Parts:
- added J19: PCF_SCREEN, TerminalBlock:TerminalBlock_MaiXu_MX126-5.0-04P_1x04_P5.00mm, symbol Connector:Conn_01x04_Pin
- added R39, R40: 4.7k, Resistor_THT:R_Axial_DIN0207_L6.3mm_D2.5mm_P10.16mm_Horizontal, symbol Device:R
Connections:
- net GND: now also J19.1 (Pin_1)
- net SCL: now also J19.4 (Pin_4), R39.2
- net SDA: now also J19.3 (Pin_3), R40.2
- net VCC: now also J19.2 (Pin_2), R39.1, R40.1

Commit message: .
Parts:
- added R1, R13, R14, R3, R4, R7: 100, Resistor_THT:R_Axial_DIN0207_L6.3mm_D2.5mm_P10.16mm_Horizontal, symbol Device:R
- SW3: value SW_Push -> SWS_Push
- renumbered U4 to AUDIO-SCREEN1
Connections:
- net DIN_GRID is gone; now on an unnamed net: AUDIO-SCREEN1.23 (PC0)
- net DAC1: now reaches AUDIO-SCREEN1.11 (PD5)
- net DAC2: now reaches AUDIO-SCREEN1.12 (PD6)
- net at AUDIO-SCREEN1.13 (PD7): now also R7.1
- net INT3: now reaches AUDIO-SCREEN1.15 (PB1)
- net INT4: now reaches AUDIO-SCREEN1.16 (PB2)
- net at AUDIO-SCREEN1.24 (PC1): now also R13.1, R14.1
- net INT1: now reaches AUDIO-SCREEN1.25 (PC2)
- net INT2: now reaches AUDIO-SCREEN1.26 (PC3)
- net at AUDIO-SCREEN1.4 (PD2): now also R1.1
- net at AUDIO-SCREEN1.5 (PD3): now also R3.1
- net at AUDIO-SCREEN1.6 (PD4): now also R4.1
- new net B_EXIT: R14.2
- new net B_START: R7.2
- new net JS_DOWN: R3.2
- new net JS_LEFT: R4.2
- new net JS_RIGHT: R13.2
- new net JS_UP: R1.2
- no-connect marks 11 -> 0
Other:
- moved on the sheet: C14, C15, J19, R39, R40, Y3

Commit message: .
Parts:
- added C9: 100nF, Capacitor_THT:C_Disc_D7.5mm_W5.0mm_P5.00mm, symbol Device:C_Small
- added TS5A23159DGSR1: CONT_UART_RED_SWT, symbol Lucas_Lib:TS5A23159DGSR
- C11, C12, C13: value C_Small -> 100nF; footprint Capacitor_THT:CP_Radial_D5.0mm_P2.50mm -> Capacitor_THT:C_Disc_D7.5mm_W5.0mm_P5.00mm
- C14, C15: value C_Small -> 20pF; footprint Capacitor_THT:CP_Radial_D5.0mm_P2.50mm -> Capacitor_THT:C_Disc_D7.5mm_W5.0mm_P5.00mm
Connections:
- net GND: now also TS5A23159DGSR1.3 (GND)
- net RXD: now also TS5A23159DGSR1.10 (COM1)
- net TXD: now also TS5A23159DGSR1.6 (COM2)
- net VCC: now also C9.1, TS5A23159DGSR1.8 (VCC)
- new net RXD_ESP: TS5A23159DGSR1.9 (NC1)
- new net RXD_TERM: TS5A23159DGSR1.2 (NO1)
- new net TXD_ESP: TS5A23159DGSR1.7 (NC2)
- new net TXD_TERM: TS5A23159DGSR1.4 (NO2)
Other:
- moved on the sheet: AUDIO-SCREEN1, C11, C12, C13, C14, C15, J19, R1, R13, R14, R3, R37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

Commit message: .
Parts:
- removed TS5A23159DGSR1: CONT_UART_RED_SWT, symbol Lucas_Lib:TS5A23159DGSR
- added C10, C16, C19, C20, C24, C25, C26: 100nF, Capacitor_THT:C_Disc_D7.5mm_W5.0mm_P5.00mm, symbol Device:C_Small
- added R15, R16, R17, R18, R19, R20, R21, R22, R5, R6: 4.7k, Resistor_THT:R_Axial_DIN0207_L6.3mm_D2.5mm_P10.16mm_Horizontal, symbol Device:R
- added TS5A23159DGSR2: PAD_1&2, Lucas_lib:TS5A23159DGSR, symbol Lucas_Lib:TS5A23159DGSR
- added TS5A23159DGSR5: PAD_3&4, Lucas_lib:TS5A23159DGSR, symbol Lucas_Lib:TS5A23159DGSR
- added U3: PCF8574AP, Package_DIP:DIP-16_W7.62mm, symbol Interface_Expansion:PCF8574AP
Connections:
- net GND: now also C9.1, C16.1, C20.2, C24.2, TS5A23159DGSR2.3 (GND), TS5A23159DGSR5.3 (GND), U3.2 (A1), U3.8 (GND)
- net RXD: now also TS5A23159DGSR2.10 (COM1), TS5A23159DGSR5.10 (COM1)
- net TXD: now also TS5A23159DGSR2.6 (COM2), TS5A23159DGSR5.6 (COM2)
- net VCC: now also C20.1, C24.1, R15.1, R16.1, R17.1, R18.1, R19.1, R20.1, R21.2, R22.2, R5.1, R6.1, TS5A23159DGSR2.8 (VCC), TS5A23159DGSR5.8 (VCC); no longer C9.1
- net at C9.2: now also U3.16 (VDD)
- new net: R19.2, U3.5 (P1)
- new net: C19.1, TS5A23159DGSR5.9 (NC1)
- new net: R17.2, U3.7 (P3)
- new net: R18.2, U3.6 (P2)
- new net: C25.1, TS5A23159DGSR2.7 (NC2)
- new net: R5.2, U3.12 (P7)
- new net: R22.1, U3.3 (A2)
- new net: C10.1, TS5A23159DGSR2.9 (NC1)
- new net: R16.2, U3.9 (P4)
- new net: R21.1, U3.1 (A0)
- new net: R15.2, U3.10 (P5)
- new net: R6.2, U3.11 (P6)
- new net: C16.2, U3.13 (~{INT})
- new net: R20.2, U3.4 (P0)
- new net: C26.1, TS5A23159DGSR5.7 (NC2)
- new net PAD_1_DIN: TS5A23159DGSR2.2 (NO1)
- new net PAD_2_DIN: TS5A23159DGSR2.4 (NO2)
- new net PAD_3_DIN: TS5A23159DGSR5.2 (NO1)
- new net PAD_4_DIN: TS5A23159DGSR5.4 (NO2)
Other:
- moved on the sheet: AUDIO-SCREEN1, C11, C12, C13, C14, C15, J19, R1, R13, R14, R3, R37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

Commit message: .
Connections:
- net SCL: now also U3.14 (SCL)
- net SDA: now also U3.15 (SDA)
- net PAD_2_SWT: now reaches R19.2, U3.5 (P1)
- net PAD_2_SWT: now also TS5A23159DGSR2.5 (IN2)
- net PAD_4_SWT: now reaches R17.2, U3.7 (P3)
- net PAD_4_SWT: now also TS5A23159DGSR5.5 (IN2)
- net PAD_3_SWT: now reaches R18.2, U3.6 (P2)
- net PAD_3_SWT: now also TS5A23159DGSR5.1 (IN1)
- net PAD_1_SWT: now reaches TS5A23159DGSR2.1 (IN1)
- net PAD_1_SWT: now also R20.2, U3.4 (P0)
Other:
- moved on the sheet: AUDIO-SCREEN1, C10, C11, C12, C13, C14, C15, C16, C19, C20, C24, C25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

Commit message: .
Parts:
- removed C10, C16, C19, C20, C24, C25, C26, C9: 100nF, Capacitor_THT:C_Disc_D7.5mm_W5.0mm_P5.00mm, symbol Device:C_Small
- removed R15, R16, R17, R18, R19, R20, R21, R22, R5, R6: 4.7k, Resistor_THT:R_Axial_DIN0207_L6.3mm_D2.5mm_P10.16mm_Horizontal, symbol Device:R
- removed SW3: SWS_Push, Button_Switch_THT:SW_PUSH_6mm, symbol Switch:SW_Push
- removed TS5A23159DGSR2: PAD_1&2, Lucas_lib:TS5A23159DGSR, symbol Lucas_Lib:TS5A23159DGSR
- removed TS5A23159DGSR5: PAD_3&4, Lucas_lib:TS5A23159DGSR, symbol Lucas_Lib:TS5A23159DGSR
- removed U3: PCF8574AP, Package_DIP:DIP-16_W7.62mm, symbol Interface_Expansion:PCF8574AP
- added BZ1: Buzzer, Buzzer_Beeper:Buzzer_12x9.5RM7.6, symbol Device:Buzzer
- added J2: Vibrator, TerminalBlock:TerminalBlock_MaiXu_MX126-5.0-02P_1x02_P5.00mm, symbol Connector:Conn_01x02_Pin
- added R41, R42: 100, Resistor_THT:R_Axial_DIN0207_L6.3mm_D2.5mm_P10.16mm_Horizontal, symbol Device:R
- C14, C15: footprint Capacitor_THT:C_Disc_D7.5mm_W5.0mm_P5.00mm -> Capacitor_THT:CP_Radial_D5.0mm_P2.50mm
Connections:
- net GND: now also R41.1, R42.1
- net VCC: now also AUDIO-SCREEN1.21 (AREF), C11.2
- net at AUDIO-SCREEN1.23 (PC0), R13.1: no longer AUDIO-SCREEN1.24 (PC1), R14.1
- net B_EXIT renamed B_EXIT_USR
- net B_SELECT renamed B_SELECT_USR
- net B_START renamed B_START_USR
- net DAC1 renamed DAC1_VIBRATOR
- net DAC1_VIBRATOR: now also J2.1 (Pin_1)
- net DAC2 renamed DAC2_BUZZER
- net DAC2_BUZZER: now also BZ1.1 (+)
- net INT1 renamed INT1_USR
- net INT2 renamed PG
- net INT3 renamed REG_EN_LOW
- net INT4: no longer names the net of AUDIO-SCREEN1.16 (PB2)
- net JS_DOWN renamed JS_DOWN_USR
- net JS_LEFT renamed JS_LEFT_USR
- net JS_RIGHT renamed JS_RIGHT_USR
- net JS_UP renamed JS_UP_USR
- net RXD renamed RXD_TERM_USR
- net SCL renamed USR_SCL
- net SDA renamed USR_SDA
- net TXD renamed TXD_TERM_USR
- new net: J2.2 (Pin_2), R42.2
- new net: BZ1.2 (-), R41.2
- new net: AUDIO-SCREEN1.24 (PC1), R14.1
- no-connect marks 0 -> 1
Other:
- moved on the sheet: AUDIO-SCREEN1, C11, C12, C13, C14, C15, J19, R1, R13, R14, R3, R37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
