File: ATMEGA-SCHEMATICS/SNAKE_GAME/ESP12E.kicad_sch (KiCad schematic)
At the start: 6 parts, among them U1 ESP-12E

Commit message: .
Parts:
- removed C1, C3, C4: 100nF, Capacitor_THT:C_Disc_D7.5mm_W5.0mm_P5.00mm, symbol Device:C_Small
- removed C2: 1uF, Capacitor_THT:C_Disc_D7.5mm_W5.0mm_P5.00mm, symbol Device:C_Small
- removed C5: C_Small, Capacitor_THT:C_Disc_D7.5mm_W5.0mm_P5.00mm, symbol Device:C_Small
- removed U1: ESP-12E, RF_Module:ESP-12E, symbol RF_Module:ESP-12E
