File: ATMEGA-SCHEMATICS/SNAKE_GAME/untitled.kicad_sch (KiCad schematic)
At the start: 0 parts

Commit message: .
Parts:
- added 220UF2: C_Polarized, Capacitor_THT:C_Disc_D3.0mm_W1.6mm_P2.50mm, symbol Device:C_Polarized
- added D2: LED, LED_THT:LED_D1.8mm_W3.3mm_H2.4mm, symbol Device:LED
- added J15: PJ-102A, Connector_BarrelJack:BarrelJack_Horizontal, symbol dk_Barrel-Power-Connectors:PJ-102A
- added J20: GROUND, TerminalBlock:TerminalBlock_MaiXu_MX126-5.0-04P_1x04_P5.00mm, symbol Connector:Conn_01x05_Pin
- added J21: VCC, TerminalBlock:TerminalBlock_MaiXu_MX126-5.0-04P_1x04_P5.00mm, symbol Connector:Conn_01x05_Pin
- added R2: 100, Resistor_THT:R_Axial_DIN0207_L6.3mm_D2.5mm_P10.16mm_Horizontal, symbol Device:R
- added U5: LM2576T-ADJ, Package_TO_SOT_THT:TO-220-5_Vertical, symbol Regulator_Switching:LM2576T-ADJ
Connections:
- new net: D2.1 (K), R2.2
- new net GND: 220UF2.2, J15.3, J20.1 (Pin_1), J20.2 (Pin_2), J20.3 (Pin_3), J20.4 (Pin_4), J20.5 (Pin_5), R2.1
- new net VCC: 220UF2.1, D2.2 (A), J15.1, J21.1 (Pin_1), J21.2 (Pin_2), J21.3 (Pin_3), J21.4 (Pin_4), J21.5 (Pin_5)
- no-connect marks 0 -> 1

Commit message: .
Parts:
- added U2: FT232RL, Package_SO:SSOP-28_5.3x10.2mm_P0.65mm, symbol Interface_USB:FT232RL
Changed lines of the file:
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@@
+	)
+	(symbol
+		(lib_id "Interface_USB:FT232RL")
+		(at 114.3 138.43 0)
+		(unit 1)
+		(exclude_from_sim no)
+		(in_bom yes)
+		(on_board yes)
+		(dnp no)
+		(fields_autoplaced yes)
+		(property "Reference" "U2"
+			(at 118.9833 111.76 0)
+			(effects
+				(font
+					(size 1.27 1.27)
+				)
+				(justify left)
+			)
+		)
+		(property "Value" "FT232RL"
+			(at 118.9833 114.3 0)
+			(effects
+				(font
+					(size 1.27 1.27)
+				)
+				(justify left)
+			)
+		)
+		(property "Footprint" "Package_SO:SSOP-28_5.3x10.2mm_P0.65mm"
+			(at 142.24 161.29 0)
+			(effects
+				(font
+					(size 1.27 1.27)
+				)
+				(hide yes)
+			)
+		)
+		(property "Datasheet" "https://www.ftdichip.com/Support/Documents/DataSheets/ICs/DS_FT232R.pdf"
+			(at 114.3 138.43 0)
+			(effects
+				(font
+					(size 1.27 1.27)
+				)
+				(hide yes)
+			)
+		)
+		(property "Description" "USB to Serial Interface, SSOP-28"
+			(at 114.3 138.43 0)
+			(effects
+				(font
+					(size 1.27 1.27)
+				)
+				(hide yes)
+			)
+		)
+		(pin "22"
+		)
+		(pin "13"
+		)
+		(pin "16"
+		)
+		(pin "26"
+		)
+		(pin "27"
+		)
+		(pin "28"
+		)
+		(pin "11"
+		)
+		(pin "2"
+		)
+		(pin "3"
+		)
+		(pin "9"
+		)
+		(pin "17"
+		)
+		(pin "15"
+		)
+		(pin "21"
+		)
+		(pin "18"
+		)
+		(pin "4"
+		)
+		(pin "12"
+		)
+		(pin "7"
+		)
+		(pin "20"
+		)
+		(pin "1"
+		)
+		(pin "25"
+		)
+		(pin "5"
+		)
+		(pin "14"
+		)
+		(pin "23"
+		)
+		(pin "6"
+		)
+		(pin "19"
+		)
+		(pin "10"
+		)
+		(instances
+			(project ""
+				(path "/6a8c7582-1032-4e02-bf22-b5197316f506/eca50252-6d94-4864-8ea2-9e0d1f0ae3a5"
+					(reference "U2")
+					(unit 1)
+				)
+			)
+		)
 	)
 	(symbol

Commit message: .
Parts:
- removed U2: FT232RL, Package_SO:SSOP-28_5.3x10.2mm_P0.65mm, symbol Interface_USB:FT232RL
- removed U5: LM2576T-ADJ, Package_TO_SOT_THT:TO-220-5_Vertical, symbol Regulator_Switching:LM2576T-ADJ
- added 47uF1: C_Polarized, Capacitor_THT:C_Disc_D3.0mm_W1.6mm_P2.50mm, symbol Device:C_Polarized
- added C77: 1uF, Capacitor_THT:C_Disc_D7.5mm_W5.0mm_P5.00mm, symbol Device:C
- added D7: V_METER- LED, LED_THT:LED_D1.8mm_W3.3mm_H2.4mm, symbol Device:LED
- added R54: 1k, Resistor_THT:R_Axial_DIN0207_L6.3mm_D2.5mm_P10.16mm_Horizontal, symbol Device:R
- added R56, R57: 4.7k, Resistor_THT:R_Axial_DIN0207_L6.3mm_D2.5mm_P10.16mm_Horizontal, symbol Device:R
- added TPS75533KCG1: ~, Package_TO_SOT_THT:TO-220-5_Vertical, symbol lucasLib:TPS75533KCG3
- R2: value 100 -> 1k
Connections:
- net GND: now also 47uF1.2, C77.2, R54.2, TPS75533KCG1.3 (GND)
- net VCC: now also R56.1, R57.1, TPS75533KCG1.2 (IN_VCC)
- new net: D7.1 (K), R54.1
- new net PG: R56.2, TPS75533KCG1.5 (FB/PG)
- new net REG_EN_LOW: C77.1, R57.2, TPS75533KCG1.1 (EN)
- new net VCC_LED_GRID: 47uF1.1, D7.2 (A), TPS75533KCG1.4 (OUTPUT)
Other:
- moved on the sheet: J20, J21
