File: ATMEGA-SCHEMATICS/SNAKE_GAME/GRID_CONTROLLER_sch.kicad_sch (KiCad schematic)
At the start: 16 parts, among them SW2 SW_Push, U3 ATmega168A-P, Y2 Crystal

Commit message: .
Parts:
- added J3: GRID, TerminalBlock:TerminalBlock_MaiXu_MX126-5.0-03P_1x03_P5.00mm, symbol Connector:Conn_01x03_Pin
- added R38: 4.7k, Resistor_THT:R_Axial_DIN0207_L6.3mm_D2.5mm_P10.16mm_Horizontal, symbol Device:R
Connections:
- net DIN_GRID: now also J3.3 (Pin_3), R38.1
- net GND: now also J3.2 (Pin_2)
- net VCC: now also J3.1 (Pin_1), R38.2

Commit message: .
Parts:
- SW2: value SW_Push -> SWG_Push
- renumbered U3 to GRID_CONTROLLER1
Connections:
- net INT3: now reaches GRID_CONTROLLER1.15 (PB1)
- net INT4: now reaches GRID_CONTROLLER1.16 (PB2)
- net INT1: now reaches GRID_CONTROLLER1.24 (PC1)
- net INT2: now reaches GRID_CONTROLLER1.25 (PC2)
- net SCL: no longer names the net of GRID_CONTROLLER1.28 (PC5)
- net SDA: no longer names the net of GRID_CONTROLLER1.27 (PC4)
- no-connect marks 5 -> 3
Other:
- moved on the sheet: J3, R38

Commit message: .
Parts:
- C6, C7, C8: footprint Capacitor_THT:CP_Radial_D5.0mm_P2.50mm -> Capacitor_THT:C_Disc_D7.5mm_W5.0mm_P5.00mm
- renumbered C9 to C1_Crystal1, C10 to C2_Crystal1
Changed lines of the file:
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@@
 			)
 		)
-		(property "Footprint" "Capacitor_THT:CP_Radial_D5.0mm_P2.50mm"
+		(property "Footprint" "Capacitor_THT:C_Disc_D7.5mm_W5.0mm_P5.00mm"
 			(at 118.11 63.5 0)
 			(effects
@@
 		(on_board yes)
 		(dnp no)
-		(property "Reference" "C10"
+		(property "Reference" "C2_Crystal1"
 			(at 170.1863 91.44 90)
 			(effects
@@
 		)
 		(property "Value" "C_Small"
-			(at 170.1863 88.9 90)
+			(at 170.18 88.646 90)
 			(effects
 				(font
@@
 			(project "SNAKE_GAME"
 				(path "/6a8c7582-1032-4e02-bf22-b5197316f506/de9d9dbb-4b49-4ecb-94cb-6f9eaf4425bf"
-					(reference "C10")
+					(reference "C2_Crystal1")
 					(unit 1)
 				)
@@
 			)
 		)
-		(property "Footprint" "Capacitor_THT:CP_Radial_D5.0mm_P2.50mm"
+		(property "Footprint" "Capacitor_THT:C_Disc_D7.5mm_W5.0mm_P5.00mm"
 			(at 143.51 53.34 0)
 			(effects
@@
 			)
 		)
-		(property "Footprint" "Capacitor_THT:CP_Radial_D5.0mm_P2.50mm"
+		(property "Footprint" "Capacitor_THT:C_Disc_D7.5mm_W5.0mm_P5.00mm"
 			(at 132.08 53.34 0)
 			(effects
@@
 		(dnp no)
 		(fields_autoplaced yes)
-		(property "Reference" "C9"
+		(property "Reference" "C1_Crystal1"
 			(at 170.1863 71.12 90)
 			(effects
@@
 			(project "SNAKE_GAME"
 				(path "/6a8c7582-1032-4e02-bf22-b5197316f506/de9d9dbb-4b49-4ecb-94cb-6f9eaf4425bf"
-					(reference "C9")
-					(unit 1)
-				)
+					(reference "C1_Crystal1")
+					(unit 1)
+				)

Commit message: .
Parts:
- added C27: 100nF, Capacitor_THT:C_Disc_D7.5mm_W5.0mm_P5.00mm, symbol Device:C_Small
- added TS5A23159DGSR6: CONT_UART_RED_SWT, Lucas_lib:TS5A23159DGSR, symbol Lucas_Lib:TS5A23159DGSR
Connections:
- net GND: now also TS5A23159DGSR6.3 (GND)
- net RXD: now also TS5A23159DGSR6.10 (COM1)
- net TXD: now also TS5A23159DGSR6.6 (COM2)
- net VCC: now also C27.1, TS5A23159DGSR6.8 (VCC)
- new net RXD_ESP: TS5A23159DGSR6.9 (NC1)
- new net RXD_TERM: TS5A23159DGSR6.2 (NO1)
- new net TXD_ESP: TS5A23159DGSR6.7 (NC2)
- new net TXD_TERM: TS5A23159DGSR6.4 (NO2)
Other:
- moved on the sheet: C1_Crystal1, C2_Crystal1, C6, C7, C8, GRID_CONTROLLER1, J3, R10, R11, R12, R25, R26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

Commit message: .
Parts:
- removed SW2: SWG_Push, Button_Switch_THT:SW_PUSH_6mm, symbol Switch:SW_Push
- removed TS5A23159DGSR6: CONT_UART_RED_SWT, Lucas_lib:TS5A23159DGSR, symbol Lucas_Lib:TS5A23159DGSR
- added 23A1024/23LC1: ~, Package_DIP:CERDIP-8_W7.62mm_SideBrazed_Socket, symbol lucasLib:23A1024
- added C22, C28: 100nF, Capacitor_THT:C_Disc_D7.5mm_W5.0mm_P5.00mm, symbol Device:C_Small
- added C24: 1uF, Capacitor_THT:C_Disc_D7.5mm_W5.0mm_P5.00mm, symbol Device:C_Small
- added C25: 22uF, Capacitor_THT:C_Disc_D7.5mm_W5.0mm_P5.00mm, symbol Device:C_Small
- added R55: 4.7k, Resistor_THT:R_Axial_DIN0207_L6.3mm_D2.5mm_P10.16mm_Horizontal, symbol Device:R
Connections:
- net GND: now also C27.2, 23A1024/23LC1.4 (GND), C22.1, C24.1, C25.1, C28.2
- net VCC: now also C6.2, GRID_CONTROLLER1.21 (AREF), 23A1024/23LC1.8 (VCC), C22.2, C24.2, C25.2, R55.1; no longer C27.1, J3.1 (Pin_1)
- net INT1_GRID: now reaches GRID_CONTROLLER1.26 (PC3)
- net SDA_GRID: now reaches GRID_CONTROLLER1.27 (PC4)
- net SCL_GRID: now reaches GRID_CONTROLLER1.28 (PC5)
- net B_EXIT renamed B_EXIT_GRID
- net B_SELECT renamed B_SELECT_GRID
- net B_START renamed B_START_GRID
- net INT1: no longer names the net of GRID_CONTROLLER1.24 (PC1)
- net INT2: no longer names the net of GRID_CONTROLLER1.25 (PC2)
- net INT3: no longer names the net of GRID_CONTROLLER1.15 (PB1)
- net INT4: no longer names the net of GRID_CONTROLLER1.16 (PB2)
- net JS_DOWN renamed JS_DOWN_GRID
- net JS_LEFT renamed JS_LEFT_GRID
- net JS_RIGHT renamed JS_RIGHT_GRID
- net JS_UP renamed JS_UP_GRID
- net MISO renamed GRID_MISO
- net GRID_MISO: now also 23A1024/23LC1.5 (SI/SIO0)
- net MOSI renamed GRID_MOSI
- net GRID_MOSI: now also 23A1024/23LC1.2 (SO/SIO1)
- net RESET renamed GRID_RESET
- net RXD renamed RXD_TERM_GRID
- net SCK renamed GRID_SCK
- net GRID_SCK: now also 23A1024/23LC1.6 (SCK)
- net TXD renamed TXD_TERM_GRID
- new net: 23A1024/23LC1.7 (HOLD/SIO3), C28.1
- new net: 23A1024/23LC1.3 (SIO2), C27.1
- new net RAM_SIGNAL: 23A1024/23LC1.1 (CS), R55.2
- new net VCC_LED_GRID: J3.1 (Pin_1)
- no-connect marks 3 -> 4
Other:
- moved on the sheet: C1_Crystal1, C2_Crystal1, C6, C7, C8, GRID_CONTROLLER1, J3, R10, R11, R12, R25, R26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

Commit message: .
Parts:
- removed R10, R11, R12, R25, R26, R8, R9: 100, Resistor_THT:R_Axial_DIN0207_L6.3mm_D2.5mm_P10.16mm_Horizontal, symbol Device:R
Connections:
- net SCL_GRID is gone; now on net DIN_GRID: GRID_CONTROLLER1.28 (PC5)
- net DIN_GRID: no longer GRID_CONTROLLER1.23 (PC0)
- net INT1_GRID: now also GRID_CONTROLLER1.23 (PC0); no longer GRID_CONTROLLER1.26 (PC3)
- net GRID_RTS: now reaches GRID_CONTROLLER1.14 (PB0)
- net RAM_CS: now reaches GRID_CONTROLLER1.15 (PB1)
- net SDA_GRID: no longer names the net of GRID_CONTROLLER1.27 (PC4)
- no-connect marks 4 -> 3
