File: ATMEGA-SCHEMATICS/SNAKE_GAME/GRID_SCHEMATICS/GRID/GRID.kicad_sch (KiCad schematic)
At the start: 8433 parts, among them J1 Conn_01x04_Pin, J10 Conn_01x04_Pin, J11 Conn_01x03_Pin, J12 Conn_01x03_Pin, J13 Conn_01x03_Pin, J14 Conn_01x03_Pin, J15 Conn_01x03_Pin, J16 Conn_01x03_Pin, J17 Conn_01x03_Pin, J18 Conn_01x03_Pin, J19 Conn_01x03_Pin, J2 Conn_01x04_Pin, J20 Conn_01x03_Pin, J21 Conn_01x03_Pin, J22 Conn_01x03_Pin, J23 Conn_01x03_Pin, J24 Conn_01x03_Pin, J25 Conn_01x03_Pin, J26 Conn_01x03_Pin, J27 Conn_01x03_Pin, J28 Conn_01x03_Pin, J29 Conn_01x04_Pin, J3 Conn_01x04_Pin, J4 Conn_01x04_Pin, J5 Conn_01x04_Pin, J6 Conn_01x04_Pin, J7 Conn_01x04_Pin, J8 Conn_01x04_Pin, J9 Conn_01x04_Pin

Commit message: .
Parts:
- removed J11, J12, J17: Conn_01x03_Pin, symbol Connector:Conn_01x03_Pin
- removed J3, J4, J5: Conn_01x04_Pin, Connector_PinHeader_2.54mm:PinHeader_1x04_P2.54mm_Vertical, symbol Connector:Conn_01x04_Pin
- added C4202, C4206, C4210, C4214, C4218, C4222, C4226, C4230, C4234, C4238: T520Y337M006ATE040, Capacitor_SMD:CP_Elec_10x10, symbol Device:C_Small
- added C4203, C4204, C4207, C4208, C4211, C4212, C4215, C4216, C4219, C4220, C4223, C4224, C4227, C4228, C4231, C4232, C4235, C4236, C4239, C4240: 16PK4700MEFC12.5X25, Capacitor_THT:CP_Radial_D5.0mm_P2.50mm, symbol Device:C_Polarized
- added J11, J12, J17: Conn_01x04_Pin, Connector_PinHeader_2.54mm:PinHeader_1x04_P2.54mm_Horizontal, symbol Connector:Conn_01x04_Pin
- added J30, J4, J5: Conn_01x03_Pin, Connector_PinHeader_2.54mm:PinHeader_1x03_P2.54mm_Vertical, symbol Connector:Conn_01x03_Pin
- J1, J10, J2, J29, J6, J7, J8, J9: footprint Connector_PinHeader_2.54mm:PinHeader_1x04_P2.54mm_Vertical -> Connector_PinHeader_2.54mm:PinHeader_1x04_P2.54mm_Horizontal
- J13, J14, J15, J16, J18, J19, J20, J21, J22, J23, J24, J25, J26, J27, J28: footprint (none) -> Connector_PinHeader_2.54mm:PinHeader_1x03_P2.54mm_Vertical
Connections:
- net CKOUT_24 is gone; now on an unnamed net: D1680.5 (CKI)
- net CKOUT_6 is gone; now on an unnamed net: D420.5 (CKI)
- net SDOUT_6 is gone; now on an unnamed net: D420.4 (SDI)
- net GND: now also D1148.6 (GND), D1154.6 (GND), D1160.6 (GND), D1166.6 (GND), D1172.6 (GND), D1178.6 (GND), D1184.6 (GND), D1190.6 (GND), D1196.6 (GND), D1202.6 (GND), D1208.6 (GND), D1214.6 (GND)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
- net VCC_1: now also C4202.1, C4203.1, C4204.1; no longer C1000.2, C1001.2, C1002.2, C1003.2, C1004.2, C1005.2, C1006.2, C1007.2, C1008.2, C1009.2, C1010.2, C1011.2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
- net at D2492.5 (CKI): now also D2491.2 (CKO); no longer D2516.2 (CKO)
- net at D2492.4 (SDI): now also D2491.3 (SDO); no longer D2516.3 (SDO)
- net at D2516.4 (SDI): now also D2515.3 (SDO); no longer D2540.3 (SDO)
- net at D2516.5 (CKI): now also D2515.2 (CKO); no longer D2540.2 (CKO)
- net at D3489.2 (CKO): now also D3490.5 (CKI); no longer D3501.5 (CKI)
- net at D3489.3 (SDO): now also D3490.4 (SDI); no longer D3501.4 (SDI)
- net at D3477.3 (SDO): now also D3478.4 (SDI); no longer D3489.4 (SDI)
- net at D3477.2 (CKO): now also D3478.5 (CKI); no longer D3489.5 (CKI)
- net at D2693.5 (CKI): now also D2692.2 (CKO); no longer D2669.2 (CKO)
- net at D2693.4 (SDI): now also D2692.3 (SDO); no longer D2669.3 (SDO)
- net at D2669.4 (SDI): now also D2668.3 (SDO); no longer D2645.3 (SDO)
- net at D2669.5 (CKI): now also D2668.2 (CKO); no longer D2645.2 (CKO)
- net at D862.2 (CKO): now also D863.5 (CKI); no longer D856.5 (CKI)
- net at D862.3 (SDO): now also D863.4 (SDI); no longer D856.4 (SDI)
- net at D862.4 (SDI): now also D861.3 (SDO); no longer D868.3 (SDO)
- net at D862.5 (CKI): now also D861.2 (CKO); no longer D868.2 (CKO)
- net at D3206.5 (CKI): now also D3205.2 (CKO); no longer D3230.2 (CKO)
- net at D3206.4 (SDI): now also D3205.3 (SDO); no longer D3230.3 (SDO)
- net at D3254.3 (SDO): now also D3255.4 (SDI); no longer D3230.4 (SDI)
- net at D3254.2 (CKO): now also D3255.5 (CKI); no longer D3230.5 (CKI)
- net at D3434.5 (CKI): now also D3433.2 (CKO); no longer D3446.2 (CKO)
- net at D3434.4 (SDI): now also D3433.3 (SDO); no longer D3446.3 (SDO)
- net at D3458.3 (SDO): now also D3459.4 (SDI); no longer D3446.4 (SDI)
- net at D3458.2 (CKO): now also D3459.5 (CKI); no longer D3446.5 (CKI)
- net at D3855.5 (CKI): now also D3854.2 (CKO); no longer D3843.2 (CKO)
- net at D3855.4 (SDI): now also D3854.3 (SDO); no longer D3843.3 (SDO)
- net at D3831.3 (SDO): now also D3832.4 (SDI); no longer D3843.4 (SDI)
- net at D3831.2 (CKO): now also D3832.5 (CKI); no longer D3843.5 (CKI)
- net at D2449.2 (CKO): now also D2450.5 (CKI); no longer D2473.5 (CKI)
- net at D2449.3 (SDO): now also D2450.4 (SDI); no longer D2473.4 (SDI)
- net at D2425.3 (SDO): now also D2426.4 (SDI); no longer D2449.4 (SDI)
- net at D2425.2 (CKO): now also D2426.5 (CKI); no longer D2449.5 (CKI)
- net at D1814.2 (CKO): now also D1815.5 (CKI); no longer D1790.5 (CKI)
- net at D1814.3 (SDO): now also D1815.4 (SDI); no longer D1790.4 (SDI)
- net at D1838.3 (SDO): now also D1839.4 (SDI); no longer D1814.4 (SDI)
- net at D1838.2 (CKO): now also D1839.5 (CKI); no longer D1814.5 (CKI)
- net at D2216.2 (CKO): now also D2217.5 (CKI); no longer D2192.5 (CKI)
- net at D2216.3 (SDO): now also D2217.4 (SDI); no longer D2192.4 (SDI)
- net at D2216.4 (SDI): now also D2215.3 (SDO); no longer D2240.3 (SDO)
- net at D2216.5 (CKI): now also D2215.2 (CKO); no longer D2240.2 (CKO)
- net at D3911.5 (CKI): now also D3910.2 (CKO); no longer D3899.2 (CKO)
- net at D3911.4 (SDI): now also D3910.3 (SDO); no longer D3899.3 (SDO)
- net at D3899.4 (SDI): now also D3898.3 (SDO); no longer D3887.3 (SDO)
- net at D3899.5 (CKI): now also D3898.2 (CKO); no longer D3887.2 (CKO)
- net at D1015.2 (CKO): now also D1016.5 (CKI); no longer D1021.5 (CKI)
- net at D1015.3 (SDO): now also D1016.4 (SDI); no longer D1021.4 (SDI)
- net at D1015.4 (SDI): now also D1014.3 (SDO); no longer D1009.3 (SDO)
- net at D1015.5 (CKI): now also D1014.2 (CKO); no longer D1009.2 (CKO)
- net at D495.5 (CKI): now also D494.2 (CKO); no longer D489.2 (CKO)
- net at D495.4 (SDI): now also D494.3 (SDO); no longer D489.3 (SDO)
- net at D483.3 (SDO): now also D484.4 (SDI); no longer D489.4 (SDI)
- net at D483.2 (CKO): now also D484.5 (CKI); no longer D489.5 (CKI)
- net at D1866.2 (CKO): now also D1867.5 (CKI); no longer D1842.5 (CKI)
- net at D1866.3 (SDO): now also D1867.4 (SDI); no longer D1842.4 (SDI)
- net at D1866.4 (SDI): now also D1865.3 (SDO); no longer D1890.3 (SDO)
- net at D1866.5 (CKI): now also D1865.2 (CKO); no longer D1890.2 (CKO)
- net at D2623.2 (CKO): now also D2624.5 (CKI); no longer D2647.5 (CKI)
- net CKOUT_1 renamed CKO_1
- net CKOUT_12 renamed CKO_6
- removed net CKOUT_18: D1260.5 (CKI), J15.3 (Pin_3)
- net CKOUT_3 renamed CKO_3
- net CKOUT_30 renamed CKO_30
- net CKOUT_36 renamed CKO_36
- net CKOUT_4 renamed CKO_4
- removed net CKOUT_42: D3354.5 (CKI), J23.3 (Pin_3)
- net CKOUT_48 renamed CKO_48
- net CKOUT_5 renamed CKO_5
- net CKOUT_54 renamed CKO_54
- removed net CKOUT_60: D4200.5 (CKI), J29.2 (Pin_2)
- net SDOUT_1 renamed SDO_1
- net SDOUT_12 renamed SDO_6
- removed net SDOUT_18: D1260.4 (SDI), J16.3 (Pin_3)
- net SDOUT_24 renamed CKO_24
- net SDOUT_3 renamed SDO_3
- net SDOUT_30 renamed SDO_30
- net SDOUT_36 renamed SDO_36
- net SDOUT_4 renamed SDO_4
- removed net SDOUT_42: D3354.4 (SDI), J24.3 (Pin_3)
- net SDOUT_48 renamed SDO_48
- net SDOUT_5 renamed SDO_5
- net SDOUT_54 renamed SDO_54
- removed net SDOUT_60: D4200.4 (SDI), J29.1 (Pin_1)
- new net: D3554.3 (SDO), D3555.4 (SDI)
- new net: D3554.2 (CKO), D3555.5 (CKI)
- new net: D537.3 (SDO), D538.4 (SDI)
- new net: D537.2 (CKO), D538.5 (CKI)
- new net: D2612.2 (CKO), D2613.5 (CKI)
- new net: D2612.3 (SDO), D2613.4 (SDI)
- new net: D3624.3 (SDO), D3625.4 (SDI)
- new net: D3624.2 (CKO), D3625.5 (CKI)
- new net: D3316.2 (CKO), D3317.5 (CKI)
- new net: D3316.3 (SDO), D3317.4 (SDI)
- new net: D3735.3 (SDO), D3736.4 (SDI)
- new net: D3735.2 (CKO), D3736.5 (CKI)
- new net: D1766.3 (SDO), D1767.4 (SDI)
- new net: D1766.2 (CKO), D1767.5 (CKI)
- new net: D269.2 (CKO), D270.5 (CKI)
- new net: D269.3 (SDO), D270.4 (SDI)
- new net: D3431.2 (CKO), D3432.5 (CKI)
- new net: D3431.3 (SDO), D3432.4 (SDI)
- new net: D1347.2 (CKO), D1348.5 (CKI)
- new net: D1347.3 (SDO), D1348.4 (SDI)
- new net: D4196.2 (CKO), D4197.5 (CKI)
- new net: D4196.3 (SDO), D4197.4 (SDI)
- new net: D1911.3 (SDO), D1912.4 (SDI)
- new net: D1911.2 (CKO), D1912.5 (CKI)
- new net: D3106.2 (CKO), D3107.5 (CKI)
- new net: D3106.3 (SDO), D3107.4 (SDI)
- new net: J17.1 (Pin_1), J30.1 (Pin_1)
- new net: D1290.3 (SDO), D1291.4 (SDI)
- new net: D1290.2 (CKO), D1291.5 (CKI)
- new net: D3213.2 (CKO), D3214.5 (CKI)
- new net: D3213.3 (SDO), D3214.4 (SDI)
- new net: D3754.3 (SDO), D3755.4 (SDI)
- new net: D3754.2 (CKO), D3755.5 (CKI)
- new net: D2916.2 (CKO), D2917.5 (CKI)
- new net: D2916.3 (SDO), D2917.4 (SDI)
- new net: D1112.3 (SDO), D1113.4 (SDI)
- new net: D1112.2 (CKO), D1113.5 (CKI)
- new net: D550.3 (SDO), D551.4 (SDI)
- new net: D550.2 (CKO), D551.5 (CKI)
- new net: D618.3 (SDO), D619.4 (SDI)
- new net: D618.2 (CKO), D619.5 (CKI)
- new net: D3388.3 (SDO), D3389.4 (SDI)
- new net: D3388.2 (CKO), D3389.5 (CKI)
- new net: D2577.3 (SDO), D2578.4 (SDI)
- new net: D2577.2 (CKO), D2578.5 (CKI)
- new net: D2142.3 (SDO), D2143.4 (SDI)
- new net: D2142.2 (CKO), D2143.5 (CKI)
- new net: D2539.2 (CKO), D2540.5 (CKI)
- new net: D2539.3 (SDO), D2540.4 (SDI)
- new net: D1217.2 (CKO), D1218.5 (CKI)
- new net: D1217.3 (SDO), D1218.4 (SDI)
- new net: D799.3 (SDO), D800.4 (SDI)
- new net: D799.2 (CKO), D800.5 (CKI)
- new net: D4032.2 (CKO), D4033.5 (CKI)
- new net: D4032.3 (SDO), D4033.4 (SDI)
- new net: D1417.3 (SDO), D1418.4 (SDI)
- new net: D1417.2 (CKO), D1418.5 (CKI)
- new net: D3992.3 (SDO), D3993.4 (SDI)
- new net: D3992.2 (CKO), D3993.5 (CKI)
- new net: D4065.2 (CKO), D4066.5 (CKI)
- new net: D4065.3 (SDO), D4066.4 (SDI)
- new net: D3572.3 (SDO), D3573.4 (SDI)
- new net: D3572.2 (CKO), D3573.5 (CKI)
- new net: D1572.3 (SDO), D1573.4 (SDI)
- new net: D1572.2 (CKO), D1573.5 (CKI)
- new net: D1824.3 (SDO), D1825.4 (SDI)
- new net: D1824.2 (CKO), D1825.5 (CKI)
- new net: D1038.2 (CKO), D1039.5 (CKI)
- new net: D1038.3 (SDO), D1039.4 (SDI)
- new net: D941.3 (SDO), D942.4 (SDI)
- new net: D941.2 (CKO), D942.5 (CKI)
- new net: D1230.3 (SDO), D1231.4 (SDI)
- new net: D1230.2 (CKO), D1231.5 (CKI)
- new net: D131.2 (CKO), D132.5 (CKI)
- new net: D131.3 (SDO), D132.4 (SDI)
- new net: D2885.3 (SDO), D2886.4 (SDI)
- new net: D2885.2 (CKO), D2886.5 (CKI)
- new net: D2653.2 (CKO), D2654.5 (CKI)
- new net: D2653.3 (SDO), D2654.4 (SDI)
- new net: D1542.3 (SDO), D1543.4 (SDI)
- new net: D1542.2 (CKO), D1543.5 (CKI)
- new net: D1147.2 (CKO), D1148.5 (CKI)
- new net: D1147.3 (SDO), D1148.4 (SDI)
- new net: D846.3 (SDO), D847.4 (SDI)
- new net: D846.2 (CKO), D847.5 (CKI)
- new net: D477.3 (SDO), D478.4 (SDI)
- new net: D477.2 (CKO), D478.5 (CKI)
- new net: D1907.2 (CKO), D1908.5 (CKI)
- new net: D1907.3 (SDO), D1908.4 (SDI)
- new net: D3100.2 (CKO), D3101.5 (CKI)
- new net: D3100.3 (SDO), D3101.4 (SDI)
- new net: D2058.2 (CKO), D2059.5 (CKI)
- new net: D2058.3 (SDO), D2059.4 (SDI)
- new net: D3175.3 (SDO), D3176.4 (SDI)
- new net: D3175.2 (CKO), D3176.5 (CKI)
- new net: D3006.3 (SDO), D3007.4 (SDI)
- new net: D3006.2 (CKO), D3007.5 (CKI)
- new net: D1555.3 (SDO), D1556.4 (SDI)
- new net: D1555.2 (CKO), D1556.5 (CKI)
- new net: D1157.3 (SDO), D1158.4 (SDI)
- new net: D1157.2 (CKO), D1158.5 (CKI)
- new net: D2077.3 (SDO), D2078.4 (SDI)
- new net: D1554.3 (SDO), D1555.4 (SDI)
- new net: D1554.2 (CKO), D1555.5 (CKI)
- new net: D369.2 (CKO), D370.5 (CKI)
- new net: D369.3 (SDO), D370.4 (SDI)
- new net: D2392.2 (CKO), D2393.5 (CKI)
- new net: D2392.3 (SDO), D2393.4 (SDI)
- new net: D697.3 (SDO), D698.4 (SDI)
- new net: D697.2 (CKO), D698.5 (CKI)
- new net: D1705.2 (CKO), D1706.5 (CKI)
- new net: D1705.3 (SDO), D1706.4 (SDI)
- new net: D558.2 (CKO), D559.5 (CKI)
- new net: D558.3 (SDO), D559.4 (SDI)
- new net: D2291.3 (SDO), D2292.4 (SDI)
- new net: D2291.2 (CKO), D2292.5 (CKI)
- new net: D2888.3 (SDO), D2889.4 (SDI)
- new net: D2888.2 (CKO), D2889.5 (CKI)
- new net: D3392.3 (SDO), D3393.4 (SDI)
- new net: D3392.2 (CKO), D3393.5 (CKI)
- new net: D2996.2 (CKO), D2997.5 (CKI)
- new net: D2996.3 (SDO), D2997.4 (SDI)
- new net: D3838.3 (SDO), D3839.4 (SDI)
- new net: D3838.2 (CKO), D3839.5 (CKI)
- new net: D2078.3 (SDO), D2079.4 (SDI)
- new net: D2078.2 (CKO), D2079.5 (CKI)
- new net: D2185.3 (SDO), D2186.4 (SDI)
- new net: D2185.2 (CKO), D2186.5 (CKI)
- new net: D489.3 (SDO), D490.4 (SDI)
- new net: D489.2 (CKO), D490.5 (CKI)
- new net: D1495.3 (SDO), D1496.4 (SDI)
- new net: D1495.2 (CKO), D1496.5 (CKI)
- new net: D2044.2 (CKO), D2045.5 (CKI)
- new net: D2044.3 (SDO), D2045.4 (SDI)
- new net: D3718.2 (CKO), D3719.5 (CKI)
- new net: D3718.3 (SDO), D3719.4 (SDI)
- new net: D3061.2 (CKO), D3062.5 (CKI)
- new net: D3061.3 (SDO), D3062.4 (SDI)
- new net: D1504.2 (CKO), D1505.5 (CKI)
- new net: D1504.3 (SDO), D1505.4 (SDI)
- new net: D3073.3 (SDO), D3074.4 (SDI)
- new net: D3073.2 (CKO), D3074.5 (CKI)
- new net: D1013.3 (SDO), D1014.4 (SDI)
- new net: D1013.2 (CKO), D1014.5 (CKI)
- new net: D3880.3 (SDO), D3881.4 (SDI)
- new net: D3880.2 (CKO), D3881.5 (CKI)
- new net: D624.2 (CKO), D625.5 (CKI)
- new net: D624.3 (SDO), D625.4 (SDI)
- new net: D1326.3 (SDO), D1327.4 (SDI)
- new net: D1326.2 (CKO), D1327.5 (CKI)
- new net: D4088.2 (CKO), D4089.5 (CKI)
- new net: D4088.3 (SDO), D4089.4 (SDI)
- new net: D3724.3 (SDO), D3725.4 (SDI)
- new net: D3724.2 (CKO), D3725.5 (CKI)
- new net: D2974.3 (SDO), D2975.4 (SDI)
- new net: D2974.2 (CKO), D2975.5 (CKI)
- new net: D3028.2 (CKO), D3029.5 (CKI)
- new net: D3028.3 (SDO), D3029.4 (SDI)
- new net: D1515.3 (SDO), D1516.4 (SDI)
- new net: D1515.2 (CKO), D1516.5 (CKI)
- new net: D1187.2 (CKO), D1188.5 (CKI)
- new net: D1187.3 (SDO), D1188.4 (SDI)
- new net: D2529.2 (CKO), D2530.5 (CKI)
- new net: D2529.3 (SDO), D2530.4 (SDI)
- new net: D816.3 (SDO), D817.4 (SDI)
- new net: D816.2 (CKO), D817.5 (CKI)
- new net: D4044.2 (CKO), D4045.5 (CKI)
- new net: D4044.3 (SDO), D4045.4 (SDI)
- new net: D3090.3 (SDO), D3091.4 (SDI)
- new net: D3090.2 (CKO), D3091.5 (CKI)
- new net: D2250.2 (CKO), D2251.5 (CKI)
- new net: D2250.3 (SDO), D2251.4 (SDI)
- new net: D2249.3 (SDO), D2250.4 (SDI)
- new net: D2249.2 (CKO), D2250.5 (CKI)
- new net: D1156.3 (SDO), D1157.4 (SDI)
- new net: D1156.2 (CKO), D1157.5 (CKI)
- new net: D370.2 (CKO), D371.5 (CKI)
- new net: D370.3 (SDO), D371.4 (SDI)
- new net: D4036.2 (CKO), D4037.5 (CKI)
- new net: D4036.3 (SDO), D4037.4 (SDI)
- new net: D1305.2 (CKO), D1306.5 (CKI)
- new net: D1305.3 (SDO), D1306.4 (SDI)
- new net: D1304.3 (SDO), D1305.4 (SDI)
- new net: D1304.2 (CKO), D1305.5 (CKI)
- new net: D3999.2 (CKO), D4000.5 (CKI)
- new net: D3999.3 (SDO), D4000.4 (SDI)
- new net: D2984.2 (CKO), D2985.5 (CKI)
- new net: D2984.3 (SDO), D2985.4 (SDI)
- new net: D1342.2 (CKO), D1343.5 (CKI)
- new net: D1342.3 (SDO), D1343.4 (SDI)
- new net: D511.2 (CKO), D512.5 (CKI)
- new net: D511.3 (SDO), D512.4 (SDI)
- new net: D2743.2 (CKO), D2744.5 (CKI)
- new net: D2743.3 (SDO), D2744.4 (SDI)
- new net: D565.3 (SDO), D566.4 (SDI)
- new net: D565.2 (CKO), D566.5 (CKI)
- new net: D3779.3 (SDO), D3780.4 (SDI)
- new net: D3779.2 (CKO), D3780.5 (CKI)
- new net: D701.2 (CKO), D702.5 (CKI)
- new net: D701.3 (SDO), D702.4 (SDI)
- new net: D609.2 (CKO), D610.5 (CKI)
- new net: D609.3 (SDO), D610.4 (SDI)
- new net: D608.3 (SDO), D609.4 (SDI)
- new net: D608.2 (CKO), D609.5 (CKI)
- new net: D3488.3 (SDO), D3489.4 (SDI)
- new net: D3488.2 (CKO), D3489.5 (CKI)
- new net: D3072.2 (CKO), D3073.5 (CKI)
- new net: D3072.3 (SDO), D3073.4 (SDI)
- new net: D2731.2 (CKO), D2732.5 (CKI)
- new net: D2731.3 (SDO), D2732.4 (SDI)
- new net: D2740.2 (CKO), D2741.5 (CKI)
- new net: D2740.3 (SDO), D2741.4 (SDI)
- new net: D3776.2 (CKO), D3777.5 (CKI)
- new net: D3776.3 (SDO), D3777.4 (SDI)
- new net: D3887.2 (CKO), D3888.5 (CKI)
- new net: D3887.3 (SDO), D3888.4 (SDI)
- new net: D434.3 (SDO), D435.4 (SDI)
- new net: D434.2 (CKO), D435.5 (CKI)
- new net: D935.3 (SDO), D936.4 (SDI)
- new net: D935.2 (CKO), D936.5 (CKI)
- new net: D408.2 (CKO), D409.5 (CKI)
- new net: D408.3 (SDO), D409.4 (SDI)
- new net: D2840.3 (SDO), D2841.4 (SDI)
- new net: D2840.2 (CKO), D2841.5 (CKI)
- new net: D1894.3 (SDO), D1895.4 (SDI)
- new net: D1894.2 (CKO), D1895.5 (CKI)
- new net: D2780.2 (CKO), D2781.5 (CKI)
- new net: D2780.3 (SDO), D2781.4 (SDI)
- new net: D1841.3 (SDO), D1842.4 (SDI)
- new net: D1841.2 (CKO), D1842.5 (CKI)
- new net: D2695.2 (CKO), D2696.5 (CKI)
- new net: D2695.3 (SDO), D2696.4 (SDI)
- new net: D1981.2 (CKO), D1982.5 (CKI)
- new net: D1981.3 (SDO), D1982.4 (SDI)
- new net: D1745.2 (CKO), D1746.5 (CKI)
- new net: D1745.3 (SDO), D1746.4 (SDI)
- new net: D883.2 (CKO), D884.5 (CKI)
- new net: D883.3 (SDO), D884.4 (SDI)
- new net: D2298.3 (SDO), D2299.4 (SDI)
- new net: D2298.2 (CKO), D2299.5 (CKI)
- new net: D1813.3 (SDO), D1814.4 (SDI)
- new net: D1813.2 (CKO), D1814.5 (CKI)
- new net: D2616.3 (SDO), D2617.4 (SDI)
- new net: D2616.2 (CKO), D2617.5 (CKI)
- new net: D1440.2 (CKO), D1441.5 (CKI)
- new net: D1440.3 (SDO), D1441.4 (SDI)
- new net: D2264.3 (SDO), D2265.4 (SDI)
- new net: D2264.2 (CKO), D2265.5 (CKI)
- new net: D2476.3 (SDO), D2477.4 (SDI)
- new net: D2476.2 (CKO), D2477.5 (CKI)
- new net: D3450.2 (CKO), D3451.5 (CKI)
- new net: D3450.3 (SDO), D3451.4 (SDI)
- new net: D1872.2 (CKO), D1873.5 (CKI)
- new net: D1872.3 (SDO), D1873.4 (SDI)
- new net: D3137.2 (CKO), D3138.5 (CKI)
- new net: D3137.3 (SDO), D3138.4 (SDI)
- new net: D4179.3 (SDO), D4180.4 (SDI)
- new net: D4179.2 (CKO), D4180.5 (CKI)
- new net: D3423.2 (CKO), D3424.5 (CKI)
- new net: D3423.3 (SDO), D3424.4 (SDI)
- new net: D2101.5 (CKI), J19.2 (Pin_2)
- new net: D4051.3 (SDO), D4052.4 (SDI)
- new net: D4051.2 (CKO), D4052.5 (CKI)
- new net: D2028.3 (SDO), D2029.4 (SDI)
- new net: D2028.2 (CKO), D2029.5 (CKI)
- new net: D262.3 (SDO), D263.4 (SDI)
- new net: D262.2 (CKO), D263.5 (CKI)
- new net: D4026.2 (CKO), D4027.5 (CKI)
- new net: D4026.3 (SDO), D4027.4 (SDI)
- new net: D3884.2 (CKO), D3885.5 (CKI)
- new net: D3884.3 (SDO), D3885.4 (SDI)
- new net: D1124.3 (SDO), D1125.4 (SDI)
- new net: D1124.2 (CKO), D1125.5 (CKI)
- new net: D2038.3 (SDO), D2039.4 (SDI)
- new net: D2038.2 (CKO), D2039.5 (CKI)
- new net: D3209.2 (CKO), D3210.5 (CKI)
- new net: D3209.3 (SDO), D3210.4 (SDI)
- new net: D685.2 (CKO), D686.5 (CKI)
- new net: D685.3 (SDO), D686.4 (SDI)
- new net: D2461.3 (SDO), D2462.4 (SDI)
- new net: D2461.2 (CKO), D2462.5 (CKI)
- new net: D1214.3 (SDO), D1215.4 (SDI)
- new net: D1214.2 (CKO), D1215.5 (CKI)
- new net: D3727.3 (SDO), D3728.4 (SDI)
- new net: D3727.2 (CKO), D3728.5 (CKI)
- new net: D3391.2 (CKO), D3392.5 (CKI)
- new net: D3391.3 (SDO), D3392.4 (SDI)
- new net: D2073.3 (SDO), D2074.4 (SDI)
- new net: D2073.2 (CKO), D2074.5 (CKI)
- new net: D1558.3 (SDO), D1559.4 (SDI)
- new net: D1558.2 (CKO), D1559.5 (CKI)
- new net: D660.3 (SDO), D661.4 (SDI)
- new net: D660.2 (CKO), D661.5 (CKI)
- new net: D3958.3 (SDO), D3959.4 (SDI)
- new net: D3958.2 (CKO), D3959.5 (CKI)
- new net: D3494.3 (SDO), D3495.4 (SDI)
- new net: D3494.2 (CKO), D3495.5 (CKI)
- new net: D2166.3 (SDO), D2167.4 (SDI)
- new net: D2166.2 (CKO), D2167.5 (CKI)
- new net: D385.2 (CKO), D386.5 (CKI)
- new net: D385.3 (SDO), D386.4 (SDI)
- new net: D384.3 (SDO), D385.4 (SDI)
- new net: D384.2 (CKO), D385.5 (CKI)
- new net: D3970.3 (SDO), D3971.4 (SDI)
- new net: D3970.2 (CKO), D3971.5 (CKI)
- new net: D3344.2 (CKO), D3345.5 (CKI)
- new net: D3344.3 (SDO), D3345.4 (SDI)
- new net: D2458.3 (SDO), D2459.4 (SDI)
- new net: D2458.2 (CKO), D2459.5 (CKI)
- new net: D108.3 (SDO), D109.4 (SDI)
- new net: D108.2 (CKO), D109.5 (CKI)
- new net: D3131.2 (CKO), D3132.5 (CKI)
- new net: D3131.3 (SDO), D3132.4 (SDI)
- new net: D2149.2 (CKO), D2150.5 (CKI)
- new net: D2149.3 (SDO), D2150.4 (SDI)
- new net: D3771.3 (SDO), D3772.4 (SDI)
- new net: D3771.2 (CKO), D3772.5 (CKI)
- new net: D2052.2 (CKO), D2053.5 (CKI)
- new net: D2052.3 (SDO), D2053.4 (SDI)
- new net: D1571.2 (CKO), D1572.5 (CKI)
- new net: D1571.3 (SDO), D1572.4 (SDI)
- new net: D927.2 (CKO), D928.5 (CKI)
- new net: D927.3 (SDO), D928.4 (SDI)
- new net: D2362.2 (CKO), D2363.5 (CKI)
- new net: D2362.3 (SDO), D2363.4 (SDI)
- new net: D2644.2 (CKO), D2645.5 (CKI)
- new net: D2644.3 (SDO), D2645.4 (SDI)
- new net: D1489.2 (CKO), D1490.5 (CKI)
- new net: D1489.3 (SDO), D1490.4 (SDI)
- new net: D1141.3 (SDO), D1142.4 (SDI)
- new net: D1141.2 (CKO), D1142.5 (CKI)
- new net: D916.2 (CKO), D917.5 (CKI)
- new net: D916.3 (SDO), D917.4 (SDI)
- new net: D3206.3 (SDO), D3207.4 (SDI)
- new net: D3206.2 (CKO), D3207.5 (CKI)
- new net: D2941.5 (CKI), J23.2 (Pin_2)
- new net: D3303.3 (SDO), D3304.4 (SDI)
- new net: D3303.2 (CKO), D3304.5 (CKI)
- new net: D3169.2 (CKO), D3170.5 (CKI)
- new net: D3169.3 (SDO), D3170.4 (SDI)
- new net: D3168.3 (SDO), D3169.4 (SDI)
- new net: D3168.2 (CKO), D3169.5 (CKI)
- new net: D2041.3 (SDO), D2042.4 (SDI)
- new net: D2041.2 (CKO), D2042.5 (CKI)
- new net: D3582.2 (CKO), D3583.5 (CKI)
- new net: D3582.3 (SDO), D3583.4 (SDI)
- new net: D2553.3 (SDO), D2554.4 (SDI)
- new net: D2553.2 (CKO), D2554.5 (CKI)
- new net: D2989.2 (CKO), D2990.5 (CKI)
- new net: D2989.3 (SDO), D2990.4 (SDI)
- new net: D1622.2 (CKO), D1623.5 (CKI)
- new net: D1622.3 (SDO), D1623.4 (SDI)
- new net: D1526.3 (SDO), D1527.4 (SDI)
- new net: D1526.2 (CKO), D1527.5 (CKI)
- new net: D3903.3 (SDO), D3904.4 (SDI)
- new net: D3903.2 (CKO), D3904.5 (CKI)
- new net: D2871.2 (CKO), D2872.5 (CKI)
- new net: D2871.3 (SDO), D2872.4 (SDI)
- new net: D834.3 (SDO), D835.4 (SDI)
- new net: D834.2 (CKO), D835.5 (CKI)
- new net: D4095.3 (SDO), D4096.4 (SDI)
- new net: D4095.2 (CKO), D4096.5 (CKI)
- new net: D2599.3 (SDO), D2600.4 (SDI)
- new net: D2599.2 (CKO), D2600.5 (CKI)
- new net: D1859.2 (CKO), D1860.5 (CKI)
- new net: D1859.3 (SDO), D1860.4 (SDI)
- new net: D1858.3 (SDO), D1859.4 (SDI)
- new net: D1858.2 (CKO), D1859.5 (CKI)
- new net: D1358.2 (CKO), D1359.5 (CKI)
- new net: D1358.3 (SDO), D1359.4 (SDI)
- new net: D1634.2 (CKO), D1635.5 (CKI)
- new net: D1634.3 (SDO), D1635.4 (SDI)
- new net: D3796.2 (CKO), D3797.5 (CKI)
- new net: D3796.3 (SDO), D3797.4 (SDI)
- new net: D3795.3 (SDO), D3796.4 (SDI)
- new net: D3795.2 (CKO), D3796.5 (CKI)
- new net: D650.3 (SDO), D651.4 (SDI)
- new net: D650.2 (CKO), D651.5 (CKI)
- new net: D920.3 (SDO), D921.4 (SDI)
- new net: D920.2 (CKO), D921.5 (CKI)
- new net: D1692.3 (SDO), D1693.4 (SDI)
- new net: D3919.2 (CKO), D3920.5 (CKI)
- new net: D3919.3 (SDO), D3920.4 (SDI)
- new net: D256.2 (CKO), D257.5 (CKI)
- new net: D256.3 (SDO), D257.4 (SDI)
- new net: D1850.2 (CKO), D1851.5 (CKI)
- new net: D1850.3 (SDO), D1851.4 (SDI)
- new net: D3770.3 (SDO), D3771.4 (SDI)
- new net: D3770.2 (CKO), D3771.5 (CKI)
- new net: D2443.3 (SDO), D2444.4 (SDI)
- new net: D2443.2 (CKO), D2444.5 (CKI)
- new net: D3544.2 (CKO), D3545.5 (CKI)
- new net: D3544.3 (SDO), D3545.4 (SDI)
- new net: D4084.3 (SDO), D4085.4 (SDI)
- new net: D4084.2 (CKO), D4085.5 (CKI)
- new net: D1534.2 (CKO), D1535.5 (CKI)
- new net: D1534.3 (SDO), D1535.4 (SDI)
- new net: D1247.2 (CKO), D1248.5 (CKI)
- new net: D1247.3 (SDO), D1248.4 (SDI)
- new net: D3692.2 (CKO), D3693.5 (CKI)
- new net: D3692.3 (SDO), D3693.4 (SDI)
- new net: D1660.2 (CKO), D1661.5 (CKI)
- new net: D1660.3 (SDO), D1661.4 (SDI)
- new net: D2236.2 (CKO), D2237.5 (CKI)
- new net: D2236.3 (SDO), D2237.4 (SDI)
- new net: D2932.3 (SDO), D2933.4 (SDI)
- new net: D2932.2 (CKO), D2933.5 (CKI)
- new net: D3032.2 (CKO), D3033.5 (CKI)
- new net: D3032.3 (SDO), D3033.4 (SDI)
- new net: D2061.2 (CKO), D2062.5 (CKI)
- new net: D2061.3 (SDO), D2062.4 (SDI)
- new net: D713.3 (SDO), D714.4 (SDI)
- new net: D713.2 (CKO), D714.5 (CKI)
- new net: D887.2 (CKO), D888.5 (CKI)
- new net: D887.3 (SDO), D888.4 (SDI)
- new net: D3387.2 (CKO), D3388.5 (CKI)
- new net: D3387.3 (SDO), D3388.4 (SDI)
- new net: D4146.2 (CKO), D4147.5 (CKI)
- new net: D4146.3 (SDO), D4147.4 (SDI)
- new net: D3462.3 (SDO), D3463.4 (SDI)
- new net: D3462.2 (CKO), D3463.5 (CKI)
- new net: D1926.3 (SDO), D1927.4 (SDI)
- new net: D1926.2 (CKO), D1927.5 (CKI)
- new net: D89.2 (CKO), D90.5 (CKI)
- new net: D89.3 (SDO), D90.4 (SDI)
- new net: D993.2 (CKO), D994.5 (CKI)
- new net: D993.3 (SDO), D994.4 (SDI)
- new net: D3144.2 (CKO), D3145.5 (CKI)
- new net: D3144.3 (SDO), D3145.4 (SDI)
- new net: D3602.3 (SDO), D3603.4 (SDI)
- new net: D3602.2 (CKO), D3603.5 (CKI)
- new net: D893.2 (CKO), D894.5 (CKI)
- new net: D893.3 (SDO), D894.4 (SDI)
- new net: D2025.3 (SDO), D2026.4 (SDI)
- new net: D2025.2 (CKO), D2026.5 (CKI)
- new net: D2448.3 (SDO), D2449.4 (SDI)
- new net: D2448.2 (CKO), D2449.5 (CKI)
- new net: D3764.3 (SDO), D3765.4 (SDI)
- new net: D3764.2 (CKO), D3765.5 (CKI)
- new net: D1967.2 (CKO), D1968.5 (CKI)
- new net: D1967.3 (SDO), D1968.4 (SDI)
- new net: D1966.3 (SDO), D1967.4 (SDI)
- new net: D1966.2 (CKO), D1967.5 (CKI)
- new net: D3822.3 (SDO), D3823.4 (SDI)
- new net: D3822.2 (CKO), D3823.5 (CKI)
- new net: D1763.2 (CKO), D1764.5 (CKI)
- new net: D1763.3 (SDO), D1764.4 (SDI)
- new net: D990.3 (SDO), D991.4 (SDI)
- new net: D990.2 (CKO), D991.5 (CKI)
- new net: D554.3 (SDO), D555.4 (SDI)
- new net: D554.2 (CKO), D555.5 (CKI)
- new net: D1706.2 (CKO), D1707.5 (CKI)
- new net: D1706.3 (SDO), D1707.4 (SDI)
- new net: D2516.3 (SDO), D2517.4 (SDI)
- new net: D2516.2 (CKO), D2517.5 (CKI)
- new net: D1270.2 (CKO), D1271.5 (CKI)
- new net: D1270.3 (SDO), D1271.4 (SDI)
- new net: D1005.2 (CKO), D1006.5 (CKI)
- new net: D1005.3 (SDO), D1006.4 (SDI)
- new net: D1613.2 (CKO), D1614.5 (CKI)
- new net: D1613.3 (SDO), D1614.4 (SDI)
- new net: D3515.3 (SDO), D3516.4 (SDI)
- new net: D3515.2 (CKO), D3516.5 (CKI)
- new net: D3648.3 (SDO), D3649.4 (SDI)
- new net: D3648.2 (CKO), D3649.5 (CKI)
- new net: D952.2 (CKO), D953.5 (CKI)
- new net: D952.3 (SDO), D953.4 (SDI)
- new net: D3623.2 (CKO), D3624.5 (CKI)
- new net: D3623.3 (SDO), D3624.4 (SDI)
- new net: D2685.2 (CKO), D2686.5 (CKI)
- new net: D2685.3 (SDO), D2686.4 (SDI)
- new net: D1248.3 (SDO), D1249.4 (SDI)
- new net: D1248.2 (CKO), D1249.5 (CKI)
- new net: D4168.2 (CKO), D4169.5 (CKI)
- new net: D4168.3 (SDO), D4169.4 (SDI)
- new net: D1184.2 (CKO), D1185.5 (CKI)
- new net: D1184.3 (SDO), D1185.4 (SDI)
- new net: D1674.3 (SDO), D1675.4 (SDI)
- new net: D1674.2 (CKO), D1675.5 (CKI)
- new net: D3842.2 (CKO), D3843.5 (CKI)
- new net: D3842.3 (SDO), D3843.4 (SDI)
- new net: D219.3 (SDO), D220.4 (SDI)
- new net: D219.2 (CKO), D220.5 (CKI)
- new net: D3563.2 (CKO), D3564.5 (CKI)
- new net: D3563.3 (SDO), D3564.4 (SDI)
- new net: D2519.2 (CKO), D2520.5 (CKI)
- new net: D2519.3 (SDO), D2520.4 (SDI)
- new net: D3700.2 (CKO), D3701.5 (CKI)
- new net: D3700.3 (SDO), D3701.4 (SDI)
- new net: D2858.3 (SDO), D2859.4 (SDI)
- new net: D2858.2 (CKO), D2859.5 (CKI)
- new net: D83.2 (CKO), D84.5 (CKI)
- new net: D83.3 (SDO), D84.4 (SDI)
- new net: D82.3 (SDO), D83.4 (SDI)
- new net: D82.2 (CKO), D83.5 (CKI)
- new net: D132.2 (CKO), D133.5 (CKI)
- new net: D132.3 (SDO), D133.4 (SDI)
- new net: D1206.2 (CKO), D1207.5 (CKI)
- new net: D1206.3 (SDO), D1207.4 (SDI)
- new net: D2031.2 (CKO), D2032.5 (CKI)
- new net: D2031.3 (SDO), D2032.4 (SDI)
- new net: D1733.3 (SDO), D1734.4 (SDI)
- new net: D1733.2 (CKO), D1734.5 (CKI)
- new net: D1087.3 (SDO), D1088.4 (SDI)
- new net: D1087.2 (CKO), D1088.5 (CKI)
- new net: D102.3 (SDO), D103.4 (SDI)
- new net: D102.2 (CKO), D103.5 (CKI)
- new net: D1541.3 (SDO), D1542.4 (SDI)
- new net: D1541.2 (CKO), D1542.5 (CKI)
- new net: D742.3 (SDO), D743.4 (SDI)
- new net: D742.2 (CKO), D743.5 (CKI)
- new net: D3140.2 (CKO), D3141.5 (CKI)
- new net: D3140.3 (SDO), D3141.4 (SDI)
- new net: D1796.3 (SDO), D1797.4 (SDI)
- new net: D1796.2 (CKO), D1797.5 (CKI)
- new net: D3409.2 (CKO), D3410.5 (CKI)
- new net: D3409.3 (SDO), D3410.4 (SDI)
- new net: D1637.2 (CKO), D1638.5 (CKI)
- new net: D1637.3 (SDO), D1638.4 (SDI)
- new net: D2805.3 (SDO), D2806.4 (SDI)
- new net: D2805.2 (CKO), D2806.5 (CKI)
- new net: D1665.2 (CKO), D1666.5 (CKI)
- new net: D1665.3 (SDO), D1666.4 (SDI)
- new net: D401.2 (CKO), D402.5 (CKI)
- new net: D401.3 (SDO), D402.4 (SDI)
- new net: D3644.2 (CKO), D3645.5 (CKI)
- new net: D3644.3 (SDO), D3645.4 (SDI)
- new net: D3643.3 (SDO), D3644.4 (SDI)
- new net: D3643.2 (CKO), D3644.5 (CKI)
- new net: D2306.3 (SDO), D2307.4 (SDI)
- new net: D2306.2 (CKO), D2307.5 (CKI)
- new net: D874.2 (CKO), D875.5 (CKI)
- new net: D874.3 (SDO), D875.4 (SDI)
- new net: D2351.3 (SDO), D2352.4 (SDI)
- new net: D2351.2 (CKO), D2352.5 (CKI)
- new net: D213.2 (CKO), D214.5 (CKI)
- new net: D213.3 (SDO), D214.4 (SDI)
- new net: D3201.3 (SDO), D3202.4 (SDI)
- new net: D3201.2 (CKO), D3202.5 (CKI)
- new net: D884.3 (SDO), D885.4 (SDI)
- new net: D884.2 (CKO), D885.5 (CKI)
- new net: D2846.3 (SDO), D2847.4 (SDI)
- new net: D2846.2 (CKO), D2847.5 (CKI)
- new net: D1034.3 (SDO), D1035.4 (SDI)
- new net: D1034.2 (CKO), D1035.5 (CKI)
- new net: D1129.3 (SDO), D1130.4 (SDI)
- new net: D1129.2 (CKO), D1130.5 (CKI)
- new net: D2546.2 (CKO), D2547.5 (CKI)
- new net: D2546.3 (SDO), D2547.4 (SDI)
- new net: D597.2 (CKO), D598.5 (CKI)
- new net: D597.3 (SDO), D598.4 (SDI)
- new net: D3038.2 (CKO), D3039.5 (CKI)
- new net: D3038.3 (SDO), D3039.4 (SDI)
- new net: D1101.3 (SDO), D1102.4 (SDI)
- new net: D1101.2 (CKO), D1102.5 (CKI)
- new net: D238.2 (CKO), D239.5 (CKI)
- new net: D238.3 (SDO), D239.4 (SDI)
- new net: D2584.2 (CKO), D2585.5 (CKI)
- new net: D2584.3 (SDO), D2585.4 (SDI)
- new net: D2583.3 (SDO), D2584.4 (SDI)
- new net: D2583.2 (CKO), D2584.5 (CKI)
- new net: D1343.2 (CKO), D1344.5 (CKI)
- new net: D1343.3 (SDO), D1344.4 (SDI)
- new net: D2507.3 (SDO), D2508.4 (SDI)
- new net: D2507.2 (CKO), D2508.5 (CKI)
- new net: D3955.2 (CKO), D3956.5 (CKI)
- new net: D3955.3 (SDO), D3956.4 (SDI)
- new net: D3184.3 (SDO), D3185.4 (SDI)
- new net: D3184.2 (CKO), D3185.5 (CKI)
- new net: D225.2 (CKO), D226.5 (CKI)
- new net: D225.3 (SDO), D226.4 (SDI)
- new net: D1023.2 (CKO), D1024.5 (CKI)
- new net: D1023.3 (SDO), D1024.4 (SDI)
- new net: D2924.3 (SDO), D2925.4 (SDI)
- new net: D2924.2 (CKO), D2925.5 (CKI)
- new net: D536.2 (CKO), D537.5 (CKI)
- new net: D536.3 (SDO), D537.4 (SDI)
- new net: D1274.2 (CKO), D1275.5 (CKI)
- new net: D1274.3 (SDO), D1275.4 (SDI)
- new net: D2879.3 (SDO), D2880.4 (SDI)
- new net: D2879.2 (CKO), D2880.5 (CKI)
- new net: D2370.3 (SDO), D2371.4 (SDI)
- new net: D2370.2 (CKO), D2371.5 (CKI)
- new net: D1167.2 (CKO), D1168.5 (CKI)
- new net: D1167.3 (SDO), D1168.4 (SDI)
- new net: D1523.2 (CKO), D1524.5 (CKI)
- new net: D1523.3 (SDO), D1524.4 (SDI)
- new net: D2428.2 (CKO), D2429.5 (CKI)
- new net: D2428.3 (SDO), D2429.4 (SDI)
- new net: D4058.3 (SDO), D4059.4 (SDI)
- new net: D4058.2 (CKO), D4059.5 (CKI)
- new net: D2336.2 (CKO), D2337.5 (CKI)
- new net: D2336.3 (SDO), D2337.4 (SDI)
- new net: D3509.2 (CKO), D3510.5 (CKI)
- new net: D3509.3 (SDO), D3510.4 (SDI)
- new net: D3508.3 (SDO), D3509.4 (SDI)
- new net: D3508.2 (CKO), D3509.5 (CKI)
- new net: D462.3 (SDO), D463.4 (SDI)
- new net: D462.2 (CKO), D463.5 (CKI)
- new net: D2488.3 (SDO), D2489.4 (SDI)
- new net: D2488.2 (CKO), D2489.5 (CKI)
- new net: D3058.2 (CKO), D3059.5 (CKI)
- new net: D3058.3 (SDO), D3059.4 (SDI)
- new net: D3834.2 (CKO), D3835.5 (CKI)
- new net: D3834.3 (SDO), D3835.4 (SDI)
- new net: D1367.3 (SDO), D1368.4 (SDI)
- new net: D1367.2 (CKO), D1368.5 (CKI)
- new net: D2540.2 (CKO), D2541.5 (CKI)
- new net: D2540.3 (SDO), D2541.4 (SDI)
- new net: D2956.3 (SDO), D2957.4 (SDI)
- new net: D2956.2 (CKO), D2957.5 (CKI)
- new net: D2680.3 (SDO), D2681.4 (SDI)
- new net: D2680.2 (CKO), D2681.5 (CKI)
- new net: D1100.2 (CKO), D1101.5 (CKI)
- new net: D1100.3 (SDO), D1101.4 (SDI)
- new net: D356.2 (CKO), D357.5 (CKI)
- new net: D356.3 (SDO), D357.4 (SDI)
- new net: D1380.2 (CKO), D1381.5 (CKI)
- new net: D1380.3 (SDO), D1381.4 (SDI)
- new net: D2689.3 (SDO), D2690.4 (SDI)
- new net: D2689.2 (CKO), D2690.5 (CKI)
- new net: D2704.3 (SDO), D2705.4 (SDI)
- new net: D2704.2 (CKO), D2705.5 (CKI)
- new net: D2343.2 (CKO), D2344.5 (CKI)
- new net: D2343.3 (SDO), D2344.4 (SDI)
- new net: D2342.3 (SDO), D2343.4 (SDI)
- new net: D2342.2 (CKO), D2343.5 (CKI)
- new net: D3020.3 (SDO), D3021.4 (SDI)
- new net: D3020.2 (CKO), D3021.5 (CKI)
- new net: D1051.3 (SDO), D1052.4 (SDI)
- new net: D1051.2 (CKO), D1052.5 (CKI)
- new net: D2737.2 (CKO), D2738.5 (CKI)
- new net: D2737.3 (SDO), D2738.4 (SDI)
- new net: D3002.2 (CKO), D3003.5 (CKI)
- new net: D3002.3 (SDO), D3003.4 (SDI)
- new net: D3001.3 (SDO), D3002.4 (SDI)
- new net: D3001.2 (CKO), D3002.5 (CKI)
- new net: D3802.3 (SDO), D3803.4 (SDI)
- new net: D3802.2 (CKO), D3803.5 (CKI)
- new net: D2045.3 (SDO), D2046.4 (SDI)
- new net: D2045.2 (CKO), D2046.5 (CKI)
- new net: D3534.2 (CKO), D3535.5 (CKI)
- new net: D3534.3 (SDO), D3535.4 (SDI)
- new net: D4057.3 (SDO), D4058.4 (SDI)
- new net: D4057.2 (CKO), D4058.5 (CKI)
- new net: D796.2 (CKO), D797.5 (CKI)
- new net: D796.3 (SDO), D797.4 (SDI)
- new net: D3112.3 (SDO), D3113.4 (SDI)
- new net: D3112.2 (CKO), D3113.5 (CKI)
- new net: D3530.3 (SDO), D3531.4 (SDI)
- new net: D3530.2 (CKO), D3531.5 (CKI)
- new net: D1039.3 (SDO), D1040.4 (SDI)
- new net: D1039.2 (CKO), D1040.5 (CKI)
- new net: D1789.3 (SDO), D1790.4 (SDI)
- new net: D1789.2 (CKO), D1790.5 (CKI)
- new net: D1999.3 (SDO), D2000.4 (SDI)
- new net: D1999.2 (CKO), D2000.5 (CKI)
- new net: D1829.2 (CKO), D1830.5 (CKI)
- new net: D1829.3 (SDO), D1830.4 (SDI)
- new net: D590.3 (SDO), D591.4 (SDI)
- new net: D590.2 (CKO), D591.5 (CKI)
- new net: D1830.2 (CKO), D1831.5 (CKI)
- new net: D1830.3 (SDO), D1831.4 (SDI)
- new net: D3230.3 (SDO), D3231.4 (SDI)
- new net: D3230.2 (CKO), D3231.5 (CKI)
- new net: D3652.2 (CKO), D3653.5 (CKI)
- new net: D3652.3 (SDO), D3653.4 (SDI)
- new net: D2268.3 (SDO), D2269.4 (SDI)
- new net: D2268.2 (CKO), D2269.5 (CKI)
- new net: D3363.2 (CKO), D3364.5 (CKI)
- new net: D3363.3 (SDO), D3364.4 (SDI)
- new net: D3978.3 (SDO), D3979.4 (SDI)
- new net: D3978.2 (CKO), D3979.5 (CKI)
- new net: D2321.2 (CKO), D2322.5 (CKI)
- new net: D2321.3 (SDO), D2322.4 (SDI)
- new net: D1128.3 (SDO), D1129.4 (SDI)
- new net: D1128.2 (CKO), D1129.5 (CKI)
- new net: D3944.2 (CKO), D3945.5 (CKI)
- new net: D3944.3 (SDO), D3945.4 (SDI)
- new net: D2786.2 (CKO), D2787.5 (CKI)
- new net: D2786.3 (SDO), D2787.4 (SDI)
- new net: D3471.3 (SDO), D3472.4 (SDI)
- new net: D3471.2 (CKO), D3472.5 (CKI)
- new net: J11.1 (Pin_1), J5.1 (Pin_1)
- new net: D1840.2 (CKO), D1841.5 (CKI)
- new net: D1840.3 (SDO), D1841.4 (SDI)
- new net: D1711.2 (CKO), D1712.5 (CKI)
- new net: D1711.3 (SDO), D1712.4 (SDI)
- new net: D3538.2 (CKO), D3539.5 (CKI)
- new net: D3538.3 (SDO), D3539.4 (SDI)
- new net: D2442.3 (SDO), D2443.4 (SDI)
- new net: D2442.2 (CKO), D2443.5 (CKI)
- new net: D2512.2 (CKO), D2513.5 (CKI)
- new net: D2512.3 (SDO), D2513.4 (SDI)
- new net: D1601.2 (CKO), D1602.5 (CKI)
- new net: D1601.3 (SDO), D1602.4 (SDI)
- new net: D2850.3 (SDO), D2851.4 (SDI)
- new net: D2850.2 (CKO), D2851.5 (CKI)
- new net: D2194.2 (CKO), D2195.5 (CKI)
- new net: D2194.3 (SDO), D2195.4 (SDI)
- new net: D1392.3 (SDO), D1393.4 (SDI)
- new net: D1392.2 (CKO), D1393.5 (CKI)
- new net: D1195.2 (CKO), D1196.5 (CKI)
- new net: D1195.3 (SDO), D1196.4 (SDI)
- new net: D3246.3 (SDO), D3247.4 (SDI)
- new net: D3246.2 (CKO), D3247.5 (CKI)
- new net: D2207.2 (CKO), D2208.5 (CKI)
- new net: D2207.3 (SDO), D2208.4 (SDI)
- new net: D2206.3 (SDO), D2207.4 (SDI)
- new net: D2206.2 (CKO), D2207.5 (CKI)
- new net: D1309.3 (SDO), D1310.4 (SDI)
- new net: D1309.2 (CKO), D1310.5 (CKI)
- new net: D2092.2 (CKO), D2093.5 (CKI)
- new net: D2092.3 (SDO), D2093.4 (SDI)
- new net: D923.3 (SDO), D924.4 (SDI)
- new net: D923.2 (CKO), D924.5 (CKI)
- new net: D1993.3 (SDO), D1994.4 (SDI)
- new net: D1993.2 (CKO), D1994.5 (CKI)
- new net: D2191.3 (SDO), D2192.4 (SDI)
- new net: D2191.2 (CKO), D2192.5 (CKI)
- new net: D1596.3 (SDO), D1597.4 (SDI)
- new net: D1596.2 (CKO), D1597.5 (CKI)
- new net: D426.2 (CKO), D427.5 (CKI)
- new net: D426.3 (SDO), D427.4 (SDI)
- new net: D3708.3 (SDO), D3709.4 (SDI)
- new net: D3708.2 (CKO), D3709.5 (CKI)
- new net: D3670.3 (SDO), D3671.4 (SDI)
- new net: D3670.2 (CKO), D3671.5 (CKI)
- new net: D1097.2 (CKO), D1098.5 (CKI)
- new net: D1097.3 (SDO), D1098.4 (SDI)
- new net: D4112.2 (CKO), D4113.5 (CKI)
- new net: D4112.3 (SDO), D4113.4 (SDI)
- new net: D3132.2 (CKO), D3133.5 (CKI)
- new net: D3132.3 (SDO), D3133.4 (SDI)
- new net: D675.2 (CKO), D676.5 (CKI)
- new net: D675.3 (SDO), D676.4 (SDI)
- new net: D1445.3 (SDO), D1446.4 (SDI)
- new net: D1445.2 (CKO), D1446.5 (CKI)
- new net: D3306.2 (CKO), D3307.5 (CKI)
- new net: D3306.3 (SDO), D3307.4 (SDI)
- new net: D725.3 (SDO), D726.4 (SDI)
- new net: D725.2 (CKO), D726.5 (CKI)
- new net: D1210.3 (SDO), D1211.4 (SDI)
- new net: D1210.2 (CKO), D1211.5 (CKI)
- new net: D2471.2 (CKO), D2472.5 (CKI)
- new net: D2471.3 (SDO), D2472.4 (SDI)
- new net: D3899.2 (CKO), D3900.5 (CKI)
- new net: D3899.3 (SDO), D3900.4 (SDI)
- new net: D1647.3 (SDO), D1648.4 (SDI)
- new net: D1647.2 (CKO), D1648.5 (CKI)
- new net: D96.3 (SDO), D97.4 (SDI)
- new net: D96.2 (CKO), D97.5 (CKI)
- new net: D1229.2 (CKO), D1230.5 (CKI)
- new net: D1229.3 (SDO), D1230.4 (SDI)
- new net: D2126.2 (CKO), D2127.5 (CKI)
- new net: D2126.3 (SDO), D2127.4 (SDI)
- new net: D1862.3 (SDO), D1863.4 (SDI)
- new net: D1862.2 (CKO), D1863.5 (CKI)
- new net: D431.2 (CKO), D432.5 (CKI)
- new net: D431.3 (SDO), D432.4 (SDI)
- new net: D2534.3 (SDO), D2535.4 (SDI)
- new net: D2534.2 (CKO), D2535.5 (CKI)
- new net: D1334.2 (CKO), D1335.5 (CKI)
- new net: D1334.3 (SDO), D1335.4 (SDI)
- new net: D218.3 (SDO), D219.4 (SDI)
- new net: D218.2 (CKO), D219.5 (CKI)
- new net: D2947.3 (SDO), D2948.4 (SDI)
- new net: D2947.2 (CKO), D2948.5 (CKI)
- new net: D2571.2 (CKO), D2572.5 (CKI)
- new net: D2571.3 (SDO), D2572.4 (SDI)
- new net: D3382.3 (SDO), D3383.4 (SDI)
- new net: D3382.2 (CKO), D3383.5 (CKI)
- new net: D2127.2 (CKO), D2128.5 (CKI)
- new net: D2127.3 (SDO), D2128.4 (SDI)
- new net: D3684.2 (CKO), D3685.5 (CKI)
- new net: D3684.3 (SDO), D3685.4 (SDI)
- new net: D3894.2 (CKO), D3895.5 (CKI)
- new net: D3894.3 (SDO), D3895.4 (SDI)
- new net: D2772.2 (CKO), D2773.5 (CKI)
- new net: D2772.3 (SDO), D2773.4 (SDI)
- new net: D1779.2 (CKO), D1780.5 (CKI)
- new net: D1779.3 (SDO), D1780.4 (SDI)
- new net: D1778.3 (SDO), D1779.4 (SDI)
- new net: D1778.2 (CKO), D1779.5 (CKI)
- new net: D1000.5 (CKI), D999.2 (CKO)
- new net: D1000.4 (SDI), D999.3 (SDO)
- new net: D2111.3 (SDO), D2112.4 (SDI)
- new net: D2111.2 (CKO), D2112.5 (CKI)
- new net: D2801.3 (SDO), D2802.4 (SDI)
- new net: D2801.2 (CKO), D2802.5 (CKI)
- new net: J11.2 (Pin_2), J4.1 (Pin_1)
- new net: D3455.3 (SDO), D3456.4 (SDI)
- new net: D3455.2 (CKO), D3456.5 (CKI)
- new net: D647.3 (SDO), D648.4 (SDI)
- new net: D647.2 (CKO), D648.5 (CKI)
- new net: D4113.3 (SDO), D4114.4 (SDI)
- new net: D4113.2 (CKO), D4114.5 (CKI)
- new net: D3607.3 (SDO), D3608.4 (SDI)
- new net: D3607.2 (CKO), D3608.5 (CKI)
- new net: D525.2 (CKO), D526.5 (CKI)
- new net: D525.3 (SDO), D526.4 (SDI)
- new net: D1118.2 (CKO), D1119.5 (CKI)
- new net: D1118.3 (SDO), D1119.4 (SDI)
- new net: D2483.2 (CKO), D2484.5 (CKI)
- new net: D2483.3 (SDO), D2484.4 (SDI)
- new net: D1946.3 (SDO), D1947.4 (SDI)
- new net: D1946.2 (CKO), D1947.5 (CKI)
- new net: D2434.2 (CKO), D2435.5 (CKI)
- new net: D2434.3 (SDO), D2435.4 (SDI)
- new net: D3214.3 (SDO), D3215.4 (SDI)
- new net: D3214.2 (CKO), D3215.5 (CKI)
- new net: D1512.3 (SDO), D1513.4 (SDI)
- new net: D1512.2 (CKO), D1513.5 (CKI)
- new net: D2941.2 (CKO), D2942.5 (CKI)
- new net: D2941.3 (SDO), D2942.4 (SDI)
- new net: D2941.4 (SDI), J24.2 (Pin_2)
- new net: D3367.2 (CKO), D3368.5 (CKI)
- new net: D3367.3 (SDO), D3368.4 (SDI)
- new net: D1671.2 (CKO), D1672.5 (CKI)
- new net: D1671.3 (SDO), D1672.4 (SDI)
- new net: D762.2 (CKO), D763.5 (CKI)
- new net: D762.3 (SDO), D763.4 (SDI)
- new net: D2787.3 (SDO), D2788.4 (SDI)
- new net: D2787.2 (CKO), D2788.5 (CKI)
- new net: D357.2 (CKO), D358.5 (CKI)
- new net: D357.3 (SDO), D358.4 (SDI)
- new net: D3412.2 (CKO), D3413.5 (CKI)
- new net: D3412.3 (SDO), D3413.4 (SDI)
- new net: D3593.2 (CKO), D3594.5 (CKI)
- new net: D3593.3 (SDO), D3594.4 (SDI)
- new net: D4161.2 (CKO), D4162.5 (CKI)
- new net: D4161.3 (SDO), D4162.4 (SDI)
- new net: D2796.3 (SDO), D2797.4 (SDI)
- new net: D2796.2 (CKO), D2797.5 (CKI)
- new net: D2472.3 (SDO), D2473.4 (SDI)
- new net: D2472.2 (CKO), D2473.5 (CKI)
- new net: D3539.2 (CKO), D3540.5 (CKI)
- new net: D3539.3 (SDO), D3540.4 (SDI)
- new net: D3174.2 (CKO), D3175.5 (CKI)
- new net: D3174.3 (SDO), D3175.4 (SDI)
- new net: D1295.2 (CKO), D1296.5 (CKI)
- new net: D1295.3 (SDO), D1296.4 (SDI)
- new net: D1987.3 (SDO), D1988.4 (SDI)
- new net: D1987.2 (CKO), D1988.5 (CKI)
- new net: D3320.3 (SDO), D3321.4 (SDI)
- new net: D3320.2 (CKO), D3321.5 (CKI)
- new net: D2627.2 (CKO), D2628.5 (CKI)
- new net: D2627.3 (SDO), D2628.4 (SDI)
- new net: D970.2 (CKO), D971.5 (CKI)
- new net: D970.3 (SDO), D971.4 (SDI)
- new net: D3929.2 (CKO), D3930.5 (CKI)
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Other:
- note removed: "BLOCK 5"
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