File: ATMEGA-SCHEMATICS/SNAKE_GAME/GRID_SCHEMATICS/GRID/GRID.kicad_pcb (KiCad board)
At the start: 2 copper layers, 55 x 35 mm, 46 parts, among them J1 Conn_01x04_Pin, J2 Conn_01x04_Pin

Commit message: .
Parts:
- removed C10, C11, C12, C13, C14, C15, C16, C17, C18, C19, C20, C21, C22, C23, C24, C25, C6, C7, C8, C9: 1uF, Capacitor_SMD:C_0603_1608Metric
- removed D1, D10, D11, D13, D14, D15, D16, D2, D21, D22, D23, D24, D25, D3, D4, D5, D6, D7, D8, D9: APA102-2020, LED_SMD:LED-APA102-2020
- removed H1, H2, H3, H4: MountingHole, MountingHole:MountingHole_2.1mm
- removed J2: Conn_01x04_Pin, Connector_PinSocket_2.54mm:PinSocket_1x04_P2.54mm_Vertical
- added C137: 1uF, Capacitor_SMD:C_0603_1608Metric, F.Cu at (-45.2, 74.2)
- added C138: 1uF, Capacitor_SMD:C_0603_1608Metric, F.Cu at (-45.2, 76.8)
- added C139: 1uF, Capacitor_SMD:C_0603_1608Metric, F.Cu at (-45.2, 79.3)
- added C140: 1uF, Capacitor_SMD:C_0603_1608Metric, F.Cu at (-45.2, 81.8)
- added C141: 1uF, Capacitor_SMD:C_0603_1608Metric, F.Cu at (-45.2, 84.3)
- added C142: 1uF, Capacitor_SMD:C_0603_1608Metric, F.Cu at (-45.2, 86.8)
- added C143: 1uF, Capacitor_SMD:C_0603_1608Metric, F.Cu at (-41.2, 44.1)
- added C144: 1uF, Capacitor_SMD:C_0603_1608Metric, F.Cu at (-41.2, 46.6)
- added C145: 1uF, Capacitor_SMD:C_0603_1608Metric, F.Cu at (-41.2, 49.1)
- added C146: 1uF, Capacitor_SMD:C_0603_1608Metric, F.Cu at (-41.2, 51.7)
- added C147: 1uF, Capacitor_SMD:C_0603_1608Metric, F.Cu at (-41.2, 54.2)
- added C148: 1uF, Capacitor_SMD:C_0603_1608Metric, F.Cu at (-41.2, 56.7)
- added C149: 1uF, Capacitor_SMD:C_0603_1608Metric, F.Cu at (-41.2, 59.2)
- added C150: 1uF, Capacitor_SMD:C_0603_1608Metric, F.Cu at (-41.2, 61.7)
- added C151: 1uF, Capacitor_SMD:C_0603_1608Metric, F.Cu at (-41.2, 64.2)
- added C152: 1uF, Capacitor_SMD:C_0603_1608Metric, F.Cu at (-41.2, 66.7)
- added C153: 1uF, Capacitor_SMD:C_0603_1608Metric, F.Cu at (-41.2, 69.2)
- added C154: 1uF, Capacitor_SMD:C_0603_1608Metric, F.Cu at (-41.2, 71.7)
- added C155: 1uF, Capacitor_SMD:C_0603_1608Metric, F.Cu at (-41.2, 74.2)
- added C156: 1uF, Capacitor_SMD:C_0603_1608Metric, F.Cu at (-41.2, 76.8)
- added C157: 1uF, Capacitor_SMD:C_0603_1608Metric, F.Cu at (-41.2, 79.3)
- added C158: 1uF, Capacitor_SMD:C_0603_1608Metric, F.Cu at (-41.2, 81.8)
- added C159: 1uF, Capacitor_SMD:C_0603_1608Metric, F.Cu at (-41.2, 84.3)
- added C160: 1uF, Capacitor_SMD:C_0603_1608Metric, F.Cu at (-41.2, 86.8)
- added C161: 1uF, Capacitor_SMD:C_0603_1608Metric, F.Cu at (-37.2, 44.1)
- added C162: 1uF, Capacitor_SMD:C_0603_1608Metric, F.Cu at (-37.2, 46.6)
- added C163: 1uF, Capacitor_SMD:C_0603_1608Metric, F.Cu at (-37.2, 49.1)
- added C164: 1uF, Capacitor_SMD:C_0603_1608Metric, F.Cu at (-37.2, 51.7)
- added C165: 1uF, Capacitor_SMD:C_0603_1608Metric, F.Cu at (-37.2, 54.2)
- added C166: 1uF, Capacitor_SMD:C_0603_1608Metric, F.Cu at (-37.2, 56.7)
- added C167: 1uF, Capacitor_SMD:C_0603_1608Metric, F.Cu at (-37.2, 59.2)
- added C168: 1uF, Capacitor_SMD:C_0603_1608Metric, F.Cu at (-37.2, 61.7)
- added C169: 1uF, Capacitor_SMD:C_0603_1608Metric, F.Cu at (-37.2, 64.2)
- added C170: 1uF, Capacitor_SMD:C_0603_1608Metric, F.Cu at (-37.2, 66.7)
- added C171: 1uF, Capacitor_SMD:C_0603_1608Metric, F.Cu at (-37.2, 69.2)
- added C172: 1uF, Capacitor_SMD:C_0603_1608Metric, F.Cu at (-37.2, 71.7)
- added C173: 1uF, Capacitor_SMD:C_0603_1608Metric, F.Cu at (-37.2, 74.2)
- added C174: 1uF, Capacitor_SMD:C_0603_1608Metric, F.Cu at (-37.2, 76.8)
- added C175: 1uF, Capacitor_SMD:C_0603_1608Metric, F.Cu at (-37.2, 79.3)
- added C176: 1uF, Capacitor_SMD:C_0603_1608Metric, F.Cu at (-37.2, 81.8)
- added C177: 1uF, Capacitor_SMD:C_0603_1608Metric, F.Cu at (-37.2, 84.3)
- added C178: 1uF, Capacitor_SMD:C_0603_1608Metric, F.Cu at (-37.2, 86.8)
- added C179: 1uF, Capacitor_SMD:C_0603_1608Metric, F.Cu at (-33.2, 44.1)
- added C180: 1uF, Capacitor_SMD:C_0603_1608Metric, F.Cu at (-33.2, 46.6)
- added C181: 1uF, Capacitor_SMD:C_0603_1608Metric, F.Cu at (-33.2, 49.1)
- added C182: 1uF, Capacitor_SMD:C_0603_1608Metric, F.Cu at (-33.2, 51.7)
- added C183: 1uF, Capacitor_SMD:C_0603_1608Metric, F.Cu at (-33.2, 54.2)
- added C184: 1uF, Capacitor_SMD:C_0603_1608Metric, F.Cu at (-33.2, 56.7)
- added C185: 1uF, Capacitor_SMD:C_0603_1608Metric, F.Cu at (-33.2, 59.2)
- added C186: 1uF, Capacitor_SMD:C_0603_1608Metric, F.Cu at (-33.2, 61.7)
- added C187: 1uF, Capacitor_SMD:C_0603_1608Metric, F.Cu at (-33.2, 64.2)
- added C188: 1uF, Capacitor_SMD:C_0603_1608Metric, F.Cu at (-33.2, 66.7)
- added C189: 1uF, Capacitor_SMD:C_0603_1608Metric, F.Cu at (-33.2, 69.2)
- added C190: 1uF, Capacitor_SMD:C_0603_1608Metric, F.Cu at (-33.2, 71.7)
- added C191: 1uF, Capacitor_SMD:C_0603_1608Metric, F.Cu at (-33.2, 74.2)
- added C192: 1uF, Capacitor_SMD:C_0603_1608Metric, F.Cu at (-33.2, 76.8)
- added C193: 1uF, Capacitor_SMD:C_0603_1608Metric, F.Cu at (-33.2, 79.3)
- added C194: 1uF, Capacitor_SMD:C_0603_1608Metric, F.Cu at (-33.2, 81.8)
- added C195: 1uF, Capacitor_SMD:C_0603_1608Metric, F.Cu at (-33.2, 84.3)
- added C196: 1uF, Capacitor_SMD:C_0603_1608Metric, F.Cu at (-33.2, 86.8)
- added C197: 1uF, Capacitor_SMD:C_0603_1608Metric, F.Cu at (-29.2, 44.1)
- added C198: 1uF, Capacitor_SMD:C_0603_1608Metric, F.Cu at (-29.2, 46.6)
- added C199: 1uF, Capacitor_SMD:C_0603_1608Metric, F.Cu at (-29.2, 49.1)
- added C200: 1uF, Capacitor_SMD:C_0603_1608Metric, F.Cu at (-29.2, 51.7)
- added C201: 1uF, Capacitor_SMD:C_0603_1608Metric, F.Cu at (-29.2, 54.2)
- added C202: 1uF, Capacitor_SMD:C_0603_1608Metric, F.Cu at (-29.2, 56.7)
- added C203: 1uF, Capacitor_SMD:C_0603_1608Metric, F.Cu at (-29.2, 59.2)
- added C204: 1uF, Capacitor_SMD:C_0603_1608Metric, F.Cu at (-29.2, 61.7)
- added C205: 1uF, Capacitor_SMD:C_0603_1608Metric, F.Cu at (-29.2, 64.2)
- added C206: 1uF, Capacitor_SMD:C_0603_1608Metric, F.Cu at (-29.2, 66.7)
- added C207: 1uF, Capacitor_SMD:C_0603_1608Metric, F.Cu at (-29.2, 69.2)
- added C208: 1uF, Capacitor_SMD:C_0603_1608Metric, F.Cu at (-29.2, 71.7)
- added C209: 1uF, Capacitor_SMD:C_0603_1608Metric, F.Cu at (-29.2, 74.2)
- added C210: 1uF, Capacitor_SMD:C_0603_1608Metric, F.Cu at (-29.2, 76.8)
- added C211: 1uF, Capacitor_SMD:C_0603_1608Metric, F.Cu at (-29.2, 79.3)
- added C212: 1uF, Capacitor_SMD:C_0603_1608Metric, F.Cu at (-29.2, 81.8)
- added C213: 1uF, Capacitor_SMD:C_0603_1608Metric, F.Cu at (-29.2, 84.3)
- added C214: 1uF, Capacitor_SMD:C_0603_1608Metric, F.Cu at (-29.2, 86.8)
- added C215: 1uF, Capacitor_SMD:C_0603_1608Metric, F.Cu at (-25.1, 44.1)
- added C216: 1uF, Capacitor_SMD:C_0603_1608Metric, F.Cu at (-25.1, 46.6)
- added C217: 1uF, Capacitor_SMD:C_0603_1608Metric, F.Cu at (-25.1, 49.1)
- added C218: 1uF, Capacitor_SMD:C_0603_1608Metric, F.Cu at (-25.1, 51.7)
- added C219: 1uF, Capacitor_SMD:C_0603_1608Metric, F.Cu at (-25.1, 54.2)
- added C220: 1uF, Capacitor_SMD:C_0603_1608Metric, F.Cu at (-25.1, 56.7)
- added C221: 1uF, Capacitor_SMD:C_0603_1608Metric, F.Cu at (-25.1, 59.2)
- added C222: 1uF, Capacitor_SMD:C_0603_1608Metric, F.Cu at (-25.1, 61.7)
- added C223: 1uF, Capacitor_SMD:C_0603_1608Metric, F.Cu at (-25.1, 64.2)
- added C224: 1uF, Capacitor_SMD:C_0603_1608Metric, F.Cu at (-25.1, 66.7)
- added C225: 1uF, Capacitor_SMD:C_0603_1608Metric, F.Cu at (-25.1, 69.2)
- added C226: 1uF, Capacitor_SMD:C_0603_1608Metric, F.Cu at (-25.1, 71.7)
- added C227: 1uF, Capacitor_SMD:C_0603_1608Metric, F.Cu at (-25.1, 74.2)
- added C228: 1uF, Capacitor_SMD:C_0603_1608Metric, F.Cu at (-25.1, 76.8)
- added C229: 1uF, Capacitor_SMD:C_0603_1608Metric, F.Cu at (-25.1, 79.3)
- added C230: 1uF, Capacitor_SMD:C_0603_1608Metric, F.Cu at (-25.1, 81.8)
- added C231: 1uF, Capacitor_SMD:C_0603_1608Metric, F.Cu at (-25.1, 84.3)
- added C232: 1uF, Capacitor_SMD:C_0603_1608Metric, F.Cu at (-25.1, 86.8)
- added C233: 1uF, Capacitor_SMD:C_0603_1608Metric, F.Cu at (-21.1, 44.1)
- added C234: 1uF, Capacitor_SMD:C_0603_1608Metric, F.Cu at (-21.1, 46.6)
- added C235: 1uF, Capacitor_SMD:C_0603_1608Metric, F.Cu at (-21.1, 49.1)
- added C236: 1uF, Capacitor_SMD:C_0603_1608Metric, F.Cu at (-21.1, 51.7)
- added C237: 1uF, Capacitor_SMD:C_0603_1608Metric, F.Cu at (-21.1, 54.2)
- added C238: 1uF, Capacitor_SMD:C_0603_1608Metric, F.Cu at (-21.1, 56.7)
- added C239: 1uF, Capacitor_SMD:C_0603_1608Metric, F.Cu at (-21.1, 59.2)
- added C240: 1uF, Capacitor_SMD:C_0603_1608Metric, F.Cu at (-21.1, 61.7)
- added C241: 1uF, Capacitor_SMD:C_0603_1608Metric, F.Cu at (-21.1, 64.2)
- added C242: 1uF, Capacitor_SMD:C_0603_1608Metric, F.Cu at (-21.1, 66.7)
- added C243: 1uF, Capacitor_SMD:C_0603_1608Metric, F.Cu at (-21.1, 69.2)
- added C244: 1uF, Capacitor_SMD:C_0603_1608Metric, F.Cu at (-21.1, 71.7)
- added C245: 1uF, Capacitor_SMD:C_0603_1608Metric, F.Cu at (-21.1, 74.2)
- added C246: 1uF, Capacitor_SMD:C_0603_1608Metric, F.Cu at (-21.1, 76.8)
- added C247: 1uF, Capacitor_SMD:C_0603_1608Metric, F.Cu at (-21.1, 79.3)
- added C248: 1uF, Capacitor_SMD:C_0603_1608Metric, F.Cu at (-21.1, 81.8)
- added C249: 1uF, Capacitor_SMD:C_0603_1608Metric, F.Cu at (-21.1, 84.3)
- added C250: 1uF, Capacitor_SMD:C_0603_1608Metric, F.Cu at (-21.1, 86.8)
- added C251: 1uF, Capacitor_SMD:C_0603_1608Metric, F.Cu at (-17.1, 44.1)
- added C252: 1uF, Capacitor_SMD:C_0603_1608Metric, F.Cu at (-17.1, 46.6)
- added C253: 1uF, Capacitor_SMD:C_0603_1608Metric, F.Cu at (-17.1, 49.1)
- added C254: 1uF, Capacitor_SMD:C_0603_1608Metric, F.Cu at (-17.1, 51.7)
- added C255: 1uF, Capacitor_SMD:C_0603_1608Metric, F.Cu at (-17.1, 54.2)
- added C256: 1uF, Capacitor_SMD:C_0603_1608Metric, F.Cu at (-17.1, 56.7)
- added C257: 1uF, Capacitor_SMD:C_0603_1608Metric, F.Cu at (-17.1, 59.2)
- added C258: 1uF, Capacitor_SMD:C_0603_1608Metric, F.Cu at (-17.1, 61.7)
- added C259: 1uF, Capacitor_SMD:C_0603_1608Metric, F.Cu at (-17.1, 64.2)
- added C26: 1uF, Capacitor_SMD:C_0603_1608Metric, F.Cu at (-53.2, 44.1)
- added C260: 1uF, Capacitor_SMD:C_0603_1608Metric, F.Cu at (-17.1, 66.7)
- added C261: 1uF, Capacitor_SMD:C_0603_1608Metric, F.Cu at (-17.1, 69.2)
- added C262: 1uF, Capacitor_SMD:C_0603_1608Metric, F.Cu at (-17.1, 71.7)
- added C263: 1uF, Capacitor_SMD:C_0603_1608Metric, F.Cu at (-17.1, 74.2)
- added C264: 1uF, Capacitor_SMD:C_0603_1608Metric, F.Cu at (-17.1, 76.8)
- added C265: 1uF, Capacitor_SMD:C_0603_1608Metric, F.Cu at (-17.1, 79.3)
- added C266: 1uF, Capacitor_SMD:C_0603_1608Metric, F.Cu at (-17.1, 81.8)
- added C267: 1uF, Capacitor_SMD:C_0603_1608Metric, F.Cu at (-17.1, 84.3)
- added C268: 1uF, Capacitor_SMD:C_0603_1608Metric, F.Cu at (-17.1, 86.8)
- added C269: 1uF, Capacitor_SMD:C_0603_1608Metric, F.Cu at (-13.1, 44.1)
- added C270: 1uF, Capacitor_SMD:C_0603_1608Metric, F.Cu at (-13.1, 46.6)
- added C271: 1uF, Capacitor_SMD:C_0603_1608Metric, F.Cu at (-13.1, 49.1)
- added C272: 1uF, Capacitor_SMD:C_0603_1608Metric, F.Cu at (-13.1, 51.7)
- added C273: 1uF, Capacitor_SMD:C_0603_1608Metric, F.Cu at (-13.1, 54.2)
- added C274: 1uF, Capacitor_SMD:C_0603_1608Metric, F.Cu at (-13.1, 56.7)
- added C275: 1uF, Capacitor_SMD:C_0603_1608Metric, F.Cu at (-13.1, 59.2)
- added C276: 1uF, Capacitor_SMD:C_0603_1608Metric, F.Cu at (-13.1, 61.7)
- added C277: 1uF, Capacitor_SMD:C_0603_1608Metric, F.Cu at (-13.1, 64.2)
- added C278: 1uF, Capacitor_SMD:C_0603_1608Metric, F.Cu at (-13.1, 66.7)
- added C279: 1uF, Capacitor_SMD:C_0603_1608Metric, F.Cu at (-13.1, 69.2)
- added C280: 1uF, Capacitor_SMD:C_0603_1608Metric, F.Cu at (-13.1, 71.7)
- added C281: 1uF, Capacitor_SMD:C_0603_1608Metric, F.Cu at (-13.1, 74.2)
- added C282: 1uF, Capacitor_SMD:C_0603_1608Metric, F.Cu at (-13.1, 76.8)
- added C283: 1uF, Capacitor_SMD:C_0603_1608Metric, F.Cu at (-13.1, 79.3)
- added C284: 1uF, Capacitor_SMD:C_0603_1608Metric, F.Cu at (-13.1, 81.8)
- added C42: 1uF, Capacitor_SMD:C_0603_1608Metric, F.Cu at (-53.2, 46.6)
- added C43: 1uF, Capacitor_SMD:C_0603_1608Metric, F.Cu at (-53.2, 49.1)
- added C44: 1uF, Capacitor_SMD:C_0603_1608Metric, F.Cu at (-53.2, 51.7)
- added C45: 1uF, Capacitor_SMD:C_0603_1608Metric, F.Cu at (-53.2, 54.2)
- added C46: 1uF, Capacitor_SMD:C_0603_1608Metric, F.Cu at (-53.2, 56.7)
- added C47: 1uF, Capacitor_SMD:C_0603_1608Metric, F.Cu at (-53.2, 59.2)
- added C48: 1uF, Capacitor_SMD:C_0603_1608Metric, F.Cu at (-53.2, 61.7)
- added C49: 1uF, Capacitor_SMD:C_0603_1608Metric, F.Cu at (-53.2, 64.2)
- added C50: 1uF, Capacitor_SMD:C_0603_1608Metric, F.Cu at (-53.2, 66.7)
- added C51: 1uF, Capacitor_SMD:C_0603_1608Metric, F.Cu at (-53.2, 69.2)
- added C52: 1uF, Capacitor_SMD:C_0603_1608Metric, F.Cu at (-53.2, 71.7)
- added C53: 1uF, Capacitor_SMD:C_0603_1608Metric, F.Cu at (-53.2, 74.2)
- added C54: 1uF, Capacitor_SMD:C_0603_1608Metric, F.Cu at (-53.2, 76.8)
- added C55: 1uF, Capacitor_SMD:C_0603_1608Metric, F.Cu at (-53.2, 79.3)
- added C56: 1uF, Capacitor_SMD:C_0603_1608Metric, F.Cu at (-53.2, 81.8)
- added C57: 1uF, Capacitor_SMD:C_0603_1608Metric, F.Cu at (-53.2, 84.3)
- added C58: 1uF, Capacitor_SMD:C_0603_1608Metric, F.Cu at (-53.2, 86.8)
- added C59: 1uF, Capacitor_SMD:C_0603_1608Metric, F.Cu at (-49.2, 44.1)
- added C60: 1uF, Capacitor_SMD:C_0603_1608Metric, F.Cu at (-49.2, 46.6)
- added C61: 1uF, Capacitor_SMD:C_0603_1608Metric, F.Cu at (-49.2, 49.1)
- added C62: 1uF, Capacitor_SMD:C_0603_1608Metric, F.Cu at (-49.2, 51.7)
- added C63: 1uF, Capacitor_SMD:C_0603_1608Metric, F.Cu at (-49.2, 54.2)
- added C64: 1uF, Capacitor_SMD:C_0603_1608Metric, F.Cu at (-49.2, 56.7)
- added C65: 1uF, Capacitor_SMD:C_0603_1608Metric, F.Cu at (-49.2, 59.2)
- added C66: 1uF, Capacitor_SMD:C_0603_1608Metric, F.Cu at (-49.2, 61.7)
- added C67: 1uF, Capacitor_SMD:C_0603_1608Metric, F.Cu at (-49.2, 64.2)
- added C68: 1uF, Capacitor_SMD:C_0603_1608Metric, F.Cu at (-49.2, 66.7)
- added C69: 1uF, Capacitor_SMD:C_0603_1608Metric, F.Cu at (-49.2, 69.2)
- added C70: 1uF, Capacitor_SMD:C_0603_1608Metric, F.Cu at (-49.2, 71.7)
- added C71: 1uF, Capacitor_SMD:C_0603_1608Metric, F.Cu at (-49.2, 74.2)
- added C72: 1uF, Capacitor_SMD:C_0603_1608Metric, F.Cu at (-49.2, 76.8)
- added C73: 1uF, Capacitor_SMD:C_0603_1608Metric, F.Cu at (-49.2, 79.3)
- added C74: 1uF, Capacitor_SMD:C_0603_1608Metric, F.Cu at (-49.2, 81.8)
- added C75: 1uF, Capacitor_SMD:C_0603_1608Metric, F.Cu at (-49.2, 84.3)
- added C76: 1uF, Capacitor_SMD:C_0603_1608Metric, F.Cu at (-49.2, 86.8)
- added C77: 1uF, Capacitor_SMD:C_0603_1608Metric, F.Cu at (-45.2, 44.1)
- added C78: 1uF, Capacitor_SMD:C_0603_1608Metric, F.Cu at (-45.2, 46.6)
- added C79: 1uF, Capacitor_SMD:C_0603_1608Metric, F.Cu at (-45.2, 49.1)
- added C80: 1uF, Capacitor_SMD:C_0603_1608Metric, F.Cu at (-45.2, 51.7)
- added C81: 1uF, Capacitor_SMD:C_0603_1608Metric, F.Cu at (-45.2, 54.2)
- added C82: 1uF, Capacitor_SMD:C_0603_1608Metric, F.Cu at (-45.2, 56.7)
- added C83: 1uF, Capacitor_SMD:C_0603_1608Metric, F.Cu at (-45.2, 59.2)
- added C84: 1uF, Capacitor_SMD:C_0603_1608Metric, F.Cu at (-45.2, 61.7)
- added C85: 1uF, Capacitor_SMD:C_0603_1608Metric, F.Cu at (-45.2, 64.2)
- added C86: 1uF, Capacitor_SMD:C_0603_1608Metric, F.Cu at (-45.2, 66.7)
- added C87: 1uF, Capacitor_SMD:C_0603_1608Metric, F.Cu at (-45.2, 69.2)
- added C88: 1uF, Capacitor_SMD:C_0603_1608Metric, F.Cu at (-45.2, 71.7)
- added D100: APA102-2020, LED_SMD:LED-APA102-2020, F.Cu at (105.8, 60.6)
- added D101: APA102-2020, LED_SMD:LED-APA102-2020, F.Cu at (101.8, 60.6)
- added D102: APA102-2020, LED_SMD:LED-APA102-2020, F.Cu at (97.8, 60.5)
- added D103: APA102-2020, LED_SMD:LED-APA102-2020, F.Cu at (93.8, 60.5)
- added D104: APA102-2020, LED_SMD:LED-APA102-2020, F.Cu at (89.6, 60.5)
- added D105: APA102-2020, LED_SMD:LED-APA102-2020, F.Cu at (85.6, 60.5)
- added D106: APA102-2020, LED_SMD:LED-APA102-2020, F.Cu at (85.6, 64.3)
- added D107: APA102-2020, LED_SMD:LED-APA102-2020, F.Cu at (89.6, 64.3)
- added D108: APA102-2020, LED_SMD:LED-APA102-2020, F.Cu at (93.6, 64.3)
- added D109: APA102-2020, LED_SMD:LED-APA102-2020, F.Cu at (97.6, 64.3)
- added D110: APA102-2020, LED_SMD:LED-APA102-2020, F.Cu at (102.1, 64.3)
- added D111: APA102-2020, LED_SMD:LED-APA102-2020, F.Cu at (106.1, 64.3)
- added D112: APA102-2020, LED_SMD:LED-APA102-2020, F.Cu at (110.2, 64.2)
- added D113: APA102-2020, LED_SMD:LED-APA102-2020, F.Cu at (114.2, 64.2)
- added D114: APA102-2020, LED_SMD:LED-APA102-2020, F.Cu at (118.0, 64.3)
- added D115: APA102-2020, LED_SMD:LED-APA102-2020, F.Cu at (122.3, 64.3)
- added D116: APA102-2020, LED_SMD:LED-APA102-2020, F.Cu at (126.6, 64.2)
- added D117: APA102-2020, LED_SMD:LED-APA102-2020, F.Cu at (130.8, 64.3)
- added D118: APA102-2020, LED_SMD:LED-APA102-2020, F.Cu at (134.6, 64.2)
- added D119: APA102-2020, LED_SMD:LED-APA102-2020, F.Cu at (102.0, 91.8)
- added D120: APA102-2020, LED_SMD:LED-APA102-2020, F.Cu at (138.8, 64.2)
- added D121: APA102-2020, LED_SMD:LED-APA102-2020, F.Cu at (106.1, 91.8)
- added D122: APA102-2020, LED_SMD:LED-APA102-2020, F.Cu at (138.8, 68.2)
- added D123: APA102-2020, LED_SMD:LED-APA102-2020, F.Cu at (110.2, 91.8)
- added D124: APA102-2020, LED_SMD:LED-APA102-2020, F.Cu at (134.6, 68.2)
- added D125: APA102-2020, LED_SMD:LED-APA102-2020, F.Cu at (114.1, 91.8)
- added D126: APA102-2020, LED_SMD:LED-APA102-2020, F.Cu at (130.8, 68.2)
- added D127: APA102-2020, LED_SMD:LED-APA102-2020, F.Cu at (118.0, 91.8)
- added D128: APA102-2020, LED_SMD:LED-APA102-2020, F.Cu at (126.6, 68.2)
- added D129: APA102-2020, LED_SMD:LED-APA102-2020, F.Cu at (122.3, 91.8)
- added D130: APA102-2020, LED_SMD:LED-APA102-2020, F.Cu at (122.3, 68.2)
- added D131: APA102-2020, LED_SMD:LED-APA102-2020, F.Cu at (126.6, 91.8)
- added D132: APA102-2020, LED_SMD:LED-APA102-2020, F.Cu at (118.0, 68.1)
- added D133: APA102-2020, LED_SMD:LED-APA102-2020, F.Cu at (130.8, 91.8)
- added D134: APA102-2020, LED_SMD:LED-APA102-2020, F.Cu at (114.2, 68.1)
- added D135: APA102-2020, LED_SMD:LED-APA102-2020, F.Cu at (134.6, 91.8)
- added D136: APA102-2020, LED_SMD:LED-APA102-2020, F.Cu at (110.2, 68.1)
- added D137: APA102-2020, LED_SMD:LED-APA102-2020, F.Cu at (138.8, 91.8)
- added D138: APA102-2020, LED_SMD:LED-APA102-2020, F.Cu at (106.1, 68.1)
- added D139: APA102-2020, LED_SMD:LED-APA102-2020, F.Cu at (138.8, 88.0)
- added D140: APA102-2020, LED_SMD:LED-APA102-2020, F.Cu at (102.1, 68.1)
- added D141: APA102-2020, LED_SMD:LED-APA102-2020, F.Cu at (134.6, 88.0)
- added D142: APA102-2020, LED_SMD:LED-APA102-2020, F.Cu at (97.6, 68.2)
- added D143: APA102-2020, LED_SMD:LED-APA102-2020, F.Cu at (130.8, 88.0)
- added D144: APA102-2020, LED_SMD:LED-APA102-2020, F.Cu at (93.6, 68.2)
- added D145: APA102-2020, LED_SMD:LED-APA102-2020, F.Cu at (126.6, 88.0)
- added D146: APA102-2020, LED_SMD:LED-APA102-2020, F.Cu at (89.6, 68.1)
- added D147: APA102-2020, LED_SMD:LED-APA102-2020, F.Cu at (122.3, 88.0)
- added D148: APA102-2020, LED_SMD:LED-APA102-2020, F.Cu at (85.6, 68.1)
- added D149: APA102-2020, LED_SMD:LED-APA102-2020, F.Cu at (118.0, 88.0)
- added D150: APA102-2020, LED_SMD:LED-APA102-2020, F.Cu at (85.6, 72.1)
- added D151: APA102-2020, LED_SMD:LED-APA102-2020, F.Cu at (114.1, 88.0)
- added D152: APA102-2020, LED_SMD:LED-APA102-2020, F.Cu at (89.6, 72.1)
- added D153: APA102-2020, LED_SMD:LED-APA102-2020, F.Cu at (110.2, 88.0)
- added D154: APA102-2020, LED_SMD:LED-APA102-2020, F.Cu at (93.6, 72.1)
- added D155: APA102-2020, LED_SMD:LED-APA102-2020, F.Cu at (106.1, 88.0)
- added D156: APA102-2020, LED_SMD:LED-APA102-2020, F.Cu at (97.6, 72.1)
- added D157: APA102-2020, LED_SMD:LED-APA102-2020, F.Cu at (102.0, 88.0)
- added D158: APA102-2020, LED_SMD:LED-APA102-2020, F.Cu at (102.0, 72.1)
- added D159: APA102-2020, LED_SMD:LED-APA102-2020, F.Cu at (97.6, 88.0)
- added D160: APA102-2020, LED_SMD:LED-APA102-2020, F.Cu at (106.1, 72.1)
- added D161: APA102-2020, LED_SMD:LED-APA102-2020, F.Cu at (93.6, 88.0)
- added D162: APA102-2020, LED_SMD:LED-APA102-2020, F.Cu at (110.2, 72.1)
- added D163: APA102-2020, LED_SMD:LED-APA102-2020, F.Cu at (89.6, 88.0)
- added D164: APA102-2020, LED_SMD:LED-APA102-2020, F.Cu at (114.1, 72.1)
- added D165: APA102-2020, LED_SMD:LED-APA102-2020, F.Cu at (85.6, 88.1)
- added D166: APA102-2020, LED_SMD:LED-APA102-2020, F.Cu at (118.0, 72.1)
- added D167: APA102-2020, LED_SMD:LED-APA102-2020, F.Cu at (85.6, 84.1)
- added D168: APA102-2020, LED_SMD:LED-APA102-2020, F.Cu at (122.3, 72.1)
- added D169: APA102-2020, LED_SMD:LED-APA102-2020, F.Cu at (89.6, 84.1)
- added D17: APA102-2020, LED_SMD:LED-APA102-2020, F.Cu at (85.6, 41.1)
- added D170: APA102-2020, LED_SMD:LED-APA102-2020, F.Cu at (126.6, 72.1)
- added D171: APA102-2020, LED_SMD:LED-APA102-2020, F.Cu at (93.6, 84.1)
- added D172: APA102-2020, LED_SMD:LED-APA102-2020, F.Cu at (130.8, 72.1)
- added D173: APA102-2020, LED_SMD:LED-APA102-2020, F.Cu at (97.6, 84.1)
- added D174: APA102-2020, LED_SMD:LED-APA102-2020, F.Cu at (134.6, 72.1)
- added D175: APA102-2020, LED_SMD:LED-APA102-2020, F.Cu at (102.0, 84.1)
- added D176: APA102-2020, LED_SMD:LED-APA102-2020, F.Cu at (138.8, 72.1)
- added D177: APA102-2020, LED_SMD:LED-APA102-2020, F.Cu at (106.1, 84.1)
- added D178: APA102-2020, LED_SMD:LED-APA102-2020, F.Cu at (138.8, 75.9)
- added D179: APA102-2020, LED_SMD:LED-APA102-2020, F.Cu at (110.2, 84.1)
- added D18: APA102-2020, LED_SMD:LED-APA102-2020, F.Cu at (89.6, 41.0)
- added D180: APA102-2020, LED_SMD:LED-APA102-2020, F.Cu at (134.6, 75.9)
- added D181: APA102-2020, LED_SMD:LED-APA102-2020, F.Cu at (114.2, 84.1)
- added D182: APA102-2020, LED_SMD:LED-APA102-2020, F.Cu at (130.8, 75.9)
- added D183: APA102-2020, LED_SMD:LED-APA102-2020, F.Cu at (118.0, 84.1)
- added D184: APA102-2020, LED_SMD:LED-APA102-2020, F.Cu at (126.6, 75.9)
- added D185: APA102-2020, LED_SMD:LED-APA102-2020, F.Cu at (122.3, 84.1)
- added D186: APA102-2020, LED_SMD:LED-APA102-2020, F.Cu at (122.3, 75.9)
- added D187: APA102-2020, LED_SMD:LED-APA102-2020, F.Cu at (126.6, 84.1)
- added D188: APA102-2020, LED_SMD:LED-APA102-2020, F.Cu at (118.0, 75.9)
- added D189: APA102-2020, LED_SMD:LED-APA102-2020, F.Cu at (130.8, 84.1)
- added D19: APA102-2020, LED_SMD:LED-APA102-2020, F.Cu at (93.6, 41.0)
- added D190: APA102-2020, LED_SMD:LED-APA102-2020, F.Cu at (114.1, 76.0)
- added D191: APA102-2020, LED_SMD:LED-APA102-2020, F.Cu at (134.6, 84.1)
- added D192: APA102-2020, LED_SMD:LED-APA102-2020, F.Cu at (110.2, 76.0)
- added D193: APA102-2020, LED_SMD:LED-APA102-2020, F.Cu at (138.8, 84.1)
- added D194: APA102-2020, LED_SMD:LED-APA102-2020, F.Cu at (106.1, 76.0)
- added D195: APA102-2020, LED_SMD:LED-APA102-2020, F.Cu at (138.8, 80.0)
- added D196: APA102-2020, LED_SMD:LED-APA102-2020, F.Cu at (102.0, 76.0)
- added D197: APA102-2020, LED_SMD:LED-APA102-2020, F.Cu at (134.6, 80.0)
- added D198: APA102-2020, LED_SMD:LED-APA102-2020, F.Cu at (97.6, 76.0)
- added D199: APA102-2020, LED_SMD:LED-APA102-2020, F.Cu at (130.8, 79.9)
- added D20: APA102-2020, LED_SMD:LED-APA102-2020, F.Cu at (97.6, 41.0)
- added D200: APA102-2020, LED_SMD:LED-APA102-2020, F.Cu at (93.6, 76.0)
- added D201: APA102-2020, LED_SMD:LED-APA102-2020, F.Cu at (126.6, 79.9)
- added D202: APA102-2020, LED_SMD:LED-APA102-2020, F.Cu at (89.6, 76.0)
- added D203: APA102-2020, LED_SMD:LED-APA102-2020, F.Cu at (122.3, 79.9)
- added D204: APA102-2020, LED_SMD:LED-APA102-2020, F.Cu at (85.6, 76.0)
- added D205: APA102-2020, LED_SMD:LED-APA102-2020, F.Cu at (118.0, 79.9)
- added D206: APA102-2020, LED_SMD:LED-APA102-2020, F.Cu at (85.6, 79.9)
- added D207: APA102-2020, LED_SMD:LED-APA102-2020, F.Cu at (114.2, 80.0)
- added D208: APA102-2020, LED_SMD:LED-APA102-2020, F.Cu at (89.6, 79.9)
- added D209: APA102-2020, LED_SMD:LED-APA102-2020, F.Cu at (110.2, 79.9)
- added D210: APA102-2020, LED_SMD:LED-APA102-2020, F.Cu at (93.6, 79.8)
- added D211: APA102-2020, LED_SMD:LED-APA102-2020, F.Cu at (106.1, 79.9)
- added D212: APA102-2020, LED_SMD:LED-APA102-2020, F.Cu at (97.6, 79.9)
- added D213: APA102-2020, LED_SMD:LED-APA102-2020, F.Cu at (102.0, 79.9)
- added D214: APA102-2020, LED_SMD:LED-APA102-2020, F.Cu at (97.6, 91.8)
- added D218: APA102-2020, LED_SMD:LED-APA102-2020, F.Cu at (93.6, 91.8)
- added D222: APA102-2020, LED_SMD:LED-APA102-2020, F.Cu at (89.6, 91.8)
- added D226: APA102-2020, LED_SMD:LED-APA102-2020, F.Cu at (85.6, 91.8)
- added D26: APA102-2020, LED_SMD:LED-APA102-2020, F.Cu at (101.6, 41.1)
- added D27: APA102-2020, LED_SMD:LED-APA102-2020, F.Cu at (105.6, 41.1)
- added D28: APA102-2020, LED_SMD:LED-APA102-2020, F.Cu at (110.1, 41.1)
- added D29: APA102-2020, LED_SMD:LED-APA102-2020, F.Cu at (114.1, 41.0)
- added D30: APA102-2020, LED_SMD:LED-APA102-2020, F.Cu at (118.1, 41.0)
- added D31: APA102-2020, LED_SMD:LED-APA102-2020, F.Cu at (122.1, 41.0)
- added D32: APA102-2020, LED_SMD:LED-APA102-2020, F.Cu at (126.1, 41.0)
- added D33: APA102-2020, LED_SMD:LED-APA102-2020, F.Cu at (130.3, 41.0)
- added D34: APA102-2020, LED_SMD:LED-APA102-2020, F.Cu at (134.6, 41.0)
- added D35: APA102-2020, LED_SMD:LED-APA102-2020, F.Cu at (138.8, 41.0)
- added D36: APA102-2020, LED_SMD:LED-APA102-2020, F.Cu at (138.8, 45.0)
- added D37: APA102-2020, LED_SMD:LED-APA102-2020, F.Cu at (134.6, 45.0)
- added D38: APA102-2020, LED_SMD:LED-APA102-2020, F.Cu at (130.3, 45.0)
- added D39: APA102-2020, LED_SMD:LED-APA102-2020, F.Cu at (126.0, 45.0)
- added D40: APA102-2020, LED_SMD:LED-APA102-2020, F.Cu at (122.1, 45.0)
- added D41: APA102-2020, LED_SMD:LED-APA102-2020, F.Cu at (118.1, 45.0)
- added D42: APA102-2020, LED_SMD:LED-APA102-2020, F.Cu at (114.1, 45.0)
- added D43: APA102-2020, LED_SMD:LED-APA102-2020, F.Cu at (110.1, 45.0)
- added D44: APA102-2020, LED_SMD:LED-APA102-2020, F.Cu at (105.6, 45.0)
- added D45: APA102-2020, LED_SMD:LED-APA102-2020, F.Cu at (101.6, 45.0)
- added D46: APA102-2020, LED_SMD:LED-APA102-2020, F.Cu at (97.6, 45.0)
- added D47: APA102-2020, LED_SMD:LED-APA102-2020, F.Cu at (93.6, 45.0)
- added D48: APA102-2020, LED_SMD:LED-APA102-2020, F.Cu at (89.6, 45.0)
- added D49: APA102-2020, LED_SMD:LED-APA102-2020, F.Cu at (85.6, 45.0)
- added D50: APA102-2020, LED_SMD:LED-APA102-2020, F.Cu at (85.6, 49.0)
- added D51: APA102-2020, LED_SMD:LED-APA102-2020, F.Cu at (89.6, 49.0)
- added D52: APA102-2020, LED_SMD:LED-APA102-2020, F.Cu at (93.6, 49.0)
- added D53: APA102-2020, LED_SMD:LED-APA102-2020, F.Cu at (97.6, 49.0)
- added D54: APA102-2020, LED_SMD:LED-APA102-2020, F.Cu at (101.6, 49.0)
- added D55: APA102-2020, LED_SMD:LED-APA102-2020, F.Cu at (105.6, 49.0)
- added D56: APA102-2020, LED_SMD:LED-APA102-2020, F.Cu at (110.1, 49.0)
- added D57: APA102-2020, LED_SMD:LED-APA102-2020, F.Cu at (114.1, 49.0)
- added D58: APA102-2020, LED_SMD:LED-APA102-2020, F.Cu at (118.2, 49.0)
- added D59: APA102-2020, LED_SMD:LED-APA102-2020, F.Cu at (122.2, 49.0)
- added D60: APA102-2020, LED_SMD:LED-APA102-2020, F.Cu at (126.0, 49.0)
- added D61: APA102-2020, LED_SMD:LED-APA102-2020, F.Cu at (130.3, 49.0)
- added D62: APA102-2020, LED_SMD:LED-APA102-2020, F.Cu at (134.6, 49.0)
- added D63: APA102-2020, LED_SMD:LED-APA102-2020, F.Cu at (138.8, 49.0)
- added D64: APA102-2020, LED_SMD:LED-APA102-2020, F.Cu at (138.8, 52.8)
- added D65: APA102-2020, LED_SMD:LED-APA102-2020, F.Cu at (134.6, 52.8)
- added D66: APA102-2020, LED_SMD:LED-APA102-2020, F.Cu at (130.3, 52.8)
- added D67: APA102-2020, LED_SMD:LED-APA102-2020, F.Cu at (126.0, 52.8)
- added D68: APA102-2020, LED_SMD:LED-APA102-2020, F.Cu at (122.2, 52.8)
- added D69: APA102-2020, LED_SMD:LED-APA102-2020, F.Cu at (118.2, 52.8)
- added D70: APA102-2020, LED_SMD:LED-APA102-2020, F.Cu at (114.1, 52.8)
- added D71: APA102-2020, LED_SMD:LED-APA102-2020, F.Cu at (110.1, 52.8)
- added D72: APA102-2020, LED_SMD:LED-APA102-2020, F.Cu at (105.6, 52.8)
- added D73: APA102-2020, LED_SMD:LED-APA102-2020, F.Cu at (101.6, 52.8)
- added D74: APA102-2020, LED_SMD:LED-APA102-2020, F.Cu at (97.6, 52.8)
- added D75: APA102-2020, LED_SMD:LED-APA102-2020, F.Cu at (93.6, 52.9)
- added D76: APA102-2020, LED_SMD:LED-APA102-2020, F.Cu at (89.6, 52.9)
- added D77: APA102-2020, LED_SMD:LED-APA102-2020, F.Cu at (85.6, 52.9)
- added D78: APA102-2020, LED_SMD:LED-APA102-2020, F.Cu at (85.6, 56.9)
- added D79: APA102-2020, LED_SMD:LED-APA102-2020, F.Cu at (89.6, 56.9)
- added D80: APA102-2020, LED_SMD:LED-APA102-2020, F.Cu at (93.6, 56.9)
- added D81: APA102-2020, LED_SMD:LED-APA102-2020, F.Cu at (97.6, 56.9)
- added D82: APA102-2020, LED_SMD:LED-APA102-2020, F.Cu at (101.6, 56.9)
- added D83: APA102-2020, LED_SMD:LED-APA102-2020, F.Cu at (105.6, 56.9)
- added D84: APA102-2020, LED_SMD:LED-APA102-2020, F.Cu at (110.1, 56.9)
- added D85: APA102-2020, LED_SMD:LED-APA102-2020, F.Cu at (114.1, 56.9)
- added D86: APA102-2020, LED_SMD:LED-APA102-2020, F.Cu at (118.2, 56.9)
- added D87: APA102-2020, LED_SMD:LED-APA102-2020, F.Cu at (122.2, 56.9)
- added D88: APA102-2020, LED_SMD:LED-APA102-2020, F.Cu at (126.0, 56.9)
- added D89: APA102-2020, LED_SMD:LED-APA102-2020, F.Cu at (130.3, 56.9)
- added D90: APA102-2020, LED_SMD:LED-APA102-2020, F.Cu at (134.6, 56.8)
- added D91: APA102-2020, LED_SMD:LED-APA102-2020, F.Cu at (138.8, 56.8)
- added D92: APA102-2020, LED_SMD:LED-APA102-2020, F.Cu at (138.8, 60.6)
- added D93: APA102-2020, LED_SMD:LED-APA102-2020, F.Cu at (134.6, 60.6)
- added D94: APA102-2020, LED_SMD:LED-APA102-2020, F.Cu at (130.3, 60.6)
- added D95: APA102-2020, LED_SMD:LED-APA102-2020, F.Cu at (126.3, 60.6)
- added D96: APA102-2020, LED_SMD:LED-APA102-2020, F.Cu at (122.2, 60.6)
- added D97: APA102-2020, LED_SMD:LED-APA102-2020, F.Cu at (118.2, 60.6)
- added D98: APA102-2020, LED_SMD:LED-APA102-2020, F.Cu at (113.8, 60.6)
- added D99: APA102-2020, LED_SMD:LED-APA102-2020, F.Cu at (109.8, 60.6)
- J1: footprint Connector_PinSocket_2.54mm:PinSocket_1x04_P2.54mm_Vertical -> Connector_PinHeader_2.00mm:PinHeader_1x04_P2.00mm_Horizontal
- moved J1 76.0 mm to (-9.09, 44.9)
Routing:
- net GND: track 356.9 -> 0.00 mm, vias 6 -> 0
- net VCC: track 232.7 -> 0.00 mm, vias 18 -> 0
- net Net-(D17-SDI): track 27.0 -> 0.00 mm, vias 1 -> 0
- net Net-(D2-SDO): track 20.7 -> 0.00 mm, vias 2 -> 0
- net Net-(D17-CKI): track 16.7 -> 0.00 mm, vias 1 -> 0
- net Net-(D2-CKO): track 15.1 -> 0.00 mm, vias 2 -> 0
- net Net-(D4-SDI): track 15.0 -> 0.00 mm, vias 2 -> 0
- net Net-(D23-CKO): track 13.4 -> 0.00 mm
- net Net-(D4-CKI): track 10.3 -> 0.00 mm, vias 2 -> 0
- net Net-(D23-SDO): track 6.59 -> 0.00 mm
- net Net-(D10-SDO): track 4.70 -> 0.00 mm
- net Net-(D10-CKO): track 4.70 -> 0.00 mm
- net Net-(D25-CKO): track 4.54 -> 0.00 mm
- net Net-(D25-SDO): track 4.54 -> 0.00 mm
- net Net-(D11-SDO): track 4.45 -> 0.00 mm
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- removed copper zone on B.Cu, net GND
- removed copper zone on F.Cu, net VCC
Other:
- board outline removed

Commit message: ...
Parts:
- added J2: Conn_01x04_Pin, Connector_PinHeader_2.54mm:PinHeader_1x04_P2.54mm_Vertical, F.Cu at (78.7, 52.7)
- added R1: R, Resistor_SMD:R_0402_1005Metric, F.Cu at (81.8, 39.2)
- added R2: R, Resistor_SMD:R_0402_1005Metric, F.Cu at (81.8, 42.5)
- C137, C138, C139, C140, C141, C142, C143, C144, C145, C146, C147, C148, C149, C150, C151, C152, C153, C154, C155, C156, C157, C158, C159, C160, C161, C162, C163, C164, C165, C166, C167, C168, C169, C170, C171, C172, C173, C174, C175, C176, C177, C178, C179, C180, C181, C182, C183, C184, C185, C186, C187, C188, C189, C190, C191, C192, C193, C194, C195, C196, C197, C198, C199, C200, C201, C202, C203, C204, C205, C206, C207, C208, C209, C210, C211, C212, C213, C214, C215, C216, C217, C218, C219, C220, C221, C222, C223, C224, C225, C226, C227, C228, C229, C230, C231, C232, C233, C234, C235, C236, C237, C238, C239, C240, C241, C242, C243, C244, C245, C246, C247, C248, C249, C250, C251, C252, C253, C254, C255, C256, C257, C258, C259, C26, C260, C261, C262, C263, C264, C265, C266, C267, C268, C269, C270, C271, C272, C273, C274, C275, C276, C277, C278, C279, C280, C281, C282, C283, C284, C42, C43, C44, C45, C46, C47, C48, C49, C50, C51, C52, C53, C54, C55, C56, C57, C58, C59, C60, C61, C62, C63, C64, C65, C66, C67, C68, C69, C70, C71, C72, C73, C74, C75, C76, C77, C78, C79, C80, C81, C82, C83, C84, C85, C86, C87, C88, J1: moved to B.Cu
- moved C160 183.4 mm to (141.1, 65.8), turned to 90 degrees
- moved C46 180.7 mm to (127.5, 56.8), turned to -90 degrees
- moved C44 180.7 mm to (127.5, 52.8), turned to 90 degrees
- moved C87 177.1 mm to (131.8, 72.3), turned to -90 degrees
- moved C178 173.7 mm to (135.9, 72.2), turned to -90 degrees
- moved C171 173.1 mm to (135.9, 68.2), turned to 90 degrees
- moved C64 172.9 mm to (123.7, 56.8), turned to -90 degrees
- moved C47 172.8 mm to (119.6, 60.4), turned to 90 degrees
- moved C62 172.8 mm to (123.6, 52.8), turned to 90 degrees
- moved C196 170.6 mm to (135.9, 64.5), turned to 90 degrees
- moved C142 170.4 mm to (123.8, 64.5), turned to -90 degrees
- moved C76 170.2 mm to (119.6, 64.5), turned to -90 degrees
- moved C177 170.2 mm to (131.9, 64.6), turned to -90 degrees
- moved C159 170.2 mm to (127.9, 64.5), turned to -90 degrees
- moved C58 170.2 mm to (115.5, 64.4), turned to -90 degrees
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Routing:
- net GND: track 0.00 -> 1113.1 mm, vias 0 -> 201
- net VCC: track 0.00 -> 809.3 mm, vias 0 -> 107
- net Net-(D17-CKI): track 0.00 -> 22.3 mm
- net Net-(D17-SDI): track 0.00 -> 20.8 mm
- net Net-(D63-SDO): track 0.00 -> 11.2 mm
- net Net-(D120-SDO): track 0.00 -> 11.1 mm
- net Net-(D91-SDO): track 0.00 -> 11.0 mm
- net Net-(D176-SDO): track 0.00 -> 10.7 mm
- net Net-(D193-SDI): track 0.00 -> 10.6 mm
- net Net-(D137-SDI): track 0.00 -> 10.4 mm
- net Net-(D120-CKO): track 0.00 -> 8.95 mm
- net Net-(D35-SDO): track 0.00 -> 8.80 mm
- net Net-(D91-CKO): track 0.00 -> 8.64 mm
- net Net-(D137-CKI): track 0.00 -> 8.25 mm
- net Net-(D63-CKO): track 0.00 -> 8.22 mm
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- added copper zone on B.Cu, net GND
- added copper zone on In1.Cu, net GND
- added copper zone on In2.Cu, net VCC
Other:
- board outline added: 73 x 57 mm
- copper layers 2 -> 4

Commit message: SPI
Parts:
- added H1: MountingHole, MountingHole:ToolingHole_1.152mm, F.Cu at (143.2, 39.4)
- added H2: MountingHole, MountingHole:ToolingHole_1.152mm, F.Cu at (143.1, 94.4)
- added H3: MountingHole, MountingHole:ToolingHole_1.152mm, F.Cu at (71.9, 39.2)
- added H4: MountingHole, MountingHole:ToolingHole_1.152mm, F.Cu at (72.0, 94.3)
- R1, R2: moved to B.Cu
- moved C258 1.14 mm to (128.6, 60.7)
- moved C137 1.14 mm to (112.6, 80.5)
- moved C138 1.14 mm to (108.7, 84.3)
- moved C142 1.14 mm to (124.9, 64.8)
- moved C150 1.14 mm to (100.6, 64.6)
- moved C152 1.14 mm to (96.7, 76.2)
- moved C157 1.14 mm to (108.7, 88.3)
- moved C161 1.14 mm to (108.7, 41.4)
- moved C162 1.14 mm to (116.5, 45.3)
- moved C164 1.14 mm to (112.5, 53.1)
- moved C166 1.14 mm to (112.7, 57.2)
- moved C167 1.14 mm to (104.6, 60.7)
- moved C169 1.14 mm to (88.6, 72.3)
- moved C171 1.14 mm to (137.0, 68.5)
- moved C172 1.14 mm to (129.0, 76.4)
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Routing:
- net Net-(D17-SDI): track 20.8 -> 23.7 mm
- net Net-(D17-CKI): track 22.3 -> 24.8 mm
Other:
- board text added: "PCB_GRID-V1-14X14-APA102-2020 SNAKE-CSF25"

Commit message: .
Parts:
- added J3: Conn_01x04_Pin, Connector_PinHeader_2.54mm:PinHeader_1x04_P2.54mm_Vertical, F.Cu at (80.0, 81.6)
- H1, H2, H3, H4: footprint MountingHole:ToolingHole_1.152mm -> MountingHole:MountingHole_2.1mm
Connections:
- D226 pad 2: unconnected-(D226-CKO-Pad2) -> Net-(D226-CKO)
- D226 pad 3: unconnected-(D226-SDO-Pad3) -> Net-(D226-SDO)
Routing:
- net Net-(D226-SDO): track 0.00 -> 23.5 mm
- net Net-(D226-CKO): track 0.00 -> 15.2 mm
