File: ATMEGA-SCHEMATICS/SNAKE_GAME/GRID_SCHEMATICS/GRID/GRID.kicad_pcb (KiCad board)
At the start: 4 copper layers, 73 x 57 mm, 401 parts, among them J1 Conn_01x04_Pin, J2 Conn_01x04_Pin, J3 Conn_01x04_Pin

Commit message: .
Parts:
- removed J3: Conn_01x04_Pin, Connector_PinHeader_2.54mm:PinHeader_1x04_P2.54mm_Vertical
- H1, H2, H3, H4: footprint MountingHole:MountingHole_2.1mm -> MountingHole:ToolingHole_1.152mm
Connections:
- D226 pad 2: Net-(D226-CKO) -> unconnected-(D226-CKO-Pad2)
- D226 pad 3: Net-(D226-SDO) -> unconnected-(D226-SDO-Pad3)
Routing:
- net Net-(D226-SDO): track 23.5 -> 0.00 mm
- net Net-(D226-CKO): track 15.2 -> 0.00 mm
