File: ATMEGA-SCHEMATICS/SNAKE_GAME/GRID_SCHEMATICS/GRID/GRID.kicad_pcb (KiCad board)
At the start: 4 copper layers, 73 x 57 mm, 400 parts, among them J1 Conn_01x04_Pin, J2 Conn_01x04_Pin

Commit message: .
Parts:
- removed D100, D101, D102, D103, D104, D105, D106, D107, D108, D109, D110, D111, D112, D113, D114, D115, D116, D117, D118, D119, D120, D121, D122, D123, D124, D125, D126, D127, D128, D129, D130, D131, D132, D133, D134, D135, D136, D137, D138, D139, D140, D141, D142, D143, D144, D145, D146, D147, D148, D149, D150, D151, D152, D153, D154, D155, D156, D157, D158, D159, D160, D161, D162, D163, D164, D165, D166, D167, D168, D169, D17, D170, D171, D172, D173, D174, D175, D176, D177, D178, D179, D18, D180, D181, D182, D183, D184, D185, D186, D187, D188, D189, D19, D190, D191, D192, D193, D194, D195, D196, D197, D198, D199, D20, D200, D201, D202, D203, D204, D205, D206, D207, D208, D209, D210, D211, D212, D213, D214, D218, D222, D226, D26, D27, D28, D29, D30, D31, D32, D33, D34, D35, D36, D37, D38, D39, D40, D41, D42, D43, D44, D45, D46, D47, D48, D49, D50, D51, D52, D53, D54, D55, D56, D57, D58, D59, D60, D61, D62, D63, D64, D65, D66, D67, D68, D69, D70, D71, D72, D73, D74, D75, D76, D77, D78, D79, D80, D81, D82, D83, D84, D85, D86, D87, D88, D89, D90, D91, D92, D93, D94, D95, D96, D97, D98, D99: APA102-2020, LED_SMD:LED-APA102-2020
- removed R1, R2: R, Resistor_SMD:R_0402_1005Metric
- added C1: 1uF, Capacitor_SMD:C_0603_1608Metric, F.Cu at (1251.6, 23.5)
- added C10: 1uF, Capacitor_SMD:C_0603_1608Metric, F.Cu at (1251.6, 46.1)
- added C100: 1uF, Capacitor_SMD:C_0603_1608Metric, F.Cu at (1255.6, 68.7)
- added C1000: 1uF, Capacitor_SMD:C_0603_1608Metric, F.Cu at (1299.7, 91.3)
- added C1001: 1uF, Capacitor_SMD:C_0603_1608Metric, F.Cu at (1299.7, 93.8)
- added C1002: 1uF, Capacitor_SMD:C_0603_1608Metric, F.Cu at (1299.7, 96.3)
- added C1003: 1uF, Capacitor_SMD:C_0603_1608Metric, F.Cu at (1299.7, 98.8)
- added C1004: 1uF, Capacitor_SMD:C_0603_1608Metric, F.Cu at (1299.7, 101.3)
- added C1005: 1uF, Capacitor_SMD:C_0603_1608Metric, F.Cu at (1299.7, 103.8)
- added C1006: 1uF, Capacitor_SMD:C_0603_1608Metric, F.Cu at (1299.7, 106.3)
- added C1007: 1uF, Capacitor_SMD:C_0603_1608Metric, F.Cu at (1299.7, 108.8)
- added C1008: 1uF, Capacitor_SMD:C_0603_1608Metric, F.Cu at (1299.7, 111.3)
- added C1009: 1uF, Capacitor_SMD:C_0603_1608Metric, F.Cu at (1299.7, 113.9)
- added C101: 1uF, Capacitor_SMD:C_0603_1608Metric, F.Cu at (1255.6, 71.2)
- added C1010: 1uF, Capacitor_SMD:C_0603_1608Metric, F.Cu at (1299.7, 116.4)
- added C1011: 1uF, Capacitor_SMD:C_0603_1608Metric, F.Cu at (1299.7, 118.9)
- added C1012: 1uF, Capacitor_SMD:C_0603_1608Metric, F.Cu at (1299.7, 121.4)
- added C1013: 1uF, Capacitor_SMD:C_0603_1608Metric, F.Cu at (1299.7, 123.9)
- added C1014: 1uF, Capacitor_SMD:C_0603_1608Metric, F.Cu at (1299.7, 126.4)
- added C1015: 1uF, Capacitor_SMD:C_0603_1608Metric, F.Cu at (1299.7, 128.9)
- added C1016: 1uF, Capacitor_SMD:C_0603_1608Metric, F.Cu at (1299.7, 131.4)
- added C1017: 1uF, Capacitor_SMD:C_0603_1608Metric, F.Cu at (1299.7, 133.9)
- added C1018: 1uF, Capacitor_SMD:C_0603_1608Metric, F.Cu at (1299.7, 136.4)
- added C1019: 1uF, Capacitor_SMD:C_0603_1608Metric, F.Cu at (1299.7, 139.0)
- added C102: 1uF, Capacitor_SMD:C_0603_1608Metric, F.Cu at (1255.6, 73.7)
- added C1020: 1uF, Capacitor_SMD:C_0603_1608Metric, F.Cu at (1299.7, 141.5)
- added C1021: 1uF, Capacitor_SMD:C_0603_1608Metric, F.Cu at (1299.7, 144.0)
- added C1022: 1uF, Capacitor_SMD:C_0603_1608Metric, F.Cu at (1299.7, 146.5)
- added C1023: 1uF, Capacitor_SMD:C_0603_1608Metric, F.Cu at (1299.7, 149.0)
- added C1024: 1uF, Capacitor_SMD:C_0603_1608Metric, F.Cu at (1299.7, 151.5)
- added C1025: 1uF, Capacitor_SMD:C_0603_1608Metric, F.Cu at (1299.7, 154.0)
- added C1026: 1uF, Capacitor_SMD:C_0603_1608Metric, F.Cu at (1299.7, 156.5)
- added C1027: 1uF, Capacitor_SMD:C_0603_1608Metric, F.Cu at (1299.7, 159.0)
- added C1028: 1uF, Capacitor_SMD:C_0603_1608Metric, F.Cu at (1299.7, 161.5)
- added C1029: 1uF, Capacitor_SMD:C_0603_1608Metric, F.Cu at (1299.7, 164.1)
- added C103: 1uF, Capacitor_SMD:C_0603_1608Metric, F.Cu at (1255.6, 76.2)
- added C1030: 1uF, Capacitor_SMD:C_0603_1608Metric, F.Cu at (1299.7, 166.6)
- added C1031: 1uF, Capacitor_SMD:C_0603_1608Metric, F.Cu at (1299.7, 169.1)
- added C1032: 1uF, Capacitor_SMD:C_0603_1608Metric, F.Cu at (1299.7, 171.6)
- added C1033: 1uF, Capacitor_SMD:C_0603_1608Metric, F.Cu at (1299.7, 174.1)
- added C1034: 1uF, Capacitor_SMD:C_0603_1608Metric, F.Cu at (1299.7, 176.6)
- added C1035: 1uF, Capacitor_SMD:C_0603_1608Metric, F.Cu at (1299.7, 179.1)
- added C1036: 1uF, Capacitor_SMD:C_0603_1608Metric, F.Cu at (1299.7, 181.6)
- added C1037: 1uF, Capacitor_SMD:C_0603_1608Metric, F.Cu at (1299.7, 184.1)
- added C1038: 1uF, Capacitor_SMD:C_0603_1608Metric, F.Cu at (1299.7, 186.6)
- added C1039: 1uF, Capacitor_SMD:C_0603_1608Metric, F.Cu at (1299.7, 189.2)
- added C104: 1uF, Capacitor_SMD:C_0603_1608Metric, F.Cu at (1255.6, 78.7)
- added C1040: 1uF, Capacitor_SMD:C_0603_1608Metric, F.Cu at (1299.7, 191.7)
- added C1041: 1uF, Capacitor_SMD:C_0603_1608Metric, F.Cu at (1299.7, 194.2)
- added C1042: 1uF, Capacitor_SMD:C_0603_1608Metric, F.Cu at (1299.7, 196.7)
- added C1043: 1uF, Capacitor_SMD:C_0603_1608Metric, F.Cu at (1299.7, 199.2)
- added C1044: 1uF, Capacitor_SMD:C_0603_1608Metric, F.Cu at (1299.7, 201.7)
- added C1045: 1uF, Capacitor_SMD:C_0603_1608Metric, F.Cu at (1299.7, 204.2)
- added C1046: 1uF, Capacitor_SMD:C_0603_1608Metric, F.Cu at (1299.7, 206.7)
- added C1047: 1uF, Capacitor_SMD:C_0603_1608Metric, F.Cu at (1299.7, 209.2)
- added C1048: 1uF, Capacitor_SMD:C_0603_1608Metric, F.Cu at (1299.7, 211.7)
- added C1049: 1uF, Capacitor_SMD:C_0603_1608Metric, F.Cu at (1299.7, 214.3)
- added C105: 1uF, Capacitor_SMD:C_0603_1608Metric, F.Cu at (1255.6, 81.2)
- added C1050: 1uF, Capacitor_SMD:C_0603_1608Metric, F.Cu at (1299.7, 216.8)
- added C1051: 1uF, Capacitor_SMD:C_0603_1608Metric, F.Cu at (1299.7, 219.3)
- added C1052: 1uF, Capacitor_SMD:C_0603_1608Metric, F.Cu at (1299.7, 221.8)
- added C1053: 1uF, Capacitor_SMD:C_0603_1608Metric, F.Cu at (1299.7, 224.3)
- added C1054: 1uF, Capacitor_SMD:C_0603_1608Metric, F.Cu at (1303.7, 23.5)
- added C1055: 1uF, Capacitor_SMD:C_0603_1608Metric, F.Cu at (1303.7, 26.0)
- added C1056: 1uF, Capacitor_SMD:C_0603_1608Metric, F.Cu at (1303.7, 28.5)
- added C1057: 1uF, Capacitor_SMD:C_0603_1608Metric, F.Cu at (1303.7, 31.0)
- added C1058: 1uF, Capacitor_SMD:C_0603_1608Metric, F.Cu at (1303.7, 33.5)
- added C1059: 1uF, Capacitor_SMD:C_0603_1608Metric, F.Cu at (1303.7, 36.0)
- added C106: 1uF, Capacitor_SMD:C_0603_1608Metric, F.Cu at (1255.6, 83.7)
- added C1060: 1uF, Capacitor_SMD:C_0603_1608Metric, F.Cu at (1303.7, 38.6)
- added C1061: 1uF, Capacitor_SMD:C_0603_1608Metric, F.Cu at (1303.7, 41.1)
- added C1062: 1uF, Capacitor_SMD:C_0603_1608Metric, F.Cu at (1303.7, 43.6)
- added C1063: 1uF, Capacitor_SMD:C_0603_1608Metric, F.Cu at (1303.7, 46.1)
- added C1064: 1uF, Capacitor_SMD:C_0603_1608Metric, F.Cu at (1303.7, 48.6)
- added C1065: 1uF, Capacitor_SMD:C_0603_1608Metric, F.Cu at (1303.7, 51.1)
- added C1066: 1uF, Capacitor_SMD:C_0603_1608Metric, F.Cu at (1303.7, 53.6)
- added C1067: 1uF, Capacitor_SMD:C_0603_1608Metric, F.Cu at (1303.7, 56.1)
- added C1068: 1uF, Capacitor_SMD:C_0603_1608Metric, F.Cu at (1303.7, 58.6)
- added C1069: 1uF, Capacitor_SMD:C_0603_1608Metric, F.Cu at (1303.7, 61.1)
- added C107: 1uF, Capacitor_SMD:C_0603_1608Metric, F.Cu at (1255.6, 86.2)
- added C1070: 1uF, Capacitor_SMD:C_0603_1608Metric, F.Cu at (1303.7, 63.7)
- added C1071: 1uF, Capacitor_SMD:C_0603_1608Metric, F.Cu at (1303.7, 66.2)
- added C1072: 1uF, Capacitor_SMD:C_0603_1608Metric, F.Cu at (1303.7, 68.7)
- added C1073: 1uF, Capacitor_SMD:C_0603_1608Metric, F.Cu at (1303.7, 71.2)
- added C1074: 1uF, Capacitor_SMD:C_0603_1608Metric, F.Cu at (1303.7, 73.7)
- added C1075: 1uF, Capacitor_SMD:C_0603_1608Metric, F.Cu at (1303.7, 76.2)
- added C1076: 1uF, Capacitor_SMD:C_0603_1608Metric, F.Cu at (1303.7, 78.7)
- added C1077: 1uF, Capacitor_SMD:C_0603_1608Metric, F.Cu at (1303.7, 81.2)
- added C1078: 1uF, Capacitor_SMD:C_0603_1608Metric, F.Cu at (1303.7, 83.7)
- added C1079: 1uF, Capacitor_SMD:C_0603_1608Metric, F.Cu at (1303.7, 86.2)
- added C108: 1uF, Capacitor_SMD:C_0603_1608Metric, F.Cu at (1255.6, 88.8)
- added C1080: 1uF, Capacitor_SMD:C_0603_1608Metric, F.Cu at (1303.7, 88.8)
- added C1081: 1uF, Capacitor_SMD:C_0603_1608Metric, F.Cu at (1303.7, 91.3)
- added C1082: 1uF, Capacitor_SMD:C_0603_1608Metric, F.Cu at (1303.7, 93.8)
- added C1083: 1uF, Capacitor_SMD:C_0603_1608Metric, F.Cu at (1303.7, 96.3)
- added C1084: 1uF, Capacitor_SMD:C_0603_1608Metric, F.Cu at (1303.7, 98.8)
- added C1085: 1uF, Capacitor_SMD:C_0603_1608Metric, F.Cu at (1303.7, 101.3)
- added C1086: 1uF, Capacitor_SMD:C_0603_1608Metric, F.Cu at (1303.7, 103.8)
- added C1087: 1uF, Capacitor_SMD:C_0603_1608Metric, F.Cu at (1303.7, 106.3)
- added C1088: 1uF, Capacitor_SMD:C_0603_1608Metric, F.Cu at (1303.7, 108.8)
- added C1089: 1uF, Capacitor_SMD:C_0603_1608Metric, F.Cu at (1303.7, 111.3)
- added C109: 1uF, Capacitor_SMD:C_0603_1608Metric, F.Cu at (1255.6, 91.3)
- added C1090: 1uF, Capacitor_SMD:C_0603_1608Metric, F.Cu at (1303.7, 113.9)
- added C1091: 1uF, Capacitor_SMD:C_0603_1608Metric, F.Cu at (1303.7, 116.4)
- added C1092: 1uF, Capacitor_SMD:C_0603_1608Metric, F.Cu at (1303.7, 118.9)
- added C1093: 1uF, Capacitor_SMD:C_0603_1608Metric, F.Cu at (1303.7, 121.4)
- added C1094: 1uF, Capacitor_SMD:C_0603_1608Metric, F.Cu at (1303.7, 123.9)
- added C1095: 1uF, Capacitor_SMD:C_0603_1608Metric, F.Cu at (1303.7, 126.4)
- added C1096: 1uF, Capacitor_SMD:C_0603_1608Metric, F.Cu at (1303.7, 128.9)
- added C1097: 1uF, Capacitor_SMD:C_0603_1608Metric, F.Cu at (1303.7, 131.4)
- added C1098: 1uF, Capacitor_SMD:C_0603_1608Metric, F.Cu at (1303.7, 133.9)
- added C1099: 1uF, Capacitor_SMD:C_0603_1608Metric, F.Cu at (1303.7, 136.4)
- added C11: 1uF, Capacitor_SMD:C_0603_1608Metric, F.Cu at (1251.6, 48.6)
- added C110: 1uF, Capacitor_SMD:C_0603_1608Metric, F.Cu at (1255.6, 93.8)
- added C1100: 1uF, Capacitor_SMD:C_0603_1608Metric, F.Cu at (1303.7, 139.0)
- added C1101: 1uF, Capacitor_SMD:C_0603_1608Metric, F.Cu at (1303.7, 141.5)
- added C1102: 1uF, Capacitor_SMD:C_0603_1608Metric, F.Cu at (1303.7, 144.0)
- added C1103: 1uF, Capacitor_SMD:C_0603_1608Metric, F.Cu at (1303.7, 146.5)
- added C1104: 1uF, Capacitor_SMD:C_0603_1608Metric, F.Cu at (1303.7, 149.0)
- added C1105: 1uF, Capacitor_SMD:C_0603_1608Metric, F.Cu at (1303.7, 151.5)
- added C1106: 1uF, Capacitor_SMD:C_0603_1608Metric, F.Cu at (1303.7, 154.0)
- added C1107: 1uF, Capacitor_SMD:C_0603_1608Metric, F.Cu at (1303.7, 156.5)
- added C1108: 1uF, Capacitor_SMD:C_0603_1608Metric, F.Cu at (1303.7, 159.0)
- added C1109: 1uF, Capacitor_SMD:C_0603_1608Metric, F.Cu at (1303.7, 161.5)
- added C111: 1uF, Capacitor_SMD:C_0603_1608Metric, F.Cu at (1255.6, 96.3)
- added C1110: 1uF, Capacitor_SMD:C_0603_1608Metric, F.Cu at (1303.7, 164.1)
- added C1111: 1uF, Capacitor_SMD:C_0603_1608Metric, F.Cu at (1303.7, 166.6)
- added C1112: 1uF, Capacitor_SMD:C_0603_1608Metric, F.Cu at (1303.7, 169.1)
- added C1113: 1uF, Capacitor_SMD:C_0603_1608Metric, F.Cu at (1303.7, 171.6)
- added C1114: 1uF, Capacitor_SMD:C_0603_1608Metric, F.Cu at (1303.7, 174.1)
- added C1115: 1uF, Capacitor_SMD:C_0603_1608Metric, F.Cu at (1303.7, 176.6)
- added C1116: 1uF, Capacitor_SMD:C_0603_1608Metric, F.Cu at (1303.7, 179.1)
- added C1117: 1uF, Capacitor_SMD:C_0603_1608Metric, F.Cu at (1303.7, 181.6)
- added C1118: 1uF, Capacitor_SMD:C_0603_1608Metric, F.Cu at (1303.7, 184.1)
- added C1119: 1uF, Capacitor_SMD:C_0603_1608Metric, F.Cu at (1303.7, 186.6)
- added C112: 1uF, Capacitor_SMD:C_0603_1608Metric, F.Cu at (1255.6, 98.8)
- added C1120: 1uF, Capacitor_SMD:C_0603_1608Metric, F.Cu at (1303.7, 189.2)
- added C1121: 1uF, Capacitor_SMD:C_0603_1608Metric, F.Cu at (1303.7, 191.7)
- added C1122: 1uF, Capacitor_SMD:C_0603_1608Metric, F.Cu at (1303.7, 194.2)
- added C1123: 1uF, Capacitor_SMD:C_0603_1608Metric, F.Cu at (1303.7, 196.7)
- added C1124: 1uF, Capacitor_SMD:C_0603_1608Metric, F.Cu at (1303.7, 199.2)
- added C1125: 1uF, Capacitor_SMD:C_0603_1608Metric, F.Cu at (1303.7, 201.7)
- added C1126: 1uF, Capacitor_SMD:C_0603_1608Metric, F.Cu at (1303.7, 204.2)
- added C1127: 1uF, Capacitor_SMD:C_0603_1608Metric, F.Cu at (1303.7, 206.7)
- added C1128: 1uF, Capacitor_SMD:C_0603_1608Metric, F.Cu at (1303.7, 209.2)
- added C1129: 1uF, Capacitor_SMD:C_0603_1608Metric, F.Cu at (1303.7, 211.7)
- added C113: 1uF, Capacitor_SMD:C_0603_1608Metric, F.Cu at (1255.6, 101.3)
- added C1130: 1uF, Capacitor_SMD:C_0603_1608Metric, F.Cu at (1303.7, 214.3)
- added C1131: 1uF, Capacitor_SMD:C_0603_1608Metric, F.Cu at (1303.7, 216.8)
- added C1132: 1uF, Capacitor_SMD:C_0603_1608Metric, F.Cu at (1303.7, 219.3)
- added C1133: 1uF, Capacitor_SMD:C_0603_1608Metric, F.Cu at (1303.7, 221.8)
- added C1134: 1uF, Capacitor_SMD:C_0603_1608Metric, F.Cu at (1303.7, 224.3)
- added C1135: 1uF, Capacitor_SMD:C_0603_1608Metric, F.Cu at (1307.7, 23.5)
- added C1136: 1uF, Capacitor_SMD:C_0603_1608Metric, F.Cu at (1307.7, 26.0)
- added C1137: 1uF, Capacitor_SMD:C_0603_1608Metric, F.Cu at (1307.7, 28.5)
- added C1138: 1uF, Capacitor_SMD:C_0603_1608Metric, F.Cu at (1307.7, 31.0)
- added C1139: 1uF, Capacitor_SMD:C_0603_1608Metric, F.Cu at (1307.7, 33.5)
- added C114: 1uF, Capacitor_SMD:C_0603_1608Metric, F.Cu at (1255.6, 103.8)
- added C1140: 1uF, Capacitor_SMD:C_0603_1608Metric, F.Cu at (1307.7, 36.0)
- added C1141: 1uF, Capacitor_SMD:C_0603_1608Metric, F.Cu at (1307.7, 38.6)
- added C1142: 1uF, Capacitor_SMD:C_0603_1608Metric, F.Cu at (1307.7, 41.1)
- added C1143: 1uF, Capacitor_SMD:C_0603_1608Metric, F.Cu at (1307.7, 43.6)
- added C1144: 1uF, Capacitor_SMD:C_0603_1608Metric, F.Cu at (1307.7, 46.1)
- added C1145: 1uF, Capacitor_SMD:C_0603_1608Metric, F.Cu at (1307.7, 48.6)
- added C1146: 1uF, Capacitor_SMD:C_0603_1608Metric, F.Cu at (1307.7, 51.1)
- added C1147: 1uF, Capacitor_SMD:C_0603_1608Metric, F.Cu at (1307.7, 53.6)
- added C1148: 1uF, Capacitor_SMD:C_0603_1608Metric, F.Cu at (1307.7, 56.1)
- added C1149: 1uF, Capacitor_SMD:C_0603_1608Metric, F.Cu at (1307.7, 58.6)
- added C115: 1uF, Capacitor_SMD:C_0603_1608Metric, F.Cu at (1255.6, 106.3)
- added C1150: 1uF, Capacitor_SMD:C_0603_1608Metric, F.Cu at (1307.7, 61.1)
- added C1151: 1uF, Capacitor_SMD:C_0603_1608Metric, F.Cu at (1307.7, 63.7)
- added C1152: 1uF, Capacitor_SMD:C_0603_1608Metric, F.Cu at (1307.7, 66.2)
- added C1153: 1uF, Capacitor_SMD:C_0603_1608Metric, F.Cu at (1307.7, 68.7)
- added C1154: 1uF, Capacitor_SMD:C_0603_1608Metric, F.Cu at (1307.7, 71.2)
- added C1155: 1uF, Capacitor_SMD:C_0603_1608Metric, F.Cu at (1307.7, 73.7)
- added C1156: 1uF, Capacitor_SMD:C_0603_1608Metric, F.Cu at (1307.7, 76.2)
- added C1157: 1uF, Capacitor_SMD:C_0603_1608Metric, F.Cu at (1307.7, 78.7)
- added C1158: 1uF, Capacitor_SMD:C_0603_1608Metric, F.Cu at (1307.7, 81.2)
- added C1159: 1uF, Capacitor_SMD:C_0603_1608Metric, F.Cu at (1307.7, 83.7)
- added C116: 1uF, Capacitor_SMD:C_0603_1608Metric, F.Cu at (1255.6, 108.8)
- added C1160: 1uF, Capacitor_SMD:C_0603_1608Metric, F.Cu at (1307.7, 86.2)
- added C1161: 1uF, Capacitor_SMD:C_0603_1608Metric, F.Cu at (1307.7, 88.8)
- added C1162: 1uF, Capacitor_SMD:C_0603_1608Metric, F.Cu at (1307.7, 91.3)
- added C1163: 1uF, Capacitor_SMD:C_0603_1608Metric, F.Cu at (1307.7, 93.8)
- added C1164: 1uF, Capacitor_SMD:C_0603_1608Metric, F.Cu at (1307.7, 96.3)
- added C1165: 1uF, Capacitor_SMD:C_0603_1608Metric, F.Cu at (1307.7, 98.8)
- added C1166: 1uF, Capacitor_SMD:C_0603_1608Metric, F.Cu at (1307.7, 101.3)
- added C1167: 1uF, Capacitor_SMD:C_0603_1608Metric, F.Cu at (1307.7, 103.8)
- added C1168: 1uF, Capacitor_SMD:C_0603_1608Metric, F.Cu at (1307.7, 106.3)
- added C1169: 1uF, Capacitor_SMD:C_0603_1608Metric, F.Cu at (1307.7, 108.8)
- added C117: 1uF, Capacitor_SMD:C_0603_1608Metric, F.Cu at (1255.6, 111.3)
- added C1170: 1uF, Capacitor_SMD:C_0603_1608Metric, F.Cu at (1307.7, 111.3)
- added C1171: 1uF, Capacitor_SMD:C_0603_1608Metric, F.Cu at (1307.7, 113.9)
- added C1172: 1uF, Capacitor_SMD:C_0603_1608Metric, F.Cu at (1307.7, 116.4)
- added C1173: 1uF, Capacitor_SMD:C_0603_1608Metric, F.Cu at (1307.7, 118.9)
- added C1174: 1uF, Capacitor_SMD:C_0603_1608Metric, F.Cu at (1307.7, 121.4)
- added C1175: 1uF, Capacitor_SMD:C_0603_1608Metric, F.Cu at (1307.7, 123.9)
- added C1176: 1uF, Capacitor_SMD:C_0603_1608Metric, F.Cu at (1307.7, 126.4)
- added C1177: 1uF, Capacitor_SMD:C_0603_1608Metric, F.Cu at (1307.7, 128.9)
- added C1178: 1uF, Capacitor_SMD:C_0603_1608Metric, F.Cu at (1307.7, 131.4)
- added C1179: 1uF, Capacitor_SMD:C_0603_1608Metric, F.Cu at (1307.7, 133.9)
- added C118: 1uF, Capacitor_SMD:C_0603_1608Metric, F.Cu at (1255.6, 113.9)
- added C1180: 1uF, Capacitor_SMD:C_0603_1608Metric, F.Cu at (1307.7, 136.4)
- added C1181: 1uF, Capacitor_SMD:C_0603_1608Metric, F.Cu at (1307.7, 139.0)
- added C1182: 1uF, Capacitor_SMD:C_0603_1608Metric, F.Cu at (1307.7, 141.5)
- added C1183: 1uF, Capacitor_SMD:C_0603_1608Metric, F.Cu at (1307.7, 144.0)
- added C1184: 1uF, Capacitor_SMD:C_0603_1608Metric, F.Cu at (1307.7, 146.5)
- added C1185: 1uF, Capacitor_SMD:C_0603_1608Metric, F.Cu at (1307.7, 149.0)
- added C1186: 1uF, Capacitor_SMD:C_0603_1608Metric, F.Cu at (1307.7, 151.5)
- added C1187: 1uF, Capacitor_SMD:C_0603_1608Metric, F.Cu at (1307.7, 154.0)
- added C1188: 1uF, Capacitor_SMD:C_0603_1608Metric, F.Cu at (1307.7, 156.5)
- added C1189: 1uF, Capacitor_SMD:C_0603_1608Metric, F.Cu at (1307.7, 159.0)
- added C119: 1uF, Capacitor_SMD:C_0603_1608Metric, F.Cu at (1255.6, 116.4)
- added C1190: 1uF, Capacitor_SMD:C_0603_1608Metric, F.Cu at (1307.7, 161.5)
- added C1191: 1uF, Capacitor_SMD:C_0603_1608Metric, F.Cu at (1307.7, 164.1)
- added C1192: 1uF, Capacitor_SMD:C_0603_1608Metric, F.Cu at (1307.7, 166.6)
- added C1193: 1uF, Capacitor_SMD:C_0603_1608Metric, F.Cu at (1307.7, 169.1)
- added C1194: 1uF, Capacitor_SMD:C_0603_1608Metric, F.Cu at (1307.7, 171.6)
- added C1195: 1uF, Capacitor_SMD:C_0603_1608Metric, F.Cu at (1307.7, 174.1)
- added C1196: 1uF, Capacitor_SMD:C_0603_1608Metric, F.Cu at (1307.7, 176.6)
- added C1197: 1uF, Capacitor_SMD:C_0603_1608Metric, F.Cu at (1307.7, 179.1)
- added C1198: 1uF, Capacitor_SMD:C_0603_1608Metric, F.Cu at (1307.7, 181.6)
- added C1199: 1uF, Capacitor_SMD:C_0603_1608Metric, F.Cu at (1307.7, 184.1)
- added C12: 1uF, Capacitor_SMD:C_0603_1608Metric, F.Cu at (1251.6, 51.1)
- added C120: 1uF, Capacitor_SMD:C_0603_1608Metric, F.Cu at (1255.6, 118.9)
- added C1200: 1uF, Capacitor_SMD:C_0603_1608Metric, F.Cu at (1307.7, 186.6)
- added C1201: 1uF, Capacitor_SMD:C_0603_1608Metric, F.Cu at (1307.7, 189.2)
- added C1202: 1uF, Capacitor_SMD:C_0603_1608Metric, F.Cu at (1307.7, 191.7)
- added C1203: 1uF, Capacitor_SMD:C_0603_1608Metric, F.Cu at (1307.7, 194.2)
- added C1204: 1uF, Capacitor_SMD:C_0603_1608Metric, F.Cu at (1307.7, 196.7)
- added C1205: 1uF, Capacitor_SMD:C_0603_1608Metric, F.Cu at (1307.7, 199.2)
- added C1206: 1uF, Capacitor_SMD:C_0603_1608Metric, F.Cu at (1307.7, 201.7)
- added C1207: 1uF, Capacitor_SMD:C_0603_1608Metric, F.Cu at (1307.7, 204.2)
- added C1208: 1uF, Capacitor_SMD:C_0603_1608Metric, F.Cu at (1307.7, 206.7)
- added C1209: 1uF, Capacitor_SMD:C_0603_1608Metric, F.Cu at (1307.7, 209.2)
- added C121: 1uF, Capacitor_SMD:C_0603_1608Metric, F.Cu at (1255.6, 121.4)
- added C1210: 1uF, Capacitor_SMD:C_0603_1608Metric, F.Cu at (1307.7, 211.7)
- added C1211: 1uF, Capacitor_SMD:C_0603_1608Metric, F.Cu at (1307.7, 214.3)
- added C1212: 1uF, Capacitor_SMD:C_0603_1608Metric, F.Cu at (1307.7, 216.8)
- added C1213: 1uF, Capacitor_SMD:C_0603_1608Metric, F.Cu at (1307.7, 219.3)
- added C1214: 1uF, Capacitor_SMD:C_0603_1608Metric, F.Cu at (1307.7, 221.8)
- added C1215: 1uF, Capacitor_SMD:C_0603_1608Metric, F.Cu at (1307.7, 224.3)
- added C1216: 1uF, Capacitor_SMD:C_0603_1608Metric, F.Cu at (1311.8, 23.5)
- added C1217: 1uF, Capacitor_SMD:C_0603_1608Metric, F.Cu at (1311.8, 26.0)
- added C1218: 1uF, Capacitor_SMD:C_0603_1608Metric, F.Cu at (1311.8, 28.5)
- added C1219: 1uF, Capacitor_SMD:C_0603_1608Metric, F.Cu at (1311.8, 31.0)
- added C122: 1uF, Capacitor_SMD:C_0603_1608Metric, F.Cu at (1255.6, 123.9)
- added C1220: 1uF, Capacitor_SMD:C_0603_1608Metric, F.Cu at (1311.8, 33.5)
- added C1221: 1uF, Capacitor_SMD:C_0603_1608Metric, F.Cu at (1311.8, 36.0)
- added C1222: 1uF, Capacitor_SMD:C_0603_1608Metric, F.Cu at (1311.8, 38.6)
- added C1223: 1uF, Capacitor_SMD:C_0603_1608Metric, F.Cu at (1311.8, 41.1)
- added C1224: 1uF, Capacitor_SMD:C_0603_1608Metric, F.Cu at (1311.8, 43.6)
- added C1225: 1uF, Capacitor_SMD:C_0603_1608Metric, F.Cu at (1311.8, 46.1)
- added C1226: 1uF, Capacitor_SMD:C_0603_1608Metric, F.Cu at (1311.8, 48.6)
- added C1227: 1uF, Capacitor_SMD:C_0603_1608Metric, F.Cu at (1311.8, 51.1)
- added C1228: 1uF, Capacitor_SMD:C_0603_1608Metric, F.Cu at (1311.8, 53.6)
- added C1229: 1uF, Capacitor_SMD:C_0603_1608Metric, F.Cu at (1311.8, 56.1)
- added C123: 1uF, Capacitor_SMD:C_0603_1608Metric, F.Cu at (1255.6, 126.4)
- added C1230: 1uF, Capacitor_SMD:C_0603_1608Metric, F.Cu at (1311.8, 58.6)
- added C1231: 1uF, Capacitor_SMD:C_0603_1608Metric, F.Cu at (1311.8, 61.1)
- added C1232: 1uF, Capacitor_SMD:C_0603_1608Metric, F.Cu at (1311.8, 63.7)
- added C1233: 1uF, Capacitor_SMD:C_0603_1608Metric, F.Cu at (1311.8, 66.2)
- added C1234: 1uF, Capacitor_SMD:C_0603_1608Metric, F.Cu at (1311.8, 68.7)
- added C1235: 1uF, Capacitor_SMD:C_0603_1608Metric, F.Cu at (1311.8, 71.2)
- added C1236: 1uF, Capacitor_SMD:C_0603_1608Metric, F.Cu at (1311.8, 73.7)
- added C1237: 1uF, Capacitor_SMD:C_0603_1608Metric, F.Cu at (1311.8, 76.2)
- added C1238: 1uF, Capacitor_SMD:C_0603_1608Metric, F.Cu at (1311.8, 78.7)
- added C1239: 1uF, Capacitor_SMD:C_0603_1608Metric, F.Cu at (1311.8, 81.2)
- added C124: 1uF, Capacitor_SMD:C_0603_1608Metric, F.Cu at (1255.6, 128.9)
- added C1240: 1uF, Capacitor_SMD:C_0603_1608Metric, F.Cu at (1311.8, 83.7)
- added C1241: 1uF, Capacitor_SMD:C_0603_1608Metric, F.Cu at (1311.8, 86.2)
- added C1242: 1uF, Capacitor_SMD:C_0603_1608Metric, F.Cu at (1311.8, 88.8)
- added C1243: 1uF, Capacitor_SMD:C_0603_1608Metric, F.Cu at (1311.8, 91.3)
- added C1244: 1uF, Capacitor_SMD:C_0603_1608Metric, F.Cu at (1311.8, 93.8)
- added C1245: 1uF, Capacitor_SMD:C_0603_1608Metric, F.Cu at (1311.8, 96.3)
- added C1246: 1uF, Capacitor_SMD:C_0603_1608Metric, F.Cu at (1311.8, 98.8)
- added C1247: 1uF, Capacitor_SMD:C_0603_1608Metric, F.Cu at (1311.8, 101.3)
- added C1248: 1uF, Capacitor_SMD:C_0603_1608Metric, F.Cu at (1311.8, 103.8)
- added C1249: 1uF, Capacitor_SMD:C_0603_1608Metric, F.Cu at (1311.8, 106.3)
- added C125: 1uF, Capacitor_SMD:C_0603_1608Metric, F.Cu at (1255.6, 131.4)
- added C1250: 1uF, Capacitor_SMD:C_0603_1608Metric, F.Cu at (1311.8, 108.8)
- added C1251: 1uF, Capacitor_SMD:C_0603_1608Metric, F.Cu at (1311.8, 111.3)
- added C1252: 1uF, Capacitor_SMD:C_0603_1608Metric, F.Cu at (1311.8, 113.9)
- added C1253: 1uF, Capacitor_SMD:C_0603_1608Metric, F.Cu at (1311.8, 116.4)
- added C1254: 1uF, Capacitor_SMD:C_0603_1608Metric, F.Cu at (1311.8, 118.9)
- added C1255: 1uF, Capacitor_SMD:C_0603_1608Metric, F.Cu at (1311.8, 121.4)
- added C1256: 1uF, Capacitor_SMD:C_0603_1608Metric, F.Cu at (1311.8, 123.9)
- added C1257: 1uF, Capacitor_SMD:C_0603_1608Metric, F.Cu at (1311.8, 126.4)
- added C1258: 1uF, Capacitor_SMD:C_0603_1608Metric, F.Cu at (1311.8, 128.9)
- added C1259: 1uF, Capacitor_SMD:C_0603_1608Metric, F.Cu at (1311.8, 131.4)
- added C126: 1uF, Capacitor_SMD:C_0603_1608Metric, F.Cu at (1255.6, 133.9)
- added C1260: 1uF, Capacitor_SMD:C_0603_1608Metric, F.Cu at (1311.8, 133.9)
- added C1261: 1uF, Capacitor_SMD:C_0603_1608Metric, F.Cu at (1311.8, 136.4)
- added C1262: 1uF, Capacitor_SMD:C_0603_1608Metric, F.Cu at (1311.8, 139.0)
- added C1263: 1uF, Capacitor_SMD:C_0603_1608Metric, F.Cu at (1311.8, 141.5)
- added C1264: 1uF, Capacitor_SMD:C_0603_1608Metric, F.Cu at (1311.8, 144.0)
- added C1265: 1uF, Capacitor_SMD:C_0603_1608Metric, F.Cu at (1311.8, 146.5)
- added C1266: 1uF, Capacitor_SMD:C_0603_1608Metric, F.Cu at (1311.8, 149.0)
- added C1267: 1uF, Capacitor_SMD:C_0603_1608Metric, F.Cu at (1311.8, 151.5)
- added C1268: 1uF, Capacitor_SMD:C_0603_1608Metric, F.Cu at (1311.8, 154.0)
- added C1269: 1uF, Capacitor_SMD:C_0603_1608Metric, F.Cu at (1311.8, 156.5)
- added C127: 1uF, Capacitor_SMD:C_0603_1608Metric, F.Cu at (1255.6, 136.4)
- added C1270: 1uF, Capacitor_SMD:C_0603_1608Metric, F.Cu at (1311.8, 159.0)
- added C1271: 1uF, Capacitor_SMD:C_0603_1608Metric, F.Cu at (1311.8, 161.5)
- added C1272: 1uF, Capacitor_SMD:C_0603_1608Metric, F.Cu at (1311.8, 164.1)
- added C1273: 1uF, Capacitor_SMD:C_0603_1608Metric, F.Cu at (1311.8, 166.6)
- added C1274: 1uF, Capacitor_SMD:C_0603_1608Metric, F.Cu at (1311.8, 169.1)
- added C1275: 1uF, Capacitor_SMD:C_0603_1608Metric, F.Cu at (1311.8, 171.6)
- added C1276: 1uF, Capacitor_SMD:C_0603_1608Metric, F.Cu at (1311.8, 174.1)
- added C1277: 1uF, Capacitor_SMD:C_0603_1608Metric, F.Cu at (1311.8, 176.6)
- added C1278: 1uF, Capacitor_SMD:C_0603_1608Metric, F.Cu at (1311.8, 179.1)
- added C1279: 1uF, Capacitor_SMD:C_0603_1608Metric, F.Cu at (1311.8, 181.6)
- added C128: 1uF, Capacitor_SMD:C_0603_1608Metric, F.Cu at (1255.6, 139.0)
- added C1280: 1uF, Capacitor_SMD:C_0603_1608Metric, F.Cu at (1311.8, 184.1)
- added C1281: 1uF, Capacitor_SMD:C_0603_1608Metric, F.Cu at (1311.8, 186.6)
- added C1282: 1uF, Capacitor_SMD:C_0603_1608Metric, F.Cu at (1311.8, 189.2)
- added C1283: 1uF, Capacitor_SMD:C_0603_1608Metric, F.Cu at (1311.8, 191.7)
- added C1284: 1uF, Capacitor_SMD:C_0603_1608Metric, F.Cu at (1311.8, 194.2)
- added C1285: 1uF, Capacitor_SMD:C_0603_1608Metric, F.Cu at (1311.8, 196.7)
- added C1286: 1uF, Capacitor_SMD:C_0603_1608Metric, F.Cu at (1311.8, 199.2)
- added C1287: 1uF, Capacitor_SMD:C_0603_1608Metric, F.Cu at (1311.8, 201.7)
- added C1288: 1uF, Capacitor_SMD:C_0603_1608Metric, F.Cu at (1311.8, 204.2)
- added C1289: 1uF, Capacitor_SMD:C_0603_1608Metric, F.Cu at (1311.8, 206.7)
- added C129: 1uF, Capacitor_SMD:C_0603_1608Metric, F.Cu at (1255.6, 141.5)
- added C1290: 1uF, Capacitor_SMD:C_0603_1608Metric, F.Cu at (1311.8, 209.2)
- added C1291: 1uF, Capacitor_SMD:C_0603_1608Metric, F.Cu at (1311.8, 211.7)
- added C1292: 1uF, Capacitor_SMD:C_0603_1608Metric, F.Cu at (1311.8, 214.3)
- added C1293: 1uF, Capacitor_SMD:C_0603_1608Metric, F.Cu at (1311.8, 216.8)
- added C1294: 1uF, Capacitor_SMD:C_0603_1608Metric, F.Cu at (1311.8, 219.3)
- added C1295: 1uF, Capacitor_SMD:C_0603_1608Metric, F.Cu at (1311.8, 221.8)
- added C1296: 1uF, Capacitor_SMD:C_0603_1608Metric, F.Cu at (1311.8, 224.3)
- added C1297: 1uF, Capacitor_SMD:C_0603_1608Metric, F.Cu at (1315.8, 23.5)
- added C1298: 1uF, Capacitor_SMD:C_0603_1608Metric, F.Cu at (1315.8, 26.0)
- added C1299: 1uF, Capacitor_SMD:C_0603_1608Metric, F.Cu at (1315.8, 28.5)
- added C13: 1uF, Capacitor_SMD:C_0603_1608Metric, F.Cu at (1251.6, 53.6)
- added C130: 1uF, Capacitor_SMD:C_0603_1608Metric, F.Cu at (1255.6, 144.0)
- added C1300: 1uF, Capacitor_SMD:C_0603_1608Metric, F.Cu at (1315.8, 31.0)
- added C1301: 1uF, Capacitor_SMD:C_0603_1608Metric, F.Cu at (1315.8, 33.5)
- added C1302: 1uF, Capacitor_SMD:C_0603_1608Metric, F.Cu at (1315.8, 36.0)
- added C1303: 1uF, Capacitor_SMD:C_0603_1608Metric, F.Cu at (1315.8, 38.6)
- added C1304: 1uF, Capacitor_SMD:C_0603_1608Metric, F.Cu at (1315.8, 41.1)
- added C1305: 1uF, Capacitor_SMD:C_0603_1608Metric, F.Cu at (1315.8, 43.6)
- added C1306: 1uF, Capacitor_SMD:C_0603_1608Metric, F.Cu at (1315.8, 46.1)
- added C1307: 1uF, Capacitor_SMD:C_0603_1608Metric, F.Cu at (1315.8, 48.6)
- added C1308: 1uF, Capacitor_SMD:C_0603_1608Metric, F.Cu at (1315.8, 51.1)
- added C1309: 1uF, Capacitor_SMD:C_0603_1608Metric, F.Cu at (1315.8, 53.6)
- added C131: 1uF, Capacitor_SMD:C_0603_1608Metric, F.Cu at (1255.6, 146.5)
- added C1310: 1uF, Capacitor_SMD:C_0603_1608Metric, F.Cu at (1315.8, 56.1)
- added C1311: 1uF, Capacitor_SMD:C_0603_1608Metric, F.Cu at (1315.8, 58.6)
- added C1312: 1uF, Capacitor_SMD:C_0603_1608Metric, F.Cu at (1315.8, 61.1)
- added C1313: 1uF, Capacitor_SMD:C_0603_1608Metric, F.Cu at (1315.8, 63.7)
- added C1314: 1uF, Capacitor_SMD:C_0603_1608Metric, F.Cu at (1315.8, 66.2)
- added C1315: 1uF, Capacitor_SMD:C_0603_1608Metric, F.Cu at (1315.8, 68.7)
- added C1316: 1uF, Capacitor_SMD:C_0603_1608Metric, F.Cu at (1315.8, 71.2)
- added C1317: 1uF, Capacitor_SMD:C_0603_1608Metric, F.Cu at (1315.8, 73.7)
- added C1318: 1uF, Capacitor_SMD:C_0603_1608Metric, F.Cu at (1315.8, 76.2)
- added C1319: 1uF, Capacitor_SMD:C_0603_1608Metric, F.Cu at (1315.8, 78.7)
- added C132: 1uF, Capacitor_SMD:C_0603_1608Metric, F.Cu at (1255.6, 149.0)
- added C1320: 1uF, Capacitor_SMD:C_0603_1608Metric, F.Cu at (1315.8, 81.2)
- added C1321: 1uF, Capacitor_SMD:C_0603_1608Metric, F.Cu at (1315.8, 83.7)
- added C1322: 1uF, Capacitor_SMD:C_0603_1608Metric, F.Cu at (1315.8, 86.2)
- added C1323: 1uF, Capacitor_SMD:C_0603_1608Metric, F.Cu at (1315.8, 88.8)
- added C1324: 1uF, Capacitor_SMD:C_0603_1608Metric, F.Cu at (1315.8, 91.3)
- added C1325: 1uF, Capacitor_SMD:C_0603_1608Metric, F.Cu at (1315.8, 93.8)
- added C1326: 1uF, Capacitor_SMD:C_0603_1608Metric, F.Cu at (1315.8, 96.3)
- added C1327: 1uF, Capacitor_SMD:C_0603_1608Metric, F.Cu at (1315.8, 98.8)
- added C1328: 1uF, Capacitor_SMD:C_0603_1608Metric, F.Cu at (1315.8, 101.3)
- added C1329: 1uF, Capacitor_SMD:C_0603_1608Metric, F.Cu at (1315.8, 103.8)
- added C133: 1uF, Capacitor_SMD:C_0603_1608Metric, F.Cu at (1255.6, 151.5)
- added C1330: 1uF, Capacitor_SMD:C_0603_1608Metric, F.Cu at (1315.8, 106.3)
- added C1331: 1uF, Capacitor_SMD:C_0603_1608Metric, F.Cu at (1315.8, 108.8)
- added C1332: 1uF, Capacitor_SMD:C_0603_1608Metric, F.Cu at (1315.8, 111.3)
- added C1333: 1uF, Capacitor_SMD:C_0603_1608Metric, F.Cu at (1315.8, 113.9)
- added C1334: 1uF, Capacitor_SMD:C_0603_1608Metric, F.Cu at (1315.8, 116.4)
- added C1335: 1uF, Capacitor_SMD:C_0603_1608Metric, F.Cu at (1315.8, 118.9)
- added C1336: 1uF, Capacitor_SMD:C_0603_1608Metric, F.Cu at (1315.8, 121.4)
- added C1337: 1uF, Capacitor_SMD:C_0603_1608Metric, F.Cu at (1315.8, 123.9)
- added C1338: 1uF, Capacitor_SMD:C_0603_1608Metric, F.Cu at (1315.8, 126.4)
- added C1339: 1uF, Capacitor_SMD:C_0603_1608Metric, F.Cu at (1315.8, 128.9)
- added C134: 1uF, Capacitor_SMD:C_0603_1608Metric, F.Cu at (1255.6, 154.0)
- added C1340: 1uF, Capacitor_SMD:C_0603_1608Metric, F.Cu at (1315.8, 131.4)
- added C1341: 1uF, Capacitor_SMD:C_0603_1608Metric, F.Cu at (1315.8, 133.9)
- added C1342: 1uF, Capacitor_SMD:C_0603_1608Metric, F.Cu at (1315.8, 136.4)
- added C1343: 1uF, Capacitor_SMD:C_0603_1608Metric, F.Cu at (1315.8, 139.0)
- added C1344: 1uF, Capacitor_SMD:C_0603_1608Metric, F.Cu at (1315.8, 141.5)
- added C1345: 1uF, Capacitor_SMD:C_0603_1608Metric, F.Cu at (1315.8, 144.0)
- added C1346: 1uF, Capacitor_SMD:C_0603_1608Metric, F.Cu at (1315.8, 146.5)
- added C1347: 1uF, Capacitor_SMD:C_0603_1608Metric, F.Cu at (1315.8, 149.0)
- added C1348: 1uF, Capacitor_SMD:C_0603_1608Metric, F.Cu at (1315.8, 151.5)
- added C1349: 1uF, Capacitor_SMD:C_0603_1608Metric, F.Cu at (1315.8, 154.0)
- added C135: 1uF, Capacitor_SMD:C_0603_1608Metric, F.Cu at (1255.6, 156.5)
- added C1350: 1uF, Capacitor_SMD:C_0603_1608Metric, F.Cu at (1315.8, 156.5)
- added C1351: 1uF, Capacitor_SMD:C_0603_1608Metric, F.Cu at (1315.8, 159.0)
- added C1352: 1uF, Capacitor_SMD:C_0603_1608Metric, F.Cu at (1315.8, 161.5)
- added C1353: 1uF, Capacitor_SMD:C_0603_1608Metric, F.Cu at (1315.8, 164.1)
- added C1354: 1uF, Capacitor_SMD:C_0603_1608Metric, F.Cu at (1315.8, 166.6)
- added C1355: 1uF, Capacitor_SMD:C_0603_1608Metric, F.Cu at (1315.8, 169.1)
- added C1356: 1uF, Capacitor_SMD:C_0603_1608Metric, F.Cu at (1315.8, 171.6)
- added C1357: 1uF, Capacitor_SMD:C_0603_1608Metric, F.Cu at (1315.8, 174.1)
- added C1358: 1uF, Capacitor_SMD:C_0603_1608Metric, F.Cu at (1315.8, 176.6)
- added C1359: 1uF, Capacitor_SMD:C_0603_1608Metric, F.Cu at (1315.8, 179.1)
- added C136: 1uF, Capacitor_SMD:C_0603_1608Metric, F.Cu at (1255.6, 159.0)
- added C1360: 1uF, Capacitor_SMD:C_0603_1608Metric, F.Cu at (1315.8, 181.6)
- added C1361: 1uF, Capacitor_SMD:C_0603_1608Metric, F.Cu at (1315.8, 184.1)
- added C1362: 1uF, Capacitor_SMD:C_0603_1608Metric, F.Cu at (1315.8, 186.6)
- added C1363: 1uF, Capacitor_SMD:C_0603_1608Metric, F.Cu at (1315.8, 189.2)
- added C1364: 1uF, Capacitor_SMD:C_0603_1608Metric, F.Cu at (1315.8, 191.7)
- added C1365: 1uF, Capacitor_SMD:C_0603_1608Metric, F.Cu at (1315.8, 194.2)
- added C1366: 1uF, Capacitor_SMD:C_0603_1608Metric, F.Cu at (1315.8, 196.7)
- added C1367: 1uF, Capacitor_SMD:C_0603_1608Metric, F.Cu at (1315.8, 199.2)
- added C1368: 1uF, Capacitor_SMD:C_0603_1608Metric, F.Cu at (1315.8, 201.7)
- added C1369: 1uF, Capacitor_SMD:C_0603_1608Metric, F.Cu at (1315.8, 204.2)
- added C1370: 1uF, Capacitor_SMD:C_0603_1608Metric, F.Cu at (1315.8, 206.7)
- added C1371: 1uF, Capacitor_SMD:C_0603_1608Metric, F.Cu at (1315.8, 209.2)
- added C1372: 1uF, Capacitor_SMD:C_0603_1608Metric, F.Cu at (1315.8, 211.7)
- added C1373: 1uF, Capacitor_SMD:C_0603_1608Metric, F.Cu at (1315.8, 214.3)
- added C1374: 1uF, Capacitor_SMD:C_0603_1608Metric, F.Cu at (1315.8, 216.8)
- added C1375: 1uF, Capacitor_SMD:C_0603_1608Metric, F.Cu at (1315.8, 219.3)
- added C1376: 1uF, Capacitor_SMD:C_0603_1608Metric, F.Cu at (1315.8, 221.8)
- added C1377: 1uF, Capacitor_SMD:C_0603_1608Metric, F.Cu at (1315.8, 224.3)
- added C1378: 1uF, Capacitor_SMD:C_0603_1608Metric, F.Cu at (1319.8, 23.5)
- added C1379: 1uF, Capacitor_SMD:C_0603_1608Metric, F.Cu at (1319.8, 26.0)
- added C1380: 1uF, Capacitor_SMD:C_0603_1608Metric, F.Cu at (1319.8, 28.5)
- added C1381: 1uF, Capacitor_SMD:C_0603_1608Metric, F.Cu at (1319.8, 31.0)
- added C1382: 1uF, Capacitor_SMD:C_0603_1608Metric, F.Cu at (1319.8, 33.5)
- added C1383: 1uF, Capacitor_SMD:C_0603_1608Metric, F.Cu at (1319.8, 36.0)
- added C1384: 1uF, Capacitor_SMD:C_0603_1608Metric, F.Cu at (1319.8, 38.6)
- added C1385: 1uF, Capacitor_SMD:C_0603_1608Metric, F.Cu at (1319.8, 41.1)
- added C1386: 1uF, Capacitor_SMD:C_0603_1608Metric, F.Cu at (1319.8, 43.6)
- added C1387: 1uF, Capacitor_SMD:C_0603_1608Metric, F.Cu at (1319.8, 46.1)
- added C1388: 1uF, Capacitor_SMD:C_0603_1608Metric, F.Cu at (1319.8, 48.6)
- added C1389: 1uF, Capacitor_SMD:C_0603_1608Metric, F.Cu at (1319.8, 51.1)
- added C1390: 1uF, Capacitor_SMD:C_0603_1608Metric, F.Cu at (1319.8, 53.6)
- added C1391: 1uF, Capacitor_SMD:C_0603_1608Metric, F.Cu at (1319.8, 56.1)
- added C1392: 1uF, Capacitor_SMD:C_0603_1608Metric, F.Cu at (1319.8, 58.6)
- added C1393: 1uF, Capacitor_SMD:C_0603_1608Metric, F.Cu at (1319.8, 61.1)
- added C1394: 1uF, Capacitor_SMD:C_0603_1608Metric, F.Cu at (1319.8, 63.7)
- added C1395: 1uF, Capacitor_SMD:C_0603_1608Metric, F.Cu at (1319.8, 66.2)
- added C1396: 1uF, Capacitor_SMD:C_0603_1608Metric, F.Cu at (1319.8, 68.7)
- added C1397: 1uF, Capacitor_SMD:C_0603_1608Metric, F.Cu at (1319.8, 71.2)
- added C1398: 1uF, Capacitor_SMD:C_0603_1608Metric, F.Cu at (1319.8, 73.7)
- added C1399: 1uF, Capacitor_SMD:C_0603_1608Metric, F.Cu at (1319.8, 76.2)
- added C14: 1uF, Capacitor_SMD:C_0603_1608Metric, F.Cu at (1251.6, 56.1)
- added C1400: 1uF, Capacitor_SMD:C_0603_1608Metric, F.Cu at (1319.8, 78.7)
- added C1401: 1uF, Capacitor_SMD:C_0603_1608Metric, F.Cu at (1319.8, 81.2)
- added C1402: 1uF, Capacitor_SMD:C_0603_1608Metric, F.Cu at (1319.8, 83.7)
- added C1403: 1uF, Capacitor_SMD:C_0603_1608Metric, F.Cu at (1319.8, 86.2)
- added C1404: 1uF, Capacitor_SMD:C_0603_1608Metric, F.Cu at (1319.8, 88.8)
- added C1405: 1uF, Capacitor_SMD:C_0603_1608Metric, F.Cu at (1319.8, 91.3)
- added C1406: 1uF, Capacitor_SMD:C_0603_1608Metric, F.Cu at (1319.8, 93.8)
- added C1407: 1uF, Capacitor_SMD:C_0603_1608Metric, F.Cu at (1319.8, 96.3)
- added C1408: 1uF, Capacitor_SMD:C_0603_1608Metric, F.Cu at (1319.8, 98.8)
- added C1409: 1uF, Capacitor_SMD:C_0603_1608Metric, F.Cu at (1319.8, 101.3)
- added C1410: 1uF, Capacitor_SMD:C_0603_1608Metric, F.Cu at (1319.8, 103.8)
- added C1411: 1uF, Capacitor_SMD:C_0603_1608Metric, F.Cu at (1319.8, 106.3)
- added C1412: 1uF, Capacitor_SMD:C_0603_1608Metric, F.Cu at (1319.8, 108.8)
- added C1413: 1uF, Capacitor_SMD:C_0603_1608Metric, F.Cu at (1319.8, 111.3)
- added C1414: 1uF, Capacitor_SMD:C_0603_1608Metric, F.Cu at (1319.8, 113.9)
- added C1415: 1uF, Capacitor_SMD:C_0603_1608Metric, F.Cu at (1319.8, 116.4)
- added C1416: 1uF, Capacitor_SMD:C_0603_1608Metric, F.Cu at (1319.8, 118.9)
- added C1417: 1uF, Capacitor_SMD:C_0603_1608Metric, F.Cu at (1319.8, 121.4)
- added C1418: 1uF, Capacitor_SMD:C_0603_1608Metric, F.Cu at (1319.8, 123.9)
- added C1419: 1uF, Capacitor_SMD:C_0603_1608Metric, F.Cu at (1319.8, 126.4)
- added C1420: 1uF, Capacitor_SMD:C_0603_1608Metric, F.Cu at (1319.8, 128.9)
- added C1421: 1uF, Capacitor_SMD:C_0603_1608Metric, F.Cu at (1319.8, 131.4)
- added C1422: 1uF, Capacitor_SMD:C_0603_1608Metric, F.Cu at (1319.8, 133.9)
- added C1423: 1uF, Capacitor_SMD:C_0603_1608Metric, F.Cu at (1319.8, 136.4)
- added C1424: 1uF, Capacitor_SMD:C_0603_1608Metric, F.Cu at (1319.8, 139.0)
- added C1425: 1uF, Capacitor_SMD:C_0603_1608Metric, F.Cu at (1319.8, 141.5)
- added C1426: 1uF, Capacitor_SMD:C_0603_1608Metric, F.Cu at (1319.8, 144.0)
- added C1427: 1uF, Capacitor_SMD:C_0603_1608Metric, F.Cu at (1319.8, 146.5)
- added C1428: 1uF, Capacitor_SMD:C_0603_1608Metric, F.Cu at (1319.8, 149.0)
- added C1429: 1uF, Capacitor_SMD:C_0603_1608Metric, F.Cu at (1319.8, 151.5)
- added C1430: 1uF, Capacitor_SMD:C_0603_1608Metric, F.Cu at (1319.8, 154.0)
- added C1431: 1uF, Capacitor_SMD:C_0603_1608Metric, F.Cu at (1319.8, 156.5)
- added C1432: 1uF, Capacitor_SMD:C_0603_1608Metric, F.Cu at (1319.8, 159.0)
- added C1433: 1uF, Capacitor_SMD:C_0603_1608Metric, F.Cu at (1319.8, 161.5)
- added C1434: 1uF, Capacitor_SMD:C_0603_1608Metric, F.Cu at (1319.8, 164.1)
- added C1435: 1uF, Capacitor_SMD:C_0603_1608Metric, F.Cu at (1319.8, 166.6)
- added C1436: 1uF, Capacitor_SMD:C_0603_1608Metric, F.Cu at (1319.8, 169.1)
- added C1437: 1uF, Capacitor_SMD:C_0603_1608Metric, F.Cu at (1319.8, 171.6)
- added C1438: 1uF, Capacitor_SMD:C_0603_1608Metric, F.Cu at (1319.8, 174.1)
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Connections:
- C137 pad 2: VCC -> VCC_1
- C138 pad 2: VCC -> VCC_1
- C139 pad 2: VCC -> VCC_1
- C140 pad 2: VCC -> VCC_1
- C141 pad 2: VCC -> VCC_1
- C142 pad 2: VCC -> VCC_1
- C143 pad 2: VCC -> VCC_1
- C144 pad 2: VCC -> VCC_1
- C145 pad 2: VCC -> VCC_1
- C146 pad 2: VCC -> VCC_1
- C147 pad 2: VCC -> VCC_1
- C148 pad 2: VCC -> VCC_1
- C149 pad 2: VCC -> VCC_1
- C150 pad 2: VCC -> VCC_1
- C151 pad 2: VCC -> VCC_1
- C152 pad 2: VCC -> VCC_1
- C153 pad 2: VCC -> VCC_1
- C154 pad 2: VCC -> VCC_1
- C155 pad 2: VCC -> VCC_1
- C156 pad 2: VCC -> VCC_1
- C157 pad 2: VCC -> VCC_1
- C158 pad 2: VCC -> VCC_1
- C159 pad 2: VCC -> VCC_1
- C160 pad 2: VCC -> VCC_1
- C161 pad 2: VCC -> VCC_1
- C162 pad 2: VCC -> VCC_1
- C163 pad 2: VCC -> VCC_1
- C164 pad 2: VCC -> VCC_1
- C165 pad 2: VCC -> VCC_1
- C166 pad 2: VCC -> VCC_1
- C167 pad 2: VCC -> VCC_1
- C168 pad 2: VCC -> VCC_1
- C169 pad 2: VCC -> VCC_1
- C170 pad 2: VCC -> VCC_1
- C171 pad 2: VCC -> VCC_1
- C172 pad 2: VCC -> VCC_1
- C173 pad 2: VCC -> VCC_1
- C174 pad 2: VCC -> VCC_1
- C175 pad 2: VCC -> VCC_1
- C176 pad 2: VCC -> VCC_1
- C177 pad 2: VCC -> VCC_1
- C178 pad 2: VCC -> VCC_1
- C179 pad 2: VCC -> VCC_1
- C180 pad 2: VCC -> VCC_1
- C181 pad 2: VCC -> VCC_1
- C182 pad 2: VCC -> VCC_1
- C183 pad 2: VCC -> VCC_1
- C184 pad 2: VCC -> VCC_1
- C185 pad 1: VCC -> GND
- C185 pad 2: GND -> VCC_1
- C186 pad 1: VCC -> GND
- C186 pad 2: GND -> VCC_1
- C187 pad 1: VCC -> GND
- C187 pad 2: GND -> VCC_1
- C188 pad 1: VCC -> GND
- C188 pad 2: GND -> VCC_1
- C189 pad 1: VCC -> GND
- C189 pad 2: GND -> VCC_1
- C190 pad 1: VCC -> GND
- C190 pad 2: GND -> VCC_1
- C191 pad 1: VCC -> GND
- C191 pad 2: GND -> VCC_1
- C192 pad 1: VCC -> GND
- C192 pad 2: GND -> VCC_1
- C193 pad 1: VCC -> GND
- C193 pad 2: GND -> VCC_1
- C194 pad 1: VCC -> GND
- C194 pad 2: GND -> VCC_1
- C195 pad 1: VCC -> GND
- C195 pad 2: GND -> VCC_1
- C196 pad 1: VCC -> GND
- C196 pad 2: GND -> VCC_1
- C197 pad 1: VCC -> GND
- C197 pad 2: GND -> VCC_1
- C198 pad 1: VCC -> GND
- C198 pad 2: GND -> VCC_1
- C199 pad 1: VCC -> GND
- C199 pad 2: GND -> VCC_1
- C200 pad 1: VCC -> GND
- C200 pad 2: GND -> VCC_1
- C201 pad 1: VCC -> GND
- C201 pad 2: GND -> VCC_1
- C202 pad 1: VCC -> GND
- C202 pad 2: GND -> VCC_1
- C203 pad 1: VCC -> GND
- C203 pad 2: GND -> VCC_1
- C204 pad 1: VCC -> GND
- C204 pad 2: GND -> VCC_1
- C205 pad 1: VCC -> GND
- C205 pad 2: GND -> VCC_1
- C206 pad 1: VCC -> GND
- C206 pad 2: GND -> VCC_1
- C207 pad 1: VCC -> GND
- C207 pad 2: GND -> VCC_1
- C208 pad 1: VCC -> GND
- C208 pad 2: GND -> VCC_1
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Routing:
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- removed copper zone on B.Cu, net GND
- removed copper zone on In1.Cu, net GND
- removed copper zone on In2.Cu, net VCC
Other:
- board outline removed
- board text removed: "PCB_GRID-V1-14X14-APA102-2020 SNAKE-CSF25"
