File: ATMEGA-SCHEMATICS/SNAKE_GAME/PROGRAMMER/PROGRAMMER.kicad_sch (KiCad schematic)
At the start: 12 parts, among them P1 USB_C_Plug_USB2.0, U1 47pF, U1 FT232RL, U2 ATmega8-16A

Commit message: .
Other:
- removed sheet Untitled Sheet
- added sheet Power (Power.kicad_sch)
- added sheet UBS_C (USB_C.kicad_sch)

Commit message: PWR_USBC_UART_ATMEGA8
Come back to Earth - Mac Miller
Parts:
- removed C1, C3, C5: 0.1uF, symbol Device:C
- removed C2, U1: 47pF, symbol Device:C
- removed C6: 4.7uF, symbol Device:C_Polarized
- removed P1: USB_C_Plug_USB2.0, symbol Connector:USB_C_Plug_USB2.0
- removed R1: 4k7, symbol Device:R_US
- removed R2: 10k, symbol Device:R_US
- removed R3: 5.1kOHM, symbol Device:R_US
- removed U1: FT232RL, Package_SO:SSOP-28_5.3x10.2mm_P0.65mm, symbol Interface_USB:FT232RL
- removed U2: ATmega8-16A, Package_QFP:TQFP-32_7x7mm_P0.8mm, symbol MCU_Microchip_ATmega:ATmega8-16A
- added H1, H2, H3, H4, H5, H6, H7: MountingHole, MountingHole:MountingHole_3.2mm_M3, symbol Mechanical:MountingHole
Connections:
- no-connect marks 31 -> 0
Other:
- sheet UBS_C renamed power
- removed sheet Power
- sheet ATmega8A ports: added none; removed AGND, AVCC, GND, PD4, PD5, PD6, PD7, VCC
- sheet FT232RL ports: added none; removed 3V3OUT, AGND, CBUS0, CBUS1, CBUS2, CBUS3, CBUS4, GND, RESET, TEST, UBSCD-, USBCD+, VCC, VCCIO
