File: ATMEGA-SCHEMATICS/SNAKE_GAME/PROGRAMMER/ATmega8A.kicad_sch (KiCad schematic)
At the start: 1 part, among them U4 ATmega8-16A

Commit message: PWR_USBC_UART_ATMEGA8
Come back to Earth - Mac Miller
Parts:
- removed U4: ATmega8-16A, Package_QFP:TQFP-32_7x7mm_P0.8mm, symbol MCU_Microchip_ATmega:ATmega8-16A
- added C8, C9: 22pF, Capacitor_THT:CP_Radial_D5.0mm_P2.50mm, symbol Device:C_US
- added J4: Conn_01x15_Pin, Connector_PinHeader_2.54mm:PinHeader_1x15_P2.54mm_Vertical, symbol Connector:Conn_01x15_Pin
- added U5: ATmega8-16P, Package_DIP:DIP-28_W7.62mm, symbol MCU_Microchip_ATmega:ATmega8-16P
- added Y1: Crystal, Crystal:Resonator-2Pin_W6.0mm_H3.0mm, symbol Device:Crystal
Connections:
- net GND: now also C8.2, C9.2, U5.22 (AGND), U5.8 (GND)
- net PD0: now also U5.2 (PD0)
- net PD1: now also U5.3 (PD1)
- net PD2: now also U5.4 (PD2)
- net PD3: now also U5.5 (PD3)
- net PD4: now also U5.6 (PD4)
- net PD5: now also U5.11 (PD5)
- net PD6: now also J4.2 (Pin_2), U5.12 (PD6)
- net PD7: now also J4.1 (Pin_1), U5.13 (PD7)
- net VCC: now also U5.20 (AVCC), U5.21 (AREF), U5.7 (VCC)
- new net: C9.1, U5.10 (PB7/XTAL2), Y1.2
- new net: C8.1, U5.9 (PB6/XTAL1), Y1.1
- new net PB0: J4.3 (Pin_3), U5.14 (PB0)
- new net PB1: J4.4 (Pin_4), U5.15 (PB1)
- new net PB2: J4.5 (Pin_5), U5.16 (PB2)
- new net PB3: J4.6 (Pin_6), U5.17 (PB3)
- new net PB4: J4.7 (Pin_7), U5.18 (PB4)
- new net PB5: J4.8 (Pin_8), U5.19 (PB5)
- new net PC0: J4.9 (Pin_9), U5.23 (PC0)
- new net PC1: J4.10 (Pin_10), U5.24 (PC1)
- new net PC2: J4.11 (Pin_11), U5.25 (PC2)
- new net PC3: J4.12 (Pin_12), U5.26 (PC3)
- new net PC4: J4.13 (Pin_13), U5.27 (PC4)
- new net PC5: J4.14 (Pin_14), U5.28 (PC5)
- new net PC6/RESET: J4.15 (Pin_15), U5.1 (PC6/~{RESET})

Commit message: edited schematics
Parts:
- added C11, C12, C13: 0.1uF, Capacitor_THT:C_Disc_D7.5mm_W5.0mm_P5.00mm, symbol Device:C
- added J1: Conn_01x06_Pin, Connector_PinHeader_2.54mm:PinHeader_1x07_P2.54mm_Vertical, symbol Connector:Conn_01x06_Pin
Connections:
- net GND: now also C11.2, C12.2, C13.2
- net PD0: now also J1.6 (Pin_6)
- net PD1: now also J1.5 (Pin_5)
- net PD2: now also J1.4 (Pin_4)
- net PD3: now also J1.3 (Pin_3)
- net PD4: now also J1.2 (Pin_2)
- net PD5: now also J1.1 (Pin_1)
- net VCC: now also C11.1, C12.1, C13.1
Other:
- moved on the sheet: J4
