File: ATMEGA-SCHEMATICS/SNAKE_GAME/PROGRAMMER/USB_C.kicad_sch (KiCad schematic)
At the start: 1 part, among them P2 USB_C_Plug_USB2.0

Commit message: PWR_USBC_UART_ATMEGA8
Come back to Earth - Mac Miller
Parts:
- removed P2: USB_C_Plug_USB2.0, symbol Connector:USB_C_Plug_USB2.0
- added C10, C2: 47pF, Capacitor_THT:C_Disc_D7.5mm_W5.0mm_P5.00mm, symbol Device:C
- added C6: 4.7uF, Capacitor_THT:C_Disc_D7.5mm_W5.0mm_P5.00mm, symbol Device:C
- added C7: 220uF, Capacitor_THT:C_Disc_D3.0mm_W1.6mm_P2.50mm, symbol Device:C_Polarized
- added J2: Barrel_Jack_Switch_Pin3Ring, Connector_BarrelJack:BarrelJack_Horizontal, symbol Connector:Barrel_Jack_Switch_Pin3Ring
- added P1: USB_C_Plug_USB2.0, Connector_USB:USB_C_Receptacle_GCT_USB4110, symbol Connector:USB_C_Plug_USB2.0
- added R1: 5k1, Resistor_THT:R_Axial_DIN0207_L6.3mm_D2.5mm_P10.16mm_Horizontal, symbol Device:R_US
Connections:
- net D+: now also C10.2, P1.A6 (D+)
- net D-: now also C2.2, P1.A7 (D-)
- net GND: now also C10.1, C2.1, C6.1, C7.2, J2.2, J2.3, P1.A1 (GND), P1.A12 (GND), P1.B1 (GND), P1.B12 (GND), R1.1
- new net: P1.A5 (CC), R1.2
- new net USBC_VBUS: P1.A4 (VBUS), P1.A9 (VBUS), P1.B4 (VBUS), P1.B9 (VBUS)
- new net VCC: C6.2, C7.1, J2.1
- no-connect marks 0 -> 2

Commit message: edited schematics
Parts:
- removed C10, C2: 47pF, Capacitor_THT:C_Disc_D7.5mm_W5.0mm_P5.00mm, symbol Device:C
- removed P1: USB_C_Plug_USB2.0, Connector_USB:USB_C_Receptacle_GCT_USB4110, symbol Connector:USB_C_Plug_USB2.0
- removed R1: 5k1, Resistor_THT:R_Axial_DIN0207_L6.3mm_D2.5mm_P10.16mm_Horizontal, symbol Device:R_US
- added C14, C15: 47pF, Capacitor_THT:C_Disc_D7.5mm_W5.0mm_P5.00mm, symbol Device:C
- added J5: USB_A, Connector_USB:USB_A_Connfly_DS1095, symbol Connector:USB_A
Connections:
- net D+: now also C15.2, J5.3 (D+)
- net D-: now also C14.2, J5.2 (D-)
- net GND: now also C14.1, C15.1, J5.4 (GND)
- net USBC_VBUS: now also J5.1 (VBUS)
- no-connect marks 2 -> 1
