File: ATMEGA-SCHEMATICS/SNAKE_GAME/PROGRAMMER/untitled.kicad_sch (KiCad schematic)
At the start: 2 parts, among them U3 FT232RL

Commit message: PWR_USBC_UART_ATMEGA8
Come back to Earth - Mac Miller
Parts:
- added C1: 4.7uF, Capacitor_THT:C_Disc_D3.0mm_W1.6mm_P2.50mm, symbol Device:C_Polarized
- added C3, C5: 0.1uF, Capacitor_THT:C_Disc_D7.5mm_W5.0mm_P5.00mm, symbol Device:C
- added D1, D2: LED, Inductor_SMD:L_Sunlord_SWPA8040S, symbol Device:LED
- added J3: Conn_01x07_Pin, Connector_PinHeader_2.54mm:PinHeader_1x07_P2.54mm_Vertical, symbol Connector:Conn_01x07_Pin
- added R4: 4k7, Resistor_THT:R_Axial_DIN0207_L6.3mm_D2.5mm_P10.16mm_Horizontal, symbol Device:R_US
- added R6, R7: 10k, Resistor_THT:R_Axial_DIN0207_L6.3mm_D2.5mm_P10.16mm_Horizontal, symbol Device:R_US
- added R8: 270 OHM, Resistor_THT:R_Axial_DIN0207_L6.3mm_D2.5mm_P10.16mm_Horizontal, symbol Device:R_US
- added R9: 270k OHM, Resistor_THT:R_Axial_DIN0207_L6.3mm_D2.5mm_P10.16mm_Horizontal, symbol Device:R_US
- C4: footprint (none) -> Capacitor_THT:C_Disc_D7.5mm_W5.0mm_P5.00mm
Connections:
- net 3V3OUT is gone; now on net VCC: C4.1
- net AGND is gone; now on net GND: U3.25 (AGND)
- net TEST is gone; now on net GND: U3.26 (TEST)
- net VCCIO is gone; now on net VCC: U3.4 (VCCIO)
- net CBUS1: now also R9.1
- net CBUS2: now also R8.1
- net CBUS4: now also J3.1 (Pin_1)
- net GND: now also C4.2, C1.2, C3.1, C5.1, R6.2
- net VCC: now also C1.1, C5.2
- net at U3.17 (3V3OUT): now also C3.2; no longer C4.2
- net DCD: now reaches U3.10 (DCD)
- net DCD: now also J3.5 (Pin_5)
- net DTR: now reaches U3.2 (DTR)
- net DTR: now also J3.7 (Pin_7)
- net OSCI: now reaches U3.27 (OSCI)
- net OSCI: now also J3.3 (Pin_3)
- net OSCO: now reaches U3.28 (OSCO)
- net OSCO: now also J3.2 (Pin_2)
- net RI: now reaches U3.6 (RI)
- net RI: now also J3.4 (Pin_4)
- net DCR: now reaches U3.9 (DCR)
- net DCR: now also J3.6 (Pin_6)
- net CBUS0 renamed PD4
- net CBUS3 renamed PD5
- net PD5: now also R7.2
- net RESET: no longer names the net of U3.19 (~{RESET})
- net RESET: now also R4.2, R6.1
- net UBSCD- renamed D-
- net USBCD+ renamed D+
- new net: D1.1 (K), R8.2
- new net: D2.1 (K), R9.2
- new net: D1.2 (A), D2.2 (A)
- new net USBC_VBUS: R4.1
Other:
- moved on the sheet: U3

Commit message: edited schematics
Parts:
- D1, D2: footprint Inductor_SMD:L_Sunlord_SWPA8040S -> LED_THT:LED_D1.8mm_W3.3mm_H2.4mm
- R9: value 270k OHM -> 270 OHM
- U3: footprint Package_SO:SSOP-28_5.3x10.2mm_P0.65mm -> Package_DIP:DIP-28_W7.62mm
Connections:
- net VCC: now also D1.2 (A), D2.2 (A), R7.1
- net OSCI: no longer names the net of J3.3 (Pin_3)
- net OSCI: no longer U3.27 (OSCI)
- net OSCO: no longer names the net of J3.2 (Pin_2)
- net OSCO: no longer U3.28 (OSCO)
- no-connect marks 0 -> 4
Changed lines of the file:
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@@
 		(color 0 0 0 0)
 	)
+	(no_connect
+		(at 69.85 96.52)
+	)
+	(no_connect
+		(at 167.64 66.04)
+	)
+	(no_connect
+		(at 167.64 63.5)
+	)
+	(no_connect
+		(at 69.85 101.6)
+	)
 	(wire
 		(pts
@@
 	(wire
 		(pts
+			(xy 74.93 168.91) (xy 82.55 168.91)
+		)
+		(stroke
+			(width 0)
+			(type default)
+		)
+	)
+	(wire
+		(pts
 			(xy 90.17 162.56) (xy 93.98 162.56)
 		)
@@
 		(pts
 			(xy 46.99 91.44) (xy 69.85 91.44)
-		)
-		(stroke
-			(width 0)
-			(type default)
-		)
-	)
-	(wire
-		(pts
-			(xy 72.39 168.91) (xy 82.55 168.91)
 		)
 		(stroke
@@
 		)
 	)
-	(label "OSCO"
-		(at 69.85 101.6 180)
-		(effects
-			(font
-				(size 1.27 1.27)
-			)
-			(justify right bottom)
-		)
-	)
 	(label "DCD"
 		(at 167.64 58.42 180)
@@
 		)
 	)
-	(label "OSCI"
-		(at 167.64 63.5 180)
-		(effects
-			(font
-				(size 1.27 1.27)
-			)
-			(justify right bottom)
-		)
-	)
-	(label "OSCO"
-		(at 167.64 66.04 180)
-		(effects
-			(font
-				(size 1.27 1.27)
-			)
-			(justify right bottom)
-		)
-	)
 	(label "DCD"
 		(at 110.49 88.9 0)
@@
 	(label "CBUS4"
 		(at 167.64 68.58 180)
-		(effects
-			(font
-				(size 1.27 1.27)
-			)
-			(justify right bottom)
-		)
-	)
-	(label "OSCI"
-		(at 69.85 96.52 180)
 		(effects
 			(font
@@
 			)
 		)
-		(property "Value" "270k OHM"
+		(property "Value" "270 OHM"
 			(at 97.282 165.862 90)
 			(effects
@@
 	)
 	(symbol
-		(lib_id "power:PWR_FLAG")
-		(at 134.62 127 270)
-		(unit 1)
-		(exclude_from_sim no)
-		(in_bom yes)
-		(on_board yes)
-		(dnp no)
-		(fields_autoplaced yes)
-		(property "Reference" "#FLG03"
-			(at 136.525 127 0)
-			(effects
-				(font
-					(size 1.27 1.27)
-				)
-				(hide yes)
-			)
-		)
-		(property "Value" "PWR_FLAG"
-			(at 138.43 126.9999 90)
-			(effects
-				(font
-					(size 1.27 1.27)
-				)
-				(justify left)
-			)
-		)
-		(property "Footprint" ""
-			(at 134.62 127 0)
-			(effects
-				(font
-					(size 1.27 1.27)
-				)
-				(hide yes)
-			)
-		)
-		(property "Datasheet" "~"
-			(at 134.62 127 0)
-			(effects
-				(font
-					(size 1.27 1.27)
-				)
-				(hide yes)
-			)
-		)
-		(property "Description" "Special symbol for telling ERC where power comes from"
-			(at 134.62 127 0)
-			(effects
-				(font
-					(size 1.27 1.27)
-				)
-				(hide yes)
-			)
-		)
-		(pin "1"
-		)
-		(instances
-			(project "PROGRAMMER"
-				(path "/c3d4d3ca-3b0c-4b66-9122-b6670ae5401e/f80a6ea3-817f-470e-88f7-47e64e60582d"
-					(reference "#FLG03")
-					(unit 1)
-				)
-			)
-		)
-	)
-	(symbol
 		(lib_id "Device:C")
 		(at 76.2 54.61 0)
@@
 	)
 	(symbol
-		(lib_id "power:PWR_FLAG")
-		(at 72.39 168.91 90)
-		(unit 1)
-		(exclude_from_sim no)
-		(in_bom yes)
-		(on_board yes)
-		(dnp no)
-		(fields_autoplaced yes)
-		(property "Reference" "#FLG05"
-			(at 70.485 168.91 0)
-			(effects
-				(font
-					(size 1.27 1.27)
-				)
-				(hide yes)
-			)
-		)
-		(property "Value" "PWR_FLAG"
-			(at 68.58 168.9099 90)
-			(effects
-				(font
-					(size 1.27 1.27)
-				)
-				(justify left)
-			)
-		)
-		(property "Footprint" ""
-			(at 72.39 168.91 0)
-			(effects
-				(font
-					(size 1.27 1.27)
-				)
-				(hide yes)
-			)
-		)
-		(property "Datasheet" "~"
-			(at 72.39 168.91 0)
-			(effects
-				(font
-					(size 1.27 1.27)
-				)
-				(hide yes)
-			)
-		)
-		(property "Description" "Special symbol for telling ERC where power comes from"
-			(at 72.39 168.91 0)
-			(effects
-				(font
-					(size 1.27 1.27)
-				)
-				(hide yes)
-			)
-		)
-		(pin "1"
-		)
-		(instances
-			(project "PROGRAMMER"
-				(path "/c3d4d3ca-3b0c-4b66-9122-b6670ae5401e/f80a6ea3-817f-470e-88f7-47e64e60582d"
-					(reference "#FLG05")
-					(unit 1)
-				)
-			)
-		)
-	)
-	(symbol
 		(lib_id "Device:C_Polarized")
 		(at 83.82 54.61 0)
@@
 			)
 		)
-		(property "Footprint" "Inductor_SMD:L_Sunlord_SWPA8040S"
+		(property "Footprint" "LED_THT:LED_D1.8mm_W3.3mm_H2.4mm"
 			(at 86.36 175.26 0)
 			(effects
@@
 	)
 	(symbol
+		(lib_id "power:VCC")
+		(at 74.93 168.91 0)
+		(unit 1)
+		(exclude_from_sim no)
+		(in_bom yes)
+		(on_board yes)
+		(dnp no)
+		(fields_autoplaced yes)
+		(property "Reference" "#PWR019"
+			(at 74.93 172.72 0)
+			(effects
+				(font
+					(size 1.27 1.27)
+				)
+				(hide yes)
+			)
+		)
+		(property "Value" "VCC"
+			(at 74.93 163.83 0)
+			(effects
+				(font
+					(size 1.27 1.27)
+				)
+			)
+		)
+		(property "Footprint" ""
+			(at 74.93 168.91 0)
+			(effects
+				(font
+					(size 1.27 1.27)
+				)
+				(hide yes)
+			)
+		)
+		(property "Datasheet" ""
+			(at 74.93 168.91 0)
+			(effects
+				(font
+					(size 1.27 1.27)
+				)
+				(hide yes)
+			)
+		)
+		(property "Description" "Power symbol creates a global label with name \"VCC\""
+			(at 74.93 168.91 0)
+			(effects
+				(font
+					(size 1.27 1.27)
+				)
+				(hide yes)
+			)
+		)
+		(pin "1"
+		)
+		(instances
+			(project "PROGRAMMER"
+				(path "/c3d4d3ca-3b0c-4b66-9122-b6670ae5401e/f80a6ea3-817f-470e-88f7-47e64e60582d"
+					(reference "#PWR019")
+					(unit 1)
+				)
+			)
+		)
+	)
+	(symbol
+		(lib_id "power:VCC")
+		(at 134.62 127 0)
+		(unit 1)
+		(exclude_from_sim no)
+		(in_bom yes)
+		(on_board yes)
+		(dnp no)
+		(fields_autoplaced yes)
+		(property "Reference" "#PWR020"
+			(at 134.62 130.81 0)
+			(effects
+				(font
+					(size 1.27 1.27)
+				)
+				(hide yes)
+			)
+		)
+		(property "Value" "VCC"
+			(at 134.62 121.92 0)
+			(effects
+				(font
+					(size 1.27 1.27)
+				)
+			)
+		)
+		(property "Footprint" ""
+			(at 134.62 127 0)
+			(effects
+				(font
+					(size 1.27 1.27)
+				)
+				(hide yes)
+			)
+		)
+		(property "Datasheet" ""
+			(at 134.62 127 0)
+			(effects
+				(font
+					(size 1.27 1.27)
+				)
+				(hide yes)
+			)
+		)
+		(property "Description" "Power symbol creates a global label with name \"VCC\""
+			(at 134.62 127 0)
+			(effects
+				(font
+					(size 1.27 1.27)
+				)
+				(hide yes)
+			)
+		)
+		(pin "1"
+		)
+		(instances
+			(project "PROGRAMMER"
+				(path "/c3d4d3ca-3b0c-4b66-9122-b6670ae5401e/f80a6ea3-817f-470e-88f7-47e64e60582d"
+					(reference "#PWR020")
+					(unit 1)
+				)
+			)
+		)
+	)
+	(symbol
 		(lib_id "Interface_USB:FT232RL")
 		(at 90.17 91.44 0)
@@
 			)
 		)
-		(property "Footprint" "Package_SO:SSOP-28_5.3x10.2mm_P0.65mm"
+		(property "Footprint" "Package_DIP:DIP-28_W7.62mm"
 			(at 118.11 114.3 0)
 			(effects
@@
 			)
 		)
-		(property "Footprint" "Inductor_SMD:L_Sunlord_SWPA8040S"
+		(property "Footprint" "LED_THT:LED_D1.8mm_W3.3mm_H2.4mm"
 			(at 86.36 162.56 0)
 			(effects
