File: ATMEGA-SCHEMATICS/SNAKE_GAME/PCB/snake_pcb/programmer.kicad_sch (KiCad schematic)
At the start: 23 parts, among them J2 Conn_02x05_Odd_Even, J5 Conn_01x03_Pin, U3 ATmega8A-P, U4 CD4066BE, U6 CD4066BE, U7 CD4066BE, Y1 Crystal

Commit message: ..
Parts:
- removed C2: C_Polarized, symbol Device:C_Polarized
- removed J2: Conn_02x05_Odd_Even, symbol Connector_Generic:Conn_02x05_Odd_Even
- removed R1: R, symbol Device:R
- added J11: EXT_ACC_PROG, symbol Connector_Generic:Conn_02x05_Odd_Even
- added SW1: PROG_SWT, Button_Switch_SMD:Nidec_Copal_CAS-120A, symbol Switch:SW_Nidec_CAS-120A1
Connections:
- net EXT_PROG: now also SW1.2 (B)
- net GND: now also J11.10 (Pin_10), J11.3 (Pin_3), J11.4 (Pin_4), J11.6 (Pin_6), J11.8 (Pin_8), SW1.1 (C)
- net MISO: now also J11.9 (Pin_9)
- net MOSI: now also J11.1 (Pin_1)
- net RESET_PROG: now also J11.5 (Pin_5)
- net SCK: now also J11.7 (Pin_7)
- net VCC: now also U3.21 (AREF), J11.2 (Pin_2), SW1.3 (A)
- no-connect marks 9 -> 17

Commit message: .
Parts:
- added J21: Conn_01x04_Pin, symbol Connector:Conn_01x04_Pin
- added J22, J23: Conn_01x06_Pin, symbol Connector:Conn_01x06_Pin
- added J24: Conn_01x05_Pin, symbol Connector:Conn_01x05_Pin
- added R22: 10K, symbol Device:R
Connections:
- net EXT_PROG: now also J23.3 (Pin_3)
- net FLASH_CS: now also J22.6 (Pin_6)
- net GAME_CS: now also J22.5 (Pin_5)
- net GAME_PROG: now also J23.2 (Pin_2)
- net GRID_CS: now also J22.4 (Pin_4)
- net GRID_PROG: now also J23.1 (Pin_1)
- net MISO: now also J24.4 (Pin_4)
- net MOSI: now also J24.3 (Pin_3)
- net RESET_PROG: now also J22.1 (Pin_1)
- net RXD_PROG: now also J22.2 (Pin_2)
- net SCK: now also J24.5 (Pin_5)
- net SRAM_CS: now also J21.1 (Pin_1)
- net TXD_PROG: now also J22.3 (Pin_3)
- net VCC: now also R22.1
- net PD6: now reaches U3.12 (PD6)
- net PD6: now also J21.2 (Pin_2)
- net PD7: now reaches U3.13 (PD7)
- net PD7: now also J21.3 (Pin_3)
- net PB0: now reaches U3.14 (PB0)
- net PB0: now also J21.4 (Pin_4)
- net PB1: now reaches U3.15 (PB1)
- net PB1: now also J24.1 (Pin_1)
- net PB2: now reaches U3.16 (PB2)
- net PB2: now also J24.2 (Pin_2), R22.2
- net PC3: now reaches U3.26 (PC3)
- net PC3: now also J23.4 (Pin_4)
- net PC4: now reaches U3.27 (PC4)
- net PC4: now also J23.5 (Pin_5)
- net PC5: now reaches U3.28 (PC5)
- net PC5: now also J23.6 (Pin_6)
- no-connect marks 17 -> 9

Commit message: .
Parts:
- added J1: Conn_01x02_Pin, Connector_PinSocket_2.54mm:PinSocket_1x02_P2.54mm_Vertical, symbol Connector:Conn_01x02_Pin
- added J25: Conn_01x02_Pin, Connector_PinHeader_2.54mm:PinHeader_1x02_P2.54mm_Vertical, symbol Connector:Conn_01x02_Pin
- added R35: 10K, Resistor_THT:R_Axial_DIN0207_L6.3mm_D2.5mm_P10.16mm_Horizontal, symbol Device:R
- added SW4: SW_Push, Button_Switch_THT:SW_PUSH_1P1T_6x3.5mm_H4.3_APEM_MJTP1243, symbol Switch:SW_Push
- C1, C3: value C -> 22pF; footprint (none) -> Capacitor_THT:CP_Radial_D5.0mm_P2.50mm
- C14, C15, C16, C4, C5, C6, C7, C8, C9: footprint (none) -> Capacitor_THT:C_Disc_D7.5mm_W5.0mm_P5.00mm
- J11: footprint (none) -> Connector_IDC:IDC-Header_2x05_P2.54mm_Vertical
- J21: footprint (none) -> Connector_PinHeader_2.54mm:PinHeader_1x04_P2.54mm_Vertical
- J22, J23: footprint (none) -> Connector_PinHeader_2.54mm:PinHeader_1x06_P2.54mm_Vertical
- J24: footprint (none) -> Connector_PinHeader_2.54mm:PinHeader_1x05_P2.54mm_Vertical
- J5: footprint (none) -> Connector_PinSocket_2.54mm:PinSocket_1x03_P2.54mm_Vertical
- R2, R22, R3, R6: footprint (none) -> Resistor_THT:R_Axial_DIN0207_L6.3mm_D2.5mm_P10.16mm_Horizontal
- SW1: footprint Button_Switch_SMD:Nidec_Copal_CAS-120A -> Button_Switch_THT:SW_Slide_SPDT_Straight_CK_OS102011MS2Q
- Y1: footprint (none) -> Crystal:Resonator-2Pin_W6.0mm_H3.0mm
Connections:
- net PD7 is gone; now on net FLASH_CS: J21.3 (Pin_3), U3.13 (PD7)
- net FLASH_CS: no longer U3.6 (PD4)
- net GND: now also SW4.2
- net MISO: no longer J11.9 (Pin_9)
- net MISO_EXT: now also J11.9 (Pin_9)
- net MOSI: no longer J11.1 (Pin_1)
- net MOSI_EXT: now also J11.1 (Pin_1)
- net RESET_PROG: now also R35.2, SW4.1
- net RXD_PROG: now also J1.2 (Pin_2); no longer J22.2 (Pin_2), U3.2 (PD0)
- net SCK: no longer J11.7 (Pin_7)
- net SCK_EXT: now also J11.7 (Pin_7)
- net TXD_PROG: now also J25.2 (Pin_2); no longer J22.3 (Pin_3), U3.3 (PD1)
- net VCC: now also R35.1
- net EXT_PROG renamed EXT_SIGNAL
- net GAME_PROG renamed GAME_SIGNAL
- net GRID_PROG renamed GRID_SIGNAL
- net PC3 renamed CTS_PROG
- net PC4 renamed RTS_PROG
- net PD6 renamed I/O_CONVERTER
- new net RXD: J1.1 (Pin_1), J22.2 (Pin_2), U3.2 (PD0)
- new net TXD: J22.3 (Pin_3), J25.1 (Pin_1), U3.3 (PD1)
- new net XCK: U3.6 (PD4)
