File: ATMEGA-SCHEMATICS/SNAKE_GAME/PCB/snake_pcb/game.kicad_sch (KiCad schematic)
At the start: 24 parts, among them J10 LCD_SCREEN, J6 TERM_GAME, J8 Conn_01x03_Pin, J9 Conn_01x05_Pin, U2 ATmega168A-P, Y2 Crystal

Commit message: ..
Connections:
- no-connect marks 1 -> 4
Changed lines of the file:
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@@
 		(at 160.02 59.69)
+	)
+	(no_connect
+		(at 160.02 82.55)
+	)
+	(no_connect
+		(at 160.02 85.09)
+	)
+	(no_connect
+		(at 160.02 80.01)
 	)
 	(wire

Commit message: .
Parts:
- added J14: Conn_01x05_Pin, symbol Connector:Conn_01x05_Pin
- added J15: Conn_01x04_Pin, symbol Connector:Conn_01x04_Pin
- added J17, J19: Conn_01x06_Pin, symbol Connector:Conn_01x06_Pin
- added R1: 10K, symbol Device:R
Connections:
- net B_SELECT: now also J19.6 (Pin_6)
- net B_START: now also J15.2 (Pin_2)
- net B_STOP: now also J15.3 (Pin_3)
- net FLASH_CS: now also J14.1 (Pin_1)
- net FLASH_HOLD: now also J15.4 (Pin_4)
- net J_DOWN: now also J17.5 (Pin_5)
- net J_LEFT: now also J17.6 (Pin_6)
- net J_RIGHT: now also J15.1 (Pin_1)
- net J_UP: now also J17.4 (Pin_4)
- net MISO_GAME: now also J14.4 (Pin_4)
- net MOSI_GAME: now also J14.3 (Pin_3)
- net RESET_GAME: now also J17.1 (Pin_1)
- net RXD_GAME: now also J17.2 (Pin_2)
- net SCK_GAME: now also J14.5 (Pin_5)
- net SCL_GAME: now also J19.1 (Pin_1)
- net SDA_GAME: now also J19.2 (Pin_2)
- net TXD_GAME: now also J17.3 (Pin_3)
- net VCC: now also R1.1
- net PB2: now reaches U2.16 (PB2)
- net PB2: now also J14.2 (Pin_2), R1.2
- net PC1: now reaches U2.24 (PC1)
- net PC1: now also J19.5 (Pin_5)
- net PC2: now reaches U2.25 (PC2)
- net PC2: now also J19.4 (Pin_4)
- net PC3: now reaches U2.26 (PC3)
- net PC3: now also J19.3 (Pin_3)
- no-connect marks 4 -> 0

Commit message: ...
Parts:
- added C29: 4.7uF, symbol Device:C
- added C30, C32, C33, C34, C35, C36, C37, C38, C39: 100nF, symbol Device:C
- added CS_HOLD_SHIFTER, MISO_SHIFTER, MOSI_CLK_SHIFTER, WP_SHIFTER: ~, symbol lucasLib:SN74LXC2T45
- added R24, R25, R26: 10K, symbol Device:R
- added U8: MX25L3233FM1, Package_SO:SOP-8_3.9x4.9mm_P1.27mm, symbol Memory_Flash:MX25L3233FM1
Connections:
- net FLASH_CS: now also CS_HOLD_SHIFTER.2 (A1)
- net FLASH_HOLD: now also CS_HOLD_SHIFTER.3 (A3)
- net GND: now also C29.2, C30.2, C32.2, C33.2, C34.2, C35.2, C36.2, C37.2, C38.2, C39.2, CS_HOLD_SHIFTER.4 (GND), MISO_SHIFTER.4 (GND), MOSI_CLK_SHIFTER.4 (GND), R24.2, R26.2, U8.4 (GND), WP_SHIFTER.4 (GND)
- net MISO_GAME: now also MISO_SHIFTER.2 (A1)
- net MOSI_GAME: now also MOSI_CLK_SHIFTER.2 (A1)
- net SCK_GAME: now also MOSI_CLK_SHIFTER.3 (A3)
- net VCC: now also C29.1, C30.1, R25.2, U8.8 (VCC)
- net PC1 renamed FLASH_WP
- net FLASH_WP: now also WP_SHIFTER.2 (A1)
- new net: C38.1, WP_SHIFTER.1 (VCCA)
- new net: C32.1, MISO_SHIFTER.1 (VCCA)
- new net: C36.1, MOSI_CLK_SHIFTER.1 (VCCA)
- new net: C37.1, CS_HOLD_SHIFTER.1 (VCCA)
- new net 3.3V: C33.1, C34.1, C35.1, C39.1, CS_HOLD_SHIFTER.8 (VCCB), MISO_SHIFTER.8 (VCCB), MOSI_CLK_SHIFTER.8 (VCCB), WP_SHIFTER.8 (VCCB)
- new net CS: CS_HOLD_SHIFTER.7 (B1), R25.1, U8.1 (~{CS})
- new net HOLD: CS_HOLD_SHIFTER.6 (B2), R24.1, U8.7 (~{HOLD}/SIO3)
- new net MISO: MISO_SHIFTER.7 (B1), U8.2 (SO/SIO1)
- new net MOSI: MOSI_CLK_SHIFTER.7 (B1), U8.5 (SI/SIO0)
- new net SCK: MOSI_CLK_SHIFTER.6 (B2), U8.6 (SCLK)
- new net WP: R26.1, U8.3 (~{WP}/SIO2), WP_SHIFTER.7 (B1)
- no-connect marks 0 -> 4
Other:
- note added: "EXTERNAL_FLASH"
- note added: "GPIO_ACCESS"
- note added: "LCD_SCREEN"
- note added: "TERMINAL ACCESS"
- moved on the sheet: J10, J14, J15, J17, J19, J6

Commit message: .
Parts:
- removed J8: Conn_01x03_Pin, symbol Connector:Conn_01x03_Pin
- added J26: B_START, Connector_PinHeader_2.54mm:PinHeader_1x02_P2.54mm_Vertical, symbol Connector:Conn_01x02_Pin
- added J27: B_STOP, Connector_PinHeader_2.54mm:PinHeader_1x02_P2.54mm_Vertical, symbol Connector:Conn_01x02_Pin
- added J28: B_SELECT, Connector_PinHeader_2.54mm:PinHeader_1x02_P2.54mm_Vertical, symbol Connector:Conn_01x02_Pin
- added R27, R29: 10K, Resistor_THT:R_Axial_DIN0207_L6.3mm_D2.5mm_P10.16mm_Horizontal, symbol Device:R
- added SW3: SW_Push, Button_Switch_THT:SW_PUSH_1P1T_6x3.5mm_H4.3_APEM_MJTP1243, symbol Switch:SW_Push
- C17, C18: value C -> 22pF; footprint (none) -> Capacitor_THT:CP_Radial_D5.0mm_P2.50mm
- C19, C20, C21, C22, C29, C30, C32, C33, C34, C35, C36, C37, C38, C39: footprint (none) -> Capacitor_THT:C_Disc_D7.5mm_W5.0mm_P5.00mm
- CS_HOLD_SHIFTER1: renamed from CS_HOLD_SHIFTER; footprint (none) -> Package_DIP:DIP-8_W7.62mm
- J10: footprint (none) -> Connector_PinSocket_2.54mm:PinSocket_1x04_P2.54mm_Vertical
- J14: footprint (none) -> Connector_PinHeader_2.54mm:PinHeader_1x05_P2.54mm_Vertical
- J15: footprint (none) -> Connector_PinHeader_2.54mm:PinHeader_1x04_P2.54mm_Vertical
- J17, J19: footprint (none) -> Connector_PinHeader_2.54mm:PinHeader_1x06_P2.54mm_Vertical
- J6: footprint (none) -> Connector_PinSocket_2.54mm:PinSocket_1x03_P2.54mm_Vertical
- J9: footprint (none) -> Connector_PinSocket_2.54mm:PinSocket_1x05_P2.54mm_Vertical
- MISO_SHIFTER1: renamed from MISO_SHIFTER; footprint (none) -> Package_DIP:DIP-8_W7.62mm
- MOSI_CLK_SHIFTER1: renamed from MOSI_CLK_SHIFTER; footprint (none) -> Package_DIP:DIP-8_W7.62mm
- R1, R10, R11, R12, R13, R14, R15, R16, R17, R18, R24, R25, R26, R7, R8, R9: footprint (none) -> Resistor_THT:R_Axial_DIN0207_L6.3mm_D2.5mm_P10.16mm_Horizontal
- U8: footprint Package_SO:SOP-8_3.9x4.9mm_P1.27mm -> Package_DIP:CERDIP-8_W7.62mm_SideBrazed_Socket
- WP_SHIFTER1: renamed from WP_SHIFTER; footprint (none) -> Package_DIP:DIP-8_W7.62mm
- Y2: footprint (none) -> Crystal:Resonator-2Pin_W6.0mm_H3.0mm
Connections:
- net B_SELECT: now also R11.1, J28.1 (Pin_1); no longer R11.2
- net B_START: now also R13.1, J26.1 (Pin_1); no longer R13.2
- net B_STOP: now also R12.1, J27.1 (Pin_1); no longer R12.2
- net GND: now also J26.2 (Pin_2), J27.2 (Pin_2), J28.2 (Pin_2), SW3.2
- net J_DOWN: now also J9.2 (Pin_2), R14.1; no longer R14.2
- net J_LEFT: now also J9.3 (Pin_3), R15.1; no longer R15.2
- net J_RIGHT: now also J9.4 (Pin_4), R16.1; no longer R16.2
- net J_UP: now also J9.1 (Pin_1), R10.1; no longer R10.2
- net PC2: now also CS_HOLD_SHIFTER1.5 (DIR), MOSI_CLK_SHIFTER1.5 (DIR), WP_SHIFTER1.5 (DIR), R27.2
- net PC3: now also MISO_SHIFTER1.5 (DIR), R29.2
- net RESET_GAME: now also SW3.1
- net VCC: now also R10.2, R11.2, R12.2, R13.2, R14.2, R15.2, R16.2, R27.1, R29.1
Other:
- moved on the sheet: R10, R11, R12, R13, R14, R15, R16

Commit message: .
Parts:
- added BZ1: Buzzer, symbol Device:Buzzer
- added J8: Vibrator, Connector_PinHeader_2.54mm:PinHeader_1x02_P2.54mm_Vertical, symbol Connector:Conn_01x02_Pin
- added R40, R41: 200, Resistor_THT:R_Axial_DIN0207_L6.3mm_D2.5mm_P10.16mm_Horizontal, symbol Device:R
Connections:
- net GND: now also R40.2, R41.2
- net J_RIGHT: now also J19.4 (Pin_4), U2.25 (PC2); no longer U2.11 (PD5)
- net PC2: no longer J19.4 (Pin_4), U2.25 (PC2)
- net PC3: no longer J19.3 (Pin_3), U2.26 (PC3)
- new net: J8.1 (Pin_1), R41.1
- new net: BZ1.2 (-), R40.1
- new net BUZZER_PWM: BZ1.1 (+), U2.11 (PD5)
- new net VIBRATOR: J19.3 (Pin_3), J8.2 (Pin_2), U2.26 (PC3)
