File: ATMEGA-SCHEMATICS/SNAKE_GAME/PCB/snake_pcb/game.kicad_sch (KiCad schematic)
At the start: 60 parts, among them J10 LCD_SCREEN, J14 Conn_01x05_Pin, J15 Conn_01x04_Pin, J17 Conn_01x06_Pin, J19 Conn_01x06_Pin, J26 B_START, J27 B_STOP, J28 B_SELECT, J6 TERM_GAME, J8 Vibrator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

Commit message: .
Parts:
- C19, C29: footprint Capacitor_SMD:C_0805_2012Metric -> Capacitor_THT:C_Disc_D7.5mm_W5.0mm_P5.00mm
- C20, C21, C22, C30, C32, C33, C34, C35, C36, C37, C38, C39: footprint Capacitor_SMD:C_0402_1005Metric -> Capacitor_THT:C_Disc_D7.5mm_W5.0mm_P5.00mm
Connections:
- net 3.3V: now also C29.1, C30.1, R25.2, U8.8 (VCC)
- net VCC: now also C32.1, C36.1, C37.1, C38.1, CS_HOLD_SHIFTER1.1 (VCCA), MISO_SHIFTER1.1 (VCCA), MOSI_CLK_SHIFTER1.1 (VCCA), WP_SHIFTER1.1 (VCCA); no longer C29.1, C30.1, R25.2, U8.8 (VCC)
