File: ATMEGA-SCHEMATICS/SNAKE_GAME/PCB/snake_pcb/power.kicad_sch (KiCad schematic)
At the start: 33 parts, among them J4 Barrel_Jack_Switch, U9 AMS1117-3.3

Commit message: .
Parts:
- C2: footprint Capacitor_SMD:C_0402_1005Metric -> Capacitor_THT:C_Disc_D7.5mm_W5.0mm_P5.00mm
- C44, C45, C46, C48, C77: footprint Capacitor_SMD:C_0805_2012Metric -> Capacitor_THT:C_Disc_D7.5mm_W5.0mm_P5.00mm
Changed lines of the file:
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@@
 	)
 	(junction
-		(at 71.12 76.2)
+		(at 62.23 49.53)
 		(diameter 0)
 		(color 0 0 0 0)
@@
 	)
 	(junction
-		(at 68.58 50.8)
-		(diameter 0)
-		(color 0 0 0 0)
-	)
-	(junction
 		(at 250.19 151.13)
 		(diameter 0)
@@
 	(wire
 		(pts
-			(xy 71.12 72.39) (xy 71.12 76.2)
-		)
-		(stroke
-			(width 0)
-			(type default)
-		)
-	)
-	(wire
-		(pts
 			(xy 57.15 160.02) (xy 57.15 166.37)
 		)
@@
 	(wire
 		(pts
-			(xy 68.58 50.8) (xy 82.55 50.8)
+			(xy 66.04 50.8) (xy 82.55 50.8)
 		)
 		(stroke
@@
 	(wire
 		(pts
-			(xy 63.5 50.8) (xy 60.96 48.26)
+			(xy 63.5 50.8) (xy 62.23 49.53)
 		)
 		(stroke
@@
 	(wire
 		(pts
-			(xy 66.04 50.8) (xy 68.58 50.8)
-		)
-		(stroke
-			(width 0)
-			(type default)
-		)
-	)
-	(wire
-		(pts
 			(xy 74.93 43.18) (xy 82.55 43.18)
 		)
@@
 	(wire
 		(pts
+			(xy 62.23 49.53) (xy 60.96 48.26)
+		)
+		(stroke
+			(width 0)
+			(type default)
+		)
+	)
+	(wire
+		(pts
 			(xy 53.34 43.18) (xy 57.15 43.18)
 		)
@@
 		)
 	)
-	(global_label "3.3V"
-		(shape output)
-		(at 71.12 72.39 90)
+	(global_label "REG_EN_LOW"
+		(shape input)
+		(at 209.55 137.16 90)
 		(fields_autoplaced yes)
 		(effects
@@
 		)
 		(property "Intersheetrefs" "${INTERSHEET_REFS}"
-			(at 71.12 65.2924 90)
+			(at 209.55 122.2611 90)
 			(effects
 				(font
@@
 		)
 	)
-	(global_label "REG_EN_LOW"
-		(shape input)
-		(at 209.55 137.16 90)
+	(global_label "3.3V"
+		(shape output)
+		(at 69.85 76.2 90)
 		(fields_autoplaced yes)
 		(effects
@@
 		)
 		(property "Intersheetrefs" "${INTERSHEET_REFS}"
-			(at 209.55 122.2611 90)
+			(at 69.85 69.1024 90)
 			(effects
 				(font
@@
 			)
 		)
-		(property "Footprint" "Capacitor_SMD:C_0805_2012Metric"
+		(property "Footprint" "Capacitor_THT:C_Disc_D7.5mm_W5.0mm_P5.00mm"
 			(at 72.0852 83.82 0)
 			(effects
@@
 	)
 	(symbol
-		(lib_id "power:PWR_FLAG")
-		(at 68.58 50.8 180)
-		(unit 1)
-		(exclude_from_sim no)
-		(in_bom yes)
-		(on_board yes)
-		(dnp no)
-		(fields_autoplaced yes)
-		(property "Reference" "#FLG03"
-			(at 68.58 52.705 0)
-			(effects
-				(font
-					(size 1.27 1.27)
-				)
-				(hide yes)
-			)
-		)
-		(property "Value" "PWR_FLAG"
-			(at 68.58 55.88 0)
-			(effects
-				(font
-					(size 1.27 1.27)
-				)
-			)
-		)
-		(property "Footprint" ""
-			(at 68.58 50.8 0)
-			(effects
-				(font
-					(size 1.27 1.27)
-				)
-				(hide yes)
-			)
-		)
-		(property "Datasheet" "~"
-			(at 68.58 50.8 0)
-			(effects
-				(font
-					(size 1.27 1.27)
-				)
-				(hide yes)
-			)
-		)
-		(property "Description" "Special symbol for telling ERC where power comes from"
-			(at 68.58 50.8 0)
-			(effects
-				(font
-					(size 1.27 1.27)
-				)
-				(hide yes)
-			)
-		)
-		(pin "1"
-		)
-		(instances
-			(project "snake_pcb"
-				(path "/071b2fc6-d65a-411c-93b6-4a9f90a11c3f/f45a2180-d4ef-4236-8e82-25b6011e1113"
-					(reference "#FLG03")
-					(unit 1)
-				)
-			)
-		)
-	)
-	(symbol
 		(lib_id "Device:R")
 		(at 74.93 31.75 180)
@@
 	)
 	(symbol
+		(lib_id "power:PWR_FLAG")
+		(at 62.23 49.53 180)
+		(unit 1)
+		(exclude_from_sim no)
+		(in_bom yes)
+		(on_board yes)
+		(dnp no)
+		(fields_autoplaced yes)
+		(property "Reference" "#FLG03"
+			(at 62.23 51.435 0)
+			(effects
+				(font
+					(size 1.27 1.27)
+				)
+				(hide yes)
+			)
+		)
+		(property "Value" "PWR_FLAG"
+			(at 62.23 54.61 0)
+			(effects
+				(font
+					(size 1.27 1.27)
+				)
+			)
+		)
+		(property "Footprint" ""
+			(at 62.23 49.53 0)
+			(effects
+				(font
+					(size 1.27 1.27)
+				)
+				(hide yes)
+			)
+		)
+		(property "Datasheet" "~"
+			(at 62.23 49.53 0)
+			(effects
+				(font
+					(size 1.27 1.27)
+				)
+				(hide yes)
+			)
+		)
+		(property "Description" "Special symbol for telling ERC where power comes from"
+			(at 62.23 49.53 0)
+			(effects
+				(font
+					(size 1.27 1.27)
+				)
+				(hide yes)
+			)
+		)
+		(pin "1"
+		)
+		(instances
+			(project "snake_pcb"
+				(path "/071b2fc6-d65a-411c-93b6-4a9f90a11c3f/f45a2180-d4ef-4236-8e82-25b6011e1113"
+					(reference "#FLG03")
+					(unit 1)
+				)
+			)
+		)
+	)
+	(symbol
 		(lib_id "Device:C")
 		(at 120.65 151.13 0)
@@
 			)
 		)
-		(property "Footprint" "Capacitor_SMD:C_0805_2012Metric"
+		(property "Footprint" "Capacitor_THT:C_Disc_D7.5mm_W5.0mm_P5.00mm"
 			(at 121.6152 154.94 0)
 			(effects
@@
 			)
 		)
-		(property "Footprint" "Capacitor_SMD:C_0805_2012Metric"
+		(property "Footprint" "Capacitor_THT:C_Disc_D7.5mm_W5.0mm_P5.00mm"
 			(at 44.1452 83.82 0)
 			(effects
@@
 			)
 		)
-		(property "Footprint" "Capacitor_SMD:C_0805_2012Metric"
+		(property "Footprint" "Capacitor_THT:C_Disc_D7.5mm_W5.0mm_P5.00mm"
 			(at 210.5152 154.94 0)
 			(effects
@@
 			)
 		)
-		(property "Footprint" "Capacitor_SMD:C_0805_2012Metric"
+		(property "Footprint" "Capacitor_THT:C_Disc_D7.5mm_W5.0mm_P5.00mm"
 			(at 37.7952 154.94 0)
 			(effects
@@
 			)
 		)
-		(property "Footprint" "Capacitor_SMD:C_0402_1005Metric"
+		(property "Footprint" "Capacitor_THT:C_Disc_D7.5mm_W5.0mm_P5.00mm"
 			(at 67.0052 43.18 0)
 			(effects
