File: ATMEGA-SCHEMATICS/SNAKE_GAME/PCB/snake_pcb/snake_pcb.kicad_sch (KiCad schematic)
At the start: 1 part, among them J1 USB_A

Commit message: ...
Parts:
- removed J1: USB_A, symbol Connector:USB_A
Changed lines of the file:
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@@
 	(generator_version "9.0")
 	(paper "A4")
-	(symbol
-		(lib_id "Connector:USB_A")
-		(at 71.12 45.72 0)
-		(unit 1)
-		(exclude_from_sim no)
-		(in_bom yes)
-		(on_board yes)
-		(dnp no)
-		(fields_autoplaced yes)
-		(property "Reference" "J1"
-			(at 71.12 33.02 0)
-			(effects
-				(font
-					(size 1.27 1.27)
-				)
-			)
-		)
-		(property "Value" "USB_A"
-			(at 71.12 35.56 0)
-			(effects
-				(font
-					(size 1.27 1.27)
-				)
-			)
-		)
-		(property "Footprint" ""
-			(at 74.93 46.99 0)
-			(effects
-				(font
-					(size 1.27 1.27)
-				)
-				(hide yes)
-			)
-		)
-		(property "Datasheet" "~"
-			(at 74.93 46.99 0)
-			(effects
-				(font
-					(size 1.27 1.27)
-				)
-				(hide yes)
-			)
-		)
-		(property "Description" "USB Type A connector"
-			(at 71.12 45.72 0)
-			(effects
-				(font
-					(size 1.27 1.27)
-				)
-				(hide yes)
-			)
-		)
-		(pin "5"
-		)
-		(pin "4"
-		)
-		(pin "1"
-		)
-		(pin "3"
-		)
-		(pin "2"
-		)
-		(instances
-			(project ""
-				(path "/071b2fc6-d65a-411c-93b6-4a9f90a11c3f"
-					(reference "J1")
-					(unit 1)
-				)
-			)
-		)
-	)
 	(sheet
 		(at 190.5 85.09)
@@
 	)
 	(sheet
-		(at 144.78 38.1)
+		(at 21.59 25.4)
 		(size 21.59 25.4)
 		(exclude_from_sim no)
@@
 		)
 		(property "Sheetname" "power"
-			(at 144.78 37.3884 0)
+			(at 21.59 24.6884 0)
 			(effects
 				(font
@@
 		)
 		(property "Sheetfile" "power.kicad_sch"
-			(at 144.78 64.0846 0)
+			(at 21.59 51.3846 0)
 			(effects
 				(font

Commit message: .
Other:
- sheet converter ports: added CLOCK, CTS_CONV, RTS_CONV, RXD_CONV, TXD_CONV, WAKE_UP; removed none
- sheet game ports: added FLASH_CS, MISO_GAME, MOSI_GAME, RESET_GAME, SCK_GAME, SCL_GAME, SDA_GAME; removed none
- sheet grid ports: added MISO_GRID, MOSI_GRID, RESET_GRID, SCK_GRID, SCL_GRID, SDA_GRID, SRAM_CS; removed none
- sheet programmer ports: added CTS_PROG, FLASH_CS, GAME_CS, GRID_CS, I/O_CONVERTER, MISO_GAME, MISO_GRID, MOSI_GAME, MOSI_GRID, RTS_PROG, RXD_PROG, SCK_GAME, SCK_GRID, SRAM_CS, TXD_PROG, XCK; removed none

Commit message: .
Parts:
- added H1, H2, H3, H4, H5, H6: MountingHole, MountingHole:MountingHole_2.1mm, symbol Mechanical:MountingHole
