File: ATMEGA-SCHEMATICS/SNAKE_GAME/PCB/snake_pcb/snake_pcb.kicad_pcb (KiCad board)
At the start: 2 copper layers, 240 x 195 mm, 170 parts, among them J1 Conn_01x02_Pin, J10 LCD_SCREEN, J11 EXT_ACC_PROG, J12 JUMPER, J13 Conn_01x04_Pin, J14 Conn_01x05_Pin, J15 Conn_01x04_Pin, J16 Conn_01x06_Pin, J17 Conn_01x06_Pin, J18 Conn_01x05_Pin, J19 Conn_01x06_Pin, J20 Conn_01x06_Pin, J21 Conn_01x04_Pin, J22 Conn_01x06_Pin, J23 Conn_01x06_Pin, J24 Conn_01x05_Pin, J25 Conn_01x02_Pin, J26 B_START, J27 B_STOP, J28 B_SELECT, J29 GRID, J3 USB_A, J4 Barrel_Jack_Switch, J5 Conn_01x03_Pin, J6 TERM_GAME, J7 TERM_GRID, J8 Vibrator, J9 Conn_01x05_Pin, SW1 PROG_SWT, SW2 SW_Push, SW3 SW_Push, SW4 SW_Push, SW5 SW_Push, U1 ATmega168A-P, U10 PCF8574AP, U2 ATmega168A-P, U3 ATmega8A-P, U4 CD4066BE, U5 FT232RL, U6 CD4066BE, U7 CD4066BE, U8 MX25L3233FM1, U9 AMS1117-3.3, Y1 Crystal, Y2 Crystal, Y3 Crystal

Commit message: .
Parts:
- moved 220uF1 353.6 mm to (383.0, 186.3)
- moved 23A1024/23LC1 353.6 mm to (287.9, 142.1)
- moved 4.7uF1 353.6 mm to (374.8, 185.5)
- moved 47uF1 353.6 mm to (175.8, 155.5)
- moved 47uF2 353.6 mm to (175.2, 125.7)
- moved 47uF3 353.6 mm to (175.0, 183.8)
- moved BZ1 353.6 mm to (317.2, 297.0)
- moved C1 353.6 mm to (303.0, 158.5)
- moved C10 353.6 mm to (334.0, 254.0)
- moved C11 353.6 mm to (334.0, 248.5)
- moved C12 353.6 mm to (360.9, 268.2)
- moved C13 353.6 mm to (360.8, 274.3)
- moved C14 353.6 mm to (312.0, 214.0)
- moved C15 353.6 mm to (246.0, 214.5)
- moved C16 353.6 mm to (283.8, 213.7)
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Connections:
- J20 pad 5: /grid/PC1 -> REG_EN_LOW
- U1 pad 24: /grid/PC1 -> REG_EN_LOW
Routing:
- net REG_EN_LOW: track 130.9 -> 238.9 mm, vias 0 -> 1
- net /grid/PC1: track 6.55 -> 0.00 mm
