File: ATMEGA-SCHEMATICS/SNAKE_GAME/PCB/snake_pcb/grid.kicad_sch (KiCad schematic)
At the start: 12 parts, among them J7 TERM_GRID, U1 ATmega168A-P, Y3 Crystal

Commit message: ..
Parts:
- added J12: JUMPER, symbol Connector:Conn_01x02_Pin
- added J2: GRID, symbol Connector:Conn_01x03_Pin
Connections:
- net GND: now also J2.1 (Pin_1)
- net TXD_GRID: now also J12.2 (Pin_2)
- net USART_CLK: now reaches U1.6 (PD4)
- net USART_CLK: now also J2.3 (Pin_3)
- new net: J12.1 (Pin_1), J2.2 (Pin_2)
- no-connect marks 1 -> 6
Other:
- moved on the sheet: J7

Commit message: .
Parts:
- added J13: Conn_01x04_Pin, symbol Connector:Conn_01x04_Pin
- added J16, J20: Conn_01x06_Pin, symbol Connector:Conn_01x06_Pin
- added J18: Conn_01x05_Pin, symbol Connector:Conn_01x05_Pin
- added R21: 10K, symbol Device:R
Connections:
- net B_SELECT: now also J20.6 (Pin_6)
- net MISO_GAME: now also J18.4 (Pin_4)
- net MOSI_GAME: now also J18.3 (Pin_3)
- net RXD_GRID: now also J16.2 (Pin_2)
- net SCK_GAME: now also J18.5 (Pin_5)
- net SCL_GRID: now also J20.1 (Pin_1)
- net SDA_GRID: now also J20.2 (Pin_2)
- net TXD_GRID: now also J16.3 (Pin_3)
- net USART_CLK: now also J16.6 (Pin_6)
- net VCC: now also R21.1
- net PD5: now reaches U1.11 (PD5)
- net PD5: now also J13.1 (Pin_1)
- net PD6: now reaches U1.12 (PD6)
- net PD6: now also J13.2 (Pin_2)
- net PD7: now reaches U1.13 (PD7)
- net PD7: now also J13.3 (Pin_3)
- net PB2: now reaches U1.16 (PB2)
- net PB2: now also J18.2 (Pin_2), R21.2
- net PC1: now reaches U1.24 (PC1)
- net PC1: now also J20.5 (Pin_5)
- net PC2: now reaches U1.25 (PC2)
- net PC2: now also J20.4 (Pin_4)
- net PC3: now reaches U1.26 (PC3)
- net PC3: now also J20.3 (Pin_3)
- net PD2: now reaches U1.4 (PD2)
- net PD2: now also J16.4 (Pin_4)
- net PD3: now reaches U1.5 (PD3)
- net PD3: now also J16.5 (Pin_5)
- net FLASH_CS renamed SRAM_CS
- net SRAM_CS: now also J18.1 (Pin_1)
- net FLASH_HOLD renamed SRAM_HOLD
- net SRAM_HOLD: now also J13.4 (Pin_4)
- new net RESET_GAME: J16.1 (Pin_1)
- no-connect marks 6 -> 0

Commit message: .
Parts:
- added 23A1024/23LC1: ~, Package_DIP:CERDIP-8_W7.62mm_SideBrazed_Socket, symbol lucasLib:23A1024
- added C31: 4.7uF, Capacitor_THT:C_Disc_D7.5mm_W5.0mm_P5.00mm, symbol Device:C
- added C40: 100nF, Capacitor_THT:C_Disc_D7.5mm_W5.0mm_P5.00mm, symbol Device:C
- added C41: 100nF, Capacitor_THT:C_Disc_D7.5mm_W5.0mm_P5.00mm, symbol Device:C_Small
- added SW2: SW_Push, Button_Switch_THT:SW_PUSH_1P1T_6x3.5mm_H4.3_APEM_MJTP1243, symbol Switch:SW_Push
- C23, C24, C25, C26: footprint (none) -> Capacitor_THT:C_Disc_D7.5mm_W5.0mm_P5.00mm
- C27, C28: value C -> 22pF; footprint (none) -> Capacitor_THT:CP_Radial_D5.0mm_P2.50mm
- J12: footprint (none) -> Connector_PinHeader_2.54mm:PinHeader_1x02_P2.54mm_Vertical
- J13: footprint (none) -> Connector_PinHeader_2.54mm:PinHeader_1x04_P2.54mm_Vertical
- J16, J20: footprint (none) -> Connector_PinHeader_2.54mm:PinHeader_1x06_P2.54mm_Vertical
- J18: footprint (none) -> Connector_PinHeader_2.54mm:PinHeader_1x05_P2.54mm_Vertical
- J2: footprint (none) -> Connector_PinHeader_2.54mm:PinHeader_1x03_P2.54mm_Vertical
- J7: footprint (none) -> Connector_PinSocket_2.54mm:PinSocket_1x03_P2.54mm_Vertical
- R19, R20, R21, R23: footprint (none) -> Resistor_THT:R_Axial_DIN0207_L6.3mm_D2.5mm_P10.16mm_Horizontal
- Y3: footprint (none) -> Crystal:Resonator-2Pin_W6.0mm_H3.0mm
Connections:
- net RESET_GAME is gone; now on net RESET_GRID: J16.1 (Pin_1)
- net GND: now also 23A1024/23LC1.4 (GND), C31.1, C40.1, C41.2, SW2.2
- net RESET_GRID: now also SW2.1
- net SRAM_CS: now also 23A1024/23LC1.1 (CS)
- net SRAM_HOLD: now also 23A1024/23LC1.7 (HOLD/SIO3)
- net VCC: now also 23A1024/23LC1.8 (VCC), C31.2, C40.2
- net MISO_GAME renamed MISO_GRID
- net MISO_GRID: now also 23A1024/23LC1.2 (SO/SIO1)
- net MOSI_GAME renamed MOSI_GRID
- net MOSI_GRID: now also 23A1024/23LC1.5 (SI/SIO0)
- net SCK_GAME renamed SCK_GRID
- net SCK_GRID: now also 23A1024/23LC1.6 (SCK)
- new net: 23A1024/23LC1.3 (SIO2), C41.1

Commit message: ...
Parts:
- removed J2: GRID, Connector_PinHeader_2.54mm:PinHeader_1x03_P2.54mm_Vertical, symbol Connector:Conn_01x03_Pin
- added J29: GRID, Connector_PinHeader_2.54mm:PinHeader_1x04_P2.54mm_Vertical, symbol Connector:Conn_01x04_Pin
- C23, C31: footprint Capacitor_THT:C_Disc_D7.5mm_W5.0mm_P5.00mm -> Capacitor_SMD:C_0805_2012Metric
- C24, C25, C26, C40, C41: footprint Capacitor_THT:C_Disc_D7.5mm_W5.0mm_P5.00mm -> Capacitor_SMD:C_0402_1005Metric
Connections:
- net GND: now also J29.1 (Pin_1)
- net USART_CLK: now also J29.3 (Pin_3)
- net at J12.1 (Pin_1): now also J29.2 (Pin_2)
- new net VCC_LED_GRID: J29.4 (Pin_4)
Changed lines of the file:
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@@
+		)
+	)
+	(global_label "VCC_LED_GRID"
+		(shape input)
+		(at 237.49 115.57 90)
+		(fields_autoplaced yes)
+		(effects
+			(font
+				(size 1.27 1.27)
+			)
+			(justify left)
+		)
+		(property "Intersheetrefs" "${INTERSHEET_REFS}"
+			(at 237.49 99.1591 90)
+			(effects
+				(font
+					(size 1.27 1.27)
+				)
+				(justify left)
+				(hide yes)
+			)
 		)
 	)
@@
 	)
 	(symbol
+		(lib_id "Connector:Conn_01x04_Pin")
+		(at 242.57 120.65 180)
+		(unit 1)
+		(exclude_from_sim no)
+		(in_bom yes)
+		(on_board yes)
+		(dnp no)
+		(fields_autoplaced yes)
+		(property "Reference" "J29"
+			(at 243.84 118.1099 0)
+			(effects
+				(font
+					(size 1.27 1.27)
+				)
+				(justify right)
+			)
+		)
+		(property "Value" "GRID"
+			(at 243.84 120.6499 0)
+			(effects
+				(font
+					(size 1.27 1.27)
+				)
+				(justify right)
+			)
+		)
+		(property "Footprint" "Connector_PinHeader_2.54mm:PinHeader_1x04_P2.54mm_Vertical"
+			(at 242.57 120.65 0)
+			(effects
+				(font
+					(size 1.27 1.27)
+				)
+				(hide yes)
+			)
+		)
+		(property "Datasheet" "~"
+			(at 242.57 120.65 0)
+			(effects
+				(font
+					(size 1.27 1.27)
+				)
+				(hide yes)
+			)
+		)
+		(property "Description" "Generic connector, single row, 01x04, script generated"
+			(at 242.57 120.65 0)
+			(effects
+				(font
+					(size 1.27 1.27)
+				)
+				(hide yes)
+			)
+		)
+		(pin "1"
+		)
+		(pin "4"
+		)
+		(pin "2"
+		)
+		(pin "3"
+		)
+		(instances
+			(project ""
+				(path "/071b2fc6-d65a-411c-93b6-4a9f90a11c3f/5fd9a7fb-d9b8-4dd1-97f8-12c5ea1daca5"
+					(reference "J29")
+					(unit 1)
+				)
+			)
+		)
+	)
+	(symbol
 		(lib_id "Connector:Conn_01x02_Pin")
 		(at 214.63 107.95 270)
@@
 			)
 		)
-		(property "Footprint" "Capacitor_THT:C_Disc_D7.5mm_W5.0mm_P5.00mm"
+		(property "Footprint" "Capacitor_SMD:C_0402_1005Metric"
 			(at 119.0752 52.07 0)
 			(effects
@@
 			)
 		)
-		(property "Footprint" "Capacitor_THT:C_Disc_D7.5mm_W5.0mm_P5.00mm"
+		(property "Footprint" "Capacitor_SMD:C_0402_1005Metric"
 			(at 127.9652 52.07 0)
 			(effects
@@
 			)
 		)
-		(property "Footprint" "Capacitor_THT:C_Disc_D7.5mm_W5.0mm_P5.00mm"
+		(property "Footprint" "Capacitor_SMD:C_0402_1005Metric"
 			(at 201.93 62.23 0)
 			(effects
@@
 			)
 		)
-		(property "Footprint" "Capacitor_THT:C_Disc_D7.5mm_W5.0mm_P5.00mm"
+		(property "Footprint" "Capacitor_SMD:C_0805_2012Metric"
 			(at 227.6348 44.45 0)
 			(effects
@@
 	)
 	(symbol
-		(lib_id "Connector:Conn_01x03_Pin")
-		(at 242.57 120.65 180)
-		(unit 1)
-		(exclude_from_sim no)
-		(in_bom yes)
-		(on_board yes)
-		(dnp no)
-		(fields_autoplaced yes)
-		(property "Reference" "J2"
-			(at 243.84 119.3799 0)
-			(effects
-				(font
-					(size 1.27 1.27)
-				)
-				(justify right)
-			)
-		)
-		(property "Value" "GRID"
-			(at 243.84 121.9199 0)
-			(effects
-				(font
-					(size 1.27 1.27)
-				)
-				(justify right)
-			)
-		)
-		(property "Footprint" "Connector_PinHeader_2.54mm:PinHeader_1x03_P2.54mm_Vertical"
-			(at 242.57 120.65 0)
-			(effects
-				(font
-					(size 1.27 1.27)
-				)
-				(hide yes)
-			)
-		)
-		(property "Datasheet" "~"
-			(at 242.57 120.65 0)
-			(effects
-				(font
-					(size 1.27 1.27)
-				)
-				(hide yes)
-			)
-		)
-		(property "Description" "Generic connector, single row, 01x03, script generated"
-			(at 242.57 120.65 0)
-			(effects
-				(font
-					(size 1.27 1.27)
-				)
-				(hide yes)
-			)
-		)
-		(pin "1"
-		)
-		(pin "2"
-		)
-		(pin "3"
-		)
-		(instances
-			(project "snake_pcb"
-				(path "/071b2fc6-d65a-411c-93b6-4a9f90a11c3f/5fd9a7fb-d9b8-4dd1-97f8-12c5ea1daca5"
-					(reference "J2")
-					(unit 1)
-				)
-			)
-		)
-	)
-	(symbol
 		(lib_id "Device:C")
 		(at 105.41 55.88 0)
@@
 			)
 		)
-		(property "Footprint" "Capacitor_THT:C_Disc_D7.5mm_W5.0mm_P5.00mm"
+		(property "Footprint" "Capacitor_SMD:C_0402_1005Metric"
 			(at 106.3752 52.07 0)
 			(effects
@@
 			)
 		)
-		(property "Footprint" "Capacitor_THT:C_Disc_D7.5mm_W5.0mm_P5.00mm"
+		(property "Footprint" "Capacitor_SMD:C_0805_2012Metric"
 			(at 94.9452 52.07 0)
 			(effects
@@
 			)
 		)
-		(property "Footprint" "Capacitor_THT:C_Disc_D7.5mm_W5.0mm_P5.00mm"
+		(property "Footprint" "Capacitor_SMD:C_0402_1005Metric"
 			(at 216.2048 44.45 0)
 			(effects

Commit message: .
Parts:
- C23, C31: footprint Capacitor_SMD:C_0805_2012Metric -> Capacitor_THT:C_Disc_D7.5mm_W5.0mm_P5.00mm
- C24, C25, C26, C40, C41: footprint Capacitor_SMD:C_0402_1005Metric -> Capacitor_THT:C_Disc_D7.5mm_W5.0mm_P5.00mm
Changed lines of the file:
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@@
 			)
 		)
-		(property "Footprint" "Capacitor_SMD:C_0402_1005Metric"
+		(property "Footprint" "Capacitor_THT:C_Disc_D7.5mm_W5.0mm_P5.00mm"
 			(at 119.0752 52.07 0)
 			(effects
@@
 			)
 		)
-		(property "Footprint" "Capacitor_SMD:C_0402_1005Metric"
+		(property "Footprint" "Capacitor_THT:C_Disc_D7.5mm_W5.0mm_P5.00mm"
 			(at 127.9652 52.07 0)
 			(effects
@@
 			)
 		)
-		(property "Footprint" "Capacitor_SMD:C_0402_1005Metric"
+		(property "Footprint" "Capacitor_THT:C_Disc_D7.5mm_W5.0mm_P5.00mm"
 			(at 201.93 62.23 0)
 			(effects
@@
 			)
 		)
-		(property "Footprint" "Capacitor_SMD:C_0805_2012Metric"
+		(property "Footprint" "Capacitor_THT:C_Disc_D7.5mm_W5.0mm_P5.00mm"
 			(at 227.6348 44.45 0)
 			(effects
@@
 			)
 		)
-		(property "Footprint" "Capacitor_SMD:C_0402_1005Metric"
+		(property "Footprint" "Capacitor_THT:C_Disc_D7.5mm_W5.0mm_P5.00mm"
 			(at 106.3752 52.07 0)
 			(effects
@@
 			)
 		)
-		(property "Footprint" "Capacitor_SMD:C_0805_2012Metric"
+		(property "Footprint" "Capacitor_THT:C_Disc_D7.5mm_W5.0mm_P5.00mm"
 			(at 94.9452 52.07 0)
 			(effects
@@
 			)
 		)
-		(property "Footprint" "Capacitor_SMD:C_0402_1005Metric"
+		(property "Footprint" "Capacitor_THT:C_Disc_D7.5mm_W5.0mm_P5.00mm"
 			(at 216.2048 44.45 0)
 			(effects

Commit message: .
Connections:
- net PC1 renamed REG_EN_LOW
Changed lines of the file:
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@@
+	(wire
+		(pts
+			(xy 146.05 95.25) (xy 152.4 95.25)
+		)
+		(stroke
+			(width 0)
+			(type default)
+		)
+	)
 	(wire
 		(pts
@@
 		(pts
 			(xy 208.28 133.35) (xy 215.9 133.35)
+		)
+		(stroke
+			(width 0)
+			(type default)
+		)
+	)
+	(wire
+		(pts
+			(xy 92.71 115.57) (xy 100.33 115.57)
 		)
 		(stroke
@@
 		)
 	)
-	(label "PC1"
-		(at 92.71 115.57 0)
-		(effects
-			(font
-				(size 1.27 1.27)
-			)
-			(justify left bottom)
-		)
-	)
 	(label "PC2"
 		(at 92.71 113.03 0)
@@
 		)
 	)
-	(label "PC1"
-		(at 146.05 95.25 0)
-		(effects
-			(font
-				(size 1.27 1.27)
-			)
-			(justify left bottom)
-		)
-	)
 	(label "USART_CLK"
 		(at 92.71 96.52 0)
@@
 		)
 	)
+	(global_label "REG_EN_LOW"
+		(shape input)
+		(at 100.33 115.57 0)
+		(fields_autoplaced yes)
+		(effects
+			(font
+				(size 1.27 1.27)
+			)
+			(justify left)
+		)
+		(property "Intersheetrefs" "${INTERSHEET_REFS}"
+			(at 115.2289 115.57 0)
+			(effects
+				(font
+					(size 1.27 1.27)
+				)
+				(justify left)
+				(hide yes)
+			)
+		)
+	)
+	(global_label "REG_EN_LOW"
+		(shape input)
+		(at 152.4 95.25 0)
+		(fields_autoplaced yes)
+		(effects
+			(font
+				(size 1.27 1.27)
+			)
+			(justify left)
+		)
+		(property "Intersheetrefs" "${INTERSHEET_REFS}"
+			(at 167.2989 95.25 0)
+			(effects
+				(font
+					(size 1.27 1.27)
+				)
+				(justify left)
+				(hide yes)
+			)
+		)
+	)
