File: ATMEGA-SCHEMATICS/SNAKE_GAME/PCB/snake_pcb_v2/converter.kicad_sch (KiCad schematic)
At the start: 16 parts, among them J3 USB_A, SW5 SW_Push, U5 FT232RL

Commit message: ...
Parts:
- removed U5: FT232RL, Package_DIP:DIP-28_W15.24mm_LongPads, symbol Interface_USB:FT232RL
- added U3: FT232RL, Package_SO:SSOP-28_5.3x10.2mm_P0.65mm, symbol Interface_USB:FT232RL
- C42, C43: footprint Capacitor_THT:C_Disc_D7.5mm_W5.0mm_P5.00mm -> Capacitor_SMD:C_0402_1005Metric
- D1, D2: footprint LED_THT:LED_D1.8mm_W3.3mm_H2.4mm -> LED_SMD:LED_0603_1608Metric
- R31, R32, R33, R4, R5: footprint Resistor_THT:R_Axial_DIN0207_L6.3mm_D2.5mm_P10.16mm_Horizontal -> Resistor_SMD:R_0402_1005Metric
Connections:
- net CLOCK: now also U3.23 (CBUS0)
- net CTS_CONV: now also U3.11 (CTS)
- net D+: now also U3.15 (USBD+)
- net D-: now also U3.16 (USBD-)
- net GND: now also U3.18 (GND), U3.21 (GND), U3.25 (AGND), U3.26 (TEST), U3.7 (GND)
- net RTS_CONV: now also U3.3 (RTS)
- net RXD_CONV: now also U3.5 (RXD)
- net TXD_CONV: now also U3.1 (TXD)
- net VCC: now also U3.20 (VCC), U3.4 (VCCIO)
- net WAKE_UP: now also U3.14 (CBUS3)
- net at D2.1 (K): now also U3.13 (CBUS2)
- net at C13.1: now also U3.17 (3V3OUT)
- net at R4.1, R5.2, SW5.1: now also U3.19 (~{RESET})
- net at D1.1 (K): now also U3.22 (CBUS1)
Changed lines of the file:
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@@
+	)
+	(junction
+		(at 149.86 71.12)
+		(diameter 0)
+		(color 0 0 0 0)
+	)
+	(junction
+		(at 149.86 121.92)
+		(diameter 0)
+		(color 0 0 0 0)
+	)
+	(junction
+		(at 100.33 81.28)
+		(diameter 0)
+		(color 0 0 0 0)
+	)
+	(junction
+		(at 90.17 81.28)
+		(diameter 0)
+		(color 0 0 0 0)
+	)
+	(junction
+		(at 173.99 111.76)
+		(diameter 0)
+		(color 0 0 0 0)
 	)
 	(junction
@@
 	)
 	(junction
-		(at 100.33 81.28)
-		(diameter 0)
-		(color 0 0 0 0)
-	)
-	(junction
-		(at 90.17 81.28)
-		(diameter 0)
-		(color 0 0 0 0)
-	)
-	(junction
-		(at 173.99 111.76)
-		(diameter 0)
-		(color 0 0 0 0)
-	)
-	(junction
 		(at 205.74 102.87)
 		(diameter 0)
@@
 	)
 	(junction
-		(at 149.86 71.12)
-		(diameter 0)
-		(color 0 0 0 0)
-	)
-	(junction
 		(at 125.73 59.69)
 		(diameter 0)
@@
 	)
 	(junction
-		(at 149.86 121.92)
-		(diameter 0)
-		(color 0 0 0 0)
-	)
-	(junction
 		(at 104.14 86.36)
 		(diameter 0)
@@
 	(wire
 		(pts
+			(xy 149.86 121.92) (xy 152.4 121.92)
+		)
+		(stroke
+			(width 0)
+			(type default)
+		)
+	)
+	(wire
+		(pts
 			(xy 167.64 86.36) (xy 170.18 86.36)
 		)
@@
 		(pts
 			(xy 167.64 111.76) (xy 173.99 111.76)
-		)
-		(stroke
-			(width 0)
-			(type default)
-		)
-	)
-	(wire
-		(pts
-			(xy 149.86 121.92) (xy 152.4 121.92)
 		)
 		(stroke
@@
 	)
 	(symbol
-		(lib_id "Interface_USB:FT232RL")
-		(at 147.32 96.52 0)
-		(unit 1)
-		(exclude_from_sim no)
-		(in_bom yes)
-		(on_board yes)
-		(dnp no)
-		(fields_autoplaced yes)
-		(property "Reference" "U5"
-			(at 152.0033 69.85 0)
-			(effects
-				(font
-					(size 1.27 1.27)
-				)
-				(justify left)
-			)
-		)
-		(property "Value" "FT232RL"
-			(at 152.0033 72.39 0)
-			(effects
-				(font
-					(size 1.27 1.27)
-				)
-				(justify left)
-			)
-		)
-		(property "Footprint" "Package_DIP:DIP-28_W15.24mm_LongPads"
-			(at 175.26 119.38 0)
-			(effects
-				(font
-					(size 1.27 1.27)
-				)
-				(hide yes)
-			)
-		)
-		(property "Datasheet" "https://www.ftdichip.com/Support/Documents/DataSheets/ICs/DS_FT232R.pdf"
-			(at 147.32 96.52 0)
-			(effects
-				(font
-					(size 1.27 1.27)
-				)
-				(hide yes)
-			)
-		)
-		(property "Description" "USB to Serial Interface, SSOP-28"
-			(at 147.32 96.52 0)
-			(effects
-				(font
-					(size 1.27 1.27)
-				)
-				(hide yes)
-			)
-		)
-		(pin "4"
-		)
-		(pin "28"
-		)
-		(pin "3"
-		)
-		(pin "23"
-		)
-		(pin "11"
-		)
-		(pin "22"
-		)
-		(pin "7"
-		)
-		(pin "26"
-		)
-		(pin "1"
-		)
-		(pin "19"
-		)
-		(pin "16"
-		)
-		(pin "10"
-		)
-		(pin "15"
-		)
-		(pin "17"
-		)
-		(pin "6"
-		)
-		(pin "20"
-		)
-		(pin "2"
-		)
-		(pin "9"
-		)
-		(pin "13"
-		)
-		(pin "5"
-		)
-		(pin "25"
-		)
-		(pin "21"
-		)
-		(pin "18"
-		)
-		(pin "12"
-		)
-		(pin "14"
-		)
-		(pin "27"
-		)
-		(instances
-			(project "snake_pcb"
-				(path "/071b2fc6-d65a-411c-93b6-4a9f90a11c3f/56e9ae98-bada-4e2a-9fa4-047d2506f55b"
-					(reference "U5")
-					(unit 1)
-				)
-			)
-		)
-	)
-	(symbol
 		(lib_id "power:GND")
 		(at 111.76 80.01 0)
@@
 			)
 		)
-		(property "Footprint" "Capacitor_THT:C_Disc_D7.5mm_W5.0mm_P5.00mm"
+		(property "Footprint" "Capacitor_SMD:C_0402_1005Metric"
 			(at 95.5548 96.52 0)
 			(effects
@@
 			)
 		)
-		(property "Footprint" "Resistor_THT:R_Axial_DIN0207_L6.3mm_D2.5mm_P10.16mm_Horizontal"
+		(property "Footprint" "Resistor_SMD:R_0402_1005Metric"
 			(at 201.93 107.442 90)
 			(effects
@@
 			)
 		)
-		(property "Footprint" "LED_THT:LED_D1.8mm_W3.3mm_H2.4mm"
+		(property "Footprint" "LED_SMD:LED_0603_1608Metric"
 			(at 194.31 109.22 0)
 			(effects
@@
 			)
 		)
-		(property "Footprint" "Resistor_THT:R_Axial_DIN0207_L6.3mm_D2.5mm_P10.16mm_Horizontal"
+		(property "Footprint" "Resistor_SMD:R_0402_1005Metric"
 			(at 105.41 83.058 90)
 			(effects
@@
 			)
 		)
-		(property "Footprint" "Resistor_THT:R_Axial_DIN0207_L6.3mm_D2.5mm_P10.16mm_Horizontal"
+		(property "Footprint" "Resistor_SMD:R_0402_1005Metric"
 			(at 201.93 104.648 90)
 			(effects
@@
 			)
 		)
-		(property "Footprint" "Resistor_THT:R_Axial_DIN0207_L6.3mm_D2.5mm_P10.16mm_Horizontal"
+		(property "Footprint" "Resistor_SMD:R_0402_1005Metric"
 			(at 95.25 83.058 90)
 			(effects
@@
 			)
 		)
-		(property "Footprint" "Resistor_THT:R_Axial_DIN0207_L6.3mm_D2.5mm_P10.16mm_Horizontal"
+		(property "Footprint" "Resistor_SMD:R_0402_1005Metric"
 			(at 175.768 115.57 90)
 			(effects
@@
 			)
 		)
-		(property "Footprint" "LED_THT:LED_D1.8mm_W3.3mm_H2.4mm"
+		(property "Footprint" "LED_SMD:LED_0603_1608Metric"
 			(at 194.31 102.87 0)
 			(effects
@@
 				(path "/071b2fc6-d65a-411c-93b6-4a9f90a11c3f/56e9ae98-bada-4e2a-9fa4-047d2506f55b"
 					(reference "D1")
+					(unit 1)
+				)
+			)
+		)
+	)
+	(symbol
+		(lib_id "Interface_USB:FT232RL")
+		(at 147.32 96.52 0)
+		(unit 1)
+		(exclude_from_sim no)
+		(in_bom yes)
+		(on_board yes)
+		(dnp no)
+		(fields_autoplaced yes)
+		(property "Reference" "U3"
+			(at 152.0033 69.85 0)
+			(effects
+				(font
+					(size 1.27 1.27)
+				)
+				(justify left)
+			)
+		)
+		(property "Value" "FT232RL"
+			(at 152.0033 72.39 0)
+			(effects
+				(font
+					(size 1.27 1.27)
+				)
+				(justify left)
+			)
+		)
+		(property "Footprint" "Package_SO:SSOP-28_5.3x10.2mm_P0.65mm"
+			(at 175.26 119.38 0)
+			(effects
+				(font
+					(size 1.27 1.27)
+				)
+				(hide yes)
+			)
+		)
+		(property "Datasheet" "https://www.ftdichip.com/Support/Documents/DataSheets/ICs/DS_FT232R.pdf"
+			(at 147.32 96.52 0)
+			(effects
+				(font
+					(size 1.27 1.27)
+				)
+				(hide yes)
+			)
+		)
+		(property "Description" "USB to Serial Interface, SSOP-28"
+			(at 147.32 96.52 0)
+			(effects
+				(font
+					(size 1.27 1.27)
+				)
+				(hide yes)
+			)
+		)
+		(pin "27"
+		)
+		(pin "28"
+		)
+		(pin "22"
+		)
+		(pin "13"
+		)
+		(pin "7"
+		)
+		(pin "20"
+		)
+		(pin "11"
+		)
+		(pin "2"
+		)
+		(pin "14"
+		)
+		(pin "12"
+		)
+		(pin "23"
+		)
+		(pin "5"
+		)
+		(pin "3"
+		)
+		(pin "25"
+		)
+		(pin "9"
+		)
+		(pin "10"
+		)
+		(pin "6"
+		)
+		(pin "18"
+		)
+		(pin "21"
+		)
+		(pin "1"
+		)
+		(pin "4"
+		)
+		(pin "17"
+		)
+		(pin "16"
+		)
+		(pin "15"
+		)
+		(pin "19"
+		)
+		(pin "26"
+		)
+		(instances
+			(project ""
+				(path "/071b2fc6-d65a-411c-93b6-4a9f90a11c3f/56e9ae98-bada-4e2a-9fa4-047d2506f55b"
+					(reference "U3")
 					(unit 1)
 				)
@@
 			)
 		)
-		(property "Footprint" "Capacitor_THT:C_Disc_D7.5mm_W5.0mm_P5.00mm"
+		(property "Footprint" "Capacitor_SMD:C_0402_1005Metric"
 			(at 103.1748 93.98 0)
 			(effects
