File: ATMEGA-SCHEMATICS/SNAKE_GAME/PCB/snake_pcb_v2/game.kicad_sch (KiCad schematic)
At the start: 60 parts, among them J10 LCD_SCREEN, J14 Conn_01x05_Pin, J15 Conn_01x04_Pin, J17 Conn_01x06_Pin, J19 Conn_01x06_Pin, J26 B_START, J27 B_STOP, J28 B_SELECT, J6 TERM_GAME, J8 Vibrator, J9 Conn_01x05_Pin, SW3 SW_Push, U10 PCF8574AP, U2 ATmega168A-P, U8 MX25L3233FM1, Y2 Crystal

Commit message: ...
Parts:
- removed C19: 4.7uF, Capacitor_SMD:C_0805_2012Metric, symbol Device:C
- removed C20, C21, C22: 100nF, Capacitor_SMD:C_0402_1005Metric, symbol Device:C
- removed R1, R18: 10K, Resistor_THT:R_Axial_DIN0207_L6.3mm_D2.5mm_P10.16mm_Horizontal, symbol Device:R
- removed SW3: SW_Push, Button_Switch_THT:SW_PUSH_1P1T_6x3.5mm_H4.3_APEM_MJTP1243, symbol Switch:SW_Push
- removed U2: ATmega168A-P, Package_DIP:DIP-28_W7.62mm, symbol MCU_Microchip_ATmega:ATmega168A-P
- removed U8: MX25L3233FM1, Package_DIP:CERDIP-8_W7.62mm_SideBrazed_Socket, symbol Memory_Flash:MX25L3233FM1
- removed Y2: Crystal, Crystal:Resonator-2Pin_W6.0mm_H3.0mm, symbol Device:Crystal
- added C25, C26: 22pF, Capacitor_SMD:C_0402_1005Metric, symbol Device:C
- added C27, C28, C6: 100nF, Capacitor_SMD:C_0402_1005Metric, symbol Device:C
- added R19, R20: 4K7, Resistor_SMD:R_0402_1005Metric, symbol Device:R
- added R21: 10K, Resistor_SMD:R_0402_1005Metric, symbol Device:R
- added SW2: SW_Push, Button_Switch_THT:SW_PUSH_1P1T_6x3.5mm_H4.3_APEM_MJTP1243, symbol Switch:SW_Push
- added U1: ATmega8-16A, Package_QFP:TQFP-32_7x7mm_P0.8mm, symbol MCU_Microchip_ATmega:ATmega8-16A
- added U5: MX25L3233FM1, Package_SO:JEITA_SOIC-8_3.9x4.9mm_P1.27mm, symbol Memory_Flash:MX25L3233FM1
- added Y3: Crystal, Crystal:Crystal_SMD_3225-4Pin_3.2x2.5mm_HandSoldering, symbol Device:Crystal
- C17: value 22pF -> 4.7uF; footprint Capacitor_THT:CP_Radial_D5.0mm_P2.50mm -> Capacitor_SMD:C_0805_2012Metric
- C18: value 22pF -> 100nF; footprint Capacitor_THT:CP_Radial_D5.0mm_P2.50mm -> Capacitor_SMD:C_0402_1005Metric
- R10, R11, R12, R13, R14, R15, R16, R17, R24, R25, R26, R40, R41, R42, R43, R44, R45, R46, R8: footprint Resistor_THT:R_Axial_DIN0207_L6.3mm_D2.5mm_P10.16mm_Horizontal -> Resistor_SMD:R_0402_1005Metric
- R7, R9: value 4K7 -> 10K; footprint Resistor_THT:R_Axial_DIN0207_L6.3mm_D2.5mm_P10.16mm_Horizontal -> Resistor_SMD:R_0402_1005Metric
Connections:
- net 3.3V: now also C29.1, C30.1, R25.2, U5.8 (VCC)
- net BUZZER_PWM: now also U1.9 (PD5)
- net B_SELECT: now also U1.23 (PC0)
- net B_START: now also U1.10 (PD6)
- net B_STOP: now also U1.11 (PD7)
- net CS: now also U5.1 (~{CS})
- net FLASH_CS: now also R9.2, U1.13 (PB1)
- net FLASH_HOLD: now also R8.1, U1.12 (PB0); no longer R17.1
- net FLASH_WP: now also U1.24 (PC1)
- net GND: now also R17.1, C25.2, C26.2, C27.2, C28.2, C6.2, SW2.2, U1.21 (AGND), U1.3 (GND), U1.5 (GND), U5.4 (GND); no longer U10.1 (A0)
- net HOLD: now also U5.7 (~{HOLD}/SIO3)
- net J_DOWN: now also U1.1 (PD3)
- net J_LEFT: now also U1.2 (PD4)
- net J_RIGHT: now also U1.25 (PC2)
- net J_UP: now also U1.32 (PD2)
- net MISO: now also U5.2 (SO/SIO1)
- net MISO_GAME: now also U1.16 (PB4)
- net MOSI: now also U5.5 (SI/SIO0)
- net MOSI_GAME: now also U1.15 (PB3)
- net PB2: now also R21.2, U1.14 (PB2)
- net RESET_GAME: now also R7.1, SW2.1, U1.29 (PC6/~{RESET}); no longer R8.1
- net RXD_GAME: now also U1.30 (PD0)
- net SCK: now also U5.6 (SCLK)
- net SCK_GAME: now also U1.17 (PB5)
- net SCL_GAME: now also R19.1, R20.1, U1.28 (PC5); no longer R9.1
- net SDA_GAME: now also U1.27 (PC4); no longer R7.1
- net TXD_GAME: now also U1.31 (PD1)
- net VCC: now also C17.1, C18.1, C32.1, C36.1, C37.1, C38.1, CS_HOLD_SHIFTER1.1 (VCCA), MISO_SHIFTER1.1 (VCCA), MOSI_CLK_SHIFTER1.1 (VCCA), R9.1, WP_SHIFTER1.1 (VCCA), C27.1, C28.1, C6.1, R19.2, R20.2, R21.1, U1.18 (AVCC), U1.20 (AREF), U1.4 (VCC), U1.6 (VCC); no longer C29.1, C30.1, R17.2, R25.2, R9.2
- net VIBRATOR: now also U1.26 (PC3)
- net WP: now also U5.3 (~{WP}/SIO2)
- new net: C25.1, U1.8 (PB7/XTAL2), Y3.1
- new net: R17.2, U10.1 (A0)
- new net: C26.1, U1.7 (PB6/XTAL1), Y3.2
- no-connect marks 10 -> 12
Other:
- moved on the sheet: BZ1, J26, J27, J28, J8, J9, R10, R11, R12, R13, R14, R15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
