File: ATMEGA-SCHEMATICS/SNAKE_GAME/PCB/snake_pcb_v2/programmer.kicad_sch (KiCad schematic)
At the start: 31 parts, among them J1 Conn_01x02_Pin, J11 EXT_ACC_PROG, J21 Conn_01x04_Pin, J22 Conn_01x06_Pin, J23 Conn_01x06_Pin, J24 Conn_01x05_Pin, J25 Conn_01x02_Pin, J5 Conn_01x03_Pin, SW1 PROG_SWT, SW4 SW_Push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

Commit message: ...
Parts:
- removed C6: 4.7uF, Capacitor_SMD:C_0805_2012Metric, symbol Device:C
- removed R35: 10K, Resistor_THT:R_Axial_DIN0207_L6.3mm_D2.5mm_P10.16mm_Horizontal, symbol Device:R
- removed SW4: SW_Push, Button_Switch_THT:SW_PUSH_1P1T_6x3.5mm_H4.3_APEM_MJTP1243, symbol Switch:SW_Push
- removed U3: ATmega8A-P, Package_DIP:DIP-28_W7.62mm, symbol MCU_Microchip_ATmega:ATmega8A-P
- removed Y1: Crystal, Crystal:Resonator-2Pin_W6.0mm_H3.0mm, symbol Device:Crystal
- added C19, C20: 22pF, Capacitor_SMD:C_0402_1005Metric, symbol Device:C
- added C21: 100nF, Capacitor_SMD:C_0402_1005Metric, symbol Device:C
- added R1: 10K, Resistor_SMD:R_0402_1005Metric, symbol Device:R
- added SW3: SW_Push, Button_Switch_THT:SW_PUSH_1P1T_6x3.5mm_H4.3_APEM_MJTP1243, symbol Switch:SW_Push
- added U2: ATmega8-16A, Package_QFP:TQFP-32_7x7mm_P0.8mm, symbol MCU_Microchip_ATmega:ATmega8-16A
- added Y2: 16MHz, Crystal:Crystal_SMD_3225-4Pin_3.2x2.5mm_HandSoldering, symbol Device:Crystal
- C1: value 22pF -> 4.7uF; footprint Capacitor_THT:CP_Radial_D5.0mm_P2.50mm -> Capacitor_SMD:C_0805_2012Metric
- C3: value 22pF -> 100nF; footprint Capacitor_THT:CP_Radial_D5.0mm_P2.50mm -> Capacitor_SMD:C_0402_1005Metric
- R2, R22, R3, R6: footprint Resistor_THT:R_Axial_DIN0207_L6.3mm_D2.5mm_P10.16mm_Horizontal -> Resistor_SMD:R_0402_1005Metric
Connections:
- net CTS_PROG: now also U2.26 (PC3)
- net EXT_SIGNAL: now also U2.25 (PC2)
- net FLASH_CS: now also U2.11 (PD7)
- net GAME_CS: now also U2.1 (PD3)
- net GAME_SIGNAL: now also U2.24 (PC1)
- net GND: now also C19.2, C20.2, C21.2, SW3.2, U2.21 (AGND), U2.3 (GND), U2.5 (GND)
- net GRID_CS: now also U2.32 (PD2)
- net GRID_SIGNAL: now also U2.23 (PC0)
- net I/O_CONVERTER: now also U2.10 (PD6)
- net MISO: now also U2.16 (PB4)
- net MOSI: now also U2.15 (PB3)
- net PB0: now also U2.12 (PB0)
- net PB1: now also U2.13 (PB1)
- net PB2: now also U2.14 (PB2)
- net PC5: now also U2.28 (PC5)
- net RESET_PROG: now also R1.2, SW3.1, U2.29 (PC6/~{RESET})
- net RTS_PROG: now also U2.27 (PC4)
- net RXD: now also U2.30 (PD0)
- net SCK: now also U2.17 (PB5)
- net SRAM_CS: now also U2.9 (PD5)
- net TXD: now also U2.31 (PD1)
- net VCC: now also C1.1, C3.1, C21.1, R1.1, U2.18 (AVCC), U2.20 (AREF), U2.4 (VCC), U2.6 (VCC)
- net XCK: now also U2.2 (PD4)
- new net: C20.1, U2.8 (PB7/XTAL2), Y2.1
- new net: C19.1, U2.7 (PB6/XTAL1), Y2.2
- no-connect marks 9 -> 11
Other:
- moved on the sheet: J1, J11, J25, J5

Commit message: .
Parts:
- renumbered J5 to CONV_UART1
Changed lines of the file:
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@@
 		(dnp no)
 		(fields_autoplaced yes)
-		(property "Reference" "J5"
+		(property "Reference" "CONV_UART1"
 			(at 281.94 182.8799 0)
 			(effects
@@
 			(project ""
 				(path "/071b2fc6-d65a-411c-93b6-4a9f90a11c3f/070e247b-fc65-48a1-a34b-7b6bc28073d9"
-					(reference "J5")
+					(reference "CONV_UART1")
 					(unit 1)
 				)
