File: ATMEGA-SCHEMATICS/SNAKE_GAME/PCB/snake_pcb_v2/snake_pcb_v2.kicad_pcb (KiCad board)
At the start: 4 copper layers, 160 parts, among them J1 Conn_01x02_Pin, J10 LCD_SCREEN, J11 EXT_ACC_PROG, J14 Conn_01x05_Pin, J15 Conn_01x04_Pin, J17 Conn_01x06_Pin, J19 Conn_01x06_Pin, J21 Conn_01x04_Pin, J22 Conn_01x06_Pin, J23 Conn_01x06_Pin, J24 Conn_01x05_Pin, J25 Conn_01x02_Pin, J26 B_START, J27 B_STOP, J28 B_SELECT, J3 USB_A, J4 Barrel_Jack_Switch, J5 Conn_01x03_Pin, J6 TERM_GAME, J8 Vibrator, J9 Conn_01x05_Pin, SW1 PROG_SWT, SW2 SW_Push, SW3 SW_Push, SW5 SW_Push, SW6 SW_Push, U1 ATmega8-16A, U10 PCF8574AP, U11 ATmega8-16A, U2 ATmega8-16A, U3 FT232RL, U4 CD4066BE, U5 MX25L3233FM1, U6 CD4066BE, U7 CD4066BE, U9 AMS1117-3.3, Y2 16MHz, Y3 Crystal, Y4 20MHz

Commit message: .
Parts:
- removed J10: LCD_SCREEN, Connector_PinSocket_2.54mm:PinSocket_1x04_P2.54mm_Vertical
- added C6: 100nF, Capacitor_SMD:C_0402_1005Metric, F.Cu at (134.5, 153.5)
- added LCD_SCREEN: LCD_SCREEN, Connector_PinSocket_2.54mm:PinSocket_1x04_P2.54mm_Vertical, F.Cu at (117.9, 105.0)
- moved J22 174.8 mm to (236.6, 202.0), turned to -90 degrees
- moved J21 140.7 mm to (217.3, 202.0), turned to -90 degrees
- moved U4 138.8 mm to (206.9, 138.1), turned to 90 degrees
- moved J24 134.8 mm to (203.6, 202.0), turned to -90 degrees
- moved 220uF1 134.3 mm to (235.5, 126.0)
- moved J11 133.2 mm to (187.0, 177.0), turned to -90 degrees
- moved 4.7uF1 132.7 mm to (235.2, 121.0)
- moved J1 128.6 mm to (197.2, 161.5), turned to 90 degrees
- moved C16 127.8 mm to (206.0, 127.1), turned to 180 degrees
- moved 47uF3 127.5 mm to (231.0, 102.2), turned to 180 degrees
- moved R34 125.6 mm to (233.1, 151.6)
- moved J14 124.7 mm to (151.4, 202.0), turned to 90 degrees
- moved D9 124.1 mm to (239.5, 95.5), turned to -90 degrees
- moved TPS75533KCG3 121.9 mm to (226.6, 94.5)
- moved C15 121.7 mm to (206.0, 124.1), turned to 180 degrees
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- renumbered J5 to CONV_UART1
Routing:
- net /game/FLASH_WP: track 0.00 -> 265.5 mm, vias 0 -> 1
- net /game/VIBRATOR: track 0.00 -> 261.3 mm, vias 0 -> 1
- net /game/J_RIGHT: track 0.00 -> 260.1 mm, vias 0 -> 2
- net /game/SDA_GAME: track 0.00 -> 260.0 mm, vias 0 -> 7
- net /game/B_STOP: track 0.00 -> 259.4 mm, vias 0 -> 8
- net /game/SCL_GAME: track 0.00 -> 230.1 mm, vias 0 -> 4
- net 3.3V: track 19.8 -> 248.2 mm, vias 1 -> 10
- net /game/B_START: track 0.00 -> 211.1 mm, vias 0 -> 5
- net /game/MISO_GAME: track 0.00 -> 206.6 mm, vias 0 -> 4
- net /game/RESET_GAME: track 0.00 -> 174.3 mm, vias 0 -> 9
- net /game/J_UP: track 0.00 -> 172.3 mm, vias 0 -> 2
- net /programmer/EXT_SIGNAL: track 0.00 -> 159.4 mm, vias 0 -> 3
- net /game/J_DOWN: track 0.00 -> 158.4 mm
- net /game/J_LEFT: track 0.00 -> 145.7 mm, vias 0 -> 1
- net /programmer/SCK_EXT: track 0.00 -> 145.7 mm
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- added copper zone on B.Cu, net 3.3V
- added copper zone on F.Cu, net VCC
Other:
- board text added: "RXD"
- board text added: "TXD"
