File: ATMEGA-SCHEMATICS/SNAKE_GAME/PCB/BOARDS/PROGRAMMER/programmer/untitled.kicad_sch (KiCad schematic)
At the start: 34 parts, among them J1 Conn_01x02_Pin, J11 EXT_ACC_PROG, J21 Conn_01x04_Pin, J22 Conn_01x06_Pin, J23 Conn_01x06_Pin, J24 Conn_01x05_Pin, J25 Conn_01x02_Pin, J5 Conn_01x03_Pin, SW1 PROG_SWT, SW3 SW_Push, U2 ATmega8-16A, U4 CD4066BE, U6 CD4066BE, U7 CD4066BE, U8 ATmega88-20A, Y2 16MHz

Commit message: .
Parts:
- removed C1, C15, C7, C9: 4.7uF, Capacitor_SMD:C_0805_2012Metric, symbol Device:C
- removed C14, C16, C3, C4, C5, C8: 100nF, Capacitor_SMD:C_0402_1005Metric, symbol Device:C
- removed J1: Conn_01x02_Pin, Connector_PinSocket_2.54mm:PinSocket_1x02_P2.54mm_Vertical, symbol Connector:Conn_01x02_Pin
- removed J11: EXT_ACC_PROG, Connector_IDC:IDC-Header_2x05_P2.54mm_Vertical, symbol Connector_Generic:Conn_02x05_Odd_Even
- removed J21: Conn_01x04_Pin, Connector_PinHeader_2.54mm:PinHeader_1x04_P2.54mm_Vertical, symbol Connector:Conn_01x04_Pin
- removed J22, J23: Conn_01x06_Pin, Connector_PinHeader_2.54mm:PinHeader_1x06_P2.54mm_Vertical, symbol Connector:Conn_01x06_Pin
- removed J24: Conn_01x05_Pin, Connector_PinHeader_2.54mm:PinHeader_1x05_P2.54mm_Vertical, symbol Connector:Conn_01x05_Pin
- removed J25: Conn_01x02_Pin, Connector_PinHeader_2.54mm:PinHeader_1x02_P2.54mm_Vertical, symbol Connector:Conn_01x02_Pin
- removed J5: Conn_01x03_Pin, Connector_PinSocket_2.54mm:PinSocket_1x03_P2.54mm_Vertical, symbol Connector:Conn_01x03_Pin
- removed R1, R2, R22, R3, R6: 10K, Resistor_SMD:R_0402_1005Metric, symbol Device:R
- removed SW1: PROG_SWT, Button_Switch_THT:SW_Slide_SPDT_Straight_CK_OS102011MS2Q, symbol Switch:SW_Nidec_CAS-120A1
- removed SW3: SW_Push, Button_Switch_THT:SW_PUSH_1P1T_6x3.5mm_H4.3_APEM_MJTP1243, symbol Switch:SW_Push
- removed U2: ATmega8-16A, Package_QFP:TQFP-32_7x7mm_P0.8mm, symbol MCU_Microchip_ATmega:ATmega8-16A
- removed U4, U6, U7: CD4066BE, Package_DIP:DIP-14_W7.62mm, symbol Analog_Switch:CD4066BE
- removed U8: ATmega88-20A, Package_QFP:TQFP-32_7x7mm_P0.8mm, symbol MCU_Microchip_ATmega:ATmega88-20A
- added C17, C2: 22pF, Capacitor_THT:CP_Radial_D5.0mm_P2.50mm, symbol Device:C
- added C18, C22, C23: 4.7uF, Capacitor_SMD:C_0805_2012Metric, symbol Device:C
- added C24, C25, C26: 100nF, Capacitor_SMD:C_0402_1005Metric, symbol Device:C
- added J12: EXT_ACC_PROG, Connector_IDC:IDC-Header_2x05_P2.54mm_Vertical, symbol Connector_Generic:Conn_02x05_Odd_Even
- added J26: Conn_01x04_Pin, Connector_PinHeader_2.54mm:PinHeader_1x04_P2.54mm_Vertical, symbol Connector:Conn_01x04_Pin
- added J27, J28: Conn_01x06_Pin, Connector_PinHeader_2.54mm:PinHeader_1x06_P2.54mm_Vertical, symbol Connector:Conn_01x06_Pin
- added J29: Conn_01x05_Pin, Connector_PinHeader_2.54mm:PinHeader_1x05_P2.54mm_Vertical, symbol Connector:Conn_01x05_Pin
- added J30: Conn_01x02_Pin, Connector_PinHeader_2.54mm:PinHeader_1x02_P2.54mm_Vertical, symbol Connector:Conn_01x02_Pin
- added J6: Conn_01x02_Pin, Connector_PinSocket_2.54mm:PinSocket_1x02_P2.54mm_Vertical, symbol Connector:Conn_01x02_Pin
- added J7: Conn_01x03_Pin, Connector_PinSocket_2.54mm:PinSocket_1x03_P2.54mm_Vertical, symbol Connector:Conn_01x03_Pin
- added R23, R36, R7, R8, R9: 10K, Resistor_THT:R_Axial_DIN0207_L6.3mm_D2.5mm_P10.16mm_Horizontal, symbol Device:R
- added SW2: PROG_SWT, Button_Switch_THT:SW_Slide_SPDT_Straight_CK_OS102011MS2Q, symbol Switch:SW_Nidec_CAS-120A1
- added SW6: SW_Push, Button_Switch_THT:SW_PUSH_1P1T_6x3.5mm_H4.3_APEM_MJTP1243, symbol Switch:SW_Push
- added U10, U11, U9: CD4066BE, Package_DIP:DIP-14_W7.62mm, symbol Analog_Switch:CD4066BE
- added U8: ATmega8A-P, Package_DIP:DIP-28_W7.62mm, symbol MCU_Microchip_ATmega:ATmega8A-P
- C19, C20: value 22pF -> 100nF
- C21: value 100nF -> 4.7uF; footprint Capacitor_SMD:C_0402_1005Metric -> Capacitor_SMD:C_0805_2012Metric
- Y2: value 16MHz -> Crystal; footprint Crystal:Crystal_SMD_3225-4Pin_3.2x2.5mm_HandSoldering -> Crystal:Resonator-2Pin_W6.0mm_H3.0mm
Connections:
- net CTS_PROG: now also J28.4 (Pin_4), U8.26 (PC3)
- net EXT_SIGNAL: now also J28.3 (Pin_3), R9.1, SW2.2 (B), U10.6, U11.6, U8.25 (PC2), U9.6
- net FLASH_CS: now also J26.3 (Pin_3), J27.6 (Pin_6), U8.13 (PD7)
- net GAME_CS: now also J27.5 (Pin_5), U8.5 (PD3)
- net GAME_SIGNAL: now also J28.2 (Pin_2), R8.1, U10.5, U11.5, U8.24 (PC1), U9.5
- net GND: now also C17.2, C18.2, C2.2, C22.2, C23.2, C24.2, C25.2, C26.2, J12.10 (Pin_10), J12.3 (Pin_3), J12.4 (Pin_4), J12.6 (Pin_6), J12.8 (Pin_8), J7.1 (Pin_1), R7.2, R8.2, R9.2, SW2.1 (C), SW6.2, U10.7 (V_{SS}), U11.7 (V_{SS}), U8.22 (AGND), U8.8 (GND), U9.7 (V_{SS})
- net GRID_CS: now also J27.4 (Pin_4), U8.4 (PD2)
- net GRID_SIGNAL: now also J28.1 (Pin_1), R7.1, U10.13, U11.13, U8.23 (PC0), U9.13
- net I/O_CONVERTER: now also J26.2 (Pin_2), U8.12 (PD6)
- net MISO: now also J29.4 (Pin_4), U10.1, U10.4, U10.8, U8.18 (PB4)
- net MISO_EXT: now also J12.9 (Pin_9), U10.9
- net MISO_GAME: now also U10.3
- net MISO_GRID: now also U10.2
- net MOSI: now also J29.3 (Pin_3), U8.17 (PB3), U9.1, U9.4, U9.8
- net MOSI_EXT: now also J12.1 (Pin_1), U9.9
- net MOSI_GAME: now also U9.3
- net MOSI_GRID: now also U9.2
- net PB0: now also J26.4 (Pin_4), U8.14 (PB0)
- net PB1: now also J29.1 (Pin_1), U8.15 (PB1)
- net PB2: now also J29.2 (Pin_2), R23.2, U8.16 (PB2)
- net PC5: now also J28.6 (Pin_6), U8.28 (PC5)
- net RESET_PROG: now also J12.5 (Pin_5), J27.1 (Pin_1), R36.2, SW6.1, U8.1 (PC6/~{RESET})
- net RTS_PROG: now also J28.5 (Pin_5), U8.27 (PC4)
- net RXD: now also J27.2 (Pin_2), J6.1 (Pin_1), U8.2 (PD0)
- net RXD_PROG: now also J6.2 (Pin_2), J7.3 (Pin_3)
- net SCK: now also J29.5 (Pin_5), U11.1, U11.4, U11.8, U8.19 (PB5)
- net SCK_EXT: now also J12.7 (Pin_7), U11.9
- net SCK_GAME: now also U11.3
- net SCK_GRID: now also U11.2
- net SRAM_CS: now also J26.1 (Pin_1), U8.11 (PD5)
- net TXD: now also J27.3 (Pin_3), J30.1 (Pin_1), U8.3 (PD1)
- net TXD_PROG: now also J30.2 (Pin_2), J7.2 (Pin_2)
- net VCC: now also C19.1, C20.1, C18.1, C22.1, C23.1, C24.1, C25.1, C26.1, J12.2 (Pin_2), R23.1, R36.1, SW2.3 (A), U10.14 (V_{DD}), U11.14 (V_{DD}), U8.20 (AVCC), U8.21 (AREF), U8.7 (VCC), U9.14 (V_{DD})
- net XCK: now also U8.6 (PD4)
- net at Y2.1: now also C17.1, U8.10 (PB7/XTAL2); no longer C20.1
- net at Y2.2: now also C2.1, U8.9 (PB6/XTAL1); no longer C19.1
- no-connect marks 11 -> 9
