File: ATMEGA-SCHEMATICS/SNAKE_GAME/GRID_SCHEMATICS/GRID_V2/GRID_V2.kicad_sch (KiCad schematic)
At the start: 8572 parts, among them J1 Conn_01x04_Pin, J10 Conn_01x03_Pin, J11 Conn_01x03_Pin, J12 Conn_01x04_Pin, J13 Conn_01x03_Pin, J14 Conn_01x03_Pin, J15 Conn_01x04_Pin, J16 Conn_01x03_Pin, J17 Conn_01x03_Pin, J18 Conn_01x04_Pin, J19 Conn_01x03_Pin, J20 Conn_01x03_Pin, J21 Conn_01x04_Pin, J22 Conn_01x03_Pin, J23 Conn_01x03_Pin, J24 Conn_01x04_Pin, J25 Conn_01x03_Pin, J26 Conn_01x03_Pin, J27 Conn_01x04_Pin, J28 Conn_01x03_Pin, J29 Conn_01x03_Pin, J3 Conn_01x04_Pin, J30 Conn_01x04_Pin, J4 Conn_01x04_Pin, J5 Conn_01x03_Pin, J6 Conn_01x03_Pin, J7 Conn_01x03_Pin, J8 Conn_01x03_Pin, J9 Conn_01x04_Pin

Commit message: .
Parts:
- removed C1, C10, C100, C1000, C1001, C1002, C1003, C1004, C1005, C1006, C1007, C1008, C1009, C101, C1010, C1011, C1012, C1013, C1014, C1015, C1016, C1017, C1018, C1019, C102, C1020, C1021, C1022, C1023, C1024, C1025, C1026, C1027, C1028, C1029, C103, C1030, C1031, C1032, C1033, C1034, C1035, C1036, C1037, C1038, C1039, C104, C1040, C1041, C1042, C1043, C1044, C1045, C1046, C1047, C1048, C1049, C105, C1050, C1051, C1052, C1053, C1054, C1055, C1056, C1057, C1058, C1059, C106, C1060, C1061, C1062, C1063, C1064, C1065, C1066, C1067, C1068, C1069, C107, C1070, C1071, C1072, C1073, C1074, C1075, C1076, C1077, C1078, C1079, C108, C1080, C1081, C1082, C1083, C1084, C1085, C1086, C1087, C1088, C1089, C109, C1090, C1091, C1092, C1093, C1094, C1095, C1096, C1097, C1098, C1099, C11, C110, C1100, C1101, C1102, C1103, C1104, C1105, C1106, C1107, C1108, C1109, C111, C1110, C1111, C1112, C1113, C1114, C1115, C1116, C1117, C1118, C1119, C112, C1120, C1121, C1122, C1123, C1124, C1125, C1126, C1127, C1128, C1129, C113, C1130, C1131, C1132, C1133, C1134, C1135, C1136, C1137, C1138, C1139, C114, C1140, C1141, C1142, C1143, C1144, C1145, C1146, C1147, C1148, C1149, C115, C1150, C1151, C1152, C1153, C1154, C1155, C1156, C1157, C1158, C1159, C116, C1160, C1161, C1162, C1163, C1164, C1165, C1166, C1167, C1168, C1169, C117, C1170, C1171, C1172, C1173, C1174, C1175, C1176, C1177, C1178, C1179, C118, C1180, C1181, C1182, C1183, C1184, C1185, C1186, C1187, C1188, C1189, C119, C1190, C1191, C1192, C1193, C1194, C1195, C1196, C1197, C1198, C1199, C12, C120, C1200, C1201, C1202, C1203, C1204, C1205, C1206, C1207, C1208, C1209, C121, C1210, C1211, C1212, C1213, C1214, C1215, C1216, C1217, C1218, C1219, C122, C1220, C1221, C1222, C1223, C1224, C1225, C1226, C1227, C1228, C1229, C123, C1230, C1231, C1232, C1233, C1234, C1235, C1236, C1237, C1238, C1239, C124, C1240, C1241, C1242, C1243, C1244, C1245, C1246, C1247, C1248, C1249, C125, C1250, C1251, C1252, C1253, C1254, C1255, C1256, C1257, C1258, C1259, C126, C1260, C1261, C1262, C1263, C1264, C1265, C1266, C1267, C1268, C1269, C127, C1270, C1271, C1272, C1273, C1274, C1275, C1276, C1277, C1278, C1279, C128, C1280, C1281, C1282, C1283, C1284, C1285, C1286, C1287, C1288, C1289, C129, C1290, C1291, C1292, C1293, C1294, C1295, C1296, C1297, C1298, C1299, C13, C130, C1300, C1301, C1302, C1303, C1304, C1305, C1306, C1307, C1308, C1309, C131, C1310, C1311, C1312, C1313, C1314, C1315, C1316, C1317, C1318, C1319, C132, C1320, C1321, C1322, C1323, C1324, C1325, C1326, C1327, C1328, C1329, C133, C1330, C1331, C1332, C1333, C1334, C1335, C1336, C1337, C1338, C1339, C134, C1340, C1341, C1342, C1343, C1344, C1345, C1346, C1347, C1348, C1349, C135, C1350, C1351, C1352, C1353, C1354, C1355, C1356, C1357, C1358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: 1uF, Capacitor_SMD:C_0603_1608Metric, symbol Device:C
- removed C4323, C4325, C4327, C4329, C4331, C4333, C4335, C4337, C4339: 16PK4700MEFC12.5X25, symbol Device:C_Polarized
- removed C4324, C4326, C4328, C4330, C4332, C4334, C4336, C4338, C4340: T520Y337M006ATE040, symbol Device:C_Small
- removed D1, D10, D100, D1000, D1001, D1002, D1003, D1004, D1005, D1006, D1007, D1008, D1009, D101, D1010, D1011, D1012, D1013, D1014, D1015, D1016, D1017, D1018, D1019, D102, D1020, D1021, D1022, D1023, D1024, D1025, D1026, D1027, D1028, D1029, D103, D1030, D1031, D1032, D1033, D1034, D1035, D1036, D1037, D1038, D1039, D104, D1040, D1041, D1042, D1043, D1044, D1045, D1046, D1047, D1048, D1049, D105, D1050, D1051, D1052, D1053, D1054, D1055, D1056, D1057, D1058, D1059, D106, D1060, D1061, D1062, D1063, D1064, D1065, D1066, D1067, D1068, D1069, D107, D1070, D1071, D1072, D1073, D1074, D1075, D1076, D1077, D1078, D1079, D108, D1080, D1081, D1082, D1083, D1084, D1085, D1086, D1087, D1088, D1089, D109, D1090, D1091, D1092, D1093, D1094, D1095, D1096, D1097, D1098, D1099, D11, D110, D1100, D1101, D1102, D1103, D1104, D1105, D1106, D1107, D1108, D1109, D111, D1110, D1111, D1112, D1113, D1114, D1115, D1116, D1117, D1118, D1119, D112, D1120, D1121, D1122, D1123, D1124, D1125, D1126, D1127, D1128, D1129, D113, D1130, D1131, D1132, D1133, D1134, D1135, D1136, D1137, D1138, D1139, D114, D1140, D1141, D1142, D1143, D1144, D1145, D1146, D1147, D1148, D1149, D115, D1150, D1151, D1152, D1153, D1154, D1155, D1156, D1157, D1158, D1159, D116, D1160, D1161, D1162, D1163, D1164, D1165, D1166, D1167, D1168, D1169, D117, D1170, D1171, D1172, D1173, D1174, D1175, D1176, D1177, D1178, D1179, D118, D1180, D1181, D1182, D1183, D1184, D1185, D1186, D1187, D1188, D1189, D119, D1190, D1191, D1192, D1193, D1194, D1195, D1196, D1197, D1198, D1199, D12, D120, D1200, D1201, D1202, D1203, D1204, D1205, D1206, D1207, D1208, D1209, D121, D1210, D1211, D1212, D1213, D1214, D1215, D1216, D1217, D1218, D1219, D122, D1220, D1221, D1222, D1223, D1224, D1225, D1226, D1227, D1228, D1229, D123, D1230, D1231, D1232, D1233, D1234, D1235, D1236, D1237, D1238, D1239, D124, D1240, D1241, D1242, D1243, D1244, D1245, D1246, D1247, D1248, D1249, D125, D1250, D1251, D1252, D1253, D1254, D1255, D1256, D1257, D1258, D1259, D126, D1260, D1261, D1262, D1263, D1264, D1265, D1266, D1267, D1268, D1269, D127, D1270, D1271, D1272, D1273, D1274, D1275, D1276, D1277, D1278, D1279, D128, D1280, D1281, D1282, D1283, D1284, D1285, D1286, D1287, D1288, D1289, D129, D1290, D1291, D1292, D1293, D1294, D1295, D1296, D1297, D1298, D1299, D13, D130, D1300, D1301, D1302, D1303, D1304, D1305, D1306, D1307, D1308, D1309, D131, D1310, D1311, D1312, D1313, D1314, D1315, D1316, D1317, D1318, D1319, D132, D1320, D1321, D1322, D1323, D1324, D1325, D1326, D1327, D1328, D1329, D133, D1330, D1331, D1332, D1333, D1334, D1335, D1336, D1337, D1338, D1339, D134, D1340, D1341, D1342, D1343, D1344, D1345, D1346, D1347, D1348, D1349, D135, D1350, D1351, D1352, D1353, D1354, D1355, D1356, D1357, D1358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: APA102-2020, LED_SMD:LED-APA102-2020, symbol LED:APA102-2020
- removed J1, J12, J15, J18, J21, J24, J27, J30, J4, J9: Conn_01x04_Pin, Connector_PinSocket_2.54mm:PinSocket_1x04_P2.54mm_Horizontal, symbol Connector:Conn_01x04_Pin
- removed J10, J11, J13, J14, J16, J17, J19, J20, J22, J23, J25, J26, J28, J29, J5, J6, J7, J8: Conn_01x03_Pin, Connector_PinSocket_2.54mm:PinSocket_1x03_P2.54mm_Horizontal, symbol Connector:Conn_01x03_Pin
